File: boards/a1_codec/a1_codec.kicad_sch (KiCad schematic)
At the start: 20 parts, among them U1 LM3480-3.3, U2 NAU8822, U4 74LV6T17, U6 TXS0102DCT

Commit message: Extracted LAN chip, more progress towards full schematic.
Other:
- note added: "TODO: - Replace all 402-s with 602-es - Widen power traces - Double-check power consumption on LDO"
Changed lines of the file:
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@@
     (stroke (width 0) (type default))
+  )
+  (text "TODO:\n- Replace all 402-s with 602-es\n- Widen power traces\n- Double-check power consumption on LDO\n"
+    (at 186.69 93.98 0)
+    (effects (font (size 1.27 1.27)) (justify left bottom))
   )
   (label "RLIN{slash}GPIO3" (at 76.2 168.91 180) (fields_autoplaced)
