File: boards/a1_mega/a1_mega.kicad_pcb (KiCad board)
At the start: 2 copper layers, 107 parts, among them J1 Bus_ISA_8bit, J10 DE9_Plug, J11 RJ45_Amphenol_RJMG1BD3B8K1ANR, J12 SJ1-3535NG-BE, J13 SJ1-3535NG-BE, J14 USB_A_Stacked, J2 Bus_ISA_8bit, J3 Bus_ISA_8bit, J4 Bus_ISA_8bit, J5 Conn_01x02, J6 HDMI_A, J7 Micro_SD_Card, J8 USB_A_Stacked, J9 USB_A_Stacked, U1 74LS139, U10 74AHCT245, U11 74AHCT245, U12 74AHCT245, U13 74AHCT245, U14 74AHCT245, U15 74AHCT245, U16 74LS273, U17 74LS273, U18 74LS138, U19 ESPRESSO, U2 74LS08, U20 SIMM-30, U21 SIMM-30, U22 74LS125, U23 74LS125, U24 DISCO, U25 A1_CODEC, U26 MIO, U28 MAX232, U29 DS1307+, U3 74LS08, U30 SIMM-30, U31 SIMM-30, U32 KSZ8851-11MLL, U33 74LS00, U34 A1_USBHUB, U4 74LS32, U5 74LS273, U6 74LS574, U7 74LS04, U8 74LS27, U9 74LS86, X1 CXO_DIP14, X2 24MHz, Y1 32768Hz, Y2 25MHz

Commit message: It seems motherboard is feature-complete. Routing started.
Parts:
- added C15: 1uF, Capacitor_THT:C_Disc_D4.7mm_W2.5mm_P5.00mm, F.Cu at (192.0, 112.8)
- added C16: 1uF, Capacitor_THT:C_Disc_D4.7mm_W2.5mm_P5.00mm, F.Cu at (192.0, 123.4)
- added C23: 22pF, Capacitor_THT:C_Disc_D3.4mm_W2.1mm_P2.50mm, F.Cu at (158.5, 222.7)
- added C24: 22pF, Capacitor_THT:C_Disc_D3.4mm_W2.1mm_P2.50mm, F.Cu at (158.5, 226.3)
- added C25: 1uF, Capacitor_THT:C_Disc_D4.7mm_W2.5mm_P5.00mm, F.Cu at (227.9, 233.4)
- added C26: 1uF, Capacitor_THT:C_Disc_D4.7mm_W2.5mm_P5.00mm, F.Cu at (314.7, 272.0)
- added C27: 1uF, Capacitor_THT:C_Disc_D4.7mm_W2.5mm_P5.00mm, F.Cu at (235.9, 176.5)
- added C28: 1uF, Capacitor_THT:C_Disc_D4.7mm_W2.5mm_P5.00mm, F.Cu at (187.0, 289.5)
- added C29: 1uF, Capacitor_THT:C_Disc_D4.7mm_W2.5mm_P5.00mm, F.Cu at (171.8, 289.5)
- added C30: 1uF, Capacitor_THT:C_Disc_D4.7mm_W2.5mm_P5.00mm, F.Cu at (156.0, 289.5)
- added C31: 1uF, Capacitor_THT:C_Disc_D4.7mm_W2.5mm_P5.00mm, F.Cu at (222.7, 264.9)
- added C32: 1uF, Capacitor_THT:C_Disc_D4.7mm_W2.5mm_P5.00mm, F.Cu at (223.3, 290.3)
- added C33: 1uF, Capacitor_THT:C_Disc_D4.7mm_W2.5mm_P5.00mm, F.Cu at (291.8, 101.3)
- added C34: 1uF, Capacitor_THT:C_Disc_D4.7mm_W2.5mm_P5.00mm, F.Cu at (188.8, 214.1)
- added C35: 1uF, Capacitor_THT:C_Disc_D4.7mm_W2.5mm_P5.00mm, F.Cu at (389.9, 135.7)
- added C36: 1uF, Capacitor_THT:C_Disc_D4.7mm_W2.5mm_P5.00mm, F.Cu at (235.2, 146.6)
- added C37: 1uF, Capacitor_THT:C_Disc_D4.7mm_W2.5mm_P5.00mm, F.Cu at (171.5, 263.1)
- added C38: 1uF, Capacitor_THT:C_Disc_D4.7mm_W2.5mm_P5.00mm, F.Cu at (155.6, 263.1)
- added C39: 1uF, Capacitor_THT:C_Disc_D4.7mm_W2.5mm_P5.00mm, F.Cu at (345.2, 254.7)
- added C40: 1uF, Capacitor_THT:C_Disc_D4.7mm_W2.5mm_P5.00mm, F.Cu at (271.1, 254.7)
- added C41: 1uF, Capacitor_THT:C_Disc_D4.7mm_W2.5mm_P5.00mm, F.Cu at (275.1, 184.1)
- added C42: 1uF, Capacitor_THT:C_Disc_D4.7mm_W2.5mm_P5.00mm, F.Cu at (204.6, 227.8)
- added C43: 1uF, Capacitor_THT:C_Disc_D4.7mm_W2.5mm_P5.00mm, F.Cu at (188.8, 196.3)
- added C44: 1uF, Capacitor_THT:C_Disc_D4.7mm_W2.5mm_P5.00mm, F.Cu at (202.6, 263.1)
- added C45: 1uF, Capacitor_THT:C_Disc_D4.7mm_W2.5mm_P5.00mm, F.Cu at (187.3, 263.1)
- added C46: 1uF, Capacitor_THT:C_Disc_D4.7mm_W2.5mm_P5.00mm, F.Cu at (250.7, 202.4)
- added C47: 1uF, Capacitor_THT:C_Disc_D4.7mm_W2.5mm_P5.00mm, F.Cu at (313.7, 128.1)
- added C48: 1uF, Capacitor_THT:C_Disc_D4.7mm_W2.5mm_P5.00mm, F.Cu at (299.4, 287.3)
- added C49: 1uF, Capacitor_THT:C_Disc_D4.7mm_W2.5mm_P5.00mm, F.Cu at (220.7, 158.7)
- added C50: 1uF, Capacitor_THT:C_Disc_D4.7mm_W2.5mm_P5.00mm, F.Cu at (230.8, 202.9)
- added C51: 1uF, Capacitor_THT:C_Disc_D4.7mm_W2.5mm_P5.00mm, F.Cu at (215.1, 121.7)
- added C52: 1uF, Capacitor_THT:C_Disc_D4.7mm_W2.5mm_P5.00mm, F.Cu at (250.7, 232.9)
- added C53: 1uF, Capacitor_THT:C_Disc_D4.7mm_W2.5mm_P5.00mm, F.Cu at (264.2, 152.9)
- added C54: 1uF, Capacitor_THT:C_Disc_D4.7mm_W2.5mm_P5.00mm, F.Cu at (250.2, 291.8)
- added C55: 1uF, Capacitor_THT:C_Disc_D4.7mm_W2.5mm_P5.00mm, F.Cu at (250.2, 262.3)
- added C56: 1uF, Capacitor_THT:C_Disc_D4.7mm_W2.5mm_P5.00mm, F.Cu at (266.7, 121.7)
- added C57: 1uF, Capacitor_THT:C_Disc_D4.7mm_W2.5mm_P5.00mm, F.Cu at (293.9, 191.7)
- added C58: 1uF, Capacitor_THT:C_Disc_D4.7mm_W2.5mm_P5.00mm, F.Cu at (263.9, 191.8)
- added C59: 1uF, Capacitor_THT:C_Disc_D4.7mm_W2.5mm_P5.00mm, F.Cu at (280.7, 219.2)
- added C60: 1uF, Capacitor_THT:C_Disc_D4.7mm_W2.5mm_P5.00mm, F.Cu at (220.7, 136.4)
- added C61: 1uF, Capacitor_THT:C_Disc_D4.7mm_W2.5mm_P5.00mm, F.Cu at (271.6, 234.9)
- added C62: 1uF, Capacitor_THT:C_Disc_D4.7mm_W2.5mm_P5.00mm, F.Cu at (345.2, 185.6)
- added C63: 1uF, Capacitor_THT:C_Disc_D4.7mm_W2.5mm_P5.00mm, F.Cu at (271.6, 185.6)
- added C64: 1uF, Capacitor_THT:C_Disc_D4.7mm_W2.5mm_P5.00mm, F.Cu at (345.2, 165.8)
- added C65: 1uF, Capacitor_THT:C_Disc_D4.7mm_W2.5mm_P5.00mm, F.Cu at (271.5, 165.8)
- added C66: 1uF, Capacitor_THT:C_Disc_D4.7mm_W2.5mm_P5.00mm, F.Cu at (323.9, 191.8)
- added C67: 1uF, Capacitor_THT:C_Disc_D4.7mm_W2.5mm_P5.00mm, F.Cu at (250.2, 172.4)
- added C68: 1uF, Capacitor_THT:C_Disc_D4.7mm_W2.5mm_P5.00mm, F.Cu at (345.2, 234.9)
- added CMC1: L_Ferrite_Coupled_Small, anachron:SCM2012FS, F.Cu at (251.4, 100.1)
- added CMC10: L_Ferrite_Coupled_Small, anachron:SCM2012FS, F.Cu at (325.1, 104.1)
- added CMC2: L_Ferrite_Coupled_Small, anachron:SCM2012FS, F.Cu at (253.4, 100.1)
- added CMC3: L_Ferrite_Coupled_Small, anachron:SCM2012FS, F.Cu at (255.3, 100.1)
- added CMC4: L_Ferrite_Coupled_Small, anachron:SCM2012FS, F.Cu at (257.2, 100.1)
- added CMC5: L_Ferrite_Coupled_Small, anachron:SCM2012FS, F.Cu at (360.7, 104.1)
- added CMC6: L_Ferrite_Coupled_Small, anachron:SCM2012FS, F.Cu at (362.6, 104.1)
- added CMC7: L_Ferrite_Coupled_Small, anachron:SCM2012FS, F.Cu at (341.0, 104.1)
- added CMC8: L_Ferrite_Coupled_Small, anachron:SCM2012FS, F.Cu at (342.9, 104.1)
- added CMC9: L_Ferrite_Coupled_Small, anachron:SCM2012FS, F.Cu at (323.2, 104.1)
- added D1: 1N5711, Diode_THT:D_DO-35_SOD27_P7.62mm_Horizontal, F.Cu at (138.4, 222.6)
- added D2: 1N5711, Diode_THT:D_DO-35_SOD27_P7.62mm_Horizontal, F.Cu at (138.4, 226.2)
- added FB10: FerriteBead_Small, Inductor_THT:L_Axial_L7.0mm_D3.3mm_P2.54mm_Vertical_Fastron_MICC, F.Cu at (306.7, 97.2)
- added FB11: FerriteBead_Small, Inductor_THT:L_Axial_L7.0mm_D3.3mm_P2.54mm_Vertical_Fastron_MICC, F.Cu at (301.0, 97.2)
- added FB12: FerriteBead_Small, Inductor_THT:L_Axial_L7.0mm_D3.3mm_P2.54mm_Vertical_Fastron_MICC, F.Cu at (312.4, 97.2)
- added FB13: FerriteBead_Small, Inductor_THT:L_Axial_L7.0mm_D3.3mm_P2.54mm_Vertical_Fastron_MICC, F.Cu at (265.4, 101.6)
- added FB14: FerriteBead_Small, Inductor_THT:L_Axial_L7.0mm_D3.3mm_P2.54mm_Vertical_Fastron_MICC, F.Cu at (262.3, 95.0)
- added FB15: FerriteBead_Small, Inductor_THT:L_Axial_L7.0mm_D3.3mm_P2.54mm_Vertical_Fastron_MICC, F.Cu at (248.9, 96.5)
- added FB16: FerriteBead_Small, Inductor_THT:L_Axial_L7.0mm_D3.3mm_P2.54mm_Vertical_Fastron_MICC, F.Cu at (234.9, 98.4)
- added FB17: FerriteBead_Small, Inductor_THT:L_Axial_L7.0mm_D3.3mm_P2.54mm_Vertical_Fastron_MICC, F.Cu at (238.8, 98.4)
- added FB18: FerriteBead_Small, Inductor_THT:L_Axial_L7.0mm_D3.3mm_P2.54mm_Vertical_Fastron_MICC, F.Cu at (231.1, 98.4)
- added FB19: FerriteBead_Small, Inductor_THT:L_Axial_L7.0mm_D3.3mm_P2.54mm_Vertical_Fastron_MICC, F.Cu at (227.3, 98.4)
- added FB2: FerriteBead_Small, Inductor_THT:L_Axial_L7.0mm_D3.3mm_P2.54mm_Vertical_Fastron_MICC, F.Cu at (351.8, 109.9)
- added FB20: FerriteBead_Small, Inductor_THT:L_Axial_L7.0mm_D3.3mm_P2.54mm_Vertical_Fastron_MICC, F.Cu at (265.3, 106.0)
- added FB3: FerriteBead_Small, Inductor_THT:L_Axial_L7.0mm_D3.3mm_P2.54mm_Vertical_Fastron_MICC, F.Cu at (346.1, 109.9)
- added FB4: FerriteBead_Small, Inductor_THT:L_Axial_L7.0mm_D3.3mm_P2.54mm_Vertical_Fastron_MICC, F.Cu at (377.8, 106.0)
- added FB5: FerriteBead_Small, Inductor_THT:L_Axial_L7.0mm_D3.3mm_P2.54mm_Vertical_Fastron_MICC, F.Cu at (365.8, 109.9)
- added FB6: FerriteBead_Small, Inductor_THT:L_Axial_L7.0mm_D3.3mm_P2.54mm_Vertical_Fastron_MICC, F.Cu at (334.0, 109.9)
- added FB7: FerriteBead_Small, Inductor_THT:L_Axial_L7.0mm_D3.3mm_P2.54mm_Vertical_Fastron_MICC, F.Cu at (328.3, 109.9)
- added FB8: FerriteBead_Small, Inductor_THT:L_Axial_L7.0mm_D3.3mm_P2.54mm_Vertical_Fastron_MICC, F.Cu at (289.6, 97.2)
- added FB9: FerriteBead_Small, Inductor_THT:L_Axial_L7.0mm_D3.3mm_P2.54mm_Vertical_Fastron_MICC, F.Cu at (295.3, 97.2)
- added J15: ATX-24, anachron:TE_1-1775099-3, F.Cu at (368.4, 183.9)
- added J16: Conn_01x01, MountingHole:MountingHole_4.3mm_M4_DIN965_Pad, F.Cu at (171.4, 91.4)
- added J17: Conn_01x01, MountingHole:MountingHole_4.3mm_M4_DIN965_Pad, F.Cu at (374.6, 114.3)
- added J18: Conn_01x01, MountingHole:MountingHole_4.3mm_M4_DIN965_Pad, F.Cu at (374.6, 246.4)
- added J19: Conn_01x01, MountingHole:MountingHole_4.3mm_M4_DIN965_Pad, F.Cu at (151.1, 246.4)
- added J20: Conn_01x01, MountingHole:MountingHole_4.3mm_M4_DIN965_Pad, F.Cu at (217.2, 91.4)
- added J21: Conn_01x01, MountingHole:MountingHole_4.3mm_M4_DIN965_Pad, F.Cu at (171.4, 246.4)
- added J22: Conn_01x01, MountingHole:MountingHole_4.3mm_M4_DIN965_Pad, F.Cu at (217.2, 246.4)
- added J23: Conn_01x01, MountingHole:MountingHole_4.3mm_M4_DIN965_Pad, F.Cu at (374.6, 318.8)
- added J24: Conn_01x01, MountingHole:MountingHole_4.3mm_M4_DIN965_Pad, F.Cu at (217.2, 318.8)
- added JP3: Jumper_2_Open, Connector_PinHeader_2.54mm:PinHeader_1x02_P2.54mm_Vertical, F.Cu at (184.0, 193.8)
- added JP4: Jumper_3_Bridged12, Connector_PinHeader_2.54mm:PinHeader_1x03_P2.54mm_Vertical, F.Cu at (213.7, 205.7)
- added Q1: 2N7000, Package_TO_SOT_THT:TO-92_Inline, F.Cu at (186.7, 218.9)
- added R22: 10k, Resistor_THT:R_Axial_DIN0204_L3.6mm_D1.6mm_P5.08mm_Horizontal, F.Cu at (179.6, 197.9)
- added R23: 10k, Resistor_THT:R_Axial_DIN0204_L3.6mm_D1.6mm_P5.08mm_Horizontal, F.Cu at (179.6, 201.0)
- added R24: 10k, Resistor_THT:R_Axial_DIN0204_L3.6mm_D1.6mm_P5.08mm_Horizontal, F.Cu at (179.6, 204.2)
- added R25: 10k, Resistor_THT:R_Axial_DIN0204_L3.6mm_D1.6mm_P5.08mm_Horizontal, F.Cu at (179.6, 207.3)
- added R26: 10k, Resistor_THT:R_Axial_DIN0204_L3.6mm_D1.6mm_P5.08mm_Horizontal, F.Cu at (179.6, 210.5)
- added R27: 10k, Resistor_THT:R_Axial_DIN0204_L3.6mm_D1.6mm_P5.08mm_Horizontal, F.Cu at (371.1, 152.6)
- added R28: 10k, Resistor_THT:R_Axial_DIN0204_L3.6mm_D1.6mm_P5.08mm_Horizontal, F.Cu at (308.1, 303.0)
- added R29: 10k, Resistor_THT:R_Axial_DIN0204_L3.6mm_D1.6mm_P5.08mm_Horizontal, F.Cu at (179.6, 213.6)
- added R4: 10k, Resistor_THT:R_Axial_DIN0204_L3.6mm_D1.6mm_P5.08mm_Horizontal, F.Cu at (347.2, 272.0)
- added SW1: SW_Push, Connector_PinHeader_2.54mm:PinHeader_1x02_P2.54mm_Vertical, F.Cu at (149.9, 223.2)
- added SW2: SW_Push, Button_Switch_THT:SW_PUSH_6mm, F.Cu at (169.3, 217.7)
- added SW3: SW_Push, Connector_PinHeader_2.54mm:PinHeader_1x02_P2.54mm_Vertical, F.Cu at (154.6, 223.2)
- added SW4: SW_Push, Button_Switch_THT:SW_PUSH_6mm, F.Cu at (169.3, 226.3)
- added U27: SST39SF040, anachron:PLCC-32_THT-Socket, F.Cu at (222.2, 272.2)
- added U35: L79L05_TO92, Package_TO_SOT_THT:TO-92_Inline, F.Cu at (195.8, 117.9)
- added U37: SST39SF040, anachron:PLCC-32_THT-Socket, F.Cu at (222.2, 297.9)
- added U38: ATtiny24-20P, Package_DIP:DIP-14_W7.62mm, F.Cu at (168.9, 198.4)
- added X3: 8MHz, Oscillator:Oscillator_DIP-14, F.Cu at (193.9, 220.4)
- added X4: 14.31818MHz, Oscillator:Oscillator_DIP-14, F.Cu at (193.4, 202.9)
- added Y3: 32768Hz, Crystal:Crystal_AT310_D3.0mm_L10.0mm_Horizontal_1EP_style2, F.Cu at (180.0, 217.0)
- C11, C12, C8, C9: footprint Capacitor_THT:C_Rect_L9.0mm_W2.5mm_P7.50mm_MKT -> Capacitor_THT:C_Disc_D3.4mm_W2.1mm_P2.50mm
- C17, C18, C19, C20, C21, C22: value 220uF -> 100uF; footprint Capacitor_THT:CP_Radial_D7.5mm_P2.50mm -> Capacitor_THT:CP_Radial_D5.0mm_P2.00mm
- C4, C5, C6, C7: footprint Capacitor_THT:C_Rect_L9.0mm_W2.5mm_P7.50mm_MKT -> Capacitor_THT:C_Disc_D4.7mm_W2.5mm_P5.00mm
- F1: value Polyfuse -> 0.5A; footprint Fuse:Fuse_Littelfuse_395Series -> Fuse:Fuse_BelFuse_0ZRE0005FF_L8.3mm_W3.8mm
- J11: value RJ45_Amphenol_RJMG1BD3B8K1ANR -> ~; footprint Connector_RJ:RJ45_Amphenol_RJMG1BD3B8K1ANR -> anachron:ARJM11D7-009-AB-EW2
- J14, J8, J9: footprint Connector_USB:USB_A_CUI_UJ2-ADH-TH_Horizontal_Stacked -> anachron:GCT_USB1035-XX-X-X-X-B_REVE
- J7: footprint Connector_Card:microSD_HC_Hirose_DM3BT-DSF-PEJS -> anachron:GCT_MEM2052-00-195-00-A_REVA
- moved U26 365.4 mm to (303.0, 298.9), turned to 90 degrees
- moved RN8 334.7 mm to (325.9, 305.0)
- moved J8 320.5 mm to (370.6, 92.5), turned to 180 degrees
- moved J9 297.3 mm to (350.5, 92.5), turned to 180 degrees
- moved C18 296.7 mm to (373.7, 104.8), turned to 180 degrees
- moved C17 293.5 mm to (368.0, 104.8), turned to 180 degrees
- moved X2 292.3 mm to (319.3, 271.2)
- moved RN10 292.0 mm to (330.9, 278.6)
- moved JP2 283.7 mm to (370.2, 132.6), turned to 180 degrees
- moved J7 283.3 mm to (357.4, 267.9), turned to 90 degrees
- moved C19 275.5 mm to (354.0, 104.8), turned to 180 degrees
- moved J14 274.6 mm to (330.2, 92.5), turned to 180 degrees
- moved C20 267.9 mm to (348.3, 104.8), turned to 180 degrees
- moved U34 258.7 mm to (317.0, 132.5), turned to 90 degrees
- moved U28 254.7 mm to (297.9, 108.9), turned to 90 degrees
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Connections:
- net /ISA/ISA_+12V renamed +12V
- net /ISA/ISA_-12V renamed -12V
- net /ISA_OSC renamed /ISA/ISA_OSC
- net /~{MIO0_SEL} renamed /~{MIO_SEL}
- net Net-(BT1-+) renamed +BATT
- F1 pad 1: Net-(J6-+5V) -> Net-(F1-Pad1)
- J10 pad 2: Net-(U28-R1IN) -> Net-(FB11-Pad2)
- J10 pad 3: Net-(U28-T1OUT) -> Net-(FB9-Pad2)
- J10 pad 4: Net-(U28-VS+) -> Net-(FB8-Pad2)
- J10 pad 7: Net-(U28-T2OUT) -> Net-(FB10-Pad2)
- J10 pad 8: Net-(U28-R2IN) -> Net-(FB12-Pad2)
- J12 pad 2: Net-(C2-Pad2) -> Net-(FB16-Pad1)
- J12 pad 3: Net-(C3-Pad2) -> Net-(FB17-Pad1)
- J13 pad 2: Net-(C1-Pad2) -> Net-(FB18-Pad1)
- J13 pad 3: Net-(C13-Pad2) -> Net-(FB19-Pad1)
- J6 pad 15: /VIDEO_DDC_SCL -> Net-(J6-SCL)
- J6 pad 16: /VIDEO_DDC_SDA -> Net-(J6-SDA)
- J6 pad 19: /VIDEO_HPD -> Net-(J6-HPD)
- J7 pad 9: unconnected-(J7-DET-Pad9) -> Net-(J7-DET)
- RN10 pad 2: /I2C_SDA -> unconnected-(RN10-R1-Pad2)
- RN10 pad 3: /I2C_SCL -> unconnected-(RN10-R2-Pad3)
- RN14 pad 8: /CPU_A1 -> /CPU_A0
- U10 pad 1: +5V -> GND
- U10 pad 11: /CPU_A0 -> /GFX_A7
- U10 pad 12: /CPU_A1 -> /GFX_A6
- U10 pad 13: /CPU_A2 -> /GFX_A5
- U10 pad 14: /CPU_A3 -> /GFX_A4
- U10 pad 15: /CPU_A4 -> /GFX_A3
- U10 pad 16: /CPU_A5 -> /GFX_A2
- U10 pad 17: /CPU_A6 -> /GFX_A1
- U10 pad 18: /CPU_A7 -> /GFX_A0
- U10 pad 2: /GFX_A7 -> /CPU_A0
- U10 pad 3: /GFX_A6 -> /CPU_A1
- U10 pad 4: /GFX_A5 -> /CPU_A2
- U10 pad 5: /GFX_A4 -> /CPU_A3
- U10 pad 6: /GFX_A3 -> /CPU_A4
- U10 pad 7: /GFX_A2 -> /CPU_A5
- U10 pad 8: /GFX_A1 -> /CPU_A6
- U10 pad 9: /GFX_A0 -> /CPU_A7
- U11 pad 1: +5V -> GND
- U11 pad 11: /CPU_A8 -> /GFX_A8
- U11 pad 12: /CPU_~{RAS_B} -> /GFX_~{RAS}
- U11 pad 13: /CPU_~{CAS_0} -> /GFX_~{CAS_0}
- U11 pad 14: /CPU_~{CAS_1} -> /GFX_~{CAS_1}
- U11 pad 15: /CPU_~{WE} -> /GFX_~{WE}
- U11 pad 5: /GFX_~{WE} -> /CPU_~{WE}
- U11 pad 6: /GFX_~{CAS_1} -> /CPU_~{CAS_1}
- U11 pad 7: /GFX_~{CAS_0} -> /CPU_~{CAS_0}
- U11 pad 8: /GFX_~{RAS} -> /CPU_~{RAS_B}
- U11 pad 9: /GFX_A8 -> /CPU_A8
- U12 pad 1: /CPU_~{WE} -> Net-(U12-A->B)
- U12 pad 11: /CPU_A1 -> /GFX_D7
- U12 pad 12: /CPU_A1 -> /GFX_D6
- U12 pad 13: /CPU_A1 -> /GFX_D5
- U12 pad 14: /CPU_A1 -> /GFX_D4
- U12 pad 15: /CPU_A1 -> /GFX_D3
- U12 pad 16: /CPU_A1 -> /GFX_D2
- U12 pad 17: /CPU_A1 -> /GFX_D1
- U12 pad 18: /CPU_A1 -> /GFX_D0
- U12 pad 2: /GFX_D7 -> /CPU_A0
- U12 pad 3: /GFX_D6 -> /CPU_A0
- U12 pad 4: /GFX_D5 -> /CPU_A0
- U12 pad 5: /GFX_D4 -> /CPU_A0
- U12 pad 6: /GFX_D3 -> /CPU_A0
- U12 pad 7: /GFX_D2 -> /CPU_A0
- U12 pad 8: /GFX_D1 -> /CPU_A0
- U12 pad 9: /GFX_D0 -> /CPU_A0
- U13 pad 11: /CPU_A1 -> /CPU_A0
- U13 pad 12: /CPU_A1 -> /CPU_A0
- U13 pad 13: /CPU_A1 -> /CPU_A0
- U13 pad 14: /CPU_A1 -> /CPU_A0
- U13 pad 15: /CPU_A1 -> /CPU_A0
- U13 pad 16: /CPU_A1 -> /CPU_A0
- U13 pad 17: /CPU_A1 -> /CPU_A0
- U13 pad 18: /CPU_A1 -> /CPU_A0
- U18 pad 10: /~{LAN_SEL} -> unconnected-(U18-O5-Pad10)
- U18 pad 11: /~{MIO1_SEL} -> /~{LAN_SEL}
- U19 pad 27: /CPU_A1 -> /CPU_A0
- U2 pad 10: unconnected-(U2-Pad10) -> Net-(U2-Pad10)
- U2 pad 14: GND -> +5V
- U2 pad 7: +5V -> GND
- U2 pad 8: unconnected-(U2-Pad8) -> ~{RST}
- U2 pad 9: unconnected-(U2-Pad9) -> Net-(R23-Pad2)
- U22 pad 8: /CPU_A1 -> /CPU_A0
- U24 pad 1: Net-(J6-D2+) -> Net-(U24-TMDS_D2+)
- U24 pad 2: Net-(J6-D2-) -> Net-(U24-TMDS_D2-)
- U24 pad 3: Net-(J6-D1+) -> Net-(U24-TMDS_D1+)
- U24 pad 31: /CPU_A1 -> /CPU_A0
- U24 pad 4: Net-(J6-D1-) -> Net-(U24-TMDS_D1-)
- U24 pad 5: Net-(J6-D0+) -> Net-(U24-TMDS_D0+)
- U24 pad 6: Net-(J6-D0-) -> Net-(U24-TMDS_D0-)
- U24 pad 7: Net-(J6-CK+) -> Net-(U24-TMDS_C+)
- U24 pad 8: Net-(J6-CK-) -> Net-(U24-TMDS_C-)
- U26 pad 2: unconnected-(U26-PC1_USBa_D--Pad2) -> Net-(J7-DET)
- U26 pad 3: unconnected-(U26-PC2_USBb_D+-Pad3) -> /~{RTC_INT}
- U29 pad 7: /CPU_~{INT} -> /~{RTC_INT}
- U33 pad 11: unconnected-(U33-Pad11) -> Net-(U12-A->B)
- U33 pad 12: unconnected-(U33-Pad12) -> +5V
- U33 pad 13: unconnected-(U33-Pad13) -> /CPU_~{WE}
- U34 pad 10: Net-(J9-D2+) -> Net-(U34-USBDN4_DP)
- U34 pad 11: Net-(J14-D1-) -> Net-(U34-USBDN5_DM)
- U34 pad 12: Net-(J14-D1+) -> Net-(U34-USBDN5_DP)
- U34 pad 21: Net-(J14-VBUS2) -> Net-(U34-VBUS6)
- U34 pad 22: Net-(J14-VBUS1) -> Net-(U34-VBUS5)
- U34 pad 23: unconnected-(U34-VBUS7-Pad23) -> Net-(U34-VBUS7)
- U34 pad 24: Net-(J8-VBUS1) -> unconnected-(U34-VBUS1-Pad24)
- U34 pad 25: Net-(J8-VBUS2) -> Net-(U34-VBUS2)
- U34 pad 26: Net-(J9-VBUS1) -> Net-(U34-VBUS3)
- U34 pad 27: Net-(J9-VBUS2) -> Net-(U34-VBUS4)
- U34 pad 3: Net-(J8-D1-) -> unconnected-(U34-USBDN1_DM-Pad3)
- U34 pad 34: Net-(J14-D2-) -> Net-(U34-USBDN6_DM)
- U34 pad 35: Net-(J14-D2+) -> Net-(U34-USBDN6_DP)
- U34 pad 36: unconnected-(U34-USBDN7_DM-Pad36) -> Net-(U34-USBDN7_DM)
- U34 pad 37: unconnected-(U34-USBDN7_DP-Pad37) -> Net-(U34-USBDN7_DP)
- U34 pad 4: Net-(J8-D1+) -> unconnected-(U34-USBDN1_DP-Pad4)
- U34 pad 5: Net-(J8-D2-) -> Net-(U34-USBDN2_DM)
- U34 pad 6: Net-(J8-D2+) -> Net-(U34-USBDN2_DP)
- U34 pad 7: Net-(J9-D1-) -> Net-(U34-USBDN3_DM)
- U34 pad 8: Net-(J9-D1+) -> Net-(U34-USBDN3_DP)
- U34 pad 9: Net-(J9-D2-) -> Net-(U34-USBDN4_DM)
- U5 pad 16: unconnected-(U5-Q6-Pad16) -> Net-(JP3-B)
- U5 pad 19: unconnected-(U5-Q7-Pad19) -> /Power/I2C_EN
- U6 pad 12: /BUF_D7 -> /BUF_D0
- U6 pad 13: /BUF_D6 -> /BUF_D1
- U6 pad 14: /BUF_D5 -> /BUF_D2
- U6 pad 15: /BUF_D4 -> /BUF_D3
- U6 pad 16: /BUF_D3 -> /BUF_D4
- U6 pad 17: /BUF_D2 -> /BUF_D5
- U6 pad 18: /BUF_D1 -> /BUF_D6
- U6 pad 19: /BUF_D0 -> /BUF_D7
- U6 pad 2: /ISA_IRQ2 -> /~{LAN_IRQ}
- U6 pad 3: /ISA_IRQ3 -> /~{ISA_IO_CH_CK}
- U6 pad 4: /ISA_IRQ4 -> /ISA_IRQ7
- U6 pad 5: /ISA_IRQ5 -> /ISA_IRQ6
- U6 pad 6: /ISA_IRQ6 -> /ISA_IRQ5
- U6 pad 7: /ISA_IRQ7 -> /ISA_IRQ4
- U6 pad 8: /~{ISA_IO_CH_CK} -> /ISA_IRQ3
- U6 pad 9: /~{LAN_IRQ} -> /ISA_IRQ2
- U7 pad 1: /CPU_A1 -> /CPU_A0
- U7 pad 10: unconnected-(U7-Pad10) -> /BUF_~{RD}
- U7 pad 11: unconnected-(U7-Pad11) -> /BUF_~{WE}
- U7 pad 12: unconnected-(U7-Pad12) -> Net-(U2-Pad10)
- U7 pad 13: unconnected-(U7-Pad13) -> Net-(J15-PWR_OK)
Routing:
- net /MIO/SER_TXD: track 0.00 -> 200.2 mm
- net /MIO/SER_RTS: track 0.00 -> 199.4 mm
- net /MIO/SER_CTS: track 0.00 -> 179.7 mm
- net /MIO/USB_D+: track 0.00 -> 179.2 mm
- net /MIO/SER_RXD: track 0.00 -> 178.1 mm
- net /MIO/USB_D-: track 0.00 -> 173.2 mm
- net /I2C_SDA: track 0.00 -> 163.2 mm
- net /MIO/USB_CLK: track 0.00 -> 162.2 mm
- net /I2C_SCL: track 0.00 -> 161.5 mm
- net Net-(J6-SDA): track 0.00 -> 93.0 mm
- net /GFX/CODEC_V3P3: track 0.00 -> 85.4 mm
- net /VIDEO_DDC_SCL: track 0.00 -> 81.6 mm
- net /GFX/HP_DET: track 0.00 -> 78.9 mm
- net /VIDEO_HPD: track 0.00 -> 76.7 mm
- net Net-(U24-TMDS_C-): track 0.00 -> 75.9 mm
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Other:
- board outline added: 243.8 x 243.8 mm
- copper layers 2 -> 4
- board text added: "Pin-1 locations for ISA slots"
- board text added: "Window Area"
