File: boards/a1_mega/a1_mega.kicad_sch (KiCad schematic)
At the start: 24 parts, among them U1 74LS139, U10 74AHCT245, U11 74AHCT245, U12 74AHCT245, U13 74AHCT245, U14 74AHCT245, U15 74AHCT245, U16 74LS273, U17 74LS273, U18 74LS138, U2 74LS08, U22 74LS125, U3 74LS08, U4 74LS32, U5 74LS273, U6 74LS574, U7 74LS04, U8 74LS27, U9 74LS86

Commit message: Extracted LAN chip, more progress towards full schematic.
Parts:
- added U35: 74LVC06, Package_DIP:DIP-14_W7.62mm_LongPads, symbol 74xx:74LS06
Changed lines of the file:
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@@
+    )
+  )
+  (symbol (lib_id "74xx:74LS06") (at 368.3 410.21 0) (unit 6)
+    (in_bom yes) (on_board yes) (dnp no) (fields_autoplaced)
+    (property "Reference" "U35" (at 368.3 401.955 0)
+      (effects (font (size 1.27 1.27)))
+    )
+    (property "Value" "74LVC06" (at 368.3 404.495 0)
+      (effects (font (size 1.27 1.27)))
+    )
+    (property "Footprint" "Package_DIP:DIP-14_W7.62mm_LongPads" (at 368.3 410.21 0)
+      (effects (font (size 1.27 1.27)) hide)
+    )
+    (property "Datasheet" "http://www.ti.com/lit/gpn/sn74LS06" (at 368.3 410.21 0)
+      (effects (font (size 1.27 1.27)) hide)
+    )
+    (pin "6")
+    (pin "11")
+    (pin "10")
+    (pin "7")
+    (pin "12")
+    (pin "4")
+    (pin "5")
+    (pin "13")
+    (pin "14")
+    (pin "3")
+    (pin "2")
+    (pin "1")
+    (pin "9")
+    (pin "8")
+    (instances
+      (project "a1_mega"
+        (path "/3257e1ae-50a8-410a-87c3-a39d96a2c51a"
+          (reference "U35") (unit 6)
+        )
+      )
     )
   )

Commit message: USB HUB 'chip' created and added; only a single MIO 'chip' is left in the design.
Parts:
- removed U35: 74LVC06, Package_DIP:DIP-14_W7.62mm_LongPads, symbol 74xx:74LS06
- removed unit 3 of U4
- removed unit 4 of U4
- removed unit 2 of U4
- removed unit 1 of U4
- added R10, R11: 10k, Resistor_THT:R_Axial_DIN0204_L3.6mm_D1.6mm_P5.08mm_Horizontal, symbol Device:R_US
- added U33: 74LS00, Package_DIP:DIP-14_W7.62mm_LongPads, symbol 74xx:74LS00
- added unit 6 of U7
Connections:
- net BUF_nCAS0 is gone; now on net CPU_~{DACK3}: U3.13
- net CPU_~{WAIT} is gone; now on net CPU_A[0..10]: RN14.8 (R7)
- net +5V: now also U9.12, R10.1, U33.14 (VCC), U33.9
- net BUF_A0: now also U33.2
- net BUF_NREN: now also U33.5, U33.8
- net BUF_nEN: now also U13.19 (CE)
- net CPU_A[0..10]: now also U7.1
- net CPU_DACK: now also U9.11; no longer U7.2
- net CPU_DRQ1: now also RN12.4 (R3); no longer RN12.5 (R4)
- net CPU_DRQ2: now also RN12.3 (R2); no longer RN12.4 (R3)
- net CPU_DRQ3: now also RN12.2 (R1); no longer RN12.3 (R2)
- net CPU_TC: now also R11.1; no longer RN12.2 (R1)
- net CPU_~{DACK1}: now also RN13.4 (R3), U3.2; no longer RN13.5 (R4), U3.1
- net CPU_~{DACK2}: now also RN13.3 (R2), U3.12; no longer RN13.4 (R3), U3.2
- net CPU_~{DACK3}: now also RN13.2 (R1); no longer RN13.3 (R2), U3.5
- net CPU_~{INT}: now also R10.2; no longer RN13.2 (R1)
- net GND: now also R11.2, U33.7 (GND)
- net nNR_DECODE_EN: now also U33.6
- net ~{LAN_IRQ}: now also U2.2; no longer U2.9
- net ~{LAN_WOL}: no longer U2.10
- net CPU_~{DACK}: now reaches U9.13
- net CPU_~{DACK}: now also U3.10, U3.6
- net at U2.8: no longer U2.2
- net BUF_nCAS: no longer names the net of U3.11
- net BUF_nCAS: now also U3.5; no longer U13.19 (CE)
- net BUF_nCAS1 renamed BUF_~{CAS}
- net BUF_~{CAS}: now also U33.1; no longer U3.12
- net BUF_nNREN renamed BUF_~{NREN}
- net BUF_~{NREN}: now also U33.10
- net CPU/BRQ: no longer names the net of U10.19 (CE), U11.19 (CE), U12.19 (CE)
- net CPU/BRQ: now also U7.2
- removed net CPU_nDACK: U3.10, U3.6, U7.1
- new net BUF_CAS: U33.3, U33.4
- new net CPU_DRQ0: RN12.5 (R4)
- new net CPU_~{DACK0}: RN13.5 (R4), U3.1
Other:
- sheet CPU ports: added DRQ_0, ~{DACK_0}; removed BRQ, ~{BGNT}
- sheet GFX ports: added ~{BUSY}; removed BUSY/BRQ, ~{WAIT}/~{BGNT}
- moved on the sheet: RN12, RN13, U2C, U3D, U7A, U7E, U9D

Commit message: It seems motherboard is feature-complete. Routing started.
Parts:
- removed unit 3 of U2
- removed unit 6 of U7
- added C25, C26, C27, C28, C29, C30, C31, C32, C33, C34, C35, C36, C37, C38, C39, C40, C41, C42, C43, C44, C45, C68: 1uF, Capacitor_THT:C_Disc_D4.7mm_W2.5mm_P5.00mm, symbol Device:C
- added J16, J17, J18, J19, J20, J21, J22, J23, J24: Conn_01x01, MountingHole:MountingHole_4.3mm_M4_DIN965_Pad, symbol Connector_Generic:Conn_01x01
- added JP3: Jumper_2_Open, Connector_PinHeader_2.54mm:PinHeader_1x02_P2.54mm_Vertical, symbol Jumper:Jumper_2_Open
- added R27: 10k, Resistor_THT:R_Axial_DIN0204_L3.6mm_D1.6mm_P5.08mm_Horizontal, symbol Device:R_US
- added U27, U37: SST39SF040, anachron:PLCC-32_THT-Socket, symbol Memory_Flash:SST39SF040
- added X3: 8MHz, Oscillator:Oscillator_DIP-14, symbol Oscillator:CXO_DIP14
Connections:
- net ~{MIO1_SEL} is gone; now on net ~{LAN_SEL}: U18.11 (O4)
- net +5V: now also U2.14 (VCC), U33.12, C25.1, C26.1, C27.1, C28.1, C29.1, C30.1, C31.1, C32.1, C33.1, C34.1, C35.1, C36.1, C37.1, C38.1, C39.1, C40.1, C41.1, C42.1, C43.1, C44.1, C45.1, C68.1, U27.32 (VCC), U37.32 (VCC), X3.1 (EN), X3.14 (Vcc); no longer U10.1 (A->B), U11.1 (A->B), U2.7 (GND)
- net BUF_A0: now also U27.12 (A0), U37.12 (A0)
- net BUF_A1: now also U27.11 (A1), U37.11 (A1)
- net BUF_A10: now also U27.23 (A10), U37.23 (A10)
- net BUF_A11: now also U27.25 (A11), U37.25 (A11)
- net BUF_A12: now also U27.4 (A12), U37.4 (A12)
- net BUF_A13: now also U27.28 (A13), U37.28 (A13)
- net BUF_A14: now also U27.29 (A14), U37.29 (A14)
- net BUF_A15: now also U27.3 (A15), U37.3 (A15)
- net BUF_A16: now also U27.2 (A16), U37.2 (A16)
- net BUF_A17: now also U27.30 (A17), U37.30 (A17)
- net BUF_A18: now also U27.1 (A18), U37.1 (A18)
- net BUF_A2: now also U27.10 (A2), U37.10 (A2)
- net BUF_A3: now also U27.9 (A3), U37.9 (A3)
- net BUF_A4: now also U27.8 (A4), U37.8 (A4)
- net BUF_A5: now also U27.7 (A5), U37.7 (A5)
- net BUF_A6: now also U27.6 (A6), U37.6 (A6)
- net BUF_A7: now also U27.5 (A7), U37.5 (A7)
- net BUF_A8: now also U27.27 (A8), U37.27 (A8)
- net BUF_A9: now also U27.26 (A9), U37.26 (A9)
- net BUF_D0: now also U6.12 (Q7), U27.13 (D0), U37.13 (D0); no longer U6.19 (Q0)
- net BUF_D1: now also U6.13 (Q6), U27.14 (D1), U37.14 (D1); no longer U6.18 (Q1)
- net BUF_D2: now also U6.14 (Q5), U27.15 (D2), U37.15 (D2); no longer U6.17 (Q2)
- net BUF_D3: now also U6.15 (Q4), U27.17 (D3), U37.17 (D3); no longer U6.16 (Q3)
- net BUF_D4: now also U6.16 (Q3), U27.18 (D4), U37.18 (D4); no longer U6.15 (Q4)
- net BUF_D5: now also U6.17 (Q2), U27.19 (D5), U37.19 (D5); no longer U6.14 (Q5)
- net BUF_D6: now also U6.18 (Q1), U27.20 (D6), U37.20 (D6); no longer U6.13 (Q6)
- net BUF_D7: now also U6.19 (Q0), U27.21 (D7), U37.21 (D7); no longer U6.12 (Q7)
- net BUF_~{WE}: now also U7.11, U27.31 (PGM), U37.31 (PGM)
- net CPU_A0: now also U10.2 (A0); no longer U10.11 (B7)
- net CPU_A1: now also U10.3 (A1); no longer U10.12 (B6)
- net CPU_A2: now also U10.4 (A2); no longer U10.13 (B5)
- net CPU_A3: now also U10.5 (A3); no longer U10.14 (B4)
- net CPU_A4: now also U10.6 (A4); no longer U10.15 (B3)
- net CPU_A5: now also U10.7 (A5); no longer U10.16 (B2)
- net CPU_A6: now also U10.8 (A6); no longer U10.17 (B1)
- net CPU_A7: now also U10.9 (A7); no longer U10.18 (B0)
- net CPU_A8: now also U11.9 (A7); no longer U11.11 (B7)
- net CPU_D0: now also U12.2 (A0); no longer U12.11 (B7)
- net CPU_D1: now also U12.3 (A1); no longer U12.12 (B6)
- net CPU_D2: now also U12.4 (A2); no longer U12.13 (B5)
- net CPU_D3: now also U12.5 (A3); no longer U12.14 (B4)
- net CPU_D4: now also U12.6 (A4); no longer U12.15 (B3)
- net CPU_D5: now also U12.7 (A5); no longer U12.16 (B2)
- net CPU_D6: now also U12.8 (A6); no longer U12.17 (B1)
- net CPU_D7: now also U12.9 (A7); no longer U12.18 (B0)
- net CPU_~{CAS_0}: now also U11.7 (A5); no longer U11.13 (B5)
- net CPU_~{CAS_1}: now also U11.6 (A4); no longer U11.14 (B4)
- net CPU_~{RAS_B}: now also U11.8 (A6); no longer U11.12 (B6)
- net CPU_~{WE}: now also U11.5 (A3), U33.13; no longer U11.15 (B3), U12.1 (A->B)
- net GFX_A0: now also U10.18 (B0); no longer U10.9 (A7)
- net GFX_A1: now also U10.17 (B1); no longer U10.8 (A6)
- net GFX_A2: now also U10.16 (B2); no longer U10.7 (A5)
- net GFX_A3: now also U10.15 (B3); no longer U10.6 (A4)
- net GFX_A4: now also U10.14 (B4); no longer U10.5 (A3)
- net GFX_A5: now also U10.13 (B5); no longer U10.4 (A2)
- net GFX_A6: now also U10.12 (B6); no longer U10.3 (A1)
- net GFX_A7: now also U10.11 (B7); no longer U10.2 (A0)
- net GFX_A8: now also U11.11 (B7); no longer U11.9 (A7)
- net GFX_D0: now also U12.18 (B0); no longer U12.9 (A7)
- net GFX_D1: now also U12.17 (B1); no longer U12.8 (A6)
- net GFX_D2: now also U12.16 (B2); no longer U12.7 (A5)
- net GFX_D3: now also U12.15 (B3); no longer U12.6 (A4)
- net GFX_D4: now also U12.14 (B4); no longer U12.5 (A3)
- net GFX_D5: now also U12.13 (B5); no longer U12.4 (A2)
- net GFX_D6: now also U12.12 (B6); no longer U12.3 (A1)
- net GFX_D7: now also U12.11 (B7); no longer U12.2 (A0)
- net GFX_~{CAS_0}: now also U11.13 (B5); no longer U11.7 (A5)
- net GFX_~{CAS_1}: now also U11.14 (B4); no longer U11.6 (A4)
- net GFX_~{RAS}: now also U11.12 (B6); no longer U11.8 (A6)
- net GFX_~{WE}: now also U11.15 (B3); no longer U11.5 (A3)
- net GND: now also U10.1 (A->B), U11.1 (A->B), U2.7 (GND), C25.2, C26.2, C27.2, C28.2, C29.2, C30.2, C31.2, C32.2, C33.2, C34.2, C35.2, C36.2, C37.2, C38.2, C39.2, C40.2, C41.2, C42.2, C43.2, C44.2, C45.2, C68.2, R27.2, U27.16 (GND), U37.16 (GND), X3.7 (GND); no longer U2.14 (VCC)
- net ISA_IRQ2: now also U6.9 (D7); no longer U6.2 (D0)
- net ISA_IRQ3: now also U6.8 (D6); no longer U6.3 (D1)
- net ISA_IRQ4: now also U6.7 (D5); no longer U6.4 (D2)
- net ISA_IRQ5: now also U6.6 (D4); no longer U6.5 (D3)
- net ISA_IRQ6: now also U6.5 (D3); no longer U6.6 (D4)
- net ISA_IRQ7: now also U6.4 (D2); no longer U6.7 (D5)
- net ~{ISA_IO_CH_CK}: now also U6.3 (D1); no longer U6.8 (D6)
- net ~{LAN_IRQ}: now also U6.2 (D0); no longer U6.9 (D7)
- net ~{LAN_SEL}: no longer U18.10 (O5)
- net ~{ROM0_SEL}: now also U27.22 (CE), U37.22 (CE)
- net at U5.16 (Q6): now also JP3.2 (B)
- net Power/I2C_EN: now reaches U5.19 (Q7)
- net BUF_~{RD}: now reaches U7.10
- net BUF_~{RD}: now also U27.24 (OE), U37.24 (OE)
- net at U33.11: now also U12.1 (A->B)
- net ~{MIO0_SEL} renamed ~{MIO_SEL}
- new net Power/PWR_OFF: JP3.1 (A), R27.1
- new net SYS_CLK: X3.8 (OUT)
Other:
- added sheet Power (power.kicad_sch)
- sheet ISA ports: added none; removed OSC
- sheet MIO ports: added none; removed DRQ1, ~{DACK1}, ~{MIO1_SEL}
- note removed: "For Ethernet, the Microchip KSZ8851-16MLL seems to be good choice. This used to be Micrel Ethernet controller with Linux and bare-metal driver support. https://ww1.microchip.com/downloads/aemDocuments/documents/OTH/ProductDocuments/DataSheets/KSZ8851-16MLL-Single-Port-Ethernet-MAC-Controller-with-8-Bit-or-16-Bit-Non-PCI-Interface-DS00002357B.pdf Another option is the ENC624J600, also from Microch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"
- note removed: "ISA OSC: 14.31818MHz"
- moved on the sheet: U22D, U2A, U2B, U2D, U2E, U5, U7A, U7E
