File: boards/a1_mega/cpu.kicad_sch (KiCad schematic)
At the start: 1 part, among them U19 ESPRESSO

Commit message: USB HUB 'chip' created and added; only a single MIO 'chip' is left in the design.
Connections:
- net BRQ renamed DRQ_0
- net ~{BGNT} renamed ~{DACK_0}
Changed lines of the file:
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@@
     (effects (font (size 1.27 1.27)) (justify left))
   )
-  (hierarchical_label "BRQ" (shape input) (at 147.32 91.44 0) (fields_autoplaced)
+  (hierarchical_label "DRQ_0" (shape input) (at 147.32 91.44 0) (fields_autoplaced)
     (effects (font (size 1.27 1.27)) (justify left))
   )
@@
     (effects (font (size 1.27 1.27)) (justify right))
   )
-  (hierarchical_label "~{BGNT}" (shape output) (at 147.32 93.98 0) (fields_autoplaced)
+  (hierarchical_label "~{DACK_0}" (shape output) (at 147.32 93.98 0) (fields_autoplaced)
     (effects (font (size 1.27 1.27)) (justify left))
   )

Commit message: It seems motherboard is feature-complete. Routing started.
Parts:
- added C46: 1uF, Capacitor_THT:C_Disc_D4.7mm_W2.5mm_P5.00mm, symbol Device:C
Connections:
- net +5V: now also C46.1
- net GND: now also C46.2
Changed lines of the file:
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@@
+    )
+  )
+  (symbol (lib_id "power:+5V") (at 186.69 86.36 0) (unit 1)
+    (in_bom yes) (on_board yes) (dnp no) (fields_autoplaced)
+    (property "Reference" "#PWR0219" (at 186.69 90.17 0)
+      (effects (font (size 1.27 1.27)) hide)
+    )
+    (property "Value" "+5V" (at 186.69 81.28 0)
+      (effects (font (size 1.27 1.27)))
+    )
+    (property "Footprint" "" (at 186.69 86.36 0)
+      (effects (font (size 1.27 1.27)) hide)
+    )
+    (property "Datasheet" "" (at 186.69 86.36 0)
+      (effects (font (size 1.27 1.27)) hide)
+    )
+    (pin "1")
+    (instances
+      (project "a1_mega"
+        (path "/3257e1ae-50a8-410a-87c3-a39d96a2c51a/894d02d2-0889-4880-8f04-ac96b9bee43e"
+          (reference "#PWR0219") (unit 1)
+        )
+      )
     )
   )
@@
         (path "/3257e1ae-50a8-410a-87c3-a39d96a2c51a/894d02d2-0889-4880-8f04-ac96b9bee43e"
           (reference "#PWR048") (unit 1)
+        )
+      )
+    )
+  )
+  (symbol (lib_id "power:GND") (at 186.69 93.98 0) (unit 1)
+    (in_bom yes) (on_board yes) (dnp no) (fields_autoplaced)
+    (property "Reference" "#PWR0220" (at 186.69 100.33 0)
+      (effects (font (size 1.27 1.27)) hide)
+    )
+    (property "Value" "GND" (at 186.69 99.06 0)
+      (effects (font (size 1.27 1.27)))
+    )
+    (property "Footprint" "" (at 186.69 93.98 0)
+      (effects (font (size 1.27 1.27)) hide)
+    )
+    (property "Datasheet" "" (at 186.69 93.98 0)
+      (effects (font (size 1.27 1.27)) hide)
+    )
+    (pin "1")
+    (instances
+      (project "a1_mega"
+        (path "/3257e1ae-50a8-410a-87c3-a39d96a2c51a/894d02d2-0889-4880-8f04-ac96b9bee43e"
+          (reference "#PWR0220") (unit 1)
         )
       )
@@
         )
       )
+    )
+  )
+  (symbol (lib_id "Device:C") (at 186.69 90.17 0) (unit 1)
+    (in_bom yes) (on_board yes) (dnp no) (fields_autoplaced)
+    (property "Reference" "C46" (at 190.5 88.9 0)
+      (effects (font (size 1.27 1.27)) (justify left))
+    )
+    (property "Value" "1uF" (at 190.5 91.44 0)
+      (effects (font (size 1.27 1.27)) (justify left))
+    )
+    (property "Footprint" "Capacitor_THT:C_Disc_D4.7mm_W2.5mm_P5.00mm" (at 187.6552 93.98 0)
+      (effects (font (size 1.27 1.27)) hide)
+    )
+    (property "Datasheet" "~" (at 186.69 90.17 0)
+      (effects (font (size 1.27 1.27)) hide)
+    )
+    (property "mpf#" "FG28X5R1H105KRT06" (at 186.69 90.17 0)
+      (effects (font (size 1.27 1.27)) hide)
+    )
+    (pin "2")
+    (pin "1")
+    (instances
+      (project "a1_mega"
+        (path "/3257e1ae-50a8-410a-87c3-a39d96a2c51a/894d02d2-0889-4880-8f04-ac96b9bee43e"
+          (reference "C46") (unit 1)
+        )
+      )
