File: boards/a1_mega/graphics.kicad_sch (KiCad schematic)
At the start: 16 parts, among them J5 Conn_01x02, J6 HDMI_A, U24 DISCO, U25 NAU8822, U35 74LVC06, X1 CXO_DIP14

Commit message: Extracted LAN chip, more progress towards full schematic.
Parts:
- removed C1: 4.7uF, Capacitor_THT:C_Rect_L9.0mm_W2.5mm_P7.50mm_MKT, symbol Device:C
- removed TP1: TestPoint_Alt, TestPoint:TestPoint_Plated_Hole_D2.0mm, symbol Connector:TestPoint
- removed U35: 74LVC06, Package_DIP:DIP-14_W7.62mm_LongPads, symbol 74xx:74LS06
- added C1, C13: 1uF, Capacitor_THT:CP_Radial_D4.0mm_P2.00mm, symbol Device:C_Polarized_Small_US
- added C14: 4.7uF, Capacitor_THT:CP_Radial_D4.0mm_P2.00mm, symbol Device:C_Polarized_Small_US
- added J12, J13: SJ1-3535NG-BE, anachron:CUI_SJ1-3535NG-BE, symbol anachron:SJ1-3535NG-BE
- added JP1: Jumper_3_Open, Connector_PinHeader_2.54mm:PinHeader_1x03_P2.54mm_Vertical, symbol Jumper:Jumper_3_Open
- added R18, R20, R21, R7: 47k, Resistor_THT:R_Axial_DIN0204_L3.6mm_D1.6mm_P5.08mm_Horizontal, symbol Device:R_US
- added R19: 220k, Resistor_THT:R_Axial_DIN0204_L3.6mm_D1.6mm_P5.08mm_Horizontal, symbol Device:R_US
- R1: value 10k -> 220k
- U25: value NAU8822 -> A1_CODEC; footprint Package_DFN_QFN:QFN-32-1EP_5x5mm_P0.5mm_EP3.1x3.1mm -> Package_DIP:DIP-32_W15.24mm_LongPads; symbol anachron:NAU8822 -> anachron:A1_CODEC
Connections:
- net +5V: now also U25.32 (VCC_5), JP1.1 (A); no longer U25.26 (VDDSPK)
- net AUDIO_SFRM: now also U25.27 (FS); no longer U25.7 (FS)
- net BUSY/BRQ: now also U24.31 (~{BUSY}); no longer U24.30 (BUSY/BRQ)
- net CODEC_SCL: now also U25.3 (SDIO); no longer U25.17 (SDIO)
- net CODEC_SDA: now also U25.2 (SCLK); no longer U25.16 (SCLK)
- net GND: now also U25.10 (AGND), U25.16 (AGND), U25.17 (AGND), U25.23 (AGND), U25.26 (AGND), U25.4 (GND), C14.2, J12.1, J13.1, R18.2, R20.2, R21.2, R7.2; no longer U25.12 (VSSD), U25.18 (MODE), U25.24 (VSSSPK), U25.28 (VSSA), U25.EP (VSS)
- net SYS_CLK: now also U24.29 (SYS_CLK), U25.28 (BCLK), U25.31 (MCLK); no longer U24.28 (SYS_CLK)
- net ~{CAS_0}: now also U24.24 (~{CAS_0}); no longer U24.23 (~{CAS_0})
- net ~{CAS_1}: now also U24.25 (~{CAS_1}); no longer U24.24 (~{CAS_1})
- net ~{INT}: now also U24.30 (~{INT}); no longer U24.29 (~{INT})
- net ~{RAS_A}: now also U24.23 (~{RAS_A}); no longer U24.22 (~{RAS_A})
- net ~{REG_SEL}: now also U24.26 (~{REG_SEL}); no longer U24.25 (~{REG_SEL})
- net ~{RST}: now also U24.28 (~{RST}); no longer U24.27 (~{RST})
- net ~{WAIT}/~{BGNT}: no longer U24.31 (~{WAIT}/~{BGNT})
- net ~{WE}: now also U24.27 (~{WE}); no longer U24.26 (~{WE})
- net at C2.1: now also U25.15 (LHP); no longer U25.30 (LHP)
- net at C2.2: now also J12.2, R18.1
- net at U25.1 (CSB/GPIO1): now also TP2.1
- net at U25.11 (RSPKOUT): now also J5.2 (Pin_2); no longer U25.8 (BCLK)
- net at J5.1 (Pin_1): now also U25.12 (LSPKOUT); no longer U25.25 (LSPKOUT)
- net at C3.1: now also U25.14 (RHP); no longer U25.29 (RHP)
- net at FB1.2: now also U25.13 (V_SPKR), C14.1; no longer U25.31 (VDDA)
- net CODEC_V3P3: now reaches U25.5 (3P3_OUT)
- net CODEC_V3P3: now also R1.1, JP1.3 (B), R19.1
- net at U25.6 (RAUXIN): now also C13.1
- net at C3.2: now also J12.3, R7.1
- removed net +3V3: FB1.1, R1.1, U25.13 (VDDC), U25.14 (VDDB)
- net AUDIO_SDATA renamed AUDIO_SDATA_OUT
- net AUDIO_SDATA_OUT: now also U25.30 (DACIN); no longer U25.10 (DACIN)
- net JACK_DET renamed HP_DET
- net HP_DET: now also U25.24 (LLIN/GPIO2), J12.4; no longer U25.3 (LLIN/GPIO2)
- new net: C13.2, J13.3, R21.1
- new net: C1.1, U25.7 (LAUXIN)
- new net: C1.2, J13.2, R20.1
- new net: FB1.1, JP1.2 (C)
- new net AUDIO_SDATA_IN: U24.22 (AUDIO_SDATA_IN), U25.29 (ADCOUT)
- new net LINE_IN_DET: J13.4, R19.2, U25.25 (RLIN/GPIO3)
Other:
- moved on the sheet: C2, C3, F1, FB1, J6, R1, R2, R3, X1

Commit message: USB HUB 'chip' created and added; only a single MIO 'chip' is left in the design.
Parts:
- U24: footprint Package_DIP:DIP-40_W15.24mm_Socket_LongPads -> anachron:DIP-40_W15.24mm_Socket
Connections:
- net BUSY/BRQ renamed ~{BUSY}
Changed lines of the file:
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@@
-    (stroke (width 0) (type default))
-  )
-  (wire (pts (xy 118.11 40.64) (xy 138.43 40.64))
     (stroke (width 0) (type default))
   )
@@
     (effects (font (size 1.27 1.27)) (justify right))
   )
-  (hierarchical_label "~{WAIT}{slash}~{BGNT}" (shape input) (at 138.43 40.64 0) (fields_autoplaced)
-    (effects (font (size 1.27 1.27)) (justify left))
-  )
-  (hierarchical_label "BUSY{slash}BRQ" (shape output) (at 138.43 38.1 0) (fields_autoplaced)
+  (hierarchical_label "~{BUSY}" (shape output) (at 138.43 38.1 0) (fields_autoplaced)
     (effects (font (size 1.27 1.27)) (justify left))
   )
@@
       (effects (font (size 1.27 1.27)) (justify left))
     )
-    (property "Footprint" "Package_DIP:DIP-40_W15.24mm_Socket_LongPads" (at 123.19 100.33 0)
-      (effects (font (size 1.27 1.27)) hide)
-    )
+    (property "Footprint" "anachron:DIP-40_W15.24mm_Socket" (at 123.19 100.33 0)
+      (effects (font (size 1.27 1.27)) hide)
+    )

Commit message: It seems motherboard is feature-complete. Routing started.
Parts:
- added C57, C58, C59: 1uF, Capacitor_THT:C_Disc_D4.7mm_W2.5mm_P5.00mm, symbol Device:C
- added CMC1, CMC2, CMC3, CMC4: L_Ferrite_Coupled_Small, anachron:SCM2012FS, symbol Device:L_Ferrite_Coupled_Small_1243
- added FB13, FB14, FB15, FB16, FB17, FB18, FB19, FB20: FerriteBead_Small, Inductor_THT:L_Axial_L7.0mm_D3.3mm_P2.54mm_Vertical_Fastron_MICC, symbol Device:FerriteBead_Small
- F1: value Polyfuse -> 0.5A; footprint Fuse:Fuse_Littelfuse_395Series -> Fuse:Fuse_BelFuse_0ZRE0005FF_L8.3mm_W3.8mm; mpf# (none) -> 0ZRC0050FF1E
Connections:
- net +5V: now also C57.1, C58.1, C59.1
- net GND: now also C57.2, C58.2, C59.2
- net VIDEO_DDC_SCL: now also FB13.1; no longer J6.15 (SCL)
- net VIDEO_DDC_SDA: now also FB14.1; no longer J6.16 (SDA)
- net VIDEO_HPD: now also FB20.1; no longer J6.19 (HPD)
- net at C3.2, R7.1: now also FB17.2; no longer J12.3
- net at C13.2, R21.1: now also FB19.2; no longer J13.3
- net at C1.2, R20.1: now also FB18.2; no longer J13.2
- net at C2.2, R18.1: now also FB16.2; no longer J12.2
- net at J6.18 (+5V): now also FB15.1; no longer F1.1
- net at U24.1 (TMDS_D2+): now also CMC1.1; no longer J6.1 (D2+)
- net at U24.7 (TMDS_C+): now also CMC4.1; no longer J6.10 (CK+)
- net at J6.12 (CK-): now also CMC4.3; no longer U24.8 (TMDS_C-)
- net at J6.3 (D2-): now also CMC1.3; no longer U24.2 (TMDS_D2-)
- net at J6.4 (D1+): now also CMC2.2; no longer U24.3 (TMDS_D1+)
- net at J6.6 (D1-): now also CMC2.3; no longer U24.4 (TMDS_D1-)
- net at U24.5 (TMDS_D0+): now also CMC3.1; no longer J6.7 (D0+)
- net at J6.9 (D0-): now also CMC3.3; no longer U24.6 (TMDS_D0-)
- new net: CMC4.2, J6.10 (CK+)
- new net: CMC4.4, U24.8 (TMDS_C-)
- new net: FB16.1, J12.2
- new net: FB17.1, J12.3
- new net: FB19.1, J13.3
- new net: FB13.2, J6.15 (SCL)
- new net: F1.1, FB15.2
- new net: FB14.2, J6.16 (SDA)
- new net: CMC1.2, J6.1 (D2+)
- new net: CMC1.4, U24.2 (TMDS_D2-)
- new net: FB18.1, J13.2
- new net: FB20.2, J6.19 (HPD)
- new net: CMC3.2, J6.7 (D0+)
- new net: CMC3.4, U24.6 (TMDS_D0-)
- new net: CMC2.1, U24.3 (TMDS_D1+)
- new net: CMC2.4, U24.4 (TMDS_D1-)
Other:
- moved on the sheet: C1, C13, F1, R20, R21
