File: boards/a1_mega/isa.kicad_sch (KiCad schematic)
At the start: 12 parts, among them J1 Bus_ISA_8bit, J2 Bus_ISA_8bit, J3 Bus_ISA_8bit, J4 Bus_ISA_8bit, U1 74LS139, U22 74LS125, U23 74LS125, U7 74LS04, U9 74LS86

Commit message: It seems motherboard is feature-complete. Routing started.
Parts:
- added C15, C16, C51, C56: 1uF, Capacitor_THT:C_Disc_D4.7mm_W2.5mm_P5.00mm, symbol Device:C
- added JP4: Jumper_3_Bridged12, Connector_PinHeader_2.54mm:PinHeader_1x03_P2.54mm_Vertical, symbol Jumper:Jumper_3_Bridged12
- added U35: L79L05_TO92, Package_TO_SOT_THT:TO-92_Inline, symbol Regulator_Linear:L79L05_TO92
- added X4: 14.31818MHz, Oscillator:Oscillator_DIP-14, symbol Oscillator:CXO_DIP14
Connections:
- net +5V: now also C51.1, C56.1, X4.1 (EN), X4.14 (Vcc)
- net GND: now also C15.2, C16.2, C51.2, C56.2, U35.1 (GND), X4.7 (GND)
- net ISA_-5V: now also C15.1, U35.3 (VO)
- net SYS_CLK: now also JP4.1 (A)
- net ISA_+12V renamed +12V
- net ISA_-12V renamed -12V
- net -12V: now also C16.1, U35.2 (VI)
- net OSC renamed ISA_OSC
- net ISA_OSC: now also JP4.2 (C)
- new net: JP4.3 (B), X4.8 (OUT)
Other:
- note added: "Optional oscillator in case there's a bunch of problems with feeding just SYS_CLK to this ISA pin."
- moved on the sheet: RN4, RN5, RN7, U22E, U23E
