File: boards/a1_mega/memory.kicad_sch (KiCad schematic)
At the start: 2 parts, among them U20 SIMM-30, U21 SIMM-30

Commit message: It seems motherboard is feature-complete. Routing started.
Parts:
- added C47, C48, C49, C50: 1uF, Capacitor_THT:C_Disc_D4.7mm_W2.5mm_P5.00mm, symbol Device:C
Connections:
- net +5V: now also C47.1, C48.1, C49.1, C50.1
- net GND: now also C47.2, C48.2, C49.2, C50.2
