File: boards/a1_mega/mio.kicad_sch (KiCad schematic)
At the start: 50 parts, among them J10 DE9_Plug, J11 RJ45_Amphenol_RJMG1BD3B8K1ANR, J7 Micro_SD_Card, J8 USB_A_Stacked, J9 USB_A_Stacked, U26 MIO, U27 MIO, U28 MAX232, U29 DS1307+, U32 KSZ8851-11MLL, U33 93CxxA, U34 74LVC245, U35 74LVC06, U37 74LVC06, X2 48MHz, Y1 32768Hz, Y2 25MHz

Commit message: Extracted LAN chip, more progress towards full schematic.
Parts:
- removed FB2, FB3: FerriteBead_Small, Inductor_THT:L_Axial_L5.3mm_D2.2mm_P7.62mm_Horizontal_Vishay_IM-1, symbol Device:FerriteBead_Small
- removed R10: 0, Resistor_THT:R_Axial_DIN0204_L3.6mm_D1.6mm_P5.08mm_Horizontal, symbol Device:R_US
- removed R11: 3.01k, Resistor_THT:R_Axial_DIN0204_L3.6mm_D1.6mm_P5.08mm_Horizontal, symbol Device:R_US
- removed U33: 93CxxA, Package_DIP:DIP-8_W7.62mm_LongPads, symbol Memory_EEPROM:93CxxC
- removed U34: 74LVC245, Package_DIP:DIP-20_W7.62mm_LongPads, symbol 74xx:74LS245
- removed U35, U37: 74LVC06, Package_DIP:DIP-14_W7.62mm_LongPads, symbol 74xx:74LS06
- R8, R9: value 1k -> 10k
- U32: footprint Package_QFP:LQFP-48_7x7mm_P0.5mm -> Package_DIP:DIP-32_W15.24mm_LongPads; symbol anachron:KSZ8851-16MLL -> anachron:A1_LAN
Connections:
- net +5V: now also R8.2, R9.2, U32.32 (VCC)
- net A0: now also U32.15 (CMD)
- net D0: now also U32.9 (D7)
- net D1: now also U32.8 (D6)
- net D2: now also U32.7 (D5)
- net D3: now also U32.6 (D4)
- net D4: now also U32.5 (D3)
- net D5: now also U32.4 (D2)
- net D6: now also U32.3 (D1)
- net D7: now also U32.2 (D0)
- net GND: now also U32.16 (GND), U32.19 (GND), U32.20 (GND), U32.24 (GND), U32.25 (GND); no longer R8.1, U32.13 (AGND), U32.18 (AGND), U32.26 (DGND), U32.30 (SD15), U32.32 (SD13), U32.33 (SD12), U32.34 (SD11), U32.35 (SD10), U32.36 (SD9), U32.37 (DGND), U32.39 (SD8), U32.7 (DGND)
- net ~{LAN_IRQ}: now also R8.1, U32.13 (~{INTR}); no longer U32.4 (~{INTR})
- net ~{LAN_SEL}: now also U32.17 (~{CS})
- net ~{LAN_WOL}: now also R9.1, U32.12 (PME); no longer U32.3 (PME)
- net ~{RST}: now also U32.18 (~{RST})
- net ~{WE}: now also U32.14 (~{WE})
- net at C8.1, Y2.1: now also U32.23 (XTAL2); no longer U32.25 (XTAL2)
- net at C9.1, Y2.2: now also U32.21 (XTAL1); no longer U32.24 (XTAL1)
- net at U32.29 (TXP1): now also J11.R1 (TD+), R16.2; no longer U32.8 (VDD1P8_OUT)
- net at J11.R3 (RD+), R14.2: now also U32.26 (RXP1); no longer U32.16 (RXP1)
- net at U32.10 (P1LED1): now also R13.1
- net at U32.11 (P1LED0): now also R12.1
- net at U32.22 (VDD3P3_A): now also C10.1, J11.R4 (TCT), J11.R5 (RCT)
- net at J11.R2 (TD-), R17.2: now also U32.30 (TXM1); no longer U32.20 (TXM1)
- net at J11.R6 (RD-), R15.2: now also U32.27 (RXM1); no longer U32.17 (RXM1)
- removed net +3V3: J11.L2, J11.L4, R9.2, U32.27 (VDDIO), U32.38 (VDDIO), U32.46 (VDDIO)
- new net: J11.L2, J11.L4, U32.1 (V3P3)
Other:
- moved on the sheet: C10, C11, C12, C8, C9, J11, R12, R13, R14, R15, R16, R17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

Commit message: USB HUB 'chip' created and added; only a single MIO 'chip' is left in the design.
Parts:
- removed F2, F3, F4, F5: Polyfuse, Fuse:Fuse_Littelfuse_395Series, symbol Device:Polyfuse
- removed R4: 10k, Resistor_THT:R_Axial_DIN0204_L3.6mm_D1.6mm_P5.08mm_Horizontal, symbol Device:R_US
- removed RN11, RN9: 15k, Resistor_THT:R_Array_SIP5, symbol Device:R_Network04_US
- removed U27: MIO, Package_DIP:DIP-40_W15.24mm_Socket_LongPads, symbol anachron:mio
- added C17, C18, C19, C20, C21, C22: 220uF, Capacitor_THT:CP_Radial_D7.5mm_P2.50mm, symbol Device:C_Polarized_Small_US
- added J14: USB_A_Stacked, Connector_USB:USB_A_CUI_UJ2-ADH-TH_Horizontal_Stacked, symbol Connector:USB_A_Stacked
- added JP2: Jumper_2_Open, Connector_PinHeader_2.54mm:PinHeader_1x02_P2.54mm_Vertical, symbol Jumper:Jumper_2_Open
- added U34: A1_USBHUB, anachron:DIP-40_W15.24mm_Socket, symbol anachron:A1_USBHUB
- U26: footprint Package_DIP:DIP-40_W15.24mm_Socket_LongPads -> anachron:DIP-40_W15.24mm_Socket
- X2: value 48MHz -> 24MHz
Connections:
- net KBD_CLK is gone; now on net VIDEO_DDC_SDA: U26.11 (PA4_SPIMISO_I2CSDA1)
- net KBD_DAT is gone; now on net VIDEO_DDC_SCL: U26.12 (PA5_SPICLK_I2CSCL1)
- net +5V: now also U34.15 (VCC), U34.16 (VCC), U34.17 (VCC), U34.18 (VCC), U34.19 (VCC), U34.40 (VCC)
- net GND: now also C17.2, C18.2, C19.2, C20.2, C21.2, C22.2, J14.4 (GND1), J14.8 (GND2), J14.9 (Shield), JP2.1 (A), U34.14 (GND), U34.20 (GND), U34.30 (GND), U34.31 (GND), U34.33 (CFG_SEL1)
- net I2C_SCL: now also RN8.5 (R4), U34.28 (SCL); no longer RN8.3 (R2)
- net I2C_SDA: now also RN8.4 (R3), U34.29 (SDA); no longer RN8.2 (R1)
- net USB_CLK: now also U34.2 (XTAL1/CLKIN)
- net VIDEO_DDC_SCL: now also RN8.3 (R2); no longer RN8.4 (R3)
- net VIDEO_DDC_SDA: now also RN8.2 (R1); no longer RN8.5 (R4)
- net VIDEO_HPD: now also U26.1 (PC0_USBa_D+)
- net ~{RST}: now also U34.32 (~{RST})
- net at J8.6 (D2-): now also U34.5 (USBDN2_DM); no longer U26.4 (PC3_USBb_D-)
- net at J8.7 (D2+): now also U34.6 (USBDN2_DP); no longer U26.3 (PC2_USBb_D+)
- net at J8.2 (D1-): now also U34.3 (USBDN1_DM); no longer U26.2 (PC1_USBa_D-)
- net at J8.3 (D1+): now also U34.4 (USBDN1_DP); no longer U26.1 (PC0_USBa_D+)
- net at J8.5 (VBUS2): now also C17.1, U34.25 (VBUS2)
- net at J9.3 (D1+): now also U34.8 (USBDN3_DP)
- net at J9.2 (D1-): now also U34.7 (USBDN3_DM)
- net at J9.7 (D2+): now also U34.10 (USBDN4_DP)
- net at J9.6 (D2-): now also U34.9 (USBDN4_DM)
- net at J9.1 (VBUS1): now also C19.1, U34.26 (VBUS3)
- net at J8.1 (VBUS1): now also C18.1, U34.24 (VBUS1)
- net USB_D+: now reaches U26.5 (PC4_USBc_D+)
- net USB_D+: now also U34.39 (USBUP_DP)
- net USB_D-: now reaches U26.6 (PC5_USBc_D-)
- net USB_D-: now also U34.38 (USBUP_DM)
- net at J9.5 (VBUS2): now also C20.1, U34.27 (VBUS4)
- new net: C21.1, J14.1 (VBUS1), U34.22 (VBUS5)
- new net: J14.2 (D1-), U34.11 (USBDN5_DM)
- new net: J14.3 (D1+), U34.12 (USBDN5_DP)
- new net: C22.1, J14.5 (VBUS2), U34.21 (VBUS6)
- new net: J14.6 (D2-), U34.34 (USBDN6_DM)
- new net: J14.7 (D2+), U34.35 (USBDN6_DP)
- new net: JP2.2 (B), U34.13 (CFG_SEL2)
- no-connect marks 0 -> 1
Other:
- moved on the sheet: BT1, C10, C11, C12, C4, C5, C6, C7, J10, J11, J7, J8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

Commit message: It seems motherboard is feature-complete. Routing started.
Parts:
- removed BT1: CR2032 holder, Battery:BatteryHolder_Keystone_103_1x20mm, symbol Device:Battery_Cell
- added C60, C61, C62, C63, C64, C65, C66: 1uF, Capacitor_THT:C_Disc_D4.7mm_W2.5mm_P5.00mm, symbol Device:C
- added CMC10, CMC5, CMC6, CMC7, CMC8, CMC9: L_Ferrite_Coupled_Small, anachron:SCM2012FS, symbol Device:L_Ferrite_Coupled_Small_1243
- added FB10, FB11, FB12, FB2, FB3, FB4, FB5, FB6, FB7, FB8, FB9: FerriteBead_Small, Inductor_THT:L_Axial_L7.0mm_D3.3mm_P2.54mm_Vertical_Fastron_MICC, symbol Device:FerriteBead_Small
- added R28, R4: 10k, Resistor_THT:R_Axial_DIN0204_L3.6mm_D1.6mm_P5.08mm_Horizontal, symbol Device:R_US
- C11, C12: footprint Capacitor_THT:C_Rect_L9.0mm_W2.5mm_P7.50mm_MKT -> Capacitor_THT:C_Disc_D3.4mm_W2.1mm_P2.50mm; mpf# (none) -> 1C25Z5U104M050B
- C17, C18, C19, C20, C21, C22: value 220uF -> 100uF; footprint Capacitor_THT:CP_Radial_D7.5mm_P2.50mm -> Capacitor_THT:CP_Radial_D5.0mm_P2.00mm
- C4, C5, C6, C7: footprint Capacitor_THT:C_Rect_L9.0mm_W2.5mm_P7.50mm_MKT -> Capacitor_THT:C_Disc_D4.7mm_W2.5mm_P5.00mm; mpf# (none) -> FG28X5R1H105KRT06
- C8, C9: footprint Capacitor_THT:C_Rect_L9.0mm_W2.5mm_P7.50mm_MKT -> Capacitor_THT:C_Disc_D3.4mm_W2.1mm_P2.50mm
- J11: value RJ45_Amphenol_RJMG1BD3B8K1ANR -> ~; footprint Connector_RJ:RJ45_Amphenol_RJMG1BD3B8K1ANR -> anachron:ARJM11D7-009-AB-EW2; mpf# (none) -> ARJM11D7-009-AB-EW2
- J14, J8, J9: footprint Connector_USB:USB_A_CUI_UJ2-ADH-TH_Horizontal_Stacked -> anachron:GCT_USB1035-XX-X-X-X-B_REVE; mpf# (none) -> USB1035-GF-P-0-B-B
- J7: footprint Connector_Card:microSD_HC_Hirose_DM3BT-DSF-PEJS -> anachron:GCT_MEM2052-00-195-00-A_REVA
- U29, Y1: now not fitted
Connections:
- net +5V: now also C60.1, C61.1, C62.1, C63.1, C64.1, C65.1, C66.1, R28.2, R4.2
- net GND: now also C60.2, C61.2, C62.2, C63.2, C64.2, C65.2, C66.2
- net I2C_SCL: no longer RN10.3 (R2)
- net I2C_SDA: no longer RN10.2 (R1)
- net ~{RTC_INT}: now also U26.3 (PC2_USBb_D+), R28.1
- net at J10.2: now also FB11.2; no longer U28.13 (R1IN)
- net at J10.3: now also FB9.2; no longer U28.14 (T1OUT)
- net at C6.2, U28.2 (VS+): now also FB8.1; no longer J10.4
- net at J10.7: now also FB10.2; no longer U28.7 (T2OUT)
- net at J10.8: now also FB12.2; no longer U28.8 (R2IN)
- net at C21.1, J14.1 (VBUS1): now also FB7.2; no longer U34.22 (VBUS5)
- net at J14.2 (D1-): now also CMC9.3; no longer U34.11 (USBDN5_DM)
- net at J14.3 (D1+): now also CMC9.2; no longer U34.12 (USBDN5_DP)
- net at C22.1, J14.5 (VBUS2): now also FB6.2; no longer U34.21 (VBUS6)
- net at J14.6 (D2-): now also CMC10.3; no longer U34.34 (USBDN6_DM)
- net at J14.7 (D2+): now also CMC10.2; no longer U34.35 (USBDN6_DP)
- net +BATT: now reaches U29.3 (VBAT)
- net at C20.1, J9.5 (VBUS2): now also FB3.2; no longer U34.27 (VBUS4)
- net at C19.1, J9.1 (VBUS1): now also FB2.2; no longer U34.26 (VBUS3)
- net at J9.2 (D1-): now also CMC7.2; no longer U34.7 (USBDN3_DM)
- net at J9.3 (D1+): now also CMC7.3; no longer U34.8 (USBDN3_DP)
- net at J9.6 (D2-): now also CMC8.2; no longer U34.9 (USBDN4_DM)
- net at J9.7 (D2+): now also CMC8.3; no longer U34.10 (USBDN4_DP)
- net at C18.1, J8.1 (VBUS1): now also FB4.2; no longer U34.24 (VBUS1)
- net at J8.2 (D1-): now also CMC5.2; no longer U34.3 (USBDN1_DM)
- net at J8.3 (D1+): now also CMC5.3; no longer U34.4 (USBDN1_DP)
- net at C17.1, J8.5 (VBUS2): now also FB5.2; no longer U34.25 (VBUS2)
- net at U34.5 (USBDN2_DM): now also CMC7.1; no longer J8.6 (D2-)
- net at U34.6 (USBDN2_DP): now also CMC7.4; no longer J8.7 (D2+)
- net at U26.2 (PC1_USBa_D-): now also J7.9 (DET), R4.1
- net at U34.23 (VBUS7): now also FB7.1
- net at U34.36 (USBDN7_DM): now also CMC9.4
- net at U34.37 (USBDN7_DP): now also CMC9.1
- new net: FB8.2, J10.4
- new net: FB9.1, U28.14 (T1OUT)
- new net: FB11.1, U28.13 (R1IN)
- new net: FB10.1, U28.7 (T2OUT)
- new net: FB12.1, U28.8 (R2IN)
- new net: FB5.1, U34.22 (VBUS5)
- new net: CMC5.1, U34.9 (USBDN4_DM)
- new net: CMC5.4, U34.10 (USBDN4_DP)
- new net: CMC8.1, U34.7 (USBDN3_DM)
- new net: CMC8.4, U34.8 (USBDN3_DP)
- new net: FB3.1, U34.26 (VBUS3)
- new net: CMC6.2, J8.6 (D2-)
- new net: CMC6.3, J8.7 (D2+)
- new net: FB4.1, U34.27 (VBUS4)
- new net: CMC10.1, U34.35 (USBDN6_DP)
- new net: CMC10.4, U34.34 (USBDN6_DM)
- new net: FB6.1, U34.21 (VBUS6)
- new net: FB2.1, U34.25 (VBUS2)
- new net: CMC6.1, U34.11 (USBDN5_DM)
- new net: CMC6.4, U34.12 (USBDN5_DP)
Other:
- note added: "Replaced by AtTiny MCU in power section"
- moved on the sheet: C17, C18, C19, C20, C21, C22, J10, J14, J7, J8, J9
