File: boards/a1_usbhub/a1_usbhub.kicad_pcb (KiCad board)
At the start: 2 copper layers, 49.4 x 15.2 mm, 32 parts, among them U1 TXS0102DCT, U2 USB2517I-JZX, U3 AP62150Z6, U4 TPS2054D, U5 TPS2054D, U6 74LVC1G17

Commit message: USB HUB is back in.
Parts:
- turned SOCKET2 to -90 degrees
Connections:
- SOCKET2 pad 1: /XTAL2 -> /VBUS6
- SOCKET2 pad 10: /USBDN4_DP -> GND
- SOCKET2 pad 11: /USBDN5_DM -> GND
- SOCKET2 pad 12: /USBDN5_DP -> /~{RST}
- SOCKET2 pad 13: /CFG_SEL2 -> /CFG_SEL1
- SOCKET2 pad 14: GND -> /USBDN6_DM
- SOCKET2 pad 15: +5V -> /USBDN6_DP
- SOCKET2 pad 16: +5V -> /USBDN7_DM
- SOCKET2 pad 17: +5V -> /USBDN7_DP
- SOCKET2 pad 18: +5V -> /USBUP_DM
- SOCKET2 pad 19: +5V -> /USBUP_DP
- SOCKET2 pad 2: /XTAL1 -> /VBUS5
- SOCKET2 pad 21: /VBUS6 -> /XTAL2
- SOCKET2 pad 22: /VBUS5 -> /XTAL1
- SOCKET2 pad 23: /VBUS7 -> /USBDN1_DM
- SOCKET2 pad 24: /VBUS1 -> /USBDN1_DP
- SOCKET2 pad 25: /VBUS2 -> /USBDN2_DM
- SOCKET2 pad 26: /VBUS3 -> /USBDN2_DP
- SOCKET2 pad 27: /VBUS4 -> /USBDN3_DM
- SOCKET2 pad 28: /SCL -> /USBDN3_DP
- SOCKET2 pad 29: /SDA -> /USBDN4_DM
- SOCKET2 pad 3: /USBDN1_DM -> /VBUS7
- SOCKET2 pad 30: GND -> /USBDN4_DP
- SOCKET2 pad 31: GND -> /USBDN5_DM
- SOCKET2 pad 32: /~{RST} -> /USBDN5_DP
- SOCKET2 pad 33: /CFG_SEL1 -> /CFG_SEL2
- SOCKET2 pad 34: /USBDN6_DM -> GND
- SOCKET2 pad 35: /USBDN6_DP -> +5V
- SOCKET2 pad 36: /USBDN7_DM -> +5V
- SOCKET2 pad 37: /USBDN7_DP -> +5V
- SOCKET2 pad 38: /USBUP_DM -> +5V
- SOCKET2 pad 39: /USBUP_DP -> +5V
- SOCKET2 pad 4: /USBDN1_DP -> /VBUS1
- SOCKET2 pad 5: /USBDN2_DM -> /VBUS2
- SOCKET2 pad 6: /USBDN2_DP -> /VBUS3
- SOCKET2 pad 7: /USBDN3_DM -> /VBUS4
- SOCKET2 pad 8: /USBDN3_DP -> /SCL
- SOCKET2 pad 9: /USBDN4_DM -> /SDA
