File: boards/a1_mini/cpu.kicad_sch (KiCad schematic)
At the start: 2 parts, among them U19 ESPRESSO

Commit message: A1 Mini (which is not all that mini anymore) is feature-complete.
We have 2 ISA slots and even all the power supplies generated from +5V included.

The +12V switcher right next to the audio output is quite a bit concerning, but
we can always say that PWR must be 12V and we directly feed that to the ISA slots.
(Not that PWR is all that clean...) A lot will depend on how I implement grounding,
something that I still have to do.
Parts:
- renumbered C46 to C20
Changed lines of the file:
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@@
   (symbol (lib_id "power:GND") (at 106.68 134.62 0) (unit 1)
     (in_bom yes) (on_board yes) (dnp no) (fields_autoplaced)
-    (property "Reference" "#PWR049" (at 106.68 140.97 0)
+    (property "Reference" "#PWR0108" (at 106.68 140.97 0)
       (effects (font (size 1.27 1.27)) hide)
     )
@@
       (project "a1_mini"
         (path "/3257e1ae-50a8-410a-87c3-a39d96a2c51a/894d02d2-0889-4880-8f04-ac96b9bee43e"
-          (reference "#PWR049") (unit 1)
+          (reference "#PWR0108") (unit 1)
         )
       )
@@
   (symbol (lib_id "power:+5V") (at 186.69 86.36 0) (unit 1)
     (in_bom yes) (on_board yes) (dnp no) (fields_autoplaced)
-    (property "Reference" "#PWR0219" (at 186.69 90.17 0)
+    (property "Reference" "#PWR0109" (at 186.69 90.17 0)
       (effects (font (size 1.27 1.27)) hide)
     )
@@
       (project "a1_mini"
         (path "/3257e1ae-50a8-410a-87c3-a39d96a2c51a/894d02d2-0889-4880-8f04-ac96b9bee43e"
-          (reference "#PWR0219") (unit 1)
+          (reference "#PWR0109") (unit 1)
         )
       )
@@
   (symbol (lib_id "power:+5V") (at 106.68 48.26 0) (unit 1)
     (in_bom yes) (on_board yes) (dnp no) (fields_autoplaced)
-    (property "Reference" "#PWR048" (at 106.68 52.07 0)
+    (property "Reference" "#PWR0107" (at 106.68 52.07 0)
       (effects (font (size 1.27 1.27)) hide)
     )
@@
       (project "a1_mini"
         (path "/3257e1ae-50a8-410a-87c3-a39d96a2c51a/894d02d2-0889-4880-8f04-ac96b9bee43e"
-          (reference "#PWR048") (unit 1)
+          (reference "#PWR0107") (unit 1)
         )
       )
@@
   (symbol (lib_id "power:GND") (at 186.69 93.98 0) (unit 1)
     (in_bom yes) (on_board yes) (dnp no) (fields_autoplaced)
-    (property "Reference" "#PWR0220" (at 186.69 100.33 0)
+    (property "Reference" "#PWR0110" (at 186.69 100.33 0)
       (effects (font (size 1.27 1.27)) hide)
     )
@@
       (project "a1_mini"
         (path "/3257e1ae-50a8-410a-87c3-a39d96a2c51a/894d02d2-0889-4880-8f04-ac96b9bee43e"
-          (reference "#PWR0220") (unit 1)
+          (reference "#PWR0110") (unit 1)
         )
       )
@@
   (symbol (lib_id "Device:C") (at 186.69 90.17 0) (unit 1)
     (in_bom yes) (on_board yes) (dnp no) (fields_autoplaced)
-    (property "Reference" "C46" (at 190.5 88.9 0)
+    (property "Reference" "C20" (at 190.5 88.9 0)
       (effects (font (size 1.27 1.27)) (justify left))
     )
@@
       (project "a1_mini"
         (path "/3257e1ae-50a8-410a-87c3-a39d96a2c51a/894d02d2-0889-4880-8f04-ac96b9bee43e"
-          (reference "C46") (unit 1)
+          (reference "C20") (unit 1)
         )
       )
