File: boards/a1_mini/a1_mini.kicad_pcb (KiCad board)
At the start: 4 copper layers, 171.4 x 204.5 mm, 192 parts, among them J1 Jack-DC, J10 DE9_Plug, J11 USB_A_Stacked, J12 SJ1-3535NG-BE, J13 SJ1-3535NG-BE, J17 Conn_01x01, J18 Conn_01x01, J20 Conn_01x01, J22 Conn_01x01, J3 Conn_01x02, J4 USB_A_Stacked, J5 Conn_01x02, J6 HDMI_A, J7 Micro_SD_Card, J8 USB_A, J9 USB_A_Stacked, SW1 SW_Push, SW2 SW_Push, SW4 SW_DPDT_x2, U1 74LS139, U10 74AHCT245, U11 74AHCT245, U12 74AHCT245, U13 74AHCT245, U14 74AHCT245, U15 KSZ8851-11MLL, U16 74LS273, U17 74LS273, U18 A1_POWER, U19 ESPRESSO, U2 74LS14, U20 SIMM-30, U21 SIMM-30, U24 DISCO, U25 A1_CODEC, U26 MIO, U27 SST39SF040, U28 MAX232, U29 DS1307+, U3 74LS08, U30 SIMM-30, U31 SIMM-30, U33 74LS00, U4 74LS126, U5 74LS273, U6 74LS574, U7 A1_USBHUB, U8 74LS273, U9 74LS86, X1 CXO_DIP14, X2 24MHz, X3 8MHz, Y1 32768Hz, Y2 25MHz

Commit message: USB HUB is back in.
Parts:
- removed C37: 1uF, Capacitor_THT:C_Disc_D4.7mm_W2.5mm_P5.00mm
- removed CMC11: L_Ferrite_Coupled_Small, anachron:SCM2012FS
- removed F2: 0.5A, Fuse:Fuse_BelFuse_0ZRE0005FF_L8.3mm_W3.8mm
- removed FB21: FerriteBead_Small, Inductor_THT:L_Axial_L7.0mm_D3.3mm_P2.54mm_Vertical_Fastron_MICC
- removed J11: USB_A_Stacked, anachron:GCT_USB1035-XX-X-X-X-B_REVE
- C10: value 100uF -> 1uF; footprint Capacitor_THT:CP_Radial_D5.0mm_P2.00mm -> Capacitor_THT:C_Disc_D4.7mm_W2.5mm_P5.00mm
- J8: value USB_A -> USB_A_Stacked; footprint Connector_USB:USB_A_Molex_67643_Horizontal -> anachron:GCT_USB1035-XX-X-X-X-B_REVE
- SW4: footprint Button_Switch_THT:SW_E-Switch_EG2219_DPDT_Angled -> Button_Switch_THT:SW_CuK_JS202011CQN_DPDT_Straight
- U7: footprint anachron:DIP-40_W15.24mm_Socket -> Package_DIP:DIP-40_W15.24mm_LongPads
- moved SW4 237.5 mm to (45.1, 217.2), turned to -90 degrees
- moved J3 226.4 mm to (54.6, 223.5), turned to -90 degrees
- moved R5 163.2 mm to (132.7, 219.7)
- moved BT1 134.9 mm to (52.9, 124.5)
- moved Y1 125.7 mm to (54.0, 133.3), turned to 90 degrees
- moved U29 123.9 mm to (57.2, 127.0)
- moved C34 121.4 mm to (68.6, 120.7), turned to -90 degrees
- moved CMC9 109.5 mm to (142.2, 44.7), turned to 90 degrees
- moved CMC8 106.7 mm to (144.5, 44.7), turned to 90 degrees
- moved J9 105.1 mm to (146.7, 34.0), turned to 180 degrees
- moved FB6 101.0 mm to (149.2, 44.5), turned to 180 degrees
- moved U7 98.5 mm to (138.4, 78.1), turned to 90 degrees
- moved C9 97.9 mm to (189.9, 146.7), turned to -90 degrees
- moved FB5 95.4 mm to (154.9, 44.5), turned to 180 degrees
- moved JP2 93.3 mm to (167.0, 55.2)
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Connections:
- net Net-(D2-K) renamed /PWR_IN
- C10 pad 1: Net-(J4-VBUS1) -> +5V
- C19 pad 1: Net-(J11-VBUS1) -> Net-(J8-VBUS1)
- C20 pad 1: Net-(J8-VBUS) -> Net-(J4-VBUS1)
- C23 pad 1: Net-(J11-VBUS2) -> Net-(J8-VBUS2)
- CMC10 pad 2: Net-(J11-D2+) -> Net-(J8-D2+)
- CMC10 pad 3: Net-(J11-D2-) -> Net-(J8-D2-)
- CMC5 pad 1: Net-(U7-USBDN2_DM) -> Net-(U7-USBDN2_DP)
- CMC5 pad 2: Net-(J4-D1-) -> Net-(J4-D1+)
- CMC5 pad 3: Net-(J4-D1+) -> Net-(J4-D1-)
- CMC5 pad 4: Net-(U7-USBDN2_DP) -> Net-(U7-USBDN2_DM)
- CMC6 pad 1: Net-(U7-USBDN3_DM) -> Net-(U7-USBDN3_DP)
- CMC6 pad 2: Net-(J4-D2-) -> Net-(J4-D2+)
- CMC6 pad 3: Net-(J4-D2+) -> Net-(J4-D2-)
- CMC6 pad 4: Net-(U7-USBDN3_DP) -> Net-(U7-USBDN3_DM)
- CMC7 pad 1: /MIO/USB_D+ -> Net-(U7-USBDN7_DP)
- CMC7 pad 4: /MIO/USB_D- -> Net-(U7-USBDN7_DM)
- CMC8 pad 1: Net-(U7-USBDN4_DM) -> Net-(U7-USBDN4_DP)
- CMC8 pad 2: Net-(J9-D1-) -> Net-(J9-D1+)
- CMC8 pad 3: Net-(J9-D1+) -> Net-(J9-D1-)
- CMC8 pad 4: Net-(U7-USBDN4_DP) -> Net-(U7-USBDN4_DM)
- CMC9 pad 1: Net-(U7-USBDN5_DM) -> Net-(U7-USBDN5_DP)
- CMC9 pad 2: Net-(J9-D2-) -> Net-(J9-D2+)
- CMC9 pad 3: Net-(J9-D2+) -> Net-(J9-D2-)
- CMC9 pad 4: Net-(U7-USBDN5_DP) -> Net-(U7-USBDN5_DM)
- FB3 pad 1: Net-(F2-Pad1) -> Net-(U7-VBUS7)
- FB3 pad 2: Net-(J8-VBUS) -> Net-(J8-VBUS1)
- FB7 pad 2: Net-(J11-VBUS2) -> Net-(J8-VBUS2)
- J8 pad 1: Net-(J8-VBUS) -> Net-(J8-VBUS1)
- J8 pad 5: GND -> Net-(J8-VBUS2)
- U3 pad 1: /CPU_~{DACK0} -> /CPU_~{NREN}
- U3 pad 10: /CPU_~{DACK} -> /CPU_~{DACK2}
- U3 pad 11: /CPU_~{DACK} -> Net-(U3-Pad11)
- U3 pad 12: Net-(U3-Pad12) -> /CPU_~{DACK1}
- U3 pad 13: Net-(U3-Pad13) -> /CPU_~{DACK0}
- U3 pad 2: /CPU_~{DACK1} -> /CPU_~{DACK}
- U3 pad 3: Net-(U3-Pad13) -> /BUF_nEN
- U3 pad 4: /CPU_~{DACK2} -> Net-(U3-Pad11)
- U3 pad 5: /CPU_~{DACK3} -> Net-(U3-Pad5)
- U3 pad 6: Net-(U3-Pad12) -> /CPU_~{DACK}
- U3 pad 8: /BUF_nEN -> Net-(U3-Pad5)
- U3 pad 9: /CPU_~{NREN} -> /CPU_~{DACK3}
- U7 pad 1: unconnected-(U7-XTAL2-Pad1) -> Net-(U7-VBUS6)
- U7 pad 10: Net-(U7-USBDN4_DP) -> GND
- U7 pad 11: Net-(U7-USBDN5_DM) -> GND
- U7 pad 12: Net-(U7-USBDN5_DP) -> ~{RST}
- U7 pad 13: Net-(JP2-B) -> GND
- U7 pad 14: GND -> Net-(U7-USBDN6_DM)
- U7 pad 15: +5V -> Net-(U7-USBDN6_DP)
- U7 pad 16: +5V -> Net-(U7-USBDN7_DM)
- U7 pad 17: +5V -> Net-(U7-USBDN7_DP)
- U7 pad 18: +5V -> /MIO/USB_D-
- U7 pad 19: +5V -> /MIO/USB_D+
- U7 pad 2: /MIO/USB_CLK -> Net-(U7-VBUS5)
- U7 pad 21: Net-(U7-VBUS6) -> unconnected-(U7-XTAL2-Pad21)
- U7 pad 22: Net-(U7-VBUS5) -> /MIO/USB_CLK
- U7 pad 23: Net-(U7-VBUS7) -> unconnected-(U7-USBDN1_DM-Pad23)
- U7 pad 25: Net-(U7-VBUS2) -> Net-(U7-USBDN2_DM)
- U7 pad 26: Net-(U7-VBUS3) -> Net-(U7-USBDN2_DP)
- U7 pad 27: Net-(U7-VBUS4) -> Net-(U7-USBDN3_DM)
- U7 pad 28: /I2C_SDA -> Net-(U7-USBDN3_DP)
- U7 pad 29: /I2C_SCL -> Net-(U7-USBDN4_DM)
- U7 pad 3: unconnected-(U7-USBDN1_DM-Pad3) -> Net-(U7-VBUS7)
- U7 pad 30: GND -> Net-(U7-USBDN4_DP)
- U7 pad 31: GND -> Net-(U7-USBDN5_DM)
- U7 pad 32: ~{RST} -> Net-(U7-USBDN5_DP)
- U7 pad 33: GND -> Net-(JP2-B)
- U7 pad 34: Net-(U7-USBDN6_DM) -> GND
- U7 pad 35: Net-(U7-USBDN6_DP) -> +5V
- U7 pad 36: Net-(U7-USBDN7_DM) -> +5V
- U7 pad 37: Net-(U7-USBDN7_DP) -> +5V
- U7 pad 38: /MIO/USB_D- -> +5V
- U7 pad 39: /MIO/USB_D+ -> +5V
- U7 pad 5: Net-(U7-USBDN2_DM) -> Net-(U7-VBUS2)
- U7 pad 6: Net-(U7-USBDN2_DP) -> Net-(U7-VBUS3)
- U7 pad 7: Net-(U7-USBDN3_DM) -> Net-(U7-VBUS4)
- U7 pad 8: Net-(U7-USBDN3_DP) -> /I2C_SDA
- U7 pad 9: Net-(U7-USBDN4_DM) -> /I2C_SCL
- Y1 pad 1: Net-(U29-X1) -> Net-(U29-X2)
- Y1 pad 2: Net-(U29-X2) -> Net-(U29-X1)
Routing:
- net +5V: track 886.0 -> 1278.7 mm
- net GND: track 942.3 -> 1323.5 mm
- net Net-(U28-R1OUT): track 15.4 -> 275.4 mm
- net /MIO/SER_RXD: track 249.2 -> 3.70 mm
- net /PWR_IN: track 34.9 -> 269.7 mm, vias 0 -> 2
- net Net-(J3-Pin_2): track 28.3 -> 253.1 mm, vias 0 -> 2
- net /MIO/USB_CLK: track 17.7 -> 210.6 mm, vias 0 -> 2
- net Net-(U7-VBUS7): track 0.00 -> 95.3 mm
- net Net-(U7-VBUS6): track 0.00 -> 91.8 mm
- net Net-(JP3-A): track 179.7 -> 95.2 mm
- net Net-(U7-VBUS2): track 0.00 -> 76.9 mm
- net Net-(U7-VBUS3): track 0.00 -> 71.2 mm
- net /MIO/USB_D+: track 270.9 -> 207.6 mm, vias 1 -> 0
- net Net-(U7-USBDN6_DP): track 0.00 -> 63.1 mm, vias 0 -> 1
- net Net-(U7-USBDN6_DM): track 0.00 -> 61.5 mm, vias 0 -> 1
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
Commit message: Added boot mode switch, reworked LAN IRQ, places LEDs better.
Parts:
- added J11: Conn_01x02, Connector_PinSocket_2.54mm:PinSocket_1x02_P2.54mm_Vertical, F.Cu at (41.9, 182.9)
- added R26: 10k, Resistor_THT:R_Axial_DIN0204_L3.6mm_D1.6mm_P5.08mm_Horizontal, F.Cu at (46.4, 186.1)
- moved R9 135.3 mm to (48.3, 221.0), turned to 90 degrees
- moved D1 125.1 mm to (53.3, 219.1), turned to 90 degrees
- moved R13 109.8 mm to (32.4, 165.1), turned to 180 degrees
- moved D3 59.8 mm to (62.2, 219.1), turned to 90 degrees
- moved R11 12.7 mm to (79.4, 208.3)
Connections:
- R13 pad 1: Net-(U26-PC3_USBb_D-) -> Net-(U5-Q3)
- R14 pad 1: /CPU_~{INT} -> /LAN_~{INT}
- U15 pad 13: /CPU_~{INT} -> /LAN_~{INT}
- U26 pad 4: Net-(U26-PC3_USBb_D-) -> /LAN_~{INT}
- U5 pad 9: unconnected-(U5-Q3-Pad9) -> Net-(U5-Q3)
- U6 pad 2: unconnected-(U6-D0-Pad2) -> Net-(J11-Pin_2)
Routing:
- net /LAN_~{INT}: track 0.00 -> 301.1 mm, vias 0 -> 6
- net /CPU_~{INT}: track 431.4 -> 298.4 mm, vias 7 -> 4
- net Net-(D3-A): track 3.59 -> 80.0 mm
- net Net-(U5-Q3): track 0.00 -> 19.7 mm
- net Net-(J11-Pin_2): track 0.00 -> 13.7 mm
- net /CPU_TC: track 292.3 -> 280.6 mm
- net Net-(U26-PC3_USBb_D-): track 5.13 -> 0.00 mm
- net /BUF_~{CAS}: track 129.4 -> 125.0 mm
- net /~{SYS_GPIO2_SEL}: track 62.1 -> 65.6 mm
- net ~{RST}: track 559.7 -> 563.2 mm
- net /BUF_D6: track 243.1 -> 240.0 mm
- net /BUF_D4: track 232.0 -> 229.1 mm
- net /BUF_D3: track 233.0 -> 230.1 mm
- net /BUF_D7: track 239.2 -> 236.3 mm
- net /BUF_D5: track 243.1 -> 240.3 mm
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
Commit message: ISA is incorporated back into mini. Not routed yet.
Parts:
- added C24: 1uF, Capacitor_THT:C_Disc_D4.7mm_W2.5mm_P5.00mm, F.Cu at (19.6, 157.5)
- added C37: 1uF, Capacitor_THT:C_Disc_D4.7mm_W2.5mm_P5.00mm, F.Cu at (5.12, 57.1)
- added C51: 1uF, Capacitor_THT:C_Disc_D4.7mm_W2.5mm_P5.00mm, F.Cu at (19.6, 229.9)
- added C56: 1uF, Capacitor_THT:C_Disc_D4.7mm_W2.5mm_P5.00mm, F.Cu at (5.12, 65.9)
- added C64: 1uF, Capacitor_THT:C_Disc_D4.7mm_W2.5mm_P5.00mm, F.Cu at (19.6, 180.3)
- added C65: 1uF, Capacitor_THT:C_Disc_D4.7mm_W2.5mm_P5.00mm, F.Cu at (14.6, 203.2)
- added J14: Bus_ISA_8bit, anachron:BUS_XT_CONN, F.Cu at (-43.2, 48.3)
- added J15: Bus_ISA_8bit, anachron:BUS_XT_CONN, F.Cu at (-22.9, 48.3)
- added J16: Bus_ISA_8bit, anachron:BUS_XT_CONN, F.Cu at (-2.54, 48.3)
- added J19: Bus_ISA_8bit, anachron:BUS_XT_CONN, F.Cu at (17.8, 48.3)
- added JP4: Jumper_3_Bridged12, Connector_PinHeader_2.54mm:PinHeader_1x03_P2.54mm_Vertical, F.Cu at (15.2, 132.1)
- added R27: 10k, Resistor_THT:R_Axial_DIN0204_L3.6mm_D1.6mm_P5.08mm_Horizontal, F.Cu at (31.1, 151.1)
- added R29: 10k, Resistor_THT:R_Axial_DIN0204_L3.6mm_D1.6mm_P5.08mm_Horizontal, F.Cu at (63.5, 165.7)
- added RN5: 10k, Resistor_THT:R_Array_SIP9, F.Cu at (-33.0, 94.0)
- added RN7: 10k, Resistor_THT:R_Array_SIP5, F.Cu at (-33.0, 61.0)
- added U22: 74LS139, Package_DIP:DIP-16_W7.62mm_LongPads, F.Cu at (13.3, 207.0)
- added U23: L79L05_TO92, Package_TO_SOT_THT:TO-92_Inline, F.Cu at (7.98, 61.2)
- added U32: 4075, Package_DIP:DIP-14_W7.62mm_LongPads, F.Cu at (13.3, 161.3)
- added U34: 74LS14, Package_DIP:DIP-14_W7.62mm_LongPads, F.Cu at (13.3, 184.1)
- added X4: 14.31818MHz, Oscillator:Oscillator_DIP-14, F.Cu at (13.3, 137.2)
Connections:
- U1 pad 5: unconnected-(U1A-O1-Pad5) -> /~{ISA_SEL}
- U24 pad 31: /CPU_~{WAIT} -> /GFX/~{BUSY}
- U4 pad 1: unconnected-(U4-Pad1) -> /GFX/~{BUSY}
- U4 pad 10: /CPU_~{WAIT} -> Net-(U10-CE)
- U4 pad 13: /CPU_~{WAIT} -> Net-(U10-CE)
- U4 pad 2: unconnected-(U4-Pad2) -> GND
- U4 pad 3: unconnected-(U4-Pad3) -> /CPU_~{WAIT}
- U4 pad 4: unconnected-(U4-Pad4) -> /ISA/~{INT}
- U4 pad 5: unconnected-(U4-Pad5) -> GND
- U4 pad 6: unconnected-(U4-Pad6) -> /CPU_~{INT}
- U6 pad 3: unconnected-(U6-D1-Pad3) -> /ISA_CH_CK
- U6 pad 4: unconnected-(U6-D2-Pad4) -> /ISA_IRQ2
- U6 pad 5: unconnected-(U6-D3-Pad5) -> /ISA_IRQ3
- U6 pad 6: unconnected-(U6-D4-Pad6) -> /ISA_IRQ4
- U6 pad 7: unconnected-(U6-D5-Pad7) -> /ISA_IRQ5
- U6 pad 8: unconnected-(U6-D6-Pad8) -> /ISA_IRQ6
- U6 pad 9: unconnected-(U6-D7-Pad9) -> /ISA_IRQ7
- U9 pad 5: /CPU_~{WAIT} -> /GFX/~{BUSY}
Routing:
- net /GFX/~{BUSY}: track 0.00 -> 309.9 mm, vias 0 -> 5
- net /CPU_~{WAIT}: track 325.6 -> 109.6 mm, vias 7 -> 2
- net /CPU_~{INT}: track 298.4 -> 377.7 mm, vias 4 -> 6
- net Net-(U10-CE): track 145.7 -> 182.8 mm, vias 3 -> 4
- net /CPU_A8: track 233.0 -> 249.3 mm
- net GND: track 1323.5 -> 1328.5 mm
- net /ISA/~{INT}: track 0.00 -> 4.07 mm
- net /BUF_NREN: track 148.6 -> 145.0 mm, vias 6 -> 4
- net /CPU_TC: track 280.6 -> 277.4 mm
- net /BUF_~{NREN}: track 179.3 -> 182.3 mm
- net /~{GFX_SEL}: track 228.0 -> 229.8 mm
- net /LAN_~{INT}: track 301.1 -> 299.7 mm
- net Net-(U5-Q0): track 48.8 -> 47.7 mm
- net /CPU_A10: track 216.5 -> 217.4 mm
- net /CPU_A9: track 223.6 -> 224.4 mm
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
Commit message: Worked in wait-states for I/O, changed I/O address decode, added GPI pull-downs.
Parts:
- removed R26: 10k, Resistor_THT:R_Axial_DIN0204_L3.6mm_D1.6mm_P5.08mm_Horizontal
- moved RN5 123.0 mm to (53.3, 181.6), turned to 180 degrees
- moved J11 36.3 mm to (5.71, 186.1)
Connections:
- net /BUF_nEN renamed /BUF_~{EN}
- R27 pad 2: /GFX/~{BUSY} -> /GFX_~{BUSY}
- RN5 pad 2: /ISA_IRQ2 -> /ISA_IRQ7
- RN5 pad 3: /ISA_IRQ7 -> /ISA_IRQ6
- RN5 pad 4: /ISA_IRQ6 -> /ISA_IRQ5
- RN5 pad 5: /ISA_IRQ5 -> /ISA_IRQ4
- RN5 pad 6: /ISA_IRQ4 -> /ISA_IRQ3
- RN5 pad 7: /ISA_IRQ3 -> /ISA_IRQ2
- RN5 pad 8: unconnected-(RN5-R7-Pad8) -> /ISA_CH_CK
- RN5 pad 9: unconnected-(RN5-R8-Pad9) -> Net-(J11-Pin_2)
- U1 pad 13: /BUF_A16 -> /BUF_A13
- U1 pad 14: /BUF_A17 -> /BUF_A12
- U10 pad 19: Net-(U10-CE) -> /GFX_BUSY
- U11 pad 19: Net-(U10-CE) -> /GFX_BUSY
- U12 pad 19: Net-(U10-CE) -> /GFX_BUSY
- U2 pad 8: unconnected-(U2-Pad8) -> Net-(U12-A->B)
- U2 pad 9: unconnected-(U2-Pad9) -> /CPU_~{WE}
- U24 pad 31: /GFX/~{BUSY} -> /GFX_~{BUSY}
- U33 pad 11: Net-(U12-A->B) -> Net-(U33-Pad11)
- U33 pad 12: +5V -> /CPU_~{NREN}
- U33 pad 13: /CPU_~{WE} -> /GFX_BUSY
- U4 pad 1: /GFX/~{BUSY} -> Net-(U33-Pad11)
- U4 pad 10: Net-(U10-CE) -> /GFX_BUSY
- U4 pad 13: Net-(U10-CE) -> /GFX_BUSY
- U9 pad 5: /GFX/~{BUSY} -> /GFX_~{BUSY}
- U9 pad 6: Net-(U10-CE) -> /GFX_BUSY
Routing:
- net /GFX/~{BUSY}: track 309.9 -> 0.00 mm, vias 5 -> 0
- net /GFX_~{BUSY}: track 0.00 -> 305.8 mm, vias 0 -> 6
- net Net-(U12-A->B): track 80.6 -> 290.0 mm, vias 2 -> 8
- net /GFX_BUSY: track 0.00 -> 186.7 mm, vias 0 -> 5
- net Net-(U10-CE): track 182.8 -> 0.00 mm, vias 4 -> 0
- net Net-(U33-Pad11): track 0.00 -> 57.8 mm, vias 0 -> 4
- net /BUF_A17: track 109.8 -> 53.3 mm, vias 3 -> 1
- net /BUF_A16: track 99.2 -> 52.2 mm, vias 3 -> 1
- net /BUF_A13: track 39.5 -> 85.0 mm
- net /BUF_A12: track 41.2 -> 76.4 mm
- net /ISA_IRQ7: track 0.00 -> 31.4 mm
- net /ISA_IRQ6: track 0.00 -> 29.5 mm
- net /ISA_IRQ5: track 0.00 -> 27.3 mm
- net /CPU_~{NREN}: track 253.7 -> 280.2 mm, vias 5 -> 6
- net /ISA_IRQ4: track 0.00 -> 24.2 mm
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Other:
- board size 171.4 x 204.5 mm -> 184.2 x 204.5 mm

Commit message: Fixed boot-select jumper polarity
Parts:
- moved J11 36.6 mm to (41.9, 191.8), turned to 180 degrees
Connections:
- J11 pad 1: GND -> +5V
Routing:
- net Net-(J11-Pin_2): track 5.07 -> 17.8 mm
- net /~{SYS_GPIO2_SEL}: track 67.6 -> 70.4 mm
- net /BUF_D7: track 234.0 -> 233.3 mm

Commit message: A1 Mini (which is not all that mini anymore) is feature-complete.
We have 2 ISA slots and even all the power supplies generated from +5V included.

The +12V switcher right next to the audio output is quite a bit concerning, but
we can always say that PWR must be 12V and we directly feed that to the ISA slots.
(Not that PWR is all that clean...) A lot will depend on how I implement grounding,
something that I still have to do.
Parts:
- removed the C30 at (87.2, 255.3)
- removed the C31 at (47.0, 255.8)
- removed the C38 at (61.6, 252.3)
- removed the C45 at (73.8, 260.2)
- removed the C47 at (41.3, 241.2)
- removed the C52 at (57.8, 169.6)
- removed the J14 at (-43.2, 48.3)
- removed the J15 at (-22.9, 48.3)
- added C58: 220uF, Capacitor_THT:CP_Radial_D7.5mm_P2.50mm, F.Cu at (17.1, 26.0)
- added C59: 220uF, Capacitor_THT:CP_Radial_D7.5mm_P2.50mm, F.Cu at (3.70, 222.2)
- added C61: 260p, Capacitor_THT:C_Disc_D4.7mm_W2.5mm_P5.00mm, F.Cu at (8.29, 40.6)
- added C62: 1000uF, Capacitor_THT:CP_Radial_D10.0mm_P5.00mm, F.Cu at (15.2, 216.0)
- added C63: 1500uF, Capacitor_THT:CP_Radial_D10.0mm_P5.00mm, F.Cu at (18.5, 36.8)
- added D4: 1N5817, Diode_THT:D_DO-41_SOD81_P10.16mm_Horizontal, F.Cu at (8.27, 213.3)
- added D5: 1N5817, Diode_THT:D_DO-41_SOD81_P10.16mm_Horizontal, F.Cu at (5.08, 40.6)
- added L1: 25uH, Inductor_THT:L_Radial_D8.7mm_P5.00mm_Fastron_07HCP, F.Cu at (11.4, 209.5)
- added L2: 18uH, Inductor_THT:L_Radial_D8.7mm_P5.00mm_Fastron_07HCP, F.Cu at (-2.54, 31.2)
- added R29: 0.244Ohm, Resistor_THT:R_Axial_DIN0204_L3.6mm_D1.6mm_P5.08mm_Horizontal, F.Cu at (5.08, 217.2)
- added R30: 0.211Ohm, Resistor_THT:R_Axial_DIN0204_L3.6mm_D1.6mm_P5.08mm_Horizontal, F.Cu at (11.4, 27.3)
- added R31: 180, Resistor_THT:R_Axial_DIN0204_L3.6mm_D1.6mm_P5.08mm_Horizontal, F.Cu at (3.81, 27.3)
- added R32: 1.5k, Resistor_THT:R_Axial_DIN0204_L3.6mm_D1.6mm_P5.08mm_Horizontal, F.Cu at (2.54, 217.2)
- added R33: 13k, Resistor_THT:R_Axial_DIN0204_L3.6mm_D1.6mm_P5.08mm_Horizontal, F.Cu at (0.00, 212.1)
- added R34: 13k, Resistor_THT:R_Axial_DIN0204_L3.6mm_D1.6mm_P5.08mm_Horizontal, F.Cu at (14.6, 37.5)
- added R35: 1.5k, Resistor_THT:R_Axial_DIN0204_L3.6mm_D1.6mm_P5.08mm_Horizontal, F.Cu at (24.1, 30.5)
- added U34: MC33063AP, Package_DIP:DIP-8_W7.62mm, F.Cu at (4.43, 201.9)
- added U35: MC33063AP, Package_DIP:DIP-8_W7.62mm, F.Cu at (3.82, 37.5)
- C60: value 1uF -> 302pF
- moved C64 140.9 mm to (17.1, 197.5), turned to -90 degrees
- moved U36 137.6 mm to (13.3, 198.8)
- moved C65 132.3 mm to (7.58, 198.1), turned to 180 degrees
- moved U32 64.1 mm to (-4.45, 145.4), turned to 90 degrees
- moved C60 61.4 mm to (-3.17, 212.1), turned to -90 degrees
- moved RN10 61.0 mm to (26.0, 45.7)
- moved C57 54.5 mm to (-5.08, 152.4), turned to -90 degrees
- moved C55 51.5 mm to (8.21, 179.7)
- moved C17 48.3 mm to (78.1, 105.4)
- moved X4 47.6 mm to (14.0, 184.8), turned to 180 degrees
- moved C54 34.5 mm to (-5.67, 134.0), turned to 0 degrees
- moved U31 28.0 mm to (-1.91, 160.7), turned to 90 degrees
- moved C56 27.8 mm to (-5.08, 167.7), turned to -90 degrees
- moved U33 21.1 mm to (-1.91, 175.9), turned to 90 degrees
- moved C40 6.70 mm to (69.2, 88.9), turned to -90 degrees
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- renumbered C25 to C1, C35 to C10, C36 to C11, C39 to C12, C40 to C13, C41 to C14, C8 to C15, C42 to C16, C43 to C17, C44 to C18, C68 to C19, C26 to C2, C46 to C20, C48 to C21, C49 to C22, C50 to C23, C57 to C24, C58 to C25, C59 to C26, C1 to C27, C13 to C28, C14 to C29, C27 to C3, C2 to C30, C3 to C31, C4 to C32, C5 to C33, C6 to C34, C7 to C35, C61 to C36, C62 to C37, C63 to C38, C11 to C39, C28 to C4, C12 to C40, C15 to C41, C16 to C42, C17 to C43, C10 to C44, C19 to C45, C20 to C46, C18 to C47, C23 to C48, C21 to C49, C29 to C5, C22 to C50, C53 to C51, C54 to C52, C55 to C53, C24 to C54, C51 to C55, C64 to C56, C65 to C57, C32 to C6, C37 to C64, C56 to C65, C9 to C7, C33 to C8, C34 to C9, CMC7 to CMC10, CMC8 to CMC7, CMC9 to CMC8, CMC10 to CMC9, D3 to D1, D1 to D2, D2 to D3, FB18 to FB1, FB8 to FB10, FB9 to FB11, FB10 to FB12, FB11 to FB13, FB12 to FB14, FB2 to FB15, FB4 to FB16, FB5 to FB17, FB6 to FB18, FB7 to FB19, FB19 to FB2, FB3 to FB20, FB1 to FB3, FB13 to FB4, FB20 to FB5, FB14 to FB6, FB16 to FB7, FB17 to FB8, FB15 to FB9, J17 to J1, J6 to J10, J12 to J11, J10 to J12, J7 to J13, J2 to J14, J8 to J15, J4 to J16, J9 to J17, J16 to J18, J18 to J2, J20 to J3, J22 to J4, J11 to J5, J1 to J6, J3 to J7, J13 to J8, J5 to J9, JP3 to JP1, JP1 to JP2, JP2 to JP3, R11 to R1, R20 to R10, R21 to R11, R1 to R12, R19 to R13, R18 to R14, R7 to R15, R2 to R16, R3 to R17, R5 to R18, R6 to R19, R10 to R2, R4 to R20, R28 to R21, R14 to R22, R15 to R23, R16 to R24, R17 to R25, R22 to R26, R23 to R27, R24 to R28, R27 to R3, R13 to R4, R9 to R5, R25 to R6, R8 to R7, R12 to R8, R29 to R9, RN13 to RN1, RN7 to RN10, RN12 to RN2, RN14 to RN3, RN5 to RN4, RN2 to RN5, RN1 to RN6, RN8 to RN7, RN4 to RN8, RN3 to RN9, SW4 to SW1, SW1 to SW2, SW2 to SW3, TP2 to TP1, U3 to U1, U11 to U10, U27 to U11, U18 to U12, U12 to U13, U13 to U14, U14 to U15, U8 to U16, U16 to U17, U17 to U18, U9 to U2, U24 to U22, U25 to U23, U28 to U24, U26 to U25, U29 to U26, U15 to U27, U7 to U28, U30 to U29, U33 to U3, U31 to U30, U34 to U31, U22 to U32, U32 to U33, U23 to U36, U5 to U4, U6 to U5, U1 to U6, U2 to U7, U4 to U8, U10 to U9, X3 to X1, X1 to X2, X2 to X3
Connections:
- C60 pad 1: +5V -> Net-(U34-TC)
- C60 pad 2: GND -> -12V
- RN10 pad 3: /ISA/~{ISA_0WS} -> /ISA/~{ISA_DACK0}
- RN10 pad 4: /CPU_~{WAIT} -> /ISA/~{ISA_0WS}
- RN10 pad 5: /ISA/~{ISA_DACK0} -> /CPU_~{WAIT}
- U33 pad 1: /ISA_IRQ7 -> /ISA_IRQ6
- U33 pad 2: /ISA_IRQ6 -> /ISA_IRQ5
- U33 pad 4: /ISA_IRQ3 -> /ISA_IRQ2
- U33 pad 5: /ISA_IRQ2 -> /ISA_IRQ3
- U33 pad 8: /ISA_IRQ5 -> /ISA_IRQ7
Routing:
- net /BUF_A19: track 0.00 -> 298.7 mm, vias 0 -> 3
- net /BUF_A16: track 52.2 -> 293.2 mm, vias 1 -> 2
- net /BUF_A18: track 62.5 -> 302.4 mm, vias 1 -> 2
- net /BUF_A15: track 43.0 -> 280.9 mm, vias 1 -> 3
- net /BUF_A17: track 53.3 -> 285.8 mm, vias 1 -> 3
- net /BUF_A12: track 76.4 -> 308.0 mm, vias 1 -> 3
- net /BUF_A14: track 56.9 -> 278.1 mm, vias 1 -> 2
- net /BUF_A13: track 85.0 -> 305.6 mm, vias 0 -> 1
- net /BUF_A8: track 62.8 -> 261.9 mm, vias 0 -> 1
- net /BUF_A11: track 73.0 -> 269.0 mm, vias 1 -> 3
- net /ISA_IRQ2: track 19.5 -> 212.6 mm, vias 0 -> 2
- net /BUF_A7: track 51.6 -> 243.8 mm, vias 0 -> 4
- net /BUF_A9: track 67.0 -> 259.0 mm, vias 2 -> 3
- net /CPU_~{WAIT}: track 109.8 -> 300.1 mm, vias 2 -> 3
- net /BUF_A10: track 70.8 -> 260.7 mm, vias 1 -> 3
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Other:
- board size 184.2 x 204.5 mm -> 201.9 x 204.5 mm

Commit message: A1 MINI is fully routed.
That is, if I add a GND fill on both layers. Which I don't, because auto-refill takes
several seconds and so it's a PITA to work with. There are a few dozen DRC errors
as well but nothing major it seems.

Worked out roughly 100ohm diff impedance for the HDMI lines
(not GND-referenced) which I think is my best shot of making it work.

long USB trace has a nice GND shield under-it, so does audio.
Again, probably my best shot at making these work.

Ethernet still needs checking just as short-put USB connections from the hub to
the connector.
Parts:
- added JP5: Jumper_2_Bridged, Connector_PinHeader_2.54mm:PinHeader_1x02_P2.54mm_Vertical, F.Cu at (28.6, 26.0)
- added JP6: Jumper_2_Open, Connector_PinHeader_2.54mm:PinHeader_1x02_P2.54mm_Vertical, F.Cu at (8.89, 44.5)
- added JP7: Jumper_2_Bridged, Connector_PinHeader_2.54mm:PinHeader_1x02_P2.54mm_Vertical, F.Cu at (37.5, 78.1)
- J5, J7, JP1: footprint Connector_PinSocket_2.54mm:PinSocket_1x02_P2.54mm_Vertical -> Connector_PinHeader_2.54mm:PinHeader_1x02_P2.54mm_Vertical
- moved C59 196.7 mm to (17.1, 26.0), turned to -90 degrees
- moved C58 196.7 mm to (3.77, 222.2), turned to 180 degrees
- moved C51 16.8 mm to (85.8, 56.5), turned to 0 degrees
- moved JP2 10.6 mm to (50.8, 82.5)
- moved C44 10.1 mm to (189.9, 83.1), turned to 90 degrees
- moved C56 4.11 mm to (-2.50, 164.5), turned to 0 degrees
- moved C57 3.65 mm to (-2.50, 149.9), turned to 0 degrees
- moved C16 2.05 mm to (26.7, 62.3)
- moved F1 1.95 mm to (74.5, 47.0)
- moved C54 1.90 mm to (-3.77, 134.0)
- moved C42 1.32 mm to (66.7, 53.3), turned to 0 degrees
- moved U23 1.14 mm to (29.8, 74.3)
- turned C37 to 180 degrees
Connections:
- net /PWR_IN renamed PWR_IN
- C59 pad 1: +5V -> Net-(JP5-A)
- J11 pad 1: GND -> GNDA
- J8 pad 1: GND -> GNDA
- R10 pad 2: GND -> GNDA
- R11 pad 2: GND -> GNDA
- R14 pad 2: GND -> GNDA
- R15 pad 2: GND -> GNDA
- R30 pad 1: +5V -> Net-(JP5-A)
- U23 pad 10: GND -> GNDA
- U23 pad 16: GND -> GNDA
- U23 pad 17: GND -> GNDA
- U23 pad 23: GND -> GNDA
- U23 pad 26: GND -> GNDA
- U35 pad 6: +5V -> Net-(JP5-A)
- Y1 pad 3: (no net) -> GND
Routing:
- net +5V: track 1165.5 -> 2056.8 mm, vias 1 -> 15
- net GND: track 1254.6 -> 1574.5 mm, vias 0 -> 6
- net /ISA/ISA_-5V: track 24.9 -> 183.6 mm, vias 0 -> 2
- net -12V: track 88.9 -> 243.8 mm, vias 0 -> 1
- net PWR_IN: track 269.7 -> 397.7 mm, vias 2 -> 3
- net +12V: track 42.3 -> 69.6 mm, vias 0 -> 1
- net Net-(JP5-A): track 0.00 -> 21.9 mm
- net /MIO/USB_D+: track 206.1 -> 222.6 mm
- net GNDA: track 0.00 -> 15.5 mm, vias 0 -> 2
- net /MIO/USB_D-: track 208.5 -> 222.8 mm
- net SYS_CLK: track 515.0 -> 527.9 mm, vias 7 -> 10
- net ~{RST}: track 587.0 -> 596.1 mm
- net /GFX_~{WE}: track 94.2 -> 101.8 mm
- net /ISA/ISA_AEN: track 129.6 -> 122.7 mm
- net /GFX_~{BUSY}: track 304.6 -> 311.2 mm
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- added copper zone on F.Cu, net GNDA
