File: boards/a1_mini/a1_mini.kicad_pcb (KiCad board)
At the start: 4 copper layers, 201.9 x 204.5 mm, 221 parts, among them J1 Conn_01x01, J10 HDMI_A, J11 SJ1-3535NG-BE, J12 DE9_Plug, J13 Micro_SD_Card, J15 USB_A_Stacked, J16 USB_A_Stacked, J17 USB_A_Stacked, J18 Bus_ISA_8bit, J19 Bus_ISA_8bit, J2 Conn_01x01, J3 Conn_01x01, J4 Conn_01x01, J5 Conn_01x02, J6 Jack-DC, J7 Conn_01x02, J8 SJ1-3535NG-BE, J9 Conn_01x02, SW1 SW_DPDT_x2, SW2 SW_Push, SW3 SW_Push, U1 74LS08, U10 74AHCT245, U11 SST39SF040, U12 A1_POWER, U13 74AHCT245, U14 74AHCT245, U15 74AHCT245, U16 74LS273, U17 74LS273, U18 74LS273, U19 ESPRESSO, U2 74LS86, U20 SIMM-30, U21 SIMM-30, U22 DISCO, U23 A1_CODEC, U24 MAX232, U25 MIO, U26 DS1307+, U27 KSZ8851-11MLL, U28 A1_USBHUB, U29 SIMM-30, U3 74LS00, U30 SIMM-30, U31 74LS14, U32 74LS139, U33 4075, U34 MC33063AP, U35 MC33063AP, U36 L79L05_TO92, U4 74LS273, U5 74LS574, U6 74LS139, U7 74LS14, U8 74LS126, U9 74AHCT245, X1 8MHz, X2 CXO_DIP14, X3 24MHz, X4 14.31818MHz, Y1 32768Hz, Y2 25MHz

Commit message: A1-MINI is fully routed. Also fully impedance controlled.
Parts:
- removed U29, U30: SIMM-30, anachron:SIMM-30
- U20, U21: value SIMM-30 -> SIMM-30x2; footprint anachron:SIMM-30 -> anachron:SIMM-30x2_VERT
- moved C43 106.7 mm to (154.9, 86.7)
- moved C60 101.4 mm to (98.1, 207.1), turned to 90 degrees
- moved R9 98.0 mm to (161.3, 159.4), turned to -90 degrees
- moved R33 95.0 mm to (94.9, 207.2), turned to 90 degrees
- moved F1 94.1 mm to (159.4, 87.5), turned to 0 degrees
- moved RN5 92.0 mm to (214.0, 68.6)
- moved C48 91.5 mm to (270.8, 61.0)
- moved C7 91.4 mm to (171.4, 57.2)
- moved JP3 91.3 mm to (250.8, 91.4), turned to -90 degrees
- moved R32 91.1 mm to (92.3, 202.1), turned to -90 degrees
- moved C58 90.9 mm to (91.1, 197.0), turned to 0 degrees
- moved FB6 90.4 mm to (178.4, 38.7)
- moved C45 89.5 mm to (270.8, 66.7)
- moved U22 89.4 mm to (170.2, 87.6)
- moved C36 88.1 mm to (183.6, 156.2)
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Connections:
- net /MIO/USB_D+ renamed /USB_MAIN_D+
- net /MIO/USB_D- renamed /USB_MAIN_D-
- net Net-(J14-RD+) renamed /ETH/ETH_RX+
- net Net-(J14-RD-) renamed /ETH/ETH_RX-
- net Net-(J14-TD+) renamed /ETH/ETH_TX+
- net Net-(J14-TD-) renamed /ETH/ETH_TX-
- net Net-(U22-TMDS_C+) renamed /GFX/TMDS_CLK+
- net Net-(U22-TMDS_C-) renamed /GFX/TMDS_CLK-
- net Net-(U22-TMDS_D0+) renamed /GFX/TMDS_D0+
- net Net-(U22-TMDS_D0-) renamed /GFX/TMDS_D0-
- net Net-(U22-TMDS_D1+) renamed /GFX/TMDS_D1+
- net Net-(U22-TMDS_D1-) renamed /GFX/TMDS_D1-
- net Net-(U22-TMDS_D2+) renamed /GFX/TMDS_D2+
- net Net-(U22-TMDS_D2-) renamed /GFX/TMDS_D2-
- net Net-(U28-USBDN2_DM) renamed /USB/USB_DN2_D-
- net Net-(U28-USBDN2_DP) renamed /USB/USB_DN2_D+
- net Net-(U28-USBDN3_DM) renamed /USB/USB_DN3_D-
- net Net-(U28-USBDN3_DP) renamed /USB/USB_DN3_D+
- net Net-(U28-USBDN4_DM) renamed /USB/USB_DN4_D-
- net Net-(U28-USBDN4_DP) renamed /USB/USB_DN4_D+
- net Net-(U28-USBDN5_DM) renamed /USB/USB_DN5_D-
- net Net-(U28-USBDN5_DP) renamed /USB/USB_DN5_D+
- net Net-(U28-USBDN6_DM) renamed /USB/USB_DN6_D-
- net Net-(U28-USBDN6_DP) renamed /USB/USB_DN6_D+
- net Net-(U28-USBDN7_DM) renamed /USB/USB_DN7_D-
- net Net-(U28-USBDN7_DP) renamed /USB/USB_DN7_D+
Routing:
- net GND: track 1574.5 -> 2646.4 mm, vias 6 -> 16
- net Net-(JP1-A): track 88.4 -> 338.0 mm, vias 0 -> 4
- net PWR_IN: track 397.7 -> 149.2 mm
- net Net-(J7-Pin_2): track 252.1 -> 366.3 mm, vias 0 -> 2
- net +5V: track 2056.8 -> 1959.3 mm, vias 15 -> 20
- net /~{LAN_SEL}: track 197.2 -> 149.6 mm, vias 2 -> 4
- net Net-(F1-Pad1): track 3.40 -> 48.1 mm
- net /MIO/USB_CLK: track 214.9 -> 178.9 mm
- net SYS_CLK: track 527.9 -> 493.1 mm
- net /I2C_SDA: track 400.2 -> 366.0 mm
- net /I2C_SCL: track 397.9 -> 364.7 mm
- net /CPU_TC: track 420.9 -> 395.4 mm, vias 4 -> 6
- net /GFX_~{RAS}: track 101.4 -> 76.6 mm, vias 2 -> 0
- net /ETH/ETH_RX-: track 102.6 -> 78.3 mm
- net Net-(U13-A->B): track 291.3 -> 267.1 mm, vias 8 -> 6
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
Commit message: 3.3V work, before abandoning the idea.
Parts:
- added C66: 1uF, Capacitor_THT:C_Disc_D4.7mm_W2.5mm_P5.00mm, F.Cu at (194.3, 209.6)
- added C67: 1uF, Capacitor_THT:C_Disc_D4.7mm_W2.5mm_P5.00mm, F.Cu at (154.9, 147.4)
- added C68: 1uF, Capacitor_THT:C_Disc_D4.7mm_W2.5mm_P5.00mm, F.Cu at (107.3, 165.8)
- added C69: 1uF, Capacitor_THT:C_Disc_D4.7mm_W2.5mm_P5.00mm, F.Cu at (107.3, 151.2)
- added C70: 1uF, Capacitor_THT:C_Disc_D4.7mm_W2.5mm_P5.00mm, F.Cu at (139.1, 158.2)
- added C71: 1uF, Capacitor_THT:C_Disc_D4.7mm_W2.5mm_P5.00mm, F.Cu at (163.2, 174.7)
- U1: value 74LS08 -> SN74AHC08N
- U10, U13, U14, U9: value 74AHCT245 -> SN74LVC245AN
- U16, U17, U18, U4: value 74LS273 -> SN74AHC574N
- U2: value 74LS86 -> SN74AHC86N
- U24: value MAX232 -> ICL3232CPZ
- U3: value 74LS00 -> SN74AHC00N
- U31, U7: value 74LS14 -> SN74AHC14N
- U32, U6: value 74LS139 -> SN74AHC139N
- U33: value 4075 -> CD74HC4075E
- U5: value 74LS574 -> SN74AHC574N
- U8: value 74LS126 -> SN74AHC126N
- moved C23 199.6 mm to (306.7, 157.5)
- moved C53 166.1 mm to (304.8, 147.4)
- moved C52 130.5 mm to (292.7, 167.0), turned to 0 degrees
- moved C25 122.7 mm to (291.8, 114.5)
- moved C37 114.7 mm to (163.2, 182.9), turned to -90 degrees
- moved C24 99.5 mm to (292.7, 150.5)
- moved C26 98.1 mm to (283.2, 155.0)
- moved C51 92.2 mm to (249.6, 113.7)
- moved C38 79.4 mm to (149.9, 118.2)
- moved C9 79.4 mm to (229.2, 117.6)
- moved C20 79.3 mm to (186.1, 142.3)
- moved C19 76.8 mm to (169.5, 115.0), turned to -90 degrees
- moved C21 66.8 mm to (234.4, 156.2), turned to 0 degrees
- moved C36 42.4 mm to (199.4, 116.9), turned to -90 degrees
- moved C13 35.5 mm to (212.1, 176.5), turned to 180 degrees
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Connections:
- C1 pad 1: +5V -> +3.3V
- C10 pad 1: +5V -> +3.3V
- C11 pad 1: +5V -> +3.3V
- C12 pad 1: +5V -> +3.3V
- C13 pad 1: +5V -> +3.3V
- C14 pad 1: +5V -> +3.3V
- C16 pad 1: +5V -> +3.3V
- C18 pad 1: +5V -> +3.3V
- C19 pad 1: +5V -> +3.3V
- C2 pad 1: +5V -> +3.3V
- C3 pad 1: +5V -> +3.3V
- C34 pad 1: +5V -> +3.3V
- C36 pad 1: +5V -> +3.3V
- C37 pad 1: +5V -> +3.3V
- C4 pad 1: +5V -> +3.3V
- C5 pad 1: +5V -> +3.3V
- C54 pad 1: +5V -> +3.3V
- C55 pad 1: +5V -> +3.3V
- C57 pad 1: +5V -> +3.3V
- C8 pad 1: +5V -> +3.3V
- C9 pad 1: +5V -> +3.3V
- J13 pad 4: +5V -> +3.3V
- J5 pad 1: +5V -> +3.3V
- R2 pad 1: +5V -> +3.3V
- R20 pad 2: +5V -> +3.3V
- R21 pad 2: +5V -> +3.3V
- R22 pad 2: +5V -> +3.3V
- R3 pad 1: +5V -> +3.3V
- R5 pad 1: +5V -> +3.3V
- R7 pad 1: +5V -> +3.3V
- R9 pad 1: +5V -> +3.3V
- RN1 pad 1: +5V -> +3.3V
- RN10 pad 1: +5V -> +3.3V
- RN3 pad 1: +5V -> +3.3V
- RN7 pad 1: +5V -> +3.3V
- RN8 pad 1: +5V -> +3.3V
- RN9 pad 1: +5V -> +3.3V
- U1 pad 14: +5V -> +3.3V
- U10 pad 20: +5V -> +3.3V
- U13 pad 20: +5V -> +3.3V
- U14 pad 20: +5V -> +3.3V
- U15 pad 1: +5V -> +3.3V
- U15 pad 20: +5V -> +3.3V
- U16 pad 1: +5V -> GND
- U16 pad 12: /BUF_A7 -> /BUF_A1
- U16 pad 13: /CPU_A6 -> /BUF_A3
- U16 pad 14: /CPU_A4 -> /BUF_A5
- U16 pad 15: /BUF_A5 -> /BUF_A7
- U16 pad 16: /BUF_A3 -> /BUF_A8
- U16 pad 17: /CPU_A2 -> /BUF_A6
- U16 pad 18: /CPU_A0 -> /BUF_A4
- U16 pad 19: /BUF_A1 -> /BUF_A2
- U16 pad 2: /BUF_A2 -> /CPU_A1
- U16 pad 20: +5V -> +3.3V
- U16 pad 3: /CPU_A1 -> /CPU_A3
- U16 pad 4: /CPU_A3 -> /CPU_A5
- U16 pad 5: /BUF_A4 -> /CPU_A7
- U16 pad 6: /BUF_A6 -> /CPU_A6
- U16 pad 7: /CPU_A5 -> /CPU_A4
- U16 pad 8: /CPU_A7 -> /CPU_A2
- U16 pad 9: /BUF_A8 -> /CPU_A0
- U17 pad 1: +5V -> GND
- U17 pad 12: unconnected-(U17-Q4-Pad12) -> /BUF_A20
- U17 pad 13: unconnected-(U17-D4-Pad13) -> /BUF_A21
- U17 pad 14: /CPU_A10 -> /BUF_A22
- U17 pad 15: /BUF_A22 -> unconnected-(U17-Q4-Pad15)
- U17 pad 16: /BUF_A21 -> unconnected-(U17-Q3-Pad16)
- U17 pad 17: /CPU_A9 -> unconnected-(U17-Q2-Pad17)
- U17 pad 18: /CPU_A8 -> unconnected-(U17-Q1-Pad18)
- U17 pad 19: /BUF_A20 -> unconnected-(U17-Q0-Pad19)
- U17 pad 20: +5V -> +3.3V
- U17 pad 7: unconnected-(U17-D2-Pad7) -> /CPU_A10
- U17 pad 8: unconnected-(U17-D3-Pad8) -> /CPU_A9
- U17 pad 9: unconnected-(U17-Q3-Pad9) -> /CPU_A8
- U18 pad 1: +5V -> GND
- U18 pad 12: /BUF_A18 -> /BUF_A12
- U18 pad 13: /CPU_A6 -> /BUF_A14
- U18 pad 14: /CPU_A4 -> /BUF_A16
- U18 pad 15: /BUF_A16 -> /BUF_A18
- U18 pad 16: /BUF_A14 -> /BUF_A19
- U18 pad 17: /CPU_A2 -> /BUF_A17
- U18 pad 18: /CPU_A0 -> /BUF_A15
- U18 pad 19: /BUF_A12 -> /BUF_A13
- U18 pad 2: /BUF_A13 -> /CPU_A1
- U18 pad 20: +5V -> +3.3V
- U18 pad 3: /CPU_A1 -> /CPU_A3
- U18 pad 4: /CPU_A3 -> /CPU_A5
- U18 pad 5: /BUF_A15 -> /CPU_A7
- U18 pad 6: /BUF_A17 -> /CPU_A6
- U18 pad 7: /CPU_A5 -> /CPU_A4
- U18 pad 8: /CPU_A7 -> /CPU_A2
- U18 pad 9: /BUF_A19 -> /CPU_A0
- U2 pad 12: +5V -> +3.3V
- U2 pad 14: +5V -> +3.3V
- U2 pad 4: +5V -> +3.3V
- U2 pad 9: +5V -> +3.3V
- U20 pad A24: +5V -> +3.3V
- U20 pad A28: +5V -> +3.3V
- U20 pad B24: +5V -> +3.3V
- U20 pad B28: +5V -> +3.3V
- U21 pad A24: +5V -> +3.3V
- U21 pad A28: +5V -> +3.3V
- U21 pad B24: +5V -> +3.3V
- U21 pad B28: +5V -> +3.3V
- U24 pad 16: +5V -> +3.3V
- U3 pad 14: +5V -> +3.3V
- U3 pad 9: +5V -> +3.3V
- U31 pad 14: +5V -> +3.3V
- U32 pad 16: +5V -> +3.3V
- U4 pad 12: unconnected-(U4-Q4-Pad12) -> Net-(U4-Q7)
- U4 pad 13: /BUF_D1 -> unconnected-(U4-Q6-Pad13)
- U4 pad 14: /BUF_D3 -> unconnected-(U4-Q5-Pad14)
- U4 pad 16: unconnected-(U4-Q6-Pad16) -> Net-(U4-Q3)
- U4 pad 17: /BUF_D5 -> unconnected-(U4-Q2-Pad17)
- U4 pad 18: /BUF_D7 -> unconnected-(U4-Q1-Pad18)
- U4 pad 19: Net-(U4-Q7) -> Net-(U4-Q0)
- U4 pad 2: Net-(U4-Q0) -> /BUF_D6
- U4 pad 20: +5V -> +3.3V
- U4 pad 3: /BUF_D6 -> /BUF_D4
- U4 pad 4: /BUF_D4 -> /BUF_D2
- U4 pad 5: unconnected-(U4-Q1-Pad5) -> /BUF_D0
- U4 pad 6: unconnected-(U4-Q2-Pad6) -> /BUF_D1
- U4 pad 7: /BUF_D2 -> /BUF_D3
- U4 pad 8: /BUF_D0 -> /BUF_D5
- U4 pad 9: Net-(U4-Q3) -> /BUF_D7
- U5 pad 20: +5V -> +3.3V
- U6 pad 16: +5V -> +3.3V
- U7 pad 14: +5V -> +3.3V
- U8 pad 14: +5V -> +3.3V
- U9 pad 20: +5V -> +3.3V
- X1 pad 1: +5V -> +3.3V
- X1 pad 14: +5V -> +3.3V
- X2 pad 1: +5V -> +3.3V
- X2 pad 14: +5V -> +3.3V
- X3 pad 1: +5V -> +3.3V
- X3 pad 14: +5V -> +3.3V
- X4 pad 1: +5V -> +3.3V
- X4 pad 14: +5V -> +3.3V
Routing:
- net +5V: track 1959.3 -> 739.8 mm, vias 20 -> 12
- net +3.3V: track 0.00 -> 1078.2 mm, vias 0 -> 13
- net GND: track 2646.4 -> 2662.7 mm, vias 16 -> 17
- net /~{MIO_SEL}: track 194.7 -> 200.8 mm
- net /GFX_A10: track 169.0 -> 172.1 mm
- net Net-(U3-Pad11): track 55.7 -> 57.8 mm
- net /GFX_A9: track 155.3 -> 157.3 mm
- net /BUF_A4: track 215.8 -> 216.8 mm
- net /BUF_A2: track 200.9 -> 202.0 mm
- net /BUF_A1: track 202.2 -> 203.3 mm
- net /BUF_A3: track 216.3 -> 217.4 mm
- net /BUF_NREN: track 137.1 -> 136.2 mm
- net Net-(U13-A->B): track 267.1 -> 267.7 mm
- net /GFX_BUSY: vias 5 -> 6
