File: boards/a1_mini/a1_mini.kicad_sch (KiCad schematic)
At the start: 66 parts, among them J1 Jack-DC, J17 Conn_01x01, J18 Conn_01x01, J20 Conn_01x01, J22 Conn_01x01, J3 Conn_01x02, SW1 SW_Push, SW2 SW_Push, SW4 SW_DPDT_x2, U1 74LS139, U10 74AHCT245, U11 74AHCT245, U12 74AHCT245, U13 74AHCT245, U14 74AHCT245, U16 74LS273, U17 74LS273, U18 A1_POWER, U2 74LS14, U27 SST39SF040, U3 74LS08, U33 74LS00, U4 74LS126, U5 74LS273, U6 74LS574, U8 74LS273, U9 74LS86, X3 8MHz

Commit message: USB HUB is back in.
Parts:
- removed C37: 1uF, Capacitor_THT:C_Disc_D4.7mm_W2.5mm_P5.00mm, symbol Device:C
- SW4: footprint Button_Switch_THT:SW_E-Switch_EG2219_DPDT_Angled -> Button_Switch_THT:SW_CuK_JS202011CQN_DPDT_Straight
Connections:
- net BUF_nEN: now also U3.3; no longer U3.8
- net CPU_~{DACK0}: now also U3.13; no longer U3.1
- net CPU_~{DACK1}: now also U3.12; no longer U3.2
- net CPU_~{DACK2}: now also U3.10; no longer U3.4
- net CPU_~{DACK3}: now also U3.9; no longer U3.5
- net CPU_~{DACK}: now also U3.2, U3.6; no longer U3.10, U3.11
- net CPU_~{NREN}: now also U3.1; no longer U3.9
- net PWR_IN: now reaches D2.1 (K), J1.1, R25.1, U18.6 (VIN), U18.7 (VIN)
- new net: U3.11, U3.4
- new net: U3.5, U3.8
Other:
- added sheet USB (usb.kicad_sch)
- sheet MIO ports: added USB_CLK, USB_US_D+, USB_US_D-; removed none
- moved on the sheet: U3A, U3B, U3C, U3D

Commit message: Added boot mode switch, reworked LAN IRQ, places LEDs better.
Parts:
- added D3: LED, LED_THT:LED_D5.0mm, symbol Device:LED
- added J11: Conn_01x02, Connector_PinSocket_2.54mm:PinSocket_1x02_P2.54mm_Vertical, symbol Connector_Generic:Conn_01x02
- added R13: 470, Resistor_THT:R_Axial_DIN0204_L3.6mm_D1.6mm_P5.08mm_Horizontal, symbol Device:R_US
- added R26: 10k, Resistor_THT:R_Axial_DIN0204_L3.6mm_D1.6mm_P5.08mm_Horizontal, symbol Device:R_US
Connections:
- net +5V: now also R26.1
- net GND: now also D3.1 (K), J11.1 (Pin_1)
- net at U5.9 (Q3): now also R13.1
- net at U6.2 (D0): now also J11.2 (Pin_2), R26.2
- new net: D3.2 (A), R13.2
Other:
- sheet ETH ports: added ~{INT}; removed ~{LAN_IRQ}
- sheet MIO ports: added LAN_~{INT}; removed none
- note added: "ACTIVITY LED"
- note added: "BOOT SELECT"
- note added: "PWR LED"
- note added: "PWR SWITCH"
- note added: "RESET BTN"
- moved on the sheet: U4C

Commit message: ISA is incorporated back into mini. Not routed yet.
Parts:
- removed unit 2 of U4
- added R27, R29: 10k, Resistor_THT:R_Axial_DIN0204_L3.6mm_D1.6mm_P5.08mm_Horizontal, symbol Device:R_US
- added unit 2 of U4
- U4: symbol 74xx:74LS126 -> 74xx:74LS125
Connections:
- net +5V: now also R27.1, R29.1
- net CPU_~{INT}: now also U4.6
- net CPU_~{WAIT}: now also U4.3; no longer U4.10, U4.13, U9.5
- net GND: now also U4.2, U4.5
- net at U10.19 (CE), U11.19 (CE), U12.19 (CE)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: now also U4.10, U4.13
- net ~{ISA_SEL}: now reaches U1.5 (O1)
- net GFX/~{BUSY}: now reaches U4.1
- net GFX/~{BUSY}: now also U9.5, R27.2
- net ISA_CH_CK: now reaches U6.3 (D1)
- net ISA_IRQ2: now reaches U6.4 (D2)
- net ISA_IRQ3: now reaches U6.5 (D3)
- net ISA_IRQ4: now reaches U6.6 (D4)
- net ISA_IRQ5: now reaches U6.7 (D5)
- net ISA_IRQ6: now reaches U6.8 (D6)
- net ISA_IRQ7: now reaches U6.9 (D7)
- new net ISA/~{INT}: R29.2, U4.4
Other:
- added sheet ISA (isa.kicad_sch)
- note added: "We have a problem here: The way we use ~{WAIT} on the CPU is that indiscrimately pull on it, whenever GFX needs it's bus. This works, if: - The CPU bus interface is programmed to ignore ~{WAIT} for ~{RAS_A} and ~{NREN} accesses - No one else generates ~{WAIT}-states. This latter statement is not true with ISA bus: it needs to be able to generate wait-states for ~{NREN} accesses, at which point th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"
- moved on the sheet: U10, U11, U12, U33D, U9B

Commit message: Worked in wait-states for I/O, changed I/O address decode, added GPI pull-downs.
Parts:
- removed R26: 10k, Resistor_THT:R_Axial_DIN0204_L3.6mm_D1.6mm_P5.08mm_Horizontal, symbol Device:R_US
- added RN5: 10k, Resistor_THT:R_Array_SIP9, symbol Device:R_Network08_US
Connections:
- net +5V: no longer U33.12
- net BUF_A12: now also U1.14 (A0)
- net BUF_A13: now also U1.13 (A1)
- net BUF_A16: no longer U1.13 (A1)
- net BUF_A17: no longer U1.14 (A0)
- net CPU_~{NREN}: now also U33.12
- net CPU_~{WE}: now also U2.9; no longer U33.13
- net GND: now also RN5.1 (common)
- net ISA_CH_CK: now also RN5.8 (R7)
- net ISA_IRQ2: now also RN5.7 (R6)
- net ISA_IRQ3: now also RN5.6 (R5)
- net ISA_IRQ4: now also RN5.5 (R4)
- net ISA_IRQ5: now also RN5.4 (R3)
- net ISA_IRQ6: now also RN5.3 (R2)
- net ISA_IRQ7: now also RN5.2 (R1)
- net at J11.2 (Pin_2), U6.2 (D0): now also RN5.9 (R8)
- net GFX_BUSY: now reaches U10.19 (CE), U11.19 (CE), U12.19 (CE), U4.10, U4.13, U9.6
- net GFX_BUSY: now also U33.13
- net at U2.8: now also U12.1 (A->B)
- net at U33.11: now also U4.1; no longer U12.1 (A->B)
- net BUF_nEN renamed BUF_~{EN}
- net GFX/~{BUSY} renamed GFX_~{BUSY}
- net GFX_~{BUSY}: no longer U4.1
Other:
- note added: "We disable GFX~{BUSY} propagation to CPU_~{WAIT} when we do I/O cycles. This allows for peripherals to generate their own wait-states without the GFX chip interfering all the time."
- note removed: "We have a problem here: The way we use ~{WAIT} on the CPU is that indiscrimately pull on it, whenever GFX needs it's bus. This works, if: - The CPU bus interface is programmed to ignore ~{WAIT} for ~{RAS_A} and ~{NREN} accesses - No one else generates ~{WAIT}-states. This latter statement is not true with ISA bus: it needs to be able to generate wait-states for ~{NREN} accesses, at which point th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"
- moved on the sheet: D1, D3, J17, J18, J20, J22, R13, R27, R9, U2D, U33D, U4A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

Commit message: Fixed boot-select jumper polarity
Connections:
- net +5V: now also J11.1 (Pin_1)
- net GND: no longer J11.1 (Pin_1)
Other:
- moved on the sheet: J11
Changed lines of the file:
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@@
   (junction (at 219.71 396.24) (diameter 0) (color 0 0 0 0)
   )
+  (junction (at 138.43 298.45) (diameter 0) (color 0 0 0 0)
+  )
   (junction (at 119.38 44.45) (diameter 0) (color 0 0 0 0)
   )
@@
   (junction (at 539.75 215.9) (diameter 0) (color 0 0 0 0)
   )
-  (junction (at 111.76 298.45) (diameter 0) (color 0 0 0 0)
-  )
   (junction (at 411.48 336.55) (diameter 0) (color 0 0 0 0)
   )
@@
     (stroke (width 0) (type default))
   )
-  (wire (pts (xy 111.76 340.36) (xy 111.76 298.45))
-    (stroke (width 0) (type default))
-  )
   (wire (pts (xy 293.37 280.67) (xy 293.37 292.1))
     (stroke (width 0) (type default))
@@
     (stroke (width 0) (type default))
   )
-  (wire (pts (xy 105.41 346.71) (xy 105.41 342.9))
-    (stroke (width 0) (type default))
-  )
   (wire (pts (xy 26.67 62.23) (xy 62.23 62.23))
     (stroke (width 0) (type default))
@@
     (stroke (width 0) (type default))
   )
-  (wire (pts (xy 101.6 342.9) (xy 105.41 342.9))
-    (stroke (width 0) (type default))
-  )
   (wire (pts (xy 355.6 374.65) (xy 379.73 374.65))
     (stroke (width 0) (type default))
@@
     (stroke (width 0) (type default))
   )
-  (wire (pts (xy 111.76 298.45) (xy 138.43 298.45))
-    (stroke (width 0) (type default))
-  )
   (bus (pts (xy 181.61 302.26) (xy 181.61 304.8))
     (stroke (width 0) (type default))
@@
     (stroke (width 0) (type default))
   )
+  (wire (pts (xy 146.05 295.91) (xy 146.05 292.1))
+    (stroke (width 0) (type default))
+  )
   (wire (pts (xy 438.15 149.86) (xy 453.39 149.86))
     (stroke (width 0) (type default))
@@
     (stroke (width 0) (type default))
   )
-  (wire (pts (xy 101.6 340.36) (xy 111.76 340.36))
-    (stroke (width 0) (type default))
-  )
   (wire (pts (xy 72.39 196.85) (xy 205.74 196.85))
     (stroke (width 0) (type default))
@@
     (stroke (width 0) (type default))
   )
+  (wire (pts (xy 148.59 295.91) (xy 146.05 295.91))
+    (stroke (width 0) (type default))
+  )
   (wire (pts (xy 466.09 125.73) (xy 491.49 125.73))
     (stroke (width 0) (type default))
@@
     (stroke (width 0) (type default))
   )
+  (wire (pts (xy 138.43 298.45) (xy 148.59 298.45))
+    (stroke (width 0) (type default))
+  )
   (wire (pts (xy 184.15 302.26) (xy 213.36 302.26))
     (stroke (width 0) (type default))
@@
     (stroke (width 0) (type default))
   )
-  (wire (pts (xy 87.63 298.45) (xy 111.76 298.45))
+  (wire (pts (xy 87.63 298.45) (xy 138.43 298.45))
     (stroke (width 0) (type default))
   )
@@
     (effects (font (size 1.27 1.27)) (justify left bottom))
   )
-  (text "BOOT SELECT" (at 80.01 342.9 0)
-    (effects (font (size 1.27 1.27)) (justify left bottom))
+  (text "BOOT SELECT" (at 170.18 295.91 0)
+    (effects (font (size 1.27 1.27)) (justify right bottom))
   )
   (text "One could also use the SIO10N268 ($10) which gives for UARTs and\nan FDD controller and it's in active production still.\n\nhttps://ww1.microchip.com/downloads/aemDocuments/documents/OTH/ProductDocuments/DataSheets/00001819A.pdf\n\nOr the FDC37C78 ($11), which is just a FDD controller and is not\nrecommended for new designs and is not really in stock (big surprise).\n"
@@
     )
   )
+  (symbol (lib_id "power:+5V") (at 146.05 292.1 0) (unit 1)
+    (in_bom yes) (on_board yes) (dnp no) (fields_autoplaced)
+    (property "Reference" "#PWR0149" (at 146.05 295.91 0)
+      (effects (font (size 1.27 1.27)) hide)
+    )
+    (property "Value" "+5V" (at 146.05 287.02 0)
+      (effects (font (size 1.27 1.27)))
+    )
+    (property "Footprint" "" (at 146.05 292.1 0)
+      (effects (font (size 1.27 1.27)) hide)
+    )
+    (property "Datasheet" "" (at 146.05 292.1 0)
+      (effects (font (size 1.27 1.27)) hide)
+    )
+    (pin "1")
+    (instances
+      (project "a1_mini"
+        (path "/3257e1ae-50a8-410a-87c3-a39d96a2c51a"
+          (reference "#PWR0149") (unit 1)
+        )
+      )
+    )
+  )
   (symbol (lib_id "Device:C") (at 336.55 295.91 0) (unit 1)
     (in_bom yes) (on_board yes) (dnp no)
@@
     )
   )
-  (symbol (lib_id "Connector_Generic:Conn_01x02") (at 96.52 342.9 180) (unit 1)
+  (symbol (lib_id "Connector_Generic:Conn_01x02") (at 153.67 295.91 0) (unit 1)
     (in_bom yes) (on_board yes) (dnp no) (fields_autoplaced)
-    (property "Reference" "J11" (at 96.52 334.01 0)
+    (property "Reference" "J11" (at 153.67 304.8 0)
       (effects (font (size 1.27 1.27)))
     )
-    (property "Value" "Conn_01x02" (at 96.52 336.55 0)
+    (property "Value" "Conn_01x02" (at 153.67 302.26 0)
       (effects (font (size 1.27 1.27)))
     )
-    (property "Footprint" "Connector_PinSocket_2.54mm:PinSocket_1x02_P2.54mm_Vertical" (at 96.52 342.9 0)
+    (property "Footprint" "Connector_PinSocket_2.54mm:PinSocket_1x02_P2.54mm_Vertical" (at 153.67 295.91 0)
       (effects (font (size 1.27 1.27)) hide)
     )
-    (property "Datasheet" "~" (at 96.52 342.9 0)
+    (property "Datasheet" "~" (at 153.67 295.91 0)
       (effects (font (size 1.27 1.27)) hide)
     )
@@
         )
       )
-    )
-  )
-  (symbol (lib_id "power:GND") (at 105.41 346.71 0) (unit 1)
-    (in_bom yes) (on_board yes) (dnp no)
-    (property "Reference" "#PWR0135" (at 105.41 353.06 0)
-      (effects (font (size 1.27 1.27)) hide)
-    )
-    (property "Value" "GND" (at 105.41 351.79 0)
-      (effects (font (size 1.27 1.27)))
-    )
-    (property "Footprint" "" (at 105.41 346.71 0)
-      (effects (font (size 1.27 1.27)) hide)
-    )
-    (property "Datasheet" "" (at 105.41 346.71 0)
-      (effects (font (size 1.27 1.27)) hide)
-    )
-    (pin "1")
-    (instances
-      (project "a1_mini"
-        (path "/3257e1ae-50a8-410a-87c3-a39d96a2c51a"
-          (reference "#PWR0135") (unit 1)
-        )
-      )

Commit message: A1 Mini (which is not all that mini anymore) is feature-complete.
We have 2 ISA slots and even all the power supplies generated from +5V included.

The +12V switcher right next to the audio output is quite a bit concerning, but
we can always say that PWR must be 12V and we directly feed that to the ISA slots.
(Not that PWR is all that clean...) A lot will depend on how I implement grounding,
something that I still have to do.
Parts:
- removed C30, C31, C38, C45: 1uF, Capacitor_THT:C_Disc_D4.7mm_W2.5mm_P5.00mm, symbol Device:C
- renumbered C25 to C1, C35 to C10, C36 to C11, C39 to C12, C40 to C13, C41 to C14, C8 to C15, C42 to C16, C43 to C17, C44 to C18, C68 to C19, C26 to C2, C27 to C3, C28 to C4, C29 to C5, C32 to C6, C9 to C7, C33 to C8, C34 to C9, D3 to D1, D1 to D2, D2 to D3, J17 to J1, J18 to J2, J20 to J3, J22 to J4, J11 to J5, J1 to J6, J3 to J7, JP3 to JP1, R11 to R1, R10 to R2, R27 to R3, R13 to R4, R9 to R5, R25 to R6, R8 to R7, R12 to R8, R29 to R9, RN13 to RN1, RN12 to RN2, RN14 to RN3, RN5 to RN4, RN2 to RN5, RN1 to RN6, SW4 to SW1, SW1 to SW2, SW2 to SW3, U3 to U1, U11 to U10, U27 to U11, U18 to U12, U12 to U13, U13 to U14, U14 to U15, U8 to U16, U16 to U17, U17 to U18, U9 to U2, U33 to U3, U5 to U4, U6 to U5, U1 to U6, U2 to U7, U4 to U8, U10 to U9, X3 to X1

Commit message: A1 MINI is fully routed.
That is, if I add a GND fill on both layers. Which I don't, because auto-refill takes
several seconds and so it's a PITA to work with. There are a few dozen DRC errors
as well but nothing major it seems.

Worked out roughly 100ohm diff impedance for the HDMI lines
(not GND-referenced) which I think is my best shot of making it work.

long USB trace has a nice GND shield under-it, so does audio.
Again, probably my best shot at making these work.

Ethernet still needs checking just as short-put USB connections from the hub to
the connector.
Parts:
- J5, J7, JP1: footprint Connector_PinSocket_2.54mm:PinSocket_1x02_P2.54mm_Vertical -> Connector_PinHeader_2.54mm:PinHeader_1x02_P2.54mm_Vertical
Changed lines of the file:
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@@
   (junction (at 55.88 34.29) (diameter 0) (color 0 0 0 0)
   )
+  (junction (at 210.82 374.65) (diameter 0) (color 0 0 0 0)
+  )
   (junction (at 129.54 57.15) (diameter 0) (color 0 0 0 0)
   )
@@
     (stroke (width 0) (type default))
   )
+  (wire (pts (xy 210.82 374.65) (xy 224.79 374.65))
+    (stroke (width 0) (type default))
+  )
   (wire (pts (xy 466.09 123.19) (xy 494.03 123.19))
     (stroke (width 0) (type default))
@@
     (stroke (width 0) (type default))
   )
-  (wire (pts (xy 195.58 374.65) (xy 224.79 374.65))
+  (wire (pts (xy 195.58 374.65) (xy 210.82 374.65))
     (stroke (width 0) (type default))
   )
@@
     (stroke (width 0) (type default))
   )
+  (wire (pts (xy 210.82 370.84) (xy 210.82 374.65))
+    (stroke (width 0) (type default))
+  )
   (wire (pts (xy 458.47 311.15) (xy 468.63 311.15))
     (stroke (width 0) (type default))
@@
     (stroke (width 0) (type default))
   )
+  (wire (pts (xy 214.63 370.84) (xy 210.82 370.84))
+    (stroke (width 0) (type default))
+  )
   (bus (pts (xy 335.28 196.85) (xy 335.28 199.39))
     (stroke (width 0) (type default))
@@
     (effects (font (size 1.27 1.27)) (justify left bottom))
   )
+  (global_label "PWR_IN" (shape output) (at 214.63 370.84 0) (fields_autoplaced)
+    (effects (font (size 1.27 1.27)) (justify left))
+    (property "Intersheetrefs" "${INTERSHEET_REFS}" (at 224.5095 370.84 0)
+      (effects (font (size 1.27 1.27)) (justify left) hide)
+    )
+  )
   (global_label "~{RST}" (shape output) (at 365.76 292.1 0) (fields_autoplaced)
     (effects (font (size 1.27 1.27)) (justify left))
@@
       (effects (font (size 1.27 1.27)))
     )
-    (property "Footprint" "Connector_PinSocket_2.54mm:PinSocket_1x02_P2.54mm_Vertical" (at 153.67 295.91 0)
+    (property "Footprint" "Connector_PinHeader_2.54mm:PinHeader_1x02_P2.54mm_Vertical" (at 153.67 295.91 0)
       (effects (font (size 1.27 1.27)) hide)
     )
@@
       (effects (font (size 1.27 1.27)))
     )
-    (property "Footprint" "Connector_PinSocket_2.54mm:PinSocket_1x02_P2.54mm_Vertical" (at 213.36 406.4 0)
+    (property "Footprint" "Connector_PinHeader_2.54mm:PinHeader_1x02_P2.54mm_Vertical" (at 213.36 406.4 0)
       (effects (font (size 1.27 1.27)) hide)
     )
@@
       (effects (font (size 1.27 1.27)) hide)
     )
-    (property "Footprint" "Connector_PinSocket_2.54mm:PinSocket_1x02_P2.54mm_Vertical" (at 262.89 398.78 0)
+    (property "Footprint" "Connector_PinHeader_2.54mm:PinHeader_1x02_P2.54mm_Vertical" (at 262.89 398.78 0)
       (effects (font (size 1.27 1.27)) hide)
     )

Commit message: A1-MINI is fully routed. Also fully impedance controlled.
Changed lines of the file:
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@@
+    (effects (font (size 1.27 1.27)) (justify left bottom))
+  )
+  (label "USB_MAIN_D-" (at 382.27 407.67 0) (fields_autoplaced)
     (effects (font (size 1.27 1.27)) (justify left bottom))
   )
@@
   )
   (label "BUF_D6" (at 247.65 271.78 0) (fields_autoplaced)
+    (effects (font (size 1.27 1.27)) (justify left bottom))
+  )
+  (label "USB_MAIN_D+" (at 382.27 405.13 0) (fields_autoplaced)
     (effects (font (size 1.27 1.27)) (justify left bottom))
   )
@@
     )
   )
+  (netclass_flag "" (length 2.54) (shape round) (at 369.57 407.67 0) (fields_autoplaced)
+    (effects (font (size 1.27 1.27)) (justify left bottom))
+    (property "Netclass" "USB" (at 370.2685 405.13 0)
+      (effects (font (size 1.27 1.27) italic) (justify left))
+    )
+  )
+  (netclass_flag "" (length 2.54) (shape round) (at 364.49 405.13 0) (fields_autoplaced)
+    (effects (font (size 1.27 1.27)) (justify left bottom))
+    (property "Netclass" "USB" (at 365.1885 402.59 0)
+      (effects (font (size 1.27 1.27) italic) (justify left))
+    )
+  )
