File: boards/a1_mini/a1_mini.kicad_sch (KiCad schematic)
At the start: 67 parts, among them J1 Conn_01x01, J2 Conn_01x01, J3 Conn_01x01, J4 Conn_01x01, J5 Conn_01x02, J6 Jack-DC, J7 Conn_01x02, SW1 SW_DPDT_x2, SW2 SW_Push, SW3 SW_Push, U1 74LS08, U10 74AHCT245, U11 SST39SF040, U12 A1_POWER, U13 74AHCT245, U14 74AHCT245, U15 74AHCT245, U16 74LS273, U17 74LS273, U18 74LS273, U2 74LS86, U3 74LS00, U4 74LS273, U5 74LS574, U6 74LS139, U7 74LS14, U8 74LS126, U9 74AHCT245, X1 8MHz

Commit message: Checking in stuff before the 3.3V work.
Other:
- note added: "These should be 3.3V parts to enable 3.3V DRAM modules. LVC devices with an A suffix are like that, and those still seem to come in DIP packages. So we need: SN74LVC245AN SN74AHC126N For full 3.3V conversion, 273 needs to be exchanged to 373 or even better, 574 chips. The AHC series seems to have similar properties, which is good as the SN74LVC139 is NOT available in DIP."
Changed lines of the file:
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@@
     (stroke (width 0) (type default))
+  )
+  (rectangle (start 163.83 15.24) (end 229.87 39.37)
+    (stroke (width 0) (type default))
+    (fill (type color) (color 145 253 255 1))
+  )
+  (rectangle (start 406.4 74.93) (end 443.23 132.08)
+    (stroke (width 0) (type default))
+    (fill (type color) (color 145 253 255 1))
+  )
+  (rectangle (start 105.41 15.24) (end 138.43 33.02)
+    (stroke (width 0) (type default))
+    (fill (type color) (color 145 253 255 1))
+  )
+  (rectangle (start 114.3 229.87) (end 153.67 274.32)
+    (stroke (width 0) (type default))
+    (fill (type color) (color 145 253 255 1))
+  )
+  (rectangle (start 280.67 160.02) (end 303.53 177.8)
+    (stroke (width 0) (type default))
+    (fill (type color) (color 145 253 255 1))
+  )
+  (rectangle (start 125.73 87.63) (end 260.35 144.78)
+    (stroke (width 0) (type default))
+    (fill (type color) (color 145 253 255 1))
   )
   (text "Data is captured on the falling edge of nWE | nCAS by the DRAM.\nThus, buffering either of those will not cause write-setup\nviolations. At the same time, read responses are delayed, but\nthat can be handled by slowing the clock down.\n\nSo, all in all, we can buffer control and address signals to\nthe DRAM without too much worry. Buffering data hopefully is\nnot necessary as there's only 4 loads on the bus.\n\nTons of DRAM datasheets: https://minuszerodegrees.net/memory/ram.htm\n\nEssentially everything supported page mode, no worries there.\n\nSIMM socket source: https://www.peconnectors.com/sockets-pga-cpu-and-memory/hws9594/\n"
@@
     (effects (font (size 1.27 1.27)) (justify left bottom))
   )
+  (text "These should be 3.3V parts to enable 3.3V DRAM modules.\nLVC devices with an A suffix are like that, and those\nstill seem to come in DIP packages. So we need:\nSN74LVC245AN\nSN74AHC126N\nFor full 3.3V conversion, 273 needs to be exchanged to 373 \nor even better, 574 chips.\nThe AHC series seems to have similar properties, which is good\nas the SN74LVC139 is NOT available in DIP."
+    (at 166.37 35.56 0)
+    (effects (font (size 1.27 1.27)) (justify left bottom))
+  )

Commit message: 3.3V work, before abandoning the idea.
Parts:
- added C67, C68, C69, C70, C71: 1uF, Capacitor_THT:C_Disc_D4.7mm_W2.5mm_P5.00mm, symbol Device:C
- U1: value 74LS08 -> SN74AHC08N
- U10, U13, U14, U9: value 74AHCT245 -> SN74LVC245AN
- U16, U17, U18, U4: value 74LS273 -> SN74AHC574N; symbol 74xx:74LS273 -> 74xx:74LS574
- U2: value 74LS86 -> SN74AHC86N
- U3: value 74LS00 -> SN74AHC00N
- U5: value 74LS574 -> SN74AHC574N
- U6: value 74LS139 -> SN74AHC139N
- U7: value 74LS14 -> SN74AHC14N
- U8: value 74LS126 -> SN74AHC126N
Connections:
- net +5V: no longer C1.1, C10.1, C11.1, C12.1, C13.1, C14.1, C16.1, C18.1, C19.1, C2.1, C3.1, C4.1, C5.1, C8.1, C9.1, J5.1 (Pin_1), R2.1, R3.1, R5.1, R7.1, R9.1, RN1.1 (common), RN3.1 (common), U1.14 (VCC), U10.20 (VCC), U13.20 (VCC), U14.20 (VCC), U15.1 (A->B), U15.20 (VCC), U16.1 (~{Mr}), U16.20 (VCC), U17.1 (~{Mr}), U17.20 (VCC), U18.1 (~{Mr}), U18.20 (VCC), U2.12, U2.14 (VCC), U2.4, U2.9, U3.14 (VCC), U3.9, U4.20 (VCC), U5.20 (VCC), U6.16 (VCC), U7.14 (VCC), U8.14 (VCC), U9.20 (VCC), X1.1 (EN), X1.14 (Vcc)
- net BUF_A1: now also U16.12 (Q7); no longer U16.19 (Q7)
- net BUF_A12: now also U18.12 (Q7); no longer U18.19 (Q7)
- net BUF_A13: now also U18.19 (Q0); no longer U18.2 (Q0)
- net BUF_A14: now also U18.13 (Q6); no longer U18.16 (Q6)
- net BUF_A15: now also U18.18 (Q1); no longer U18.5 (Q1)
- net BUF_A16: now also U18.14 (Q5); no longer U18.15 (Q5)
- net BUF_A17: now also U18.17 (Q2); no longer U18.6 (Q2)
- net BUF_A18: now also U18.15 (Q4); no longer U18.12 (Q4)
- net BUF_A19: now also U18.16 (Q3); no longer U18.9 (Q3)
- net BUF_A2: now also U16.19 (Q0); no longer U16.2 (Q0)
- net BUF_A20: now also U17.12 (Q7); no longer U17.19 (Q7)
- net BUF_A21: now also U17.13 (Q6); no longer U17.16 (Q6)
- net BUF_A22: now also U17.14 (Q5); no longer U17.15 (Q5)
- net BUF_A3: now also U16.13 (Q6); no longer U16.16 (Q6)
- net BUF_A4: now also U16.18 (Q1); no longer U16.5 (Q1)
- net BUF_A5: now also U16.14 (Q5); no longer U16.15 (Q5)
- net BUF_A6: now also U16.17 (Q2); no longer U16.6 (Q2)
- net BUF_A7: now also U16.15 (Q4); no longer U16.12 (Q4)
- net BUF_A8: now also U16.16 (Q3); no longer U16.9 (Q3)
- net BUF_D0: now also U4.5 (D3); no longer U4.8 (D3)
- net BUF_D1: now also U4.6 (D4); no longer U4.13 (D4)
- net BUF_D2: now also U4.4 (D2); no longer U4.7 (D2)
- net BUF_D3: now also U4.7 (D5); no longer U4.14 (D5)
- net BUF_D4: now also U4.3 (D1); no longer U4.4 (D1)
- net BUF_D5: now also U4.8 (D6); no longer U4.17 (D6)
- net BUF_D6: now also U4.2 (D0); no longer U4.3 (D0)
- net BUF_D7: now also U4.9 (D7); no longer U4.18 (D7)
- net CPU_A0: now also U16.9 (D7), U18.9 (D7); no longer U16.18 (D7), U18.18 (D7)
- net CPU_A1: now also U16.2 (D0), U18.2 (D0); no longer U16.3 (D0), U18.3 (D0)
- net CPU_A10: now also U17.7 (D5); no longer U17.14 (D5)
- net CPU_A2: now also U16.8 (D6), U18.8 (D6); no longer U16.17 (D6), U18.17 (D6)
- net CPU_A3: now also U16.3 (D1), U18.3 (D1); no longer U16.4 (D1), U18.4 (D1)
- net CPU_A4: now also U16.7 (D5), U18.7 (D5); no longer U16.14 (D5), U18.14 (D5)
- net CPU_A5: now also U16.4 (D2), U18.4 (D2); no longer U16.7 (D2), U18.7 (D2)
- net CPU_A6: now also U16.6 (D4), U18.6 (D4); no longer U16.13 (D4), U18.13 (D4)
- net CPU_A7: now also U16.5 (D3), U18.5 (D3); no longer U16.8 (D3), U18.8 (D3)
- net CPU_A8: now also U17.9 (D7); no longer U17.18 (D7)
- net CPU_A9: now also U17.8 (D6); no longer U17.17 (D6)
- net GND: now also U16.1 (OE), U17.1 (OE), U18.1 (OE), C67.2, C68.2, C69.2, C70.2, C71.2
- net at U4.12 (Q7): now also U8.12
- net at U4.16 (Q3): now also R4.1
- net at U4.19 (Q0): now also U8.9; no longer U8.12
- new net +3.3V: C1.1, C10.1, C11.1, C12.1, C13.1, C14.1, C16.1, C18.1, C19.1, C2.1, C3.1, C4.1, C5.1, C67.1, C68.1, C69.1, C70.1, C71.1, C8.1, C9.1, J5.1 (Pin_1), R2.1, R3.1, R5.1, R7.1, R9.1, RN1.1 (common), RN3.1 (common), U1.14 (VCC), U10.20 (VCC), U13.20 (VCC), U14.20 (VCC), U15.1 (A->B), U15.20 (VCC), U16.20 (VCC), U17.20 (VCC), U18.20 (VCC), U2.12, U2.14 (VCC), U2.4, U2.9, U3.14 (VCC), U3.9, U4.20 (VCC), U5.20 (VCC), U6.16 (VCC), U7.14 (VCC), U8.14 (VCC), U9.20 (VCC), X1.1 (EN), X1.14 (Vcc)
Other:
- moved on the sheet: C17, C6
