File: boards/a1_mini/usb.kicad_sch (KiCad schematic)
At the start: 24 parts, among them J4 USB_A_Stacked, J8 USB_A_Stacked, J9 USB_A_Stacked, U7 A1_USBHUB

Commit message: A1 Mini (which is not all that mini anymore) is feature-complete.
We have 2 ISA slots and even all the power supplies generated from +5V included.

The +12V switcher right next to the audio output is quite a bit concerning, but
we can always say that PWR must be 12V and we directly feed that to the ISA slots.
(Not that PWR is all that clean...) A lot will depend on how I implement grounding,
something that I still have to do.
Parts:
- renumbered C10 to C44, C19 to C45, C20 to C46, C18 to C47, C23 to C48, C21 to C49, C22 to C50, CMC7 to CMC10, CMC8 to CMC7, CMC9 to CMC8, CMC10 to CMC9, FB2 to FB15, FB4 to FB16, FB5 to FB17, FB6 to FB18, FB7 to FB19, FB3 to FB20, J8 to J15, J4 to J16, J9 to J17, JP2 to JP3, U7 to U28

Commit message: A1-MINI is fully routed. Also fully impedance controlled.
Connections:
- net USB_DN6_D-: now reaches CMC9.4, U28.14 (USBDN6_DM)
- net USB_DN6_D+: now reaches CMC9.1, U28.15 (USBDN6_DP)
- net USB_DN7_D-: now reaches CMC10.4, U28.16 (USBDN7_DM)
- net USB_DN7_D+: now reaches CMC10.1, U28.17 (USBDN7_DP)
- net USB_DN2_D-: now reaches CMC5.4, U28.25 (USBDN2_DM)
- net USB_DN2_D+: now reaches CMC5.1, U28.26 (USBDN2_DP)
- net USB_DN3_D-: now reaches CMC6.4, U28.27 (USBDN3_DM)
- net USB_DN3_D+: now reaches CMC6.1, U28.28 (USBDN3_DP)
- net USB_DN4_D-: now reaches CMC7.4, U28.29 (USBDN4_DM)
- net USB_DN4_D+: now reaches CMC7.1, U28.30 (USBDN4_DP)
- net USB_DN5_D-: now reaches CMC8.4, U28.31 (USBDN5_DM)
- net USB_DN5_D+: now reaches CMC8.1, U28.32 (USBDN5_DP)
Other:
- moved on the sheet: C44, CMC10, CMC5, CMC6, CMC7, CMC8, CMC9, JP3, U28
