File: boards/a1_mini/ethernet.kicad_sch (KiCad schematic)
At the start: 15 parts, among them U15 KSZ8851-11MLL, Y2 25MHz

Commit message: Added boot mode switch, reworked LAN IRQ, places LEDs better.
Connections:
- net ~{LAN_IRQ} renamed ~{INT}
Changed lines of the file:
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@@
     (effects (font (size 1.27 1.27)) (justify right))
   )
-  (hierarchical_label "~{LAN_IRQ}" (shape output) (at 158.115 80.01 0) (fields_autoplaced)
+  (hierarchical_label "~{INT}" (shape output) (at 158.115 80.01 0) (fields_autoplaced)
     (effects (font (size 1.27 1.27)) (justify left))
   )

Commit message: A1 Mini (which is not all that mini anymore) is feature-complete.
We have 2 ISA slots and even all the power supplies generated from +5V included.

The +12V switcher right next to the audio output is quite a bit concerning, but
we can always say that PWR must be 12V and we directly feed that to the ISA slots.
(Not that PWR is all that clean...) A lot will depend on how I implement grounding,
something that I still have to do.
Parts:
- renumbered C11 to C39, C12 to C40, C15 to C41, C16 to C42, C17 to C43, J2 to J14, R14 to R22, R15 to R23, R16 to R24, R17 to R25, R22 to R26, R23 to R27, R24 to R28, U15 to U27

Commit message: A1-MINI is fully routed. Also fully impedance controlled.
Connections:
- net ETH_RX+: now reaches J14.R3 (RD+), R25.2, U27.26 (RXP1)
- net ETH_TX+: now reaches J14.R1 (TD+), R27.2, U27.29 (TXP1)
- net ETH_TX-: now reaches J14.R2 (TD-), R28.2, U27.30 (TXM1)
- net ETH_RX-: now reaches J14.R6 (RD-), R26.2, U27.27 (RXM1)
Changed lines of the file:
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@@
+    (effects (font (size 1.27 1.27)) (justify left bottom))
+  )
+  (label "ETH_TX-" (at 146.05 95.25 0) (fields_autoplaced)
+    (effects (font (size 1.27 1.27)) (justify left bottom))
+  )
+  (label "ETH_RX+" (at 146.05 85.09 0) (fields_autoplaced)
     (effects (font (size 1.27 1.27)) (justify left bottom))
   )
   (label "CMD" (at 74.93 82.55 0) (fields_autoplaced)
+    (effects (font (size 1.27 1.27)) (justify left bottom))
+  )
+  (label "ETH_RX-" (at 146.05 87.63 0) (fields_autoplaced)
     (effects (font (size 1.27 1.27)) (justify left bottom))
   )
@@
   )
   (label "D4" (at 58.42 97.79 0) (fields_autoplaced)
+    (effects (font (size 1.27 1.27)) (justify left bottom))
+  )
+  (label "ETH_TX+" (at 146.05 92.71 0) (fields_autoplaced)
     (effects (font (size 1.27 1.27)) (justify left bottom))
   )
@@
     (effects (font (size 1.27 1.27)) (justify right))
   )
+  (netclass_flag "" (length 2.54) (shape round) (at 161.29 85.09 0) (fields_autoplaced)
+    (effects (font (size 1.27 1.27)) (justify left bottom))
+    (property "Netclass" "ETH" (at 161.9885 82.55 0)
+      (effects (font (size 1.27 1.27) italic) (justify left))
+    )
+  )
+  (netclass_flag "" (length 2.54) (shape round) (at 167.64 87.63 0) (fields_autoplaced)
+    (effects (font (size 1.27 1.27)) (justify left bottom))
+    (property "Netclass" "ETH" (at 168.3385 85.09 0)
+      (effects (font (size 1.27 1.27) italic) (justify left))
+    )
+  )
+  (netclass_flag "" (length 2.54) (shape round) (at 167.64 95.25 0) (fields_autoplaced)
+    (effects (font (size 1.27 1.27)) (justify left bottom))
+    (property "Netclass" "ETH" (at 168.3385 92.71 0)
+      (effects (font (size 1.27 1.27) italic) (justify left))
+    )
+  )
+  (netclass_flag "" (length 2.54) (shape round) (at 161.29 92.71 0) (fields_autoplaced)
+    (effects (font (size 1.27 1.27)) (justify left bottom))
+    (property "Netclass" "ETH" (at 161.9885 90.17 0)
+      (effects (font (size 1.27 1.27) italic) (justify left))
+    )
+  )
   (symbol (lib_id "Device:R_US") (at 182.245 103.505 180) (unit 1)

Commit message: 3.3V work, before abandoning the idea.
Connections:
- net +5V: no longer R22.2
- new net +3.3V: R22.2
Other:
- moved on the sheet: R22
Changed lines of the file:
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@@
   (junction (at 187.96 87.63) (diameter 0) (color 0 0 0 0)
   )
+  (junction (at 143.51 80.01) (diameter 0) (color 0 0 0 0)
+  )
   (junction (at 219.075 87.63) (diameter 0) (color 0 0 0 0)
   )
   (junction (at 155.575 106.68) (diameter 0) (color 0 0 0 0)
-  )
-  (junction (at 142.875 80.01) (diameter 0) (color 0 0 0 0)
   )
   (junction (at 196.85 111.125) (diameter 0) (color 0 0 0 0)
@@
     (stroke (width 0) (type default))
   )
+  (wire (pts (xy 143.51 80.01) (xy 158.115 80.01))
+    (stroke (width 0) (type default))
+  )
   (wire (pts (xy 271.145 49.53) (xy 271.145 80.01))
     (stroke (width 0) (type default))
@@
     (stroke (width 0) (type default))
   )
-  (wire (pts (xy 142.875 80.01) (xy 158.115 80.01))
+  (wire (pts (xy 137.16 80.01) (xy 143.51 80.01))
     (stroke (width 0) (type default))
   )
@@
     (stroke (width 0) (type default))
   )
-  (wire (pts (xy 137.16 80.01) (xy 142.875 80.01))
-    (stroke (width 0) (type default))
-  )
   (wire (pts (xy 187.96 107.315) (xy 187.96 111.125))
     (stroke (width 0) (type default))
   )
-  (wire (pts (xy 142.875 66.04) (xy 142.875 80.01))
+  (wire (pts (xy 143.51 66.04) (xy 143.51 80.01))
     (stroke (width 0) (type default))
   )
@@
     )
   )
+  (symbol (lib_id "power:+3.3V") (at 143.51 58.42 0) (unit 1)
+    (in_bom yes) (on_board yes) (dnp no) (fields_autoplaced)
+    (property "Reference" "#PWR0185" (at 143.51 62.23 0)
+      (effects (font (size 1.27 1.27)) hide)
+    )
+    (property "Value" "+3.3V" (at 143.51 53.34 0)
+      (effects (font (size 1.27 1.27)))
+    )
+    (property "Footprint" "" (at 143.51 58.42 0)
+      (effects (font (size 1.27 1.27)) hide)
+    )
+    (property "Datasheet" "" (at 143.51 58.42 0)
+      (effects (font (size 1.27 1.27)) hide)
+    )
+    (pin "1")
+    (instances
+      (project "a1_mini"
+        (path "/3257e1ae-50a8-410a-87c3-a39d96a2c51a/0237d891-a96a-4307-a4d5-070a11371520"
+          (reference "#PWR0185") (unit 1)
+        )
+      )
+    )
+  )
   (symbol (lib_id "power:GND") (at 168.275 114.3 0) (unit 1)
     (in_bom yes) (on_board yes) (dnp no) (fields_autoplaced)
@@
     )
   )
-  (symbol (lib_id "Device:R_US") (at 142.875 62.23 180) (unit 1)
-    (in_bom yes) (on_board yes) (dnp no)
-    (property "Reference" "R22" (at 140.335 64.77 90)
-      (effects (font (size 1.27 1.27)))
-    )
-    (property "Value" "10k" (at 140.335 59.69 90)
-      (effects (font (size 1.27 1.27)))
-    )
-    (property "Footprint" "Resistor_THT:R_Axial_DIN0204_L3.6mm_D1.6mm_P5.08mm_Horizontal" (at 141.859 61.976 90)
-      (effects (font (size 1.27 1.27)) hide)
-    )
-    (property "Datasheet" "~" (at 142.875 62.23 0)
+  (symbol (lib_id "Device:R_US") (at 143.51 62.23 180) (unit 1)
+    (in_bom yes) (on_board yes) (dnp no)
+    (property "Reference" "R22" (at 140.97 64.77 90)
+      (effects (font (size 1.27 1.27)))
+    )
+    (property "Value" "10k" (at 140.97 59.69 90)
+      (effects (font (size 1.27 1.27)))
+    )
+    (property "Footprint" "Resistor_THT:R_Axial_DIN0204_L3.6mm_D1.6mm_P5.08mm_Horizontal" (at 142.494 61.976 90)
+      (effects (font (size 1.27 1.27)) hide)
+    )
+    (property "Datasheet" "~" (at 143.51 62.23 0)
       (effects (font (size 1.27 1.27)) hide)
     )
@@
         )
       )
-    )
-  )
-  (symbol (lib_id "power:+5V") (at 142.875 58.42 0) (unit 1)
-    (in_bom yes) (on_board yes) (dnp no) (fields_autoplaced)
-    (property "Reference" "#PWR0185" (at 142.875 62.23 0)
-      (effects (font (size 1.27 1.27)) hide)
-    )
-    (property "Value" "+5V" (at 142.875 53.34 0)
-      (effects (font (size 1.27 1.27)))
-    )
-    (property "Footprint" "" (at 142.875 58.42 0)
-      (effects (font (size 1.27 1.27)) hide)
-    )
-    (property "Datasheet" "" (at 142.875 58.42 0)
-      (effects (font (size 1.27 1.27)) hide)
-    )
-    (pin "1")
-    (instances
-      (project "a1_mini"
-        (path "/3257e1ae-50a8-410a-87c3-a39d96a2c51a/0237d891-a96a-4307-a4d5-070a11371520"
-          (reference "#PWR0185") (unit 1)
-        )
-      )
