File: boards/a1_mini/graphics.kicad_sch (KiCad schematic)
At the start: 39 parts, among them J12 SJ1-3535NG-BE, J13 SJ1-3535NG-BE, J5 Conn_01x02, J6 HDMI_A, U24 DISCO, U25 A1_CODEC, X1 CXO_DIP14

Commit message: A1 Mini (which is not all that mini anymore) is feature-complete.
We have 2 ISA slots and even all the power supplies generated from +5V included.

The +12V switcher right next to the audio output is quite a bit concerning, but
we can always say that PWR must be 12V and we directly feed that to the ISA slots.
(Not that PWR is all that clean...) A lot will depend on how I implement grounding,
something that I still have to do.
Parts:
- renumbered C57 to C24, C58 to C25, C59 to C26, C1 to C27, C13 to C28, C14 to C29, C2 to C30, C3 to C31, FB18 to FB1, FB19 to FB2, FB1 to FB3, FB13 to FB4, FB20 to FB5, FB14 to FB6, FB16 to FB7, FB17 to FB8, FB15 to FB9, J6 to J10, J12 to J11, J13 to J8, J5 to J9, JP1 to JP2, R20 to R10, R21 to R11, R1 to R12, R19 to R13, R18 to R14, R7 to R15, R2 to R16, R3 to R17, TP2 to TP1, U24 to U22, U25 to U23, X1 to X2

Commit message: A1 MINI is fully routed.
That is, if I add a GND fill on both layers. Which I don't, because auto-refill takes
several seconds and so it's a PITA to work with. There are a few dozen DRC errors
as well but nothing major it seems.

Worked out roughly 100ohm diff impedance for the HDMI lines
(not GND-referenced) which I think is my best shot of making it work.

long USB trace has a nice GND shield under-it, so does audio.
Again, probably my best shot at making these work.

Ethernet still needs checking just as short-put USB connections from the hub to
the connector.
Parts:
- added JP7: Jumper_2_Bridged, Connector_PinHeader_2.54mm:PinHeader_1x02_P2.54mm_Vertical, symbol Jumper:Jumper_2_Open
Connections:
- net GND: now also JP7.1 (A); no longer J11.1, J8.1, R10.2, R11.2, R14.2, R15.2, U23.10 (AGND), U23.16 (AGND), U23.17 (AGND), U23.23 (AGND), U23.26 (AGND)
- new net GNDA: J11.1, J8.1, JP7.2 (B), R10.2, R11.2, R14.2, R15.2, U23.10 (AGND), U23.16 (AGND), U23.17 (AGND), U23.23 (AGND), U23.26 (AGND)
Other:
- note added: "GND and GNDA are tied inside CODEC"

Commit message: A1-MINI is fully routed. Also fully impedance controlled.
Connections:
- net TMDS_CLK+: now reaches CMC4.1, U22.7 (TMDS_C+)
- net TMDS_CLK-: now reaches CMC4.4, U22.8 (TMDS_C-)
- net TMDS_D2+: now reaches CMC1.1, U22.1 (TMDS_D2+)
- net TMDS_D2-: now reaches CMC1.4, U22.2 (TMDS_D2-)
- net TMDS_D0+: now reaches CMC3.1, U22.5 (TMDS_D0+)
- net TMDS_D0-: now reaches CMC3.4, U22.6 (TMDS_D0-)
- net TMDS_D1+: now reaches CMC2.1, U22.3 (TMDS_D1+)
- net TMDS_D1-: now reaches CMC2.4, U22.4 (TMDS_D1-)
Other:
- note added: "TMDS output is quite a bit dicey on UNIC. The power diodes add too much capacitive load and limit operations to maybe 250...300Mbps. That might be sufficient for VGA resolution but not for XGA."
Changed lines of the file:
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@@
     (stroke (width 0) (type default))
   )
+  (text "TMDS output is quite a bit dicey on UNIC. The power diodes\nadd too much capacitive load and limit operations to maybe\n250...300Mbps. That might be sufficient for VGA resolution\nbut not for XGA."
+    (at 177.8 55.88 0)
+    (effects (font (size 1.27 1.27)) (justify left bottom))
+  )
   (text "GND and GNDA are tied inside CODEC" (at 113.03 199.39 0)
+    (effects (font (size 1.27 1.27)) (justify left bottom))
+  )
+  (label "TMDS_CLK+" (at 130.81 76.2 0) (fields_autoplaced)
     (effects (font (size 1.27 1.27)) (justify left bottom))
   )
@@
     (effects (font (size 1.27 1.27)) (justify left bottom))
   )
+  (label "TMDS_D0-" (at 130.81 71.12 0) (fields_autoplaced)
+    (effects (font (size 1.27 1.27)) (justify left bottom))
+  )
   (label "AUDIO_SFRM" (at 87.63 135.89 0) (fields_autoplaced)
     (effects (font (size 1.27 1.27)) (justify left bottom))
   )
   (label "A4" (at 57.15 58.42 0) (fields_autoplaced)
+    (effects (font (size 1.27 1.27)) (justify left bottom))
+  )
+  (label "TMDS_CLK-" (at 130.81 78.74 0) (fields_autoplaced)
     (effects (font (size 1.27 1.27)) (justify left bottom))
   )
@@
     (effects (font (size 1.27 1.27)) (justify left bottom))
   )
+  (label "TMDS_D2+" (at 130.81 58.42 0) (fields_autoplaced)
+    (effects (font (size 1.27 1.27)) (justify left bottom))
+  )
   (label "AUDIO_SDATA_IN" (at 120.65 93.98 0) (fields_autoplaced)
     (effects (font (size 1.27 1.27)) (justify left bottom))
@@
     (effects (font (size 1.27 1.27)) (justify left bottom))
   )
+  (label "TMDS_D2-" (at 130.81 60.96 0) (fields_autoplaced)
+    (effects (font (size 1.27 1.27)) (justify left bottom))
+  )
   (label "AUDIO_SDATA_IN" (at 87.63 140.97 0) (fields_autoplaced)
+    (effects (font (size 1.27 1.27)) (justify left bottom))
+  )
+  (label "TMDS_D1+" (at 130.81 63.5 0) (fields_autoplaced)
     (effects (font (size 1.27 1.27)) (justify left bottom))
   )
@@
   )
   (label "A0" (at 57.15 48.26 0) (fields_autoplaced)
+    (effects (font (size 1.27 1.27)) (justify left bottom))
+  )
+  (label "TMDS_D1-" (at 130.81 66.04 0) (fields_autoplaced)
     (effects (font (size 1.27 1.27)) (justify left bottom))
   )
@@
     (effects (font (size 1.27 1.27)) (justify left bottom))
   )
+  (label "TMDS_D0+" (at 130.81 68.58 0) (fields_autoplaced)
+    (effects (font (size 1.27 1.27)) (justify left bottom))
+  )

Commit message: 3.3V work, before abandoning the idea.
Connections:
- net +5V: no longer X2.1 (EN), X2.14 (Vcc)
- new net +3.3V: X2.1 (EN), X2.14 (Vcc)
Changed lines of the file:
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@@
-    )
-  )
-  (symbol (lib_id "power:+5V") (at 181.61 34.29 0) (unit 1)
-    (in_bom yes) (on_board yes) (dnp no) (fields_autoplaced)
-    (property "Reference" "#PWR0144" (at 181.61 38.1 0)
-      (effects (font (size 1.27 1.27)) hide)
-    )
-    (property "Value" "+5V" (at 181.61 29.21 0)
-      (effects (font (size 1.27 1.27)))
-    )
-    (property "Footprint" "" (at 181.61 34.29 0)
-      (effects (font (size 1.27 1.27)) hide)
-    )
-    (property "Datasheet" "" (at 181.61 34.29 0)
-      (effects (font (size 1.27 1.27)) hide)
-    )
-    (pin "1")
-    (instances
-      (project "a1_mini"
-        (path "/3257e1ae-50a8-410a-87c3-a39d96a2c51a/ca3554d2-b22b-4135-824b-57937af5503f"
-          (reference "#PWR0144") (unit 1)
-        )
-      )
     )
   )
@@
     )
   )
+  (symbol (lib_id "power:+3.3V") (at 172.72 34.29 0) (unit 1)
+    (in_bom yes) (on_board yes) (dnp no) (fields_autoplaced)
+    (property "Reference" "#PWR0142" (at 172.72 38.1 0)
+      (effects (font (size 1.27 1.27)) hide)
+    )
+    (property "Value" "+3.3V" (at 172.72 29.21 0)
+      (effects (font (size 1.27 1.27)))
+    )
+    (property "Footprint" "" (at 172.72 34.29 0)
+      (effects (font (size 1.27 1.27)) hide)
+    )
+    (property "Datasheet" "" (at 172.72 34.29 0)
+      (effects (font (size 1.27 1.27)) hide)
+    )
+    (pin "1")
+    (instances
+      (project "a1_mini"
+        (path "/3257e1ae-50a8-410a-87c3-a39d96a2c51a/ca3554d2-b22b-4135-824b-57937af5503f"
+          (reference "#PWR0142") (unit 1)
+        )
+      )
+    )
+  )
   (symbol (lib_id "power:GNDA") (at 223.52 151.13 0) (unit 1)
     (in_bom yes) (on_board yes) (dnp no) (fields_autoplaced)
@@
         (path "/3257e1ae-50a8-410a-87c3-a39d96a2c51a/ca3554d2-b22b-4135-824b-57937af5503f"
           (reference "#PWR0149") (unit 1)
-        )
-      )
-    )
-  )
-  (symbol (lib_id "power:+5V") (at 172.72 34.29 0) (unit 1)
-    (in_bom yes) (on_board yes) (dnp no) (fields_autoplaced)
-    (property "Reference" "#PWR0142" (at 172.72 38.1 0)
-      (effects (font (size 1.27 1.27)) hide)
-    )
-    (property "Value" "+5V" (at 172.72 29.21 0)
-      (effects (font (size 1.27 1.27)))
-    )
-    (property "Footprint" "" (at 172.72 34.29 0)
-      (effects (font (size 1.27 1.27)) hide)
-    )
-    (property "Datasheet" "" (at 172.72 34.29 0)
-      (effects (font (size 1.27 1.27)) hide)
-    )
-    (pin "1")
-    (instances
-      (project "a1_mini"
-        (path "/3257e1ae-50a8-410a-87c3-a39d96a2c51a/ca3554d2-b22b-4135-824b-57937af5503f"
-          (reference "#PWR0142") (unit 1)
         )
       )
@@
         )
       )
+    )
+  )
+  (symbol (lib_id "power:+3.3V") (at 181.61 34.29 0) (unit 1)
+    (in_bom yes) (on_board yes) (dnp no) (fields_autoplaced)
+    (property "Reference" "#PWR0144" (at 181.61 38.1 0)
+      (effects (font (size 1.27 1.27)) hide)
+    )
+    (property "Value" "+3.3V" (at 181.61 29.21 0)
+      (effects (font (size 1.27 1.27)))
+    )
+    (property "Footprint" "" (at 181.61 34.29 0)
+      (effects (font (size 1.27 1.27)) hide)
+    )
+    (property "Datasheet" "" (at 181.61 34.29 0)
+      (effects (font (size 1.27 1.27)) hide)
+    )
+    (pin "1")
+    (instances
+      (project "a1_mini"
+        (path "/3257e1ae-50a8-410a-87c3-a39d96a2c51a/ca3554d2-b22b-4135-824b-57937af5503f"
+          (reference "#PWR0144") (unit 1)
+        )
+      )
