File: boards/a1_mini/isa.kicad_sch (KiCad schematic)
At the start: 19 parts, among them J1 Bus_ISA_8bit, J2 Bus_ISA_8bit, J3 Bus_ISA_8bit, J4 Bus_ISA_8bit, U1 74LS139, U22 74LS125, U23 74LS125, U35 L79L05_TO92, U7 74LS04, U9 74LS86, X4 14.31818MHz

Commit message: ISA is incorporated back into mini. Not routed yet.
Parts:
- removed RN4: 10k, Resistor_THT:R_Array_SIP4, symbol Device:R_Network03_US
- removed RN7: 10k, Resistor_THT:R_Array_SIP9, symbol Device:R_Network08_US
- removed U22, U23: 74LS125, Package_DIP:DIP-14_W7.62mm_LongPads, symbol 74xx:74LS125
- removed U7: 74LS04, Package_DIP:DIP-14_W7.62mm_LongPads, symbol 74xx:74LS04
- removed U9: 74LS86, Package_DIP:DIP-14_W7.62mm_LongPads, symbol 74xx:74LS86
- added C64, C65: 1uF, Capacitor_THT:C_Disc_D4.7mm_W2.5mm_P5.00mm, symbol Device:C
- added RN7: 10k, Resistor_THT:R_Array_SIP5, symbol Device:R_Network04_US
- added unit 2 of U22
- added U32: 4075, Package_DIP:DIP-14_W7.62mm_LongPads, symbol 4xxx:4075
- added U34: 74LS14, Package_DIP:DIP-14_W7.62mm_LongPads, symbol 74xx:74LS14
- renumbered C51 to C24, C16 to C37, C56 to C51, C15 to C56, J1 to J14, J2 to J15, J3 to J16, J4 to J19, U1 to U22, U35 to U23
Connections:
- net ISA_DRQ1 is gone; now on net DRQ1: J14.18 (DRQ1), J15.18 (DRQ1), J16.18 (DRQ1), J19.18 (DRQ1)
- net ISA_DRQ2 is gone; now on net DRQ2: J14.6 (DRQ2), J15.6 (DRQ2), J16.6 (DRQ2), J19.6 (DRQ2)
- net ISA_IOCHRDY is gone; now on net ~{WAIT}: J14.41 (IO_READY), J15.41 (IO_READY), J16.41 (IO_READY), J19.41 (IO_READY)
- net ISA_TC is gone; now on net DMA_TC: J14.27 (TC), J15.27 (TC), J16.27 (TC), J19.27 (TC)
- net ~{DMA3_EN} is gone; now on net DRQ3: J14.16 (DRQ3), J15.16 (DRQ3), J16.16 (DRQ3), J19.16 (DRQ3)
- net ~{ISA_DACK1} is gone; now on net ~{DACK1}: J14.17 (~{DACK1}), J15.17 (~{DACK1}), J16.17 (~{DACK1}), J19.17 (~{DACK1})
- net ~{ISA_DACK2} is gone; now on net ~{DACK2}: J14.26 (~{DACK2}), J15.26 (~{DACK2}), J16.26 (~{DACK2}), J19.26 (~{DACK2})
- net ~{ISA_DACK3} is gone; now on net ~{DACK3}: J14.15 (~{DACK3}), J15.15 (~{DACK3}), J16.15 (~{DACK3}), J19.15 (~{DACK3})
- net +5V: now also U22.16 (VCC), C64.1, C65.1, RN7.1 (common), U32.14 (VDD), U34.14 (VCC)
- net GND: now also U22.8 (GND), C64.2, C65.2, U32.7 (VSS), U34.7 (GND)
- net ISA_A20: now also U22.13 (A1); no longer U22.13 (A1)
- net ISA_AEN: now also U34.8
- net ISA_ALE: now also U34.12
- net ISA_IRQ2: now also RN5.2 (R1), U32.5; no longer RN5.7 (R6)
- net ISA_IRQ3: now also RN5.7 (R6), U32.4; no longer RN5.6 (R5)
- net ISA_IRQ4: now also RN5.6 (R5), U32.3; no longer RN5.5 (R4)
- net ISA_IRQ5: now also RN5.5 (R4), U32.8; no longer RN5.4 (R3)
- net ISA_IRQ6: now also RN5.4 (R3), U32.2; no longer RN5.3 (R2)
- net ISA_IRQ7: now also RN5.3 (R2), U32.1; no longer RN5.2 (R1)
- net ISA_RST: now also U34.10
- net ~{ISA_0WS}: now also RN7.3 (R2)
- net ~{ISA_DACK0}: now also RN7.5 (R4)
- net ~{ISA_IOR}: now also U22.9 (O3); no longer U22.9 (O3)
- net ~{ISA_IOW}: now also U22.10 (O2); no longer U22.10 (O2)
- net ~{ISA_IO_CH_CK}: now also RN7.2 (R1), U34.3
- net ~{ISA_MEMR}: now also U22.11 (O1); no longer U22.11 (O1)
- net ~{ISA_MEMW}: now also U22.12 (O0); no longer U22.12 (O0)
- net ~{ISA_SEL}: now also U22.15 (E), U34.13; no longer U22.15 (E)
- net ~{RST}: now also U34.11
- net ~{WAIT}: now also RN7.4 (R3)
- net ~{WE}: now also U22.14 (A0); no longer U22.14 (A0)
- new net: U32.11, U32.9
- new net: U32.10, U34.1
- new net: U32.13, U32.6
- new net CPU_~{DACK}: U34.9
- new net ISA_IO_CH_CK: U32.12, U34.4
Other:
- moved on the sheet: RN5

Commit message: Worked in wait-states for I/O, changed I/O address decode, added GPI pull-downs.
Parts:
- removed RN5: 10k, Resistor_THT:R_Array_SIP9, symbol Device:R_Network08_US
Changed lines of the file:
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@@
     (title "Anachron ISA bus interface")
   )
-  (junction (at 210.82 189.23) (diameter 0) (color 0 0 0 0)
-  )
   (junction (at 201.93 121.92) (diameter 0) (color 0 0 0 0)
   )
@@
   (junction (at 226.06 107.95) (diameter 0) (color 0 0 0 0)
   )
-  (junction (at 213.36 203.2) (diameter 0) (color 0 0 0 0)
-  )
   (junction (at 52.07 259.08) (diameter 0) (color 0 0 0 0)
   )
@@
   (junction (at 298.45 121.92) (diameter 0) (color 0 0 0 0)
   )
-  (junction (at 215.9 205.74) (diameter 0) (color 0 0 0 0)
-  )
   (junction (at 389.89 127) (diameter 0) (color 0 0 0 0)
   )
@@
   (junction (at 212.09 151.13) (diameter 0) (color 0 0 0 0)
   )
-  (junction (at 208.28 186.69) (diameter 0) (color 0 0 0 0)
-  )
   (junction (at 186.69 151.13) (diameter 0) (color 0 0 0 0)
   )
-  (junction (at 203.2 208.28) (diameter 0) (color 0 0 0 0)
-  )
   (junction (at 419.1 107.95) (diameter 0) (color 0 0 0 0)
   )
@@
   (junction (at 320.04 36.83) (diameter 0) (color 0 0 0 0)
   )
-  (junction (at 205.74 184.15) (diameter 0) (color 0 0 0 0)
-  )
   (junction (at 226.06 54.61) (diameter 0) (color 0 0 0 0)
   )
@@
     (stroke (width 0) (type default))
   )
-  (wire (pts (xy 208.28 186.69) (xy 208.28 213.36))
-    (stroke (width 0) (type default))
-  )
   (wire (pts (xy 226.06 54.61) (xy 226.06 107.95))
     (stroke (width 0) (type default))
   )
-  (wire (pts (xy 203.2 189.23) (xy 210.82 189.23))
+  (wire (pts (xy 203.2 189.23) (xy 261.62 189.23))
     (stroke (width 0) (type default))
   )
@@
     (stroke (width 0) (type default))
   )
-  (wire (pts (xy 203.2 184.15) (xy 205.74 184.15))
+  (wire (pts (xy 203.2 184.15) (xy 261.62 184.15))
     (stroke (width 0) (type default))
   )
@@
     (stroke (width 0) (type default))
   )
-  (wire (pts (xy 213.36 203.2) (xy 213.36 213.36))
-    (stroke (width 0) (type default))
-  )
   (wire (pts (xy 457.2 64.77) (xy 488.95 64.77))
     (stroke (width 0) (type default))
@@
     (stroke (width 0) (type default))
   )
-  (wire (pts (xy 215.9 205.74) (xy 261.62 205.74))
+  (wire (pts (xy 203.2 205.74) (xy 261.62 205.74))
     (stroke (width 0) (type default))
   )
@@
     (stroke (width 0) (type default))
   )
-  (wire (pts (xy 203.2 205.74) (xy 215.9 205.74))
-    (stroke (width 0) (type default))
-  )
   (wire (pts (xy 29.21 325.12) (xy 57.15 325.12))
     (stroke (width 0) (type default))
@@
     (stroke (width 0) (type default))
   )
-  (wire (pts (xy 208.28 186.69) (xy 261.62 186.69))
+  (wire (pts (xy 203.2 186.69) (xy 261.62 186.69))
     (stroke (width 0) (type default))
   )
@@
     (stroke (width 0) (type default))
   )
-  (wire (pts (xy 205.74 184.15) (xy 261.62 184.15))
-    (stroke (width 0) (type default))
-  )
   (wire (pts (xy 209.55 72.39) (xy 228.6 72.39))
     (stroke (width 0) (type default))
@@
     (stroke (width 0) (type default))
   )
-  (wire (pts (xy 210.82 189.23) (xy 210.82 213.36))
-    (stroke (width 0) (type default))
-  )
   (wire (pts (xy 306.07 44.45) (xy 325.12 44.45))
     (stroke (width 0) (type default))
@@
     (stroke (width 0) (type default))
   )
-  (wire (pts (xy 205.74 184.15) (xy 205.74 213.36))
-    (stroke (width 0) (type default))
-  )
   (wire (pts (xy 264.16 64.77) (xy 295.91 64.77))
     (stroke (width 0) (type default))
@@
     (stroke (width 0) (type default))
   )
-  (wire (pts (xy 203.2 186.69) (xy 208.28 186.69))
-    (stroke (width 0) (type default))
-  )
   (bus (pts (xy 293.37 46.99) (xy 293.37 49.53))
     (stroke (width 0) (type default))
@@
     (stroke (width 0) (type default))
   )
-  (wire (pts (xy 215.9 205.74) (xy 215.9 213.36))
-    (stroke (width 0) (type default))
-  )
   (wire (pts (xy 457.2 74.93) (xy 488.95 74.93))
     (stroke (width 0) (type default))
@@
     (stroke (width 0) (type default))
   )
-  (wire (pts (xy 210.82 189.23) (xy 261.62 189.23))
-    (stroke (width 0) (type default))
-  )
   (wire (pts (xy 360.68 62.23) (xy 392.43 62.23))
     (stroke (width 0) (type default))
@@
     (stroke (width 0) (type default))
   )
-  (wire (pts (xy 213.36 203.2) (xy 261.62 203.2))
-    (stroke (width 0) (type default))
-  )
   (bus (pts (xy 298.45 80.01) (xy 298.45 82.55))
     (stroke (width 0) (type default))
@@
     (stroke (width 0) (type default))
   )
-  (wire (pts (xy 203.2 213.36) (xy 203.2 208.28))
-    (stroke (width 0) (type default))
-  )
   (bus (pts (xy 201.93 64.77) (xy 201.93 67.31))
     (stroke (width 0) (type default))
@@
     (stroke (width 0) (type default))
   )
-  (wire (pts (xy 203.2 203.2) (xy 213.36 203.2))
+  (wire (pts (xy 203.2 203.2) (xy 261.62 203.2))
     (stroke (width 0) (type default))
   )
@@
     )
   )
-  (symbol (lib_id "power:GND") (at 203.2 223.52 0) (unit 1)
-    (in_bom yes) (on_board yes) (dnp no) (fields_autoplaced)
-    (property "Reference" "#PWR0149" (at 203.2 229.87 0)
-      (effects (font (size 1.27 1.27)) hide)
-    )
-    (property "Value" "GND" (at 203.2 228.6 0)
-      (effects (font (size 1.27 1.27)))
-    )
-    (property "Footprint" "" (at 203.2 223.52 0)
-      (effects (font (size 1.27 1.27)) hide)
-    )
-    (property "Datasheet" "" (at 203.2 223.52 0)
-      (effects (font (size 1.27 1.27)) hide)
-    )
-    (pin "1")
-    (instances
-      (project "a1_mini"
-        (path "/3257e1ae-50a8-410a-87c3-a39d96a2c51a/0c1f7d0b-482f-4d97-925a-18a42e0624c3"
-          (reference "#PWR0149") (unit 1)
-        )
-      )
-    )
-  )
   (symbol (lib_id "power:GND") (at 212.09 158.75 0) (unit 1)
     (in_bom yes) (on_board yes) (dnp no) (fields_autoplaced)
@@
         )
       )
-    )
-  )
-  (symbol (lib_id "Device:R_Network08_US") (at 213.36 218.44 0) (mirror x) (unit 1)
-    (in_bom yes) (on_board yes) (dnp no) (fields_autoplaced)
-    (property "Reference" "RN5" (at 200.66 216.916 0)
-      (effects (font (size 1.27 1.27)) (justify right))
-    )
-    (property "Value" "10k" (at 200.66 219.456 0)
-      (effects (font (size 1.27 1.27)) (justify right))
-    )
-    (property "Footprint" "Resistor_THT:R_Array_SIP9" (at 225.425 218.44 90)
-      (effects (font (size 1.27 1.27)) hide)
-    )
-    (property "Datasheet" "http://www.vishay.com/docs/31509/csc.pdf" (at 213.36 218.44 0)
-      (effects (font (size 1.27 1.27)) hide)
-    )
-    (pin "8")
-    (pin "9")
-    (pin "5")
-    (pin "7")
-    (pin "2")
-    (pin "1")
-    (pin "3")
-    (pin "4")
-    (pin "6")
-    (instances
-      (project "a1_mini"
-        (path "/3257e1ae-50a8-410a-87c3-a39d96a2c51a/0c1f7d0b-482f-4d97-925a-18a42e0624c3"
-          (reference "RN5") (unit 1)
-        )
-      )

Commit message: A1 Mini (which is not all that mini anymore) is feature-complete.
We have 2 ISA slots and even all the power supplies generated from +5V included.

The +12V switcher right next to the audio output is quite a bit concerning, but
we can always say that PWR must be 12V and we directly feed that to the ISA slots.
(Not that PWR is all that clean...) A lot will depend on how I implement grounding,
something that I still have to do.
Parts:
- removed J14, J15: Bus_ISA_8bit, anachron:BUS_XT_CONN, symbol Connector:Bus_ISA_8bit
- added C58, C59: 220uF, Capacitor_THT:CP_Radial_D7.5mm_P2.50mm, symbol Device:C_Polarized_Small_US
- added C60: 302pF, Capacitor_THT:C_Disc_D4.7mm_W2.5mm_P5.00mm, symbol Device:C
- added C61: 260p, Capacitor_THT:C_Disc_D4.7mm_W2.5mm_P5.00mm, symbol Device:C
- added C62: 1000uF, Capacitor_THT:CP_Radial_D10.0mm_P5.00mm, symbol Device:C_Polarized_Small_US
- added C63: 1500uF, Capacitor_THT:CP_Radial_D10.0mm_P5.00mm, symbol Device:C_Polarized_Small_US
- added D4, D5: 1N5817, Diode_THT:D_DO-41_SOD81_P10.16mm_Horizontal, symbol Diode:1N5817
- added L1: 25uH, Inductor_THT:L_Radial_D8.7mm_P5.00mm_Fastron_07HCP, symbol Device:L
- added L2: 18uH, Inductor_THT:L_Radial_D8.7mm_P5.00mm_Fastron_07HCP, symbol Device:L
- added R29: 0.244Ohm, Resistor_THT:R_Axial_DIN0204_L3.6mm_D1.6mm_P5.08mm_Horizontal, symbol Device:R_US
- added R30: 0.211Ohm, Resistor_THT:R_Axial_DIN0204_L3.6mm_D1.6mm_P5.08mm_Horizontal, symbol Device:R_US
- added R31: 180, Resistor_THT:R_Axial_DIN0204_L3.6mm_D1.6mm_P5.08mm_Horizontal, symbol Device:R_US
- added R32, R35: 1.5k, Resistor_THT:R_Axial_DIN0204_L3.6mm_D1.6mm_P5.08mm_Horizontal, symbol Device:R_US
- added R33, R34: 13k, Resistor_THT:R_Axial_DIN0204_L3.6mm_D1.6mm_P5.08mm_Horizontal, symbol Device:R_US
- added U34, U35: MC33063AP, Package_DIP:DIP-8_W7.62mm, symbol Regulator_Switching:MC33063AP
- renumbered C24 to C54, C51 to C55, C64 to C56, C65 to C57, C37 to C64, C56 to C65, J16 to J18, RN7 to RN10, U34 to U31, U22 to U32, U32 to U33, U23 to U36
Connections:
- net +12V: now also C63.1, D5.1 (K), R34.1
- net +5V: now also C58.1, C59.1, R29.1, R30.1, U34.6 (Vin), U35.6 (Vin)
- net -12V: now also C60.2, C62.2, D4.2 (A), R32.1, U34.4 (GND)
- net GND: now also C58.2, C59.2, C61.2, C62.1, C63.2, L1.2, R33.2, R35.2, U35.2 (SwE), U35.4 (GND)
- net ISA_IRQ2: now also U33.4; no longer U33.5
- net ISA_IRQ3: now also U33.5; no longer U33.4
- net ISA_IRQ5: now also U33.2; no longer U33.8
- net ISA_IRQ6: now also U33.1; no longer U33.2
- net ISA_IRQ7: now also U33.8; no longer U33.1
- net ~{ISA_0WS}: now also RN10.4 (R3); no longer RN10.3 (R2)
- net ~{ISA_DACK0}: now also RN10.3 (R2); no longer RN10.5 (R4)
- net ~{WAIT}: now also RN10.5 (R4); no longer RN10.4 (R3)
- new net: R31.1, U35.8 (DC)
- new net: L2.1, R30.2, R31.2, U35.7 (Ipk)
- new net: C61.1, U35.3 (TC)
- new net: R29.2, U34.1 (SwC), U34.7 (Ipk), U34.8 (DC)
- new net: R32.2, R33.1, U34.5 (Vfb)
- new net: R34.2, R35.1, U35.5 (Vfb)
- new net: D4.1 (K), L1.1, U34.2 (SwE)
- new net: C60.1, U34.3 (TC)
- new net: D5.2 (A), L2.2, U35.1 (SwC)
Other:
- note added: "Designed using http://www.nomad.ee/micros/mc34063a/index.shtml"
- moved on the sheet: C64, C65, J18, J19, U36

Commit message: A1 MINI is fully routed.
That is, if I add a GND fill on both layers. Which I don't, because auto-refill takes
several seconds and so it's a PITA to work with. There are a few dozen DRC errors
as well but nothing major it seems.

Worked out roughly 100ohm diff impedance for the HDMI lines
(not GND-referenced) which I think is my best shot of making it work.

long USB trace has a nice GND shield under-it, so does audio.
Again, probably my best shot at making these work.

Ethernet still needs checking just as short-put USB connections from the hub to
the connector.
Parts:
- added JP5: Jumper_2_Bridged, Connector_PinHeader_2.54mm:PinHeader_1x02_P2.54mm_Vertical, symbol Jumper:Jumper_2_Bridged
- added JP6: Jumper_2_Open, Connector_PinHeader_2.54mm:PinHeader_1x02_P2.54mm_Vertical, symbol Jumper:Jumper_2_Open
Connections:
- net +12V: now also JP6.2 (B)
- net +5V: now also JP5.2 (B); no longer C59.1, R30.1, U35.6 (Vin)
- new net: C59.1, JP5.1 (A), R30.1, U35.6 (Vin)
- new net PWR_IN: JP6.1 (A)
Other:
- note added: "Other supply options (dual channel): TPS6513x - this seems to fit the bill BD8316GWL - this can't generate -12, only about -9. R1283x - this seems to fit the bill MAX864 - switched capacitor +/-10V @ 100mA D81870EFV - seems to fit the bill ADP5071 - seems to fit the bill max743 - low current, expensive, but, in DIP PACKAGE!!!"
- note added: "The original PC provided several amps on +12V. We obviously can't match that, but we don't expect much load on the +12V rail either."
- note added: "The original PC supplied 0.3A on the -5V and 0.25 on the -12V rails. It had 5 expansion slots. We provide about half of that current for about half of the slots. However it is anticipated that -5V is not used at all and -12 is used by RS232 transceivers only."
Changed lines of the file:
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@@
   (junction (at 459.74 344.17) (diameter 0) (color 0 0 0 0)
   )
+  (junction (at 487.68 322.58) (diameter 0) (color 0 0 0 0)
+  )
   (junction (at 386.08 336.55) (diameter 0) (color 0 0 0 0)
   )
@@
     (stroke (width 0) (type default))
   )
-  (wire (pts (xy 375.92 320.04) (xy 375.92 336.55))
+  (wire (pts (xy 375.92 320.04) (xy 375.92 323.85))
     (stroke (width 0) (type default))
   )
@@
     (stroke (width 0) (type default))
   )
-  (wire (pts (xy 471.17 322.58) (xy 494.03 322.58))
+  (wire (pts (xy 471.17 322.58) (xy 487.68 322.58))
     (stroke (width 0) (type default))
   )
@@
     (stroke (width 0) (type default))
   )
+  (wire (pts (xy 471.17 316.23) (xy 477.52 316.23))
+    (stroke (width 0) (type default))
+  )
   (wire (pts (xy 426.72 339.09) (xy 424.18 339.09))
     (stroke (width 0) (type default))
@@
     (stroke (width 0) (type default))
   )
+  (wire (pts (xy 487.68 316.23) (xy 487.68 322.58))
+    (stroke (width 0) (type default))
+  )
   (wire (pts (xy 397.51 250.19) (xy 387.35 250.19))
     (stroke (width 0) (type default))
@@
     (stroke (width 0) (type default))
   )
+  (wire (pts (xy 487.68 322.58) (xy 494.03 322.58))
+    (stroke (width 0) (type default))
+  )
   (wire (pts (xy 138.43 44.45) (xy 157.48 44.45))
     (stroke (width 0) (type default))
@@
   )
   (wire (pts (xy 386.08 360.68) (xy 402.59 360.68))
+    (stroke (width 0) (type default))
+  )
+  (wire (pts (xy 375.92 334.01) (xy 375.92 336.55))
     (stroke (width 0) (type default))
   )
@@
   (text "Optional oscillator in case\nthere's a bunch of problems\nwith feeding just SYS_CLK\nto this ISA pin."
     (at 93.98 298.45 0)
+    (effects (font (size 1.27 1.27)) (justify left bottom))
+  )
+  (text "Other supply options (dual channel):\nTPS6513x - this seems to fit the bill\nBD8316GWL - this can't generate -12, only about -9.\nR1283x - this seems to fit the bill\nMAX864 - switched capacitor +/-10V @ 100mA\nD81870EFV - seems to fit the bill\nADP5071 - seems to fit the bill\nmax743 - low current, expensive, but, in DIP PACKAGE!!!"
+    (at 346.71 312.42 0)
+    (effects (font (size 1.27 1.27)) (justify left bottom))
+  )
+  (text "The original PC provided several amps on +12V. We obviously can't\nmatch that, but we don't expect much load on the +12V rail either.\n"
+    (at 436.88 308.61 0)
+    (effects (font (size 1.27 1.27)) (justify left bottom))
+  )
+  (text "The original PC supplied 0.3A on the -5V and 0.25 on the -12V rails.\nIt had 5 expansion slots. We provide about half of that current\nfor about half of the slots. However it is anticipated that\n-5V is not used at all and -12 is used by RS232 transceivers only."
+    (at 421.64 246.38 0)
     (effects (font (size 1.27 1.27)) (justify left bottom))
   )
@@
     (effects (font (size 1.27 1.27)) (justify right))
     (property "Intersheetrefs" "${INTERSHEET_REFS}" (at 27.8577 229.87 0)
+      (effects (font (size 1.27 1.27)) (justify right) hide)
+    )
+  )
+  (global_label "PWR_IN" (shape input) (at 471.17 316.23 180) (fields_autoplaced)
+    (effects (font (size 1.27 1.27)) (justify right))
+    (property "Intersheetrefs" "${INTERSHEET_REFS}" (at 461.2905 316.23 0)
       (effects (font (size 1.27 1.27)) (justify right) hide)
     )
@@
     )
   )
+  (symbol (lib_id "Jumper:Jumper_2_Bridged") (at 375.92 328.93 90) (unit 1)
+    (in_bom yes) (on_board yes) (dnp no) (fields_autoplaced)
+    (property "Reference" "JP5" (at 377.19 327.66 90)
+      (effects (font (size 1.27 1.27)) (justify right))
+    )
+    (property "Value" "Jumper_2_Bridged" (at 377.19 330.2 90)
+      (effects (font (size 1.27 1.27)) (justify right))
+    )
+    (property "Footprint" "Connector_PinHeader_2.54mm:PinHeader_1x02_P2.54mm_Vertical" (at 375.92 328.93 0)
+      (effects (font (size 1.27 1.27)) hide)
+    )
+    (property "Datasheet" "~" (at 375.92 328.93 0)
+      (effects (font (size 1.27 1.27)) hide)
+    )
+    (pin "2")
+    (pin "1")
+    (instances
+      (project "a1_mini"
+        (path "/3257e1ae-50a8-410a-87c3-a39d96a2c51a/0c1f7d0b-482f-4d97-925a-18a42e0624c3"
+          (reference "JP5") (unit 1)
+        )
+      )
+    )
+  )
   (symbol (lib_id "74xx:74LS14") (at 68.58 273.05 0) (unit 6)
     (in_bom yes) (on_board yes) (dnp no) (fields_autoplaced)
@@
         )
       )
+    )
+  )
+  (symbol (lib_id "Jumper:Jumper_2_Open") (at 482.6 316.23 0) (unit 1)
+    (in_bom yes) (on_board yes) (dnp no) (fields_autoplaced)
+    (property "Reference" "JP6" (at 482.6 309.88 0)
+      (effects (font (size 1.27 1.27)))
+    )
+    (property "Value" "Jumper_2_Open" (at 482.6 312.42 0)
+      (effects (font (size 1.27 1.27)))
+    )
+    (property "Footprint" "Connector_PinHeader_2.54mm:PinHeader_1x02_P2.54mm_Vertical" (at 482.6 316.23 0)
+      (effects (font (size 1.27 1.27)) hide)
+    )
+    (property "Datasheet" "~" (at 482.6 316.23 0)
+      (effects (font (size 1.27 1.27)) hide)
+    )
+    (pin "2")
+    (pin "1")
+    (instances
+      (project "a1_mini"
+        (path "/3257e1ae-50a8-410a-87c3-a39d96a2c51a/0c1f7d0b-482f-4d97-925a-18a42e0624c3"
+          (reference "JP6") (unit 1)
+        )
+      )

Commit message: Checking in stuff before the 3.3V work.
Other:
- note added: "TODO: should we add a couple of 16-bit slots, where the appropriate signals are tied down to ensure that 16-bit cards don't accidentally assume 16-bit transactions just because of floating control pins?"
Changed lines of the file:
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@@
+    (effects (font (size 1.27 1.27)) (justify left bottom))
+  )
+  (text "TODO: should we add a couple of 16-bit slots, where the appropriate\nsignals are tied down to ensure that 16-bit cards don't accidentally\nassume 16-bit transactions just because of floating control pins?"
+    (at 355.6 87.63 0)
     (effects (font (size 1.27 1.27)) (justify left bottom))
   )

Commit message: 3.3V work, before abandoning the idea.
Parts:
- U31: value 74LS14 -> SN74AHC14N
- U32: value 74LS139 -> SN74AHC139N
- U33: value 4075 -> CD74HC4075E
Connections:
- net +5V: no longer C54.1, C55.1, C57.1, RN10.1 (common), U31.14 (VCC), U32.16 (VCC), X4.1 (EN), X4.14 (Vcc)
- new net +3.3V: C54.1, C55.1, C57.1, RN10.1 (common), U31.14 (VCC), U32.16 (VCC), X4.1 (EN), X4.14 (Vcc)
Other:
- note added: "There's no good 5V tolerant, 3.3V supply variant available. It however drives a 5V tolerant gate so it's output will not be delievered to 3.3V domain."
- moved on the sheet: C56, U31C
