File: boards/a1_mini/memory.kicad_sch (KiCad schematic)
At the start: 6 parts, among them U20 SIMM-30, U21 SIMM-30

Commit message: A1 Mini (which is not all that mini anymore) is feature-complete.
We have 2 ISA slots and even all the power supplies generated from +5V included.

The +12V switcher right next to the audio output is quite a bit concerning, but
we can always say that PWR must be 12V and we directly feed that to the ISA slots.
(Not that PWR is all that clean...) A lot will depend on how I implement grounding,
something that I still have to do.
Parts:
- removed C47: 1uF, Capacitor_THT:C_Disc_D4.7mm_W2.5mm_P5.00mm, symbol Device:C
- renumbered C48 to C21, C49 to C22, C50 to C23

Commit message: A1-MINI is fully routed. Also fully impedance controlled.
Parts:
- removed U20, U21: SIMM-30, anachron:SIMM-30, symbol anachron:SIMM-30
- added U21: SIMM-30x2, anachron:SIMM-30x2_VERT, symbol anachron:SIMM-30x2
Connections:
- net +5V: now also U21.A1 (VCC), U21.A24 (A11), U21.A28 (~{CASP}), U21.A30 (VCC), U21.B1 (VCC), U21.B24 (A11), U21.B28 (~{CASP}), U21.B30 (VCC)
- net A0: now also U21.A4 (A0), U21.B4 (A0)
- net A1: now also U21.A5 (A1), U21.B5 (A1)
- net A10: now also U21.A19 (A10), U21.B19 (A10)
- net A2: now also U21.A7 (A2), U21.B7 (A2)
- net A3: now also U21.A8 (A3), U21.B8 (A3)
- net A4: now also U21.A11 (A4), U21.B11 (A4)
- net A5: now also U21.A12 (A5), U21.B12 (A5)
- net A6: now also U21.A14 (A6), U21.B14 (A6)
- net A7: now also U21.A15 (A7), U21.B15 (A7)
- net A8: now also U21.A17 (A8), U21.B17 (A8)
- net A9: now also U21.A18 (A9), U21.B18 (A9)
- net D0: now also U21.A3 (DQ0), U21.B3 (DQ0)
- net D1: now also U21.A6 (DQ1), U21.B6 (DQ1)
- net D2: now also U21.A10 (DQ2), U21.B10 (DQ2)
- net D3: now also U21.A13 (DQ3), U21.B13 (DQ3)
- net D4: now also U21.A16 (DQ4), U21.B16 (DQ4)
- net D5: now also U21.A20 (DQ5), U21.B20 (DQ5)
- net D6: now also U21.A23 (DQ6), U21.B23 (DQ6)
- net D7: now also U21.A25 (DQ7), U21.B25 (DQ7)
- net GND: now also U21.A22 (GND), U21.A29 (DP), U21.A9 (GND), U21.B22 (GND), U21.B29 (DP), U21.B9 (GND)
- net ~{CAS_0}: now also U21.B2 (~{CAS})
- net ~{CAS_1}: now also U21.A2 (~{CAS})
- net ~{RAS}: now also U21.A27 (~{RAS}), U21.B27 (~{RAS})
- net ~{WE}: now also U21.A21 (~{WE}), U21.B21 (~{WE})
Other:
- note added: "Part numbers for sockets: Molex 15-46-0330 (dual) Berg 87731-102 (dual) Autotek SMV2030-6 (dual) ???? HWS9594 (dual) ???? HWS5040 (single) ???? HWS4323 (single, plastic) AdamTech SIMM-130-VTL (single) AMP 821876-2 (single) AMP 821885-2 (dual)"

Commit message: 3.3V work, before abandoning the idea.
Connections:
- net +5V: no longer U21.A24 (A11), U21.A28 (~{CASP}), U21.B24 (A11), U21.B28 (~{CASP})
- new net +3.3V: U21.A24 (A11), U21.A28 (~{CASP}), U21.B24 (A11), U21.B28 (~{CASP})
Changed lines of the file:
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@@
+    )
+  )
+  (symbol (lib_id "power:+3.3V") (at 137.16 101.6 0) (unit 1)
+    (in_bom yes) (on_board yes) (dnp no) (fields_autoplaced)
+    (property "Reference" "#PWR0112" (at 137.16 105.41 0)
+      (effects (font (size 1.27 1.27)) hide)
+    )
+    (property "Value" "+3.3V" (at 137.16 96.52 0)
+      (effects (font (size 1.27 1.27)))
+    )
+    (property "Footprint" "" (at 137.16 101.6 0)
+      (effects (font (size 1.27 1.27)) hide)
+    )
+    (property "Datasheet" "" (at 137.16 101.6 0)
+      (effects (font (size 1.27 1.27)) hide)
+    )
+    (pin "1")
+    (instances
+      (project "a1_mini"
+        (path "/3257e1ae-50a8-410a-87c3-a39d96a2c51a/74914ce5-2001-49ca-8f09-c71b1f2944ab"
+          (reference "#PWR0112") (unit 1)
+        )
+        (path "/3257e1ae-50a8-410a-87c3-a39d96a2c51a/58d11f1c-6aae-4928-b318-2d07bb2e6df5"
+          (reference "#PWR0201") (unit 1)
+        )
+      )
     )
   )
@@
     )
   )
-  (symbol (lib_id "power:+5V") (at 187.96 27.94 0) (unit 1)
+  (symbol (lib_id "power:GND") (at 193.04 158.75 0) (unit 1)
+    (in_bom yes) (on_board yes) (dnp no) (fields_autoplaced)
+    (property "Reference" "#PWR0118" (at 193.04 165.1 0)
+      (effects (font (size 1.27 1.27)) hide)
+    )
+    (property "Value" "GND" (at 193.04 163.83 0)
+      (effects (font (size 1.27 1.27)))
+    )
+    (property "Footprint" "" (at 193.04 158.75 0)
+      (effects (font (size 1.27 1.27)) hide)
+    )
+    (property "Datasheet" "" (at 193.04 158.75 0)
+      (effects (font (size 1.27 1.27)) hide)
+    )
+    (pin "1")
+    (instances
+      (project "a1_mini"
+        (path "/3257e1ae-50a8-410a-87c3-a39d96a2c51a/74914ce5-2001-49ca-8f09-c71b1f2944ab"
+          (reference "#PWR0118") (unit 1)
+        )
+        (path "/3257e1ae-50a8-410a-87c3-a39d96a2c51a/58d11f1c-6aae-4928-b318-2d07bb2e6df5"
+          (reference "#PWR0208") (unit 1)
+        )
+      )
+    )
+  )
+  (symbol (lib_id "power:+3.3V") (at 187.96 27.94 0) (unit 1)
     (in_bom yes) (on_board yes) (dnp no) (fields_autoplaced)
     (property "Reference" "#PWR0117" (at 187.96 31.75 0)
       (effects (font (size 1.27 1.27)) hide)
     )
-    (property "Value" "+5V" (at 187.96 22.86 0)
+    (property "Value" "+3.3V" (at 187.96 22.86 0)
       (effects (font (size 1.27 1.27)))
     )
@@
         )
         (path "/3257e1ae-50a8-410a-87c3-a39d96a2c51a/58d11f1c-6aae-4928-b318-2d07bb2e6df5"
-          (reference "#PWR0207") (unit 1)
-        )
-      )
-    )
-  )
-  (symbol (lib_id "power:GND") (at 193.04 158.75 0) (unit 1)
-    (in_bom yes) (on_board yes) (dnp no) (fields_autoplaced)
-    (property "Reference" "#PWR0118" (at 193.04 165.1 0)
-      (effects (font (size 1.27 1.27)) hide)
-    )
-    (property "Value" "GND" (at 193.04 163.83 0)
-      (effects (font (size 1.27 1.27)))
-    )
-    (property "Footprint" "" (at 193.04 158.75 0)
-      (effects (font (size 1.27 1.27)) hide)
-    )
-    (property "Datasheet" "" (at 193.04 158.75 0)
-      (effects (font (size 1.27 1.27)) hide)
-    )
-    (pin "1")
-    (instances
-      (project "a1_mini"
-        (path "/3257e1ae-50a8-410a-87c3-a39d96a2c51a/74914ce5-2001-49ca-8f09-c71b1f2944ab"
-          (reference "#PWR0118") (unit 1)
-        )
-        (path "/3257e1ae-50a8-410a-87c3-a39d96a2c51a/58d11f1c-6aae-4928-b318-2d07bb2e6df5"
-          (reference "#PWR0208") (unit 1)
+          (reference "#PWR0120") (unit 1)
         )
       )
@@
         (path "/3257e1ae-50a8-410a-87c3-a39d96a2c51a/58d11f1c-6aae-4928-b318-2d07bb2e6df5"
           (reference "C52") (unit 1)
+        )
+      )
+    )
+  )
+  (symbol (lib_id "power:+3.3V") (at 137.16 27.94 0) (unit 1)
+    (in_bom yes) (on_board yes) (dnp no) (fields_autoplaced)
+    (property "Reference" "#PWR0106" (at 137.16 31.75 0)
+      (effects (font (size 1.27 1.27)) hide)
+    )
+    (property "Value" "+3.3V" (at 137.16 22.86 0)
+      (effects (font (size 1.27 1.27)))
+    )
+    (property "Footprint" "" (at 137.16 27.94 0)
+      (effects (font (size 1.27 1.27)) hide)
+    )
+    (property "Datasheet" "" (at 137.16 27.94 0)
+      (effects (font (size 1.27 1.27)) hide)
+    )
+    (pin "1")
+    (instances
+      (project "a1_mini"
+        (path "/3257e1ae-50a8-410a-87c3-a39d96a2c51a/74914ce5-2001-49ca-8f09-c71b1f2944ab"
+          (reference "#PWR0106") (unit 1)
+        )
+        (path "/3257e1ae-50a8-410a-87c3-a39d96a2c51a/58d11f1c-6aae-4928-b318-2d07bb2e6df5"
+          (reference "#PWR0111") (unit 1)
         )
       )
@@
         )
       )
-    )
-  )
-  (symbol (lib_id "power:+5V") (at 137.16 27.94 0) (unit 1)
-    (in_bom yes) (on_board yes) (dnp no) (fields_autoplaced)
-    (property "Reference" "#PWR0111" (at 137.16 31.75 0)
-      (effects (font (size 1.27 1.27)) hide)
-    )
-    (property "Value" "+5V" (at 137.16 22.86 0)
-      (effects (font (size 1.27 1.27)))
-    )
-    (property "Footprint" "" (at 137.16 27.94 0)
-      (effects (font (size 1.27 1.27)) hide)
-    )
-    (property "Datasheet" "" (at 137.16 27.94 0)
-      (effects (font (size 1.27 1.27)) hide)
-    )
-    (pin "1")
-    (instances
-      (project "a1_mini"
-        (path "/3257e1ae-50a8-410a-87c3-a39d96a2c51a/74914ce5-2001-49ca-8f09-c71b1f2944ab"
-          (reference "#PWR0111") (unit 1)
-        )
-        (path "/3257e1ae-50a8-410a-87c3-a39d96a2c51a/58d11f1c-6aae-4928-b318-2d07bb2e6df5"
-          (reference "#PWR0201") (unit 1)
-        )
-      )
-    )
-  )
-  (symbol (lib_id "power:+5V") (at 137.16 101.6 0) (unit 1)
-    (in_bom yes) (on_board yes) (dnp no) (fields_autoplaced)
-    (property "Reference" "#PWR0112" (at 137.16 105.41 0)
-      (effects (font (size 1.27 1.27)) hide)
-    )
-    (property "Value" "+5V" (at 137.16 96.52 0)
-      (effects (font (size 1.27 1.27)))
-    )
-    (property "Footprint" "" (at 137.16 101.6 0)
-      (effects (font (size 1.27 1.27)) hide)
-    )
-    (property "Datasheet" "" (at 137.16 101.6 0)
-      (effects (font (size 1.27 1.27)) hide)
-    )
-    (pin "1")
-    (instances
-      (project "a1_mini"
-        (path "/3257e1ae-50a8-410a-87c3-a39d96a2c51a/74914ce5-2001-49ca-8f09-c71b1f2944ab"
-          (reference "#PWR0112") (unit 1)
-        )
-        (path "/3257e1ae-50a8-410a-87c3-a39d96a2c51a/58d11f1c-6aae-4928-b318-2d07bb2e6df5"
-          (reference "#PWR0202") (unit 1)
-        )
-      )
