File: boards/a1_mini/mio.kicad_sch (KiCad schematic)
At the start: 58 parts, among them J10 DE9_Plug, J11 USB_A_Stacked, J4 USB_A_Stacked, J7 Micro_SD_Card, J8 USB_A, J9 USB_A_Stacked, U26 MIO, U28 MAX232, U29 DS1307+, U7 A1_USBHUB, X2 24MHz, Y1 32768Hz

Commit message: USB HUB is back in.
Parts:
- removed C10, C18, C19, C20, C21, C22, C23: 100uF, Capacitor_THT:CP_Radial_D5.0mm_P2.00mm, symbol Device:C_Polarized_Small_US
- removed CMC10, CMC11, CMC5, CMC6, CMC7, CMC8, CMC9: L_Ferrite_Coupled_Small, anachron:SCM2012FS, symbol Device:L_Ferrite_Coupled_Small_1243
- removed F2: 0.5A, Fuse:Fuse_BelFuse_0ZRE0005FF_L8.3mm_W3.8mm, symbol Device:Polyfuse
- removed FB2, FB21, FB3, FB4, FB5, FB6, FB7: FerriteBead_Small, Inductor_THT:L_Axial_L7.0mm_D3.3mm_P2.54mm_Vertical_Fastron_MICC, symbol Device:FerriteBead_Small
- removed J11, J4, J9: USB_A_Stacked, anachron:GCT_USB1035-XX-X-X-X-B_REVE, symbol Connector:USB_A_Stacked
- removed J8: USB_A, Connector_USB:USB_A_Molex_67643_Horizontal, symbol Connector:USB_A
- removed JP2: Jumper_2_Open, Connector_PinHeader_2.54mm:PinHeader_1x02_P2.54mm_Vertical, symbol Jumper:Jumper_2_Open
- removed U7: A1_USBHUB, anachron:DIP-40_W15.24mm_Socket, symbol anachron:A1_USBHUB
Connections:
- net at U29.1 (X1): now also Y1.2; no longer Y1.1
- net at U29.2 (X2): now also Y1.1; no longer Y1.2
- net USB_D+ renamed USB_US_D+
- net USB_D- renamed USB_US_D-
- no-connect marks 1 -> 0

Commit message: Added boot mode switch, reworked LAN IRQ, places LEDs better.
Parts:
- removed D3: LED, LED_THT:LED_D5.0mm, symbol Device:LED
- removed R13: 470, Resistor_THT:R_Axial_DIN0204_L3.6mm_D1.6mm_P5.08mm_Horizontal, symbol Device:R_US
Connections:
- net LAN_~{INT}: now reaches U26.4 (PC3_USBb_D-)
Changed lines of the file:
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@@
     (stroke (width 0) (type default))
   )
-  (wire (pts (xy 109.22 86.36) (xy 113.03 86.36))
+  (wire (pts (xy 109.22 86.36) (xy 124.46 86.36))
     (stroke (width 0) (type default))
   )
@@
     (stroke (width 0) (type default))
   )
-  (wire (pts (xy 113.03 88.9) (xy 109.22 88.9))
+  (wire (pts (xy 124.46 88.9) (xy 109.22 88.9))
     (stroke (width 0) (type default))
   )
@@
     (stroke (width 0) (type default))
   )
-  (wire (pts (xy 113.03 113.03) (xy 113.03 120.65))
-    (stroke (width 0) (type default))
-  )
   (wire (pts (xy 49.53 43.18) (xy 68.58 43.18))
     (stroke (width 0) (type default))
@@
   )
   (wire (pts (xy 54.61 99.06) (xy 68.58 99.06))
-    (stroke (width 0) (type default))
-  )
-  (wire (pts (xy 113.03 105.41) (xy 113.03 88.9))
     (stroke (width 0) (type default))
   )
@@
     (effects (font (size 1.27 1.27)) (justify left))
   )
+  (hierarchical_label "LAN_~{INT}" (shape input) (at 124.46 88.9 0) (fields_autoplaced)
+    (effects (font (size 1.27 1.27)) (justify left))
+  )
   (hierarchical_label "VIDEO_DDC_SDA" (shape bidirectional) (at 149.86 50.8 0) (fields_autoplaced)
     (effects (font (size 1.27 1.27)) (justify left))
@@
     (effects (font (size 1.27 1.27)) (justify left))
   )
-  (hierarchical_label "VIDEO_HPD" (shape bidirectional) (at 113.03 86.36 0) (fields_autoplaced)
+  (hierarchical_label "VIDEO_HPD" (shape bidirectional) (at 124.46 86.36 0) (fields_autoplaced)
     (effects (font (size 1.27 1.27)) (justify left))
   )
@@
     )
   )
-  (symbol (lib_id "Device:LED") (at 113.03 124.46 90) (unit 1)
-    (in_bom yes) (on_board yes) (dnp no) (fields_autoplaced)
-    (property "Reference" "D3" (at 116.84 124.7775 90)
-      (effects (font (size 1.27 1.27)) (justify right))
-    )
-    (property "Value" "LED" (at 116.84 127.3175 90)
-      (effects (font (size 1.27 1.27)) (justify right))
-    )
-    (property "Footprint" "LED_THT:LED_D5.0mm" (at 113.03 124.46 0)
-      (effects (font (size 1.27 1.27)) hide)
-    )
-    (property "Datasheet" "~" (at 113.03 124.46 0)
-      (effects (font (size 1.27 1.27)) hide)
-    )
-    (pin "2")
-    (pin "1")
-    (instances
-      (project "a1_mini"
-        (path "/3257e1ae-50a8-410a-87c3-a39d96a2c51a/d5a6ed82-5dcc-475e-b753-55c600f390da"
-          (reference "D3") (unit 1)
-        )
-      )
-    )
-  )
-  (symbol (lib_id "power:GND") (at 113.03 128.27 0) (unit 1)
-    (in_bom yes) (on_board yes) (dnp no) (fields_autoplaced)
-    (property "Reference" "#PWR069" (at 113.03 134.62 0)
-      (effects (font (size 1.27 1.27)) hide)
-    )
-    (property "Value" "GND" (at 113.03 133.35 0)
-      (effects (font (size 1.27 1.27)))
-    )
-    (property "Footprint" "" (at 113.03 128.27 0)
-      (effects (font (size 1.27 1.27)) hide)
-    )
-    (property "Datasheet" "" (at 113.03 128.27 0)
-      (effects (font (size 1.27 1.27)) hide)
-    )
-    (pin "1")
-    (instances
-      (project "a1_mini"
-        (path "/3257e1ae-50a8-410a-87c3-a39d96a2c51a/d5a6ed82-5dcc-475e-b753-55c600f390da"
-          (reference "#PWR069") (unit 1)
-        )
-      )
-    )
-  )
   (symbol (lib_id "Device:R_US") (at 251.46 100.33 180) (unit 1)
     (in_bom yes) (on_board yes) (dnp no)
@@
         )
       )
-    )
-  )
-  (symbol (lib_id "Device:R_US") (at 113.03 109.22 0) (unit 1)
-    (in_bom yes) (on_board yes) (dnp no)
-    (property "Reference" "R13" (at 111.76 115.57 90)
-      (effects (font (size 1.27 1.27)) (justify left))
-    )
-    (property "Value" "470" (at 114.3 115.57 90)
-      (effects (font (size 1.27 1.27)) (justify left))
-    )
-    (property "Footprint" "Resistor_THT:R_Axial_DIN0204_L3.6mm_D1.6mm_P5.08mm_Horizontal" (at 114.046 109.474 90)
-      (effects (font (size 1.27 1.27)) hide)
-    )
-    (property "Datasheet" "~" (at 113.03 109.22 0)
-      (effects (font (size 1.27 1.27)) hide)
-    )
-    (pin "1")
-    (pin "2")
-    (instances
-      (project "a1_mini"
-        (path "/3257e1ae-50a8-410a-87c3-a39d96a2c51a/d5a6ed82-5dcc-475e-b753-55c600f390da"
-          (reference "R13") (unit 1)
-        )
-      )

Commit message: A1 Mini (which is not all that mini anymore) is feature-complete.
We have 2 ISA slots and even all the power supplies generated from +5V included.

The +12V switcher right next to the audio output is quite a bit concerning, but
we can always say that PWR must be 12V and we directly feed that to the ISA slots.
(Not that PWR is all that clean...) A lot will depend on how I implement grounding,
something that I still have to do.
Parts:
- removed C60: 1uF, Capacitor_THT:C_Disc_D4.7mm_W2.5mm_P5.00mm, symbol Device:C
- renumbered C4 to C32, C5 to C33, C6 to C34, C7 to C35, C61 to C36, C62 to C37, C63 to C38, FB8 to FB10, FB9 to FB11, FB10 to FB12, FB11 to FB13, FB12 to FB14, J10 to J12, J7 to J13, R5 to R18, R6 to R19, R4 to R20, R28 to R21, RN8 to RN7, RN4 to RN8, RN3 to RN9, U28 to U24, U26 to U25, U29 to U26, X2 to X3

Commit message: A1 MINI is fully routed.
That is, if I add a GND fill on both layers. Which I don't, because auto-refill takes
several seconds and so it's a PITA to work with. There are a few dozen DRC errors
as well but nothing major it seems.

Worked out roughly 100ohm diff impedance for the HDMI lines
(not GND-referenced) which I think is my best shot of making it work.

long USB trace has a nice GND shield under-it, so does audio.
Again, probably my best shot at making these work.

Ethernet still needs checking just as short-put USB connections from the hub to
the connector.
Parts:
- Y1: symbol Device:Crystal -> Device:Crystal_GND3
Connections:
- net GND: now also Y1.3
Changed lines of the file:
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@@
+    )
+  )
+  (symbol (lib_id "power:GND") (at 200.66 128.27 0) (unit 1)
+    (in_bom yes) (on_board yes) (dnp no) (fields_autoplaced)
+    (property "Reference" "#PWR0135" (at 200.66 134.62 0)
+      (effects (font (size 1.27 1.27)) hide)
+    )
+    (property "Value" "GND" (at 200.66 133.35 0)
+      (effects (font (size 1.27 1.27)))
+    )
+    (property "Footprint" "" (at 200.66 128.27 0)
+      (effects (font (size 1.27 1.27)) hide)
+    )
+    (property "Datasheet" "" (at 200.66 128.27 0)
+      (effects (font (size 1.27 1.27)) hide)
+    )
+    (pin "1")
+    (instances
+      (project "a1_mini"
+        (path "/3257e1ae-50a8-410a-87c3-a39d96a2c51a/d5a6ed82-5dcc-475e-b753-55c600f390da"
+          (reference "#PWR0135") (unit 1)
+        )
+      )
     )
   )
@@
     )
   )
-  (symbol (lib_id "power:GND") (at 203.2 156.21 0) (unit 1)
-    (in_bom yes) (on_board yes) (dnp no) (fields_autoplaced)
-    (property "Reference" "#PWR0171" (at 203.2 162.56 0)
-      (effects (font (size 1.27 1.27)) hide)
-    )
-    (property "Value" "GND" (at 203.2 161.29 0)
-      (effects (font (size 1.27 1.27)))
-    )
-    (property "Footprint" "" (at 203.2 156.21 0)
-      (effects (font (size 1.27 1.27)) hide)
-    )
-    (property "Datasheet" "" (at 203.2 156.21 0)
-      (effects (font (size 1.27 1.27)) hide)
-    )
-    (pin "1")
-    (instances
-      (project "a1_mini"
-        (path "/3257e1ae-50a8-410a-87c3-a39d96a2c51a/d5a6ed82-5dcc-475e-b753-55c600f390da"
-          (reference "#PWR0171") (unit 1)
-        )
-      )
-    )
-  )
   (symbol (lib_id "power:GND") (at 88.9 106.68 0) (unit 1)
     (in_bom yes) (on_board yes) (dnp no) (fields_autoplaced)
@@
     )
   )
-  (symbol (lib_id "Device:Crystal") (at 200.66 123.19 0) (mirror y) (unit 1)
+  (symbol (lib_id "Device:Crystal_GND3") (at 200.66 123.19 0) (mirror y) (unit 1)
     (in_bom yes) (on_board yes) (dnp no)
     (property "Reference" "Y1" (at 200.66 115.57 0)
@@
     (pin "1")
     (pin "2")
+    (pin "3")
     (instances
       (project "a1_mini"
@@
         )
       )
-    )
-  )
-  (symbol (lib_id "power:+5V") (at 203.2 148.59 0) (unit 1)
-    (in_bom yes) (on_board yes) (dnp no) (fields_autoplaced)
-    (property "Reference" "#PWR0170" (at 203.2 152.4 0)
-      (effects (font (size 1.27 1.27)) hide)
-    )
-    (property "Value" "+5V" (at 203.2 143.51 0)
-      (effects (font (size 1.27 1.27)))
-    )
-    (property "Footprint" "" (at 203.2 148.59 0)
-      (effects (font (size 1.27 1.27)) hide)
-    )
-    (property "Datasheet" "" (at 203.2 148.59 0)
-      (effects (font (size 1.27 1.27)) hide)
-    )
-    (pin "1")
-    (instances
-      (project "a1_mini"
-        (path "/3257e1ae-50a8-410a-87c3-a39d96a2c51a/d5a6ed82-5dcc-475e-b753-55c600f390da"
-          (reference "#PWR0170") (unit 1)
-        )
-      )

Commit message: Checking in stuff before the 3.3V work.
Other:
- note added: "TODO: SD-card pull-ups should go to 3.3V!!!!!!"
- moved on the sheet: BT1
Changed lines of the file:
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@@
     (stroke (width 0) (type default))
   )
-  (wire (pts (xy 134.62 110.49) (xy 134.62 116.84))
+  (wire (pts (xy 181.61 102.87) (xy 181.61 109.22))
     (stroke (width 0) (type default))
   )
@@
   (wire (pts (xy 107.95 163.83) (xy 107.95 176.53))
     (stroke (width 0) (type default))
+  )
+  (text "TODO: SD-card pull-ups should go to 3.3V!!!!!!" (at 148.59 40.64 0)
+    (effects (font (size 3 3) (thickness 0.6) bold (color 255 2 0 1)) (justify left bottom))
   )
   (text "DRQ signals must be open-SOURCE and DACK must be ignored when DRQ is not active!!!"
@@
     )
   )
-  (symbol (lib_id "Device:Battery_Cell") (at 134.62 121.92 0) (unit 1)
+  (symbol (lib_id "Device:Battery_Cell") (at 181.61 114.3 0) (unit 1)
     (in_bom yes) (on_board yes) (dnp no)
-    (property "Reference" "BT1" (at 128.27 123.19 90)
-      (effects (font (size 1.27 1.27)) (justify left))
-    )
-    (property "Value" "CR2032 holder" (at 130.81 127 90)
-      (effects (font (size 1.27 1.27)) (justify left))
-    )
-    (property "Footprint" "Battery:BatteryHolder_Keystone_103_1x20mm" (at 134.62 120.396 90)
-      (effects (font (size 1.27 1.27)) hide)
-    )
-    (property "Datasheet" "~" (at 134.62 120.396 90)
+    (property "Reference" "BT1" (at 175.26 115.57 90)
+      (effects (font (size 1.27 1.27)) (justify left))
+    )
+    (property "Value" "CR2032 holder" (at 177.8 119.38 90)
+      (effects (font (size 1.27 1.27)) (justify left))
+    )
+    (property "Footprint" "Battery:BatteryHolder_Keystone_103_1x20mm" (at 181.61 112.776 90)
+      (effects (font (size 1.27 1.27)) hide)
+    )
+    (property "Datasheet" "~" (at 181.61 112.776 90)
       (effects (font (size 1.27 1.27)) hide)
     )
@@
     )
   )
-  (symbol (lib_id "power:GND") (at 134.62 124.46 0) (unit 1)
-    (in_bom yes) (on_board yes) (dnp no) (fields_autoplaced)
-    (property "Reference" "#PWR0164" (at 134.62 130.81 0)
-      (effects (font (size 1.27 1.27)) hide)
-    )
-    (property "Value" "GND" (at 134.62 129.54 0)
-      (effects (font (size 1.27 1.27)))
-    )
-    (property "Footprint" "" (at 134.62 124.46 0)
-      (effects (font (size 1.27 1.27)) hide)
-    )
-    (property "Datasheet" "" (at 134.62 124.46 0)
+  (symbol (lib_id "power:GND") (at 181.61 116.84 0) (unit 1)
+    (in_bom yes) (on_board yes) (dnp no) (fields_autoplaced)
+    (property "Reference" "#PWR0164" (at 181.61 123.19 0)
+      (effects (font (size 1.27 1.27)) hide)
+    )
+    (property "Value" "GND" (at 181.61 121.92 0)
+      (effects (font (size 1.27 1.27)))
+    )
+    (property "Footprint" "" (at 181.61 116.84 0)
+      (effects (font (size 1.27 1.27)) hide)
+    )
+    (property "Datasheet" "" (at 181.61 116.84 0)
       (effects (font (size 1.27 1.27)) hide)
     )
@@
     )
   )
-  (symbol (lib_id "power:+BATT") (at 134.62 110.49 0) (unit 1)
-    (in_bom yes) (on_board yes) (dnp no) (fields_autoplaced)
-    (property "Reference" "#PWR0163" (at 134.62 114.3 0)
-      (effects (font (size 1.27 1.27)) hide)
-    )
-    (property "Value" "+BATT" (at 134.62 105.41 0)
-      (effects (font (size 1.27 1.27)))
-    )
-    (property "Footprint" "" (at 134.62 110.49 0)
-      (effects (font (size 1.27 1.27)) hide)
-    )
-    (property "Datasheet" "" (at 134.62 110.49 0)
-      (effects (font (size 1.27 1.27)) hide)
-    )
+  (symbol (lib_id "power:+BATT") (at 181.61 102.87 0) (unit 1)
+    (in_bom yes) (on_board yes) (dnp no) (fields_autoplaced)
+    (property "Reference" "#PWR0163" (at 181.61 106.68 0)
+      (effects (font (size 1.27 1.27)) hide)
+    )
+    (property "Value" "+BATT" (at 181.61 97.79 0)
+      (effects (font (size 1.27 1.27)))
+    )
+    (property "Footprint" "" (at 181.61 102.87 0)
+      (effects (font (size 1.27 1.27)) hide)
+    )
+    (property "Datasheet" "" (at 181.61 102.87 0)
+      (effects (font (size 1.27 1.27)) hide)
+    )

Commit message: 3.3V work, before abandoning the idea.
Parts:
- added C66: 1uF, Capacitor_THT:C_Disc_D4.7mm_W2.5mm_P5.00mm, symbol Device:C
- U24: value MAX232 -> ICL3232CPZ; symbol Interface_UART:MAX232 -> Interface_UART:MAX3232
Connections:
- net +5V: now also C66.1; no longer C34.1, C36.1, C37.1, J13.4 (VDD), R20.2, R21.2, RN7.1 (common), RN8.1 (common), RN9.1 (common), U24.16 (VCC), X3.1 (EN), X3.14 (Vcc)
- net GND: now also C66.2
- new net +3.3V: C34.1, C36.1, C37.1, J13.4 (VDD), R20.2, R21.2, RN7.1 (common), RN8.1 (common), RN9.1 (common), U24.16 (VCC), X3.1 (EN), X3.14 (Vcc)
Other:
- note added: "5V operation is not a real problem as all outputs are open-drain and Vil_min is 2.2V"
- note removed: "TODO: SD-card pull-ups should go to 3.3V!!!!!!"
- moved on the sheet: C38
