File: boards/a1_micro_atx/a1_micro_atx.kicad_pcb (KiCad board)
At the start: 4 copper layers, 201.9 x 204.5 mm, 222 parts, among them J1 Conn_01x01, J10 HDMI_A, J11 SJ1-3535NG-BE, J12 DE9_Plug, J13 Micro_SD_Card, J15 USB_A_Stacked, J16 USB_A_Stacked, J17 USB_A_Stacked, J18 Bus_ISA_8bit, J19 Bus_ISA_8bit, J2 Conn_01x01, J3 Conn_01x01, J4 Conn_01x01, J5 Conn_01x02, J6 Jack-DC, J7 Conn_01x02, J8 SJ1-3535NG-BE, J9 Conn_01x02, SW1 SW_DPDT_x2, SW2 SW_Push, SW3 SW_Push, U1 74LS08, U10 74AHCT245, U11 SST39SF040, U12 A1_POWER, U13 74AHCT245, U14 74AHCT245, U15 74AHCT245, U16 74LS273, U17 74LS273, U18 74LS273, U19 ESPRESSO, U2 74LS86, U20 SIMM-30x2, U21 SIMM-30x2, U22 DISCO, U23 A1_CODEC, U24 MAX232, U25 MIO, U26 DS1307+, U27 KSZ8851-11MLL, U28 A1_USBHUB, U29 L78L33ABZ-AP, U3 74LS00, U31 74LS14, U32 74LS139, U33 4075, U34 MC33063AP, U35 MC33063AP, U36 L79L05_TO92, U4 74LS273, U5 74LS574, U6 74LS139, U7 74LS14, U8 74LS126, U9 74AHCT245, X1 8MHz, X2 CXO_DIP14, X3 24MHz, X4 14.31818MHz, Y1 32768Hz, Y2 25MHz

Commit message: Lots of ISA fixes and introduction of 16-bit slots.
These 16-bit slots only support 8-bit transfers, but they do so in a 16-bit
compatible fashion. 16-bit DMAs, upper IRQs and higher addresses are
not supported.

Th PCB is not yet updated and the schematic is ugly. Still the logic should be
there.
Parts:
- added C68: 1uF, Capacitor_THT:C_Disc_D4.7mm_W2.5mm_P5.00mm, F.Cu at (54.0, 201.6)
- added C69: 1uF, Capacitor_THT:C_Disc_D4.7mm_W2.5mm_P5.00mm, F.Cu at (58.1, 201.6)
- added C70: 1uF, Capacitor_THT:C_Disc_D4.7mm_W2.5mm_P5.00mm, F.Cu at (62.1, 201.6)
- added C71: 1uF, Capacitor_THT:C_Disc_D4.7mm_W2.5mm_P5.00mm, F.Cu at (66.2, 201.6)
- added J20: Bus_ISA_16bit, anachron:BUS_AT_CONN, F.Cu at (38.1, 45.7)
- added J21: Bus_ISA_16bit, anachron:BUS_AT_CONN, F.Cu at (58.4, 45.7)
- added J22: Conn_01x01, MountingHole:MountingHole_4.3mm_M4_DIN965_Pad, F.Cu at (66.0, 30.5)
- added J23: Conn_01x01, MountingHole:MountingHole_4.3mm_M4_DIN965_Pad, F.Cu at (66.0, 185.4)
- added J24: Conn_01x01, MountingHole:MountingHole_4.3mm_M4_DIN965_Pad, F.Cu at (45.7, 185.4)
- added U30: 74AHCT245, Package_DIP:DIP-20_W7.62mm_LongPads, F.Cu at (32.1, 236.1)
- added U37: 74AHCT245, Package_DIP:DIP-20_W7.62mm_LongPads, F.Cu at (32.1, 224.5)
- added U38: 74HCT153, Package_DIP:CERDIP-16_W7.62mm_SideBrazed_LongPads_Socket, F.Cu at (32.1, 212.8)
- added U41: 74LS00, Package_DIP:CERDIP-14_W7.62mm_SideBrazed_LongPads_Socket, F.Cu at (54.7, 212.8)
- U31: value 74LS14 -> 74AHCT14
- U32: value 74LS139 -> 74AHCT139
Connections:
- J18 pad 2: /ISA/ISA_RST -> RST
- J18 pad 33: /BUF_D7 -> /ISA/ISA_D7
- J18 pad 34: /BUF_D6 -> /ISA/ISA_D6
- J18 pad 35: /BUF_D5 -> /ISA/ISA_D5
- J18 pad 36: /BUF_D4 -> /ISA/ISA_D4
- J18 pad 37: /BUF_D3 -> /ISA/ISA_D3
- J18 pad 38: /BUF_D2 -> /ISA/ISA_D2
- J18 pad 39: /BUF_D1 -> /ISA/ISA_D1
- J18 pad 40: /BUF_D0 -> /ISA/ISA_D0
- J18 pad 42: /ISA/ISA_AEN -> /CPU_DACK
- J19 pad 2: /ISA/ISA_RST -> RST
- J19 pad 33: /BUF_D7 -> /ISA/ISA_D7
- J19 pad 34: /BUF_D6 -> /ISA/ISA_D6
- J19 pad 35: /BUF_D5 -> /ISA/ISA_D5
- J19 pad 36: /BUF_D4 -> /ISA/ISA_D4
- J19 pad 37: /BUF_D3 -> /ISA/ISA_D3
- J19 pad 38: /BUF_D2 -> /ISA/ISA_D2
- J19 pad 39: /BUF_D1 -> /ISA/ISA_D1
- J19 pad 40: /BUF_D0 -> /ISA/ISA_D0
- J19 pad 42: /ISA/ISA_AEN -> /CPU_DACK
- U3 pad 12: /CPU_~{NREN} -> /BUF_~{EN}
- U31 pad 10: /ISA/ISA_RST -> Net-(U32B-E)
- U31 pad 11: ~{RST} -> Net-(U31-Pad11)
- U31 pad 5: GND -> /BUF_A0
- U31 pad 6: unconnected-(U31-Pad6) -> /ISA/ISA_~{SBHE}
- U31 pad 8: /ISA/ISA_AEN -> /ISA/ISA_TGR16
- U31 pad 9: /CPU_~{DACK} -> /ISA/ISA_~{TGR16}
- U32 pad 1: GND -> /CPU_DACK
- U32 pad 13: /BUF_A20 -> Net-(U32A-O0)
- U32 pad 14: /BUF_~{WE} -> /BUF_DIR
- U32 pad 15: /~{ISA_SEL} -> Net-(U32B-E)
- U32 pad 3: GND -> /BUF_A20
- U32 pad 4: unconnected-(U32A-O0-Pad4) -> Net-(U32A-O0)
- U7 pad 1: GND -> ~{RST}
- U7 pad 2: unconnected-(U7-Pad2) -> RST
- U7 pad 9: /CPU_~{WE} -> /BUF_DIR
Routing:
- net GND: track 2708.7 -> 3190.6 mm
- net /ISA/ISA_D7: track 0.00 -> 195.8 mm, vias 0 -> 1
- net /ISA/ISA_D6: track 0.00 -> 190.8 mm, vias 0 -> 1
- net /ISA/ISA_D5: track 0.00 -> 185.4 mm, vias 0 -> 1
- net /ISA/ISA_D4: track 0.00 -> 179.9 mm, vias 0 -> 1
- net /ISA/ISA_D3: track 0.00 -> 174.5 mm, vias 0 -> 1
- net (no net): track 0.00 -> 174.1 mm
- net /ISA/ISA_D2: track 0.00 -> 169.1 mm, vias 0 -> 1
- net /CPU_DACK: track 10.8 -> 176.2 mm, vias 0 -> 2
- net /ISA/ISA_D1: track 0.00 -> 163.4 mm, vias 0 -> 1
- net /ISA/ISA_D0: track 0.00 -> 158.1 mm, vias 0 -> 1
- net /ISA/ISA_RST: track 131.3 -> 0.00 mm
- net /ISA/ISA_AEN: track 122.7 -> 0.00 mm, vias 2 -> 0
- net +5V: track 1960.9 -> 2077.5 mm, vias 19 -> 20
- net /ISA/~{ISA_MEMR}: track 88.2 -> 196.0 mm, vias 0 -> 2
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Other:
- board size 201.9 x 204.5 mm -> 243.8 x 204.5 mm
- board text added: "J18"
- board text added: "J19"
- board text added: "REAR"
