File: boards/a1_micro_atx/a1_micro_atx.kicad_pcb (KiCad board)
At the start: 4 copper layers, 243.8 x 204.5 mm, 235 parts, among them J1 Conn_01x01, J10 HDMI_A, J11 SJ1-3535NG-BE, J12 DE9_Plug, J13 Micro_SD_Card, J15 USB_A_Stacked, J16 USB_A_Stacked, J17 USB_A_Stacked, J18 Bus_ISA_8bit, J19 Bus_ISA_8bit, J2 Conn_01x01, J20 Bus_ISA_16bit, J21 Bus_ISA_16bit, J22 Conn_01x01, J23 Conn_01x01, J24 Conn_01x01, J3 Conn_01x01, J4 Conn_01x01, J5 Conn_01x02, J6 Jack-DC, J7 Conn_01x02, J8 SJ1-3535NG-BE, J9 Conn_01x02, SW1 SW_DPDT_x2, SW2 SW_Push, SW3 SW_Push, U1 74LS08, U10 74AHCT245, U11 SST39SF040, U12 A1_POWER, U13 74AHCT245, U14 74AHCT245, U15 74AHCT245, U16 74LS273, U17 74LS273, U18 74LS273, U19 ESPRESSO, U2 74LS86, U20 SIMM-30x2, U21 SIMM-30x2, U22 DISCO, U23 A1_CODEC, U24 MAX232, U25 MIO, U26 DS1307+, U27 KSZ8851-11MLL, U28 A1_USBHUB, U29 L78L33ABZ-AP, U3 74LS00, U30 74AHCT245, U31 74AHCT14, U32 74AHCT139, U33 4075, U34 MC33063AP, U35 MC33063AP, U36 L79L05_TO92, U37 74AHCT245, U38 74HCT153, U4 74LS273, U41 74LS00, U5 74LS574, U6 74LS139, U7 74LS14, U8 74LS126, U9 74AHCT245, X1 8MHz, X2 CXO_DIP14, X3 24MHz, X4 14.31818MHz, Y1 32768Hz, Y2 25MHz

Commit message: A1 motherboard now has 16-bit ISA slot support.
Parts:
- C58: footprint Capacitor_THT:CP_Radial_D7.5mm_P2.50mm -> Capacitor_THT:CP_Radial_D6.3mm_P2.50mm
- C59: value 220uF -> 302pF; footprint Capacitor_THT:CP_Radial_D7.5mm_P2.50mm -> Capacitor_THT:C_Disc_D4.7mm_W2.5mm_P5.00mm
- C60: value 302pF -> 100uF; footprint Capacitor_THT:C_Disc_D4.7mm_W2.5mm_P5.00mm -> Capacitor_THT:CP_Radial_D6.3mm_P2.50mm
- C61: value 260p -> 1uF
- C62: value 1000uF -> 1uF; footprint Capacitor_THT:CP_Radial_D10.0mm_P5.00mm -> Capacitor_THT:C_Disc_D4.7mm_W2.5mm_P5.00mm
- C63: value 1500uF -> 220uF; footprint Capacitor_THT:CP_Radial_D10.0mm_P5.00mm -> Capacitor_THT:CP_Radial_D6.3mm_P2.50mm
- C64: value 1uF -> 260p
- C65: value 1uF -> 100uF; footprint Capacitor_THT:C_Disc_D4.7mm_W2.5mm_P5.00mm -> Capacitor_THT:CP_Radial_D6.3mm_P2.50mm
- L1: value 25uH -> 220uH
- L2: value 18uH -> 220uH
- R30: value 0.211Ohm -> 1.5k
- R31: value 180 -> 13k
- R32: value 1.5k -> 0.211Ohm
- R33: value 13k -> 180
- U34: footprint Package_DIP:DIP-8_W7.62mm -> Package_DIP:DIP-8_W7.62mm_LongPads
- U35: value MC33063AP -> L79L05_TO92; footprint Package_DIP:DIP-8_W7.62mm -> Package_TO_SOT_THT:TO-92_Inline
- U36: value L79L05_TO92 -> MC33063AP; footprint Package_TO_SOT_THT:TO-92_Inline -> Package_DIP:DIP-8_W7.62mm_LongPads
- U38: footprint Package_DIP:CERDIP-16_W7.62mm_SideBrazed_LongPads_Socket -> Package_DIP:CERDIP-16_W7.62mm_SideBrazed_LongPads
- U41: footprint Package_DIP:CERDIP-14_W7.62mm_SideBrazed_LongPads_Socket -> Package_DIP:CERDIP-14_W7.62mm_SideBrazed_LongPads
- moved C65 189.2 mm to (74.3, 33.0)
- moved U36 186.3 mm to (89.5, 34.3), turned to 90 degrees
- moved C64 184.3 mm to (88.9, 38.1), turned to 0 degrees
- moved L1 184.0 mm to (45.7, 27.9), turned to 90 degrees
- moved C60 183.6 mm to (41.8, 32.4), turned to 180 degrees
- moved R33 183.1 mm to (88.9, 24.1), turned to 180 degrees
- moved R29 183.0 mm to (52.7, 22.9)
- moved U34 182.9 mm to (50.8, 38.8)
- moved R32 178.0 mm to (97.2, 24.1), turned to 180 degrees
- moved D4 176.7 mm to (46.4, 32.4), turned to -90 degrees
- moved C58 175.0 mm to (56.6, 25.4)
- moved C62 152.5 mm to (65.4, 51.4), turned to 0 degrees
- moved R3 132.2 mm to (243.2, 129.5)
- moved R4 58.8 mm to (139.7, 215.3), turned to -90 degrees
- moved R30 58.5 mm to (34.3, 26.7), turned to 0 degrees
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Connections:
- C59 pad 1: Net-(JP5-A) -> Net-(U34-TC)
- C59 pad 2: GND -> ISA_-12V
- C60 pad 1: Net-(U34-TC) -> GND
- C60 pad 2: -12V -> ISA_-12V
- C61 pad 1: Net-(U35-TC) -> ISA_-12V
- C62 pad 1: GND -> ISA_-5V
- C62 pad 2: -12V -> GND
- C63 pad 1: +12V -> Net-(JP5-A)
- C64 pad 1: -12V -> Net-(U36-TC)
- C65 pad 1: /ISA/ISA_-5V -> ISA_+12V
- D4 pad 2: -12V -> ISA_-12V
- D5 pad 1: +12V -> ISA_+12V
- J18 pad 5: /ISA/ISA_-5V -> ISA_-5V
- J18 pad 7: -12V -> ISA_-12V
- J18 pad 9: +12V -> ISA_+12V
- J19 pad 5: /ISA/ISA_-5V -> ISA_-5V
- J19 pad 7: -12V -> ISA_-12V
- J19 pad 9: +12V -> ISA_+12V
- J20 pad 5: /ISA/ISA_-5V -> ISA_-5V
- J20 pad 7: -12V -> ISA_-12V
- J20 pad 9: +12V -> ISA_+12V
- J21 pad 5: /ISA/ISA_-5V -> ISA_-5V
- J21 pad 7: -12V -> ISA_-12V
- J21 pad 9: +12V -> ISA_+12V
- JP6 pad 2: +12V -> ISA_+12V
- L2 pad 1: Net-(U35-Ipk) -> Net-(U36-Ipk)
- R30 pad 1: Net-(JP5-A) -> ISA_-12V
- R30 pad 2: Net-(U35-Ipk) -> Net-(U34-Vfb)
- R31 pad 1: Net-(U35-DC) -> Net-(U34-Vfb)
- R31 pad 2: Net-(U35-Ipk) -> GND
- R32 pad 1: -12V -> Net-(JP5-A)
- R32 pad 2: Net-(U34-Vfb) -> Net-(U36-Ipk)
- R33 pad 1: Net-(U34-Vfb) -> Net-(U36-DC)
- R33 pad 2: GND -> Net-(U36-Ipk)
- R34 pad 1: +12V -> ISA_+12V
- R34 pad 2: Net-(U35-Vfb) -> Net-(U36-Vfb)
- R35 pad 1: Net-(U35-Vfb) -> Net-(U36-Vfb)
- U30 pad 11: /ISA/ISA_D0 -> /ISA/ISA_D7
- U30 pad 12: /ISA/ISA_D1 -> /ISA/ISA_D6
- U30 pad 13: /ISA/ISA_D2 -> /ISA/ISA_D5
- U30 pad 14: /ISA/ISA_D3 -> /ISA/ISA_D4
- U30 pad 15: /ISA/ISA_D4 -> /ISA/ISA_D3
- U30 pad 16: /ISA/ISA_D5 -> /ISA/ISA_D2
- U30 pad 17: /ISA/ISA_D6 -> /ISA/ISA_D1
- U30 pad 18: /ISA/ISA_D7 -> /ISA/ISA_D0
- U30 pad 2: /BUF_D7 -> /BUF_D0
- U30 pad 3: /BUF_D6 -> /BUF_D1
- U30 pad 4: /BUF_D5 -> /BUF_D2
- U30 pad 5: /BUF_D4 -> /BUF_D3
- U30 pad 6: /BUF_D3 -> /BUF_D4
- U30 pad 7: /BUF_D2 -> /BUF_D5
- U30 pad 8: /BUF_D1 -> /BUF_D6
- U30 pad 9: /BUF_D0 -> /BUF_D7
- U34 pad 4: -12V -> ISA_-12V
- U35 pad 1: Net-(D5-A) -> GND
- U35 pad 2: GND -> ISA_-12V
- U35 pad 3: Net-(U35-TC) -> ISA_-5V
- U36 pad 1: GND -> Net-(D5-A)
- U36 pad 2: -12V -> GND
- U36 pad 3: /ISA/ISA_-5V -> Net-(U36-TC)
- U37 pad 10: unconnected-(U37-GND-Pad10) -> GND
- U38 pad 15: /ISA/ISA_~{TGR16} -> +5V
Routing:
- net -12V: track 279.9 -> 0.00 mm, vias 1 -> 0
- net /ISA/ISA_-5V: track 247.6 -> 0.00 mm, vias 2 -> 0
- net RST: track 0.00 -> 246.7 mm, vias 0 -> 4
- net +5V: track 2077.5 -> 2268.7 mm, vias 20 -> 21
- net (no net): track 174.1 -> 0.00 mm
- net /BUF_DIR: track 197.4 -> 355.5 mm, vias 2 -> 4
- net ISA_-12V: track 0.00 -> 136.1 mm, vias 0 -> 1
- net ISA_+12V: track 0.00 -> 116.4 mm, vias 0 -> 1
- net +12V: track 112.4 -> 0.00 mm, vias 1 -> 0
- net /ISA/ISA_TGR16: track 0.00 -> 104.0 mm, vias 0 -> 1
- net /ISA/ISA_~{MEMCS16}: track 21.4 -> 114.4 mm, vias 0 -> 2
- net Net-(U4-Q3): track 19.7 -> 111.0 mm, vias 0 -> 1
- net /ISA/ISA_~{IOCS16}: track 21.4 -> 110.9 mm, vias 0 -> 2
- net Net-(U31-Pad11): track 0.00 -> 88.7 mm, vias 0 -> 1
- net /ISA/ISA_~{TGR16}: track 0.00 -> 86.9 mm, vias 0 -> 1
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
Commit message: Rotated last DIP package, fixed up a lot of violations and warnings.
Parts:
- U28: footprint Package_DIP:DIP-40_W15.24mm_LongPads -> anachron:DIP-40_W15.24mm_Socket
- U38: footprint Package_DIP:CERDIP-16_W7.62mm_SideBrazed_LongPads -> Package_DIP:DIP-16_W7.62mm_LongPads
- U41: footprint Package_DIP:CERDIP-14_W7.62mm_SideBrazed_LongPads -> Package_DIP:DIP-14_W7.62mm_LongPads
- moved R5 19.1 mm to (113.0, 210.8), turned to 0 degrees
- moved C2 18.5 mm to (102.2, 199.4), turned to -90 degrees
- moved R7 13.5 mm to (105.4, 208.3), turned to 0 degrees
- moved U7 11.9 mm to (106.0, 205.1), turned to 90 degrees
- moved R8 8.08 mm to (113.0, 208.3), turned to 0 degrees
Routing:
- net GND: track 3275.6 -> 3204.6 mm
- net +5V: track 2268.7 -> 2240.8 mm, vias 21 -> 22
- net /BUF_~{WE}: track 297.5 -> 312.1 mm, vias 5 -> 3
- net /~{MRST}: track 192.3 -> 179.5 mm
- net Net-(D2-A): track 5.61 -> 17.8 mm
- net Net-(U13-A->B): track 267.2 -> 278.2 mm, vias 6 -> 8
- net /BUF_~{NREN}: track 185.5 -> 195.7 mm
- net ~{RST}: track 557.5 -> 567.3 mm
- net Net-(C15-Pad1): track 7.71 -> 17.1 mm
- net Net-(U4-Q3): track 111.0 -> 119.0 mm
- net /MIO/~{RTC_INT}: track 214.3 -> 221.4 mm
- net /BUF_A8: track 304.6 -> 309.9 mm
- net RST: track 246.7 -> 251.4 mm
- net /BUF_A19: track 341.4 -> 345.6 mm
- net /BUF_A9: track 301.1 -> 305.1 mm
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Other:
- board text removed: "J18"
- board text removed: "J19"

Commit message: Updated PCB to latest schematic changes.
Also removed 12V boost bypass: that option would also bypass the on-off switch; not good.
Parts:
- removed JP6: Jumper_2_Open, Connector_PinHeader_2.54mm:PinHeader_1x02_P2.54mm_Vertical
Connections:
- J18 pad 2: RST -> /ISA/ISA_RST
- J19 pad 2: RST -> /ISA/ISA_RST
- J20 pad 2: RST -> /ISA/ISA_RST
- J21 pad 2: RST -> /ISA/ISA_RST
- U3 pad 10: /BUF_~{NREN} -> Net-(U3-Pad10)
- U3 pad 12: /BUF_~{EN} -> Net-(U3-Pad12)
- U3 pad 8: /BUF_NREN -> Net-(U3-Pad12)
- U3 pad 9: +5V -> /~{GFX_SEL}
- U31 pad 8: /ISA/ISA_TGR16 -> /ISA/ISA_RST
- U31 pad 9: /ISA/ISA_~{TGR16} -> ~{RST}
- U38 pad 10: +5V -> GND
- U38 pad 11: +5V -> GND
- U38 pad 12: +5V -> GND
- U38 pad 13: +5V -> GND
- U38 pad 15: +5V -> /ISA/ISA_~{TGR16}
- U38 pad 9: unconnected-(U38-Zb-Pad9) -> /ISA/ISA_TGR16
- U7 pad 1: ~{RST} -> /BUF_~{EN}
- U7 pad 10: unconnected-(U7-Pad10) -> /BUF_NREN
- U7 pad 11: +5V -> /BUF_~{NREN}
- U7 pad 2: RST -> Net-(U3-Pad10)
Routing:
- net RST: track 251.4 -> 0.00 mm, vias 4 -> 0
- net /ISA/ISA_RST: track 0.00 -> 185.2 mm, vias 0 -> 1
- net PWR_IN: track 151.8 -> 38.9 mm, vias 3 -> 2
- net Net-(U3-Pad10): track 0.00 -> 108.0 mm, vias 0 -> 6
- net /BUF_NREN: track 140.8 -> 215.5 mm, vias 4 -> 7
- net /ISA/ISA_TGR16: track 104.0 -> 37.4 mm, vias 1 -> 0
- net /ISA/ISA_~{TGR16}: track 86.9 -> 21.8 mm, vias 1 -> 0
- net /BUF_~{NREN}: track 195.7 -> 166.9 mm, vias 4 -> 2
- net /~{GFX_SEL}: track 213.2 -> 241.7 mm, vias 6 -> 7
- net /BUF_~{EN}: track 214.6 -> 242.8 mm, vias 3 -> 4
- net ~{RST}: track 567.3 -> 586.4 mm, vias 11 -> 12
- net GNDA: track 15.5 -> 0.00 mm, vias 2 -> 0
- net Net-(U3-Pad12): track 0.00 -> 13.5 mm
- net GND: track 3204.6 -> 3217.4 mm
- net +5V: track 2240.8 -> 2230.3 mm, vias 22 -> 24
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
Commit message: Added ATX-style power button.
This also involves a management ATTiny because discrete logic just simply doesn't fit.

Power can be turned-off by I2C transactions and by press-and-hold the power SW.
The power switch can also generate an interrupt. Finally, the MCU monitors ~RST
so it can ignore I2C transactions when their pull-ups are inactive due to lack of power.
Parts:
- removed J7: Conn_01x02, Connector_PinHeader_2.54mm:PinHeader_1x02_P2.54mm_Vertical
- removed SW1: SW_DPDT_x2, Button_Switch_THT:SW_CuK_JS202011CQN_DPDT_Straight
- added C72: 1uF, Capacitor_THT:C_Disc_D4.7mm_W2.5mm_P5.00mm, F.Cu at (192.4, 64.1)
- added C73: 1uF, Capacitor_THT:C_Disc_D4.7mm_W2.5mm_P5.00mm, F.Cu at (198.1, 55.9)
- added R36: 10k, Resistor_THT:R_Axial_DIN0204_L3.6mm_D1.6mm_P5.08mm_Horizontal, F.Cu at (201.3, 57.8)
- added SW4: SW_Push, Connector_PinHeader_2.54mm:PinHeader_1x02_P2.54mm_Vertical, F.Cu at (135.9, 221.0)
- added SW5: SW_Push, Button_Switch_THT:SW_PUSH_6mm, F.Cu at (122.8, 220.4)
- added U40: L78L05_TO92, Package_TO_SOT_THT:TO-92_Inline, F.Cu at (196.2, 59.6)
- added U43: ATtiny25-20P, Package_DIP:DIP-8_W7.62mm_LongPads, F.Cu at (204.5, 63.5)
- moved JP1 66.0 mm to (204.5, 219.1), turned to -90 degrees
- moved U7 4.46 mm to (106.0, 200.7)
- moved R6 2.69 mm to (172.1, 65.4)
- moved C51 2.67 mm to (172.1, 68.6)
Connections:
- net /MIO/~{RTC_INT} renamed /I2C_~{INT}
- net Net-(J7-Pin_2) renamed /PWR_ON
- net Net-(JP1-A) renamed /PG
- D3 pad 1: PWR_IN -> /PWR_IN
- J6 pad 1: PWR_IN -> /PWR_IN
- R6 pad 1: PWR_IN -> GND
- U12 pad 6: PWR_IN -> /PWR_IN
- U12 pad 7: PWR_IN -> /PWR_IN
Routing:
- net Net-(U43-~{RESET}/PB5): track 0.00 -> 343.8 mm, vias 0 -> 4
- net /PWR_ON: track 369.8 -> 38.0 mm, vias 2 -> 0
- net /I2C_~{INT}: track 222.5 -> 340.0 mm, vias 2 -> 8
- net /~{MRST}: track 179.5 -> 117.1 mm
- net /I2C_SCL: track 364.7 -> 424.3 mm, vias 6 -> 8
- net /PG: track 336.4 -> 282.8 mm
- net /I2C_SDA: track 366.0 -> 419.0 mm, vias 6 -> 8
- net /PWR_IN: track 0.00 -> 50.0 mm, vias 0 -> 1
- net PWR_IN: track 38.9 -> 0.00 mm, vias 2 -> 0
- net GND: track 3217.4 -> 3252.9 mm
- net ~{RST}: track 586.4 -> 614.5 mm, vias 12 -> 16
- net +5V_STB: track 0.00 -> 12.5 mm
- net Net-(J13-DET): track 71.3 -> 62.2 mm, vias 1 -> 2
- net +5V: track 2230.3 -> 2237.2 mm, vias 24 -> 26
- net /BUF_NREN: track 215.5 -> 208.9 mm
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Other:
- board text added: "3.3V"
- board text added: "5V"
- board text added: "ACT"
- board text added: "POWER"
- board text added: "PWR_GOOD"
- board text added: "RESET"
- board text added: "SPKR_OUT"
- board text added: "SPKR_POWER"
