File: boards/a1_micro_atx/a1_micro_atx.kicad_pcb (KiCad board)
At the start: 4 copper layers, 243.8 x 204.5 mm, 239 parts, among them J1 Conn_01x01, J10 HDMI_A, J11 SJ1-3535NG-BE, J12 DE9_Plug, J13 Micro_SD_Card, J15 USB_A_Stacked, J16 USB_A_Stacked, J17 USB_A_Stacked, J18 Bus_ISA_8bit, J19 Bus_ISA_8bit, J2 Conn_01x01, J20 Bus_ISA_16bit, J21 Bus_ISA_16bit, J22 Conn_01x01, J23 Conn_01x01, J24 Conn_01x01, J3 Conn_01x01, J4 Conn_01x01, J5 Conn_01x02, J6 Jack-DC, J8 SJ1-3535NG-BE, J9 Conn_01x02, SW2 SW_Push, SW3 SW_Push, SW4 SW_Push, SW5 SW_Push, U1 74LS08, U10 74AHCT245, U11 SST39SF040, U12 A1_POWER, U13 74AHCT245, U14 74AHCT245, U15 74AHCT245, U16 74LS273, U17 74LS273, U18 74LS273, U19 ESPRESSO, U2 74LS86, U20 SIMM-30x2, U21 SIMM-30x2, U22 DISCO, U23 A1_CODEC, U24 MAX232, U25 MIO, U26 DS1307+, U27 KSZ8851-11MLL, U28 A1_USBHUB, U29 L78L33ABZ-AP, U3 74LS00, U30 74AHCT245, U31 74AHCT14, U32 74AHCT139, U33 4075, U34 MC33063AP, U35 L79L05_TO92, U36 MC33063AP, U37 74AHCT245, U38 74HCT153, U4 74LS273, U40 L78L05_TO92, U41 74LS00, U43 ATtiny25-20P, U5 74LS574, U6 74LS139, U7 74LS14, U8 74LS126, U9 74AHCT245, X1 8MHz, X2 CXO_DIP14, X3 24MHz, X4 14.31818MHz, Y1 32768Hz, Y2 25MHz

Commit message: Added reverse-power protection to HDMI; small cleanup
- Reverse-current protection on HDMI (via simple diode)
- Cleaned up diff-pair annotation on schematic
- Added proper 3D shape for AT connector
Parts:
- added D6: 1N5817, Diode_THT:D_DO-41_SOD81_P10.16mm_Horizontal, F.Cu at (163.8, 92.7)
Connections:
- F1 pad 2: +5V -> Net-(D6-K)
Routing:
- net +5V: track 2237.2 -> 2228.3 mm
- net Net-(D6-K): track 0.00 -> 3.91 mm
- net /GFX/AUDIO_SFRM: track 152.0 -> 154.4 mm
- net /I2C_SDA: track 419.0 -> 421.2 mm
- net /I2C_SCL: track 424.3 -> 426.3 mm
- net /~{GFX_SEL}: track 241.7 -> 241.0 mm

Commit message: Small fixes and improvements
- Speaker connector is now PC-compatible
- Added internal USB connector for the 7th USB port
- If MCU is not programmed, power defaults to ON
Parts:
- added C74: 100uF, Capacitor_THT:CP_Radial_D5.0mm_P2.00mm, F.Cu at (266.8, 136.5)
- added J7: Conn_02x05_Odd_Even, Connector_PinHeader_2.54mm:PinHeader_2x05_P2.54mm_Vertical, F.Cu at (267.3, 131.4)
- J9: footprint Connector_PinHeader_2.54mm:PinHeader_1x02_P2.54mm_Vertical -> Connector_PinHeader_2.54mm:PinHeader_1x04_P2.54mm_Vertical
- moved R19 36.2 mm to (267.3, 168.3)
- moved R6 16.5 mm to (188.6, 65.4), turned to 180 degrees
- moved C44 10.1 mm to (252.1, 90.8)
- moved FB3 5.07 mm to (120.5, 75.3)
- moved JP7 3.82 mm to (114.9, 75.3)
- moved TP1 3.08 mm to (109.6, 75.3)
- moved JP3 2.54 mm to (248.3, 91.4)
- moved J9 0.88 mm to (139.1, 75.3)
Connections:
- J9 pad 2: Net-(J9-Pin_2) -> Net-(J9-Pin_1)
- R6 pad 1: GND -> +5V_STB
- U23 pad 11: Net-(J9-Pin_2) -> Net-(J9-Pin_3)
- U28 pad 1: unconnected-(U28-VBUS6-Pad1) -> Net-(J7-Pin_1)
- U28 pad 14: unconnected-(U28-USBDN6_DM-Pad14) -> /USB/USB_DN_INT_D+
- U28 pad 15: unconnected-(U28-USBDN6_DP-Pad15) -> /USB/USB_DN_INT_D-
Routing:
- net Net-(J7-Pin_1): track 0.00 -> 101.0 mm, vias 0 -> 2
- net /USB/USB_DN_INT_D-: track 0.00 -> 49.3 mm, vias 0 -> 1
- net /USB/USB_DN_INT_D+: track 0.00 -> 48.8 mm
- net /MIO/SER_CTS: track 115.8 -> 80.2 mm
- net Net-(U24-R2OUT): track 128.2 -> 161.4 mm
- net GND: track 3252.9 -> 3283.6 mm
- net /PG: track 282.8 -> 269.7 mm
- net Net-(U43-~{RESET}/PB5): track 343.8 -> 331.1 mm
- net /VIDEO_HPD: track 307.0 -> 295.2 mm
- net /VIDEO_DDC_SCL: track 283.9 -> 272.0 mm
- net +5V_STB: track 12.5 -> 24.2 mm
- net /I2C_SDA: track 421.2 -> 410.9 mm
- net +5V: track 2228.3 -> 2218.7 mm, vias 26 -> 25
- net SYS_CLK: track 536.3 -> 527.2 mm
- net /CPU_~{INT}: track 378.4 -> 369.9 mm
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Other:
- board text added: "INT USB"

Commit message: Reversed default power-on.
The problem with defaulting to power-on-by-default is that there is a short
on transient while the MCU is booting and gets to override the pull-up. This
is mitigated now by a pull-down and an override jumper. The existence of the
jumper now necessitates an open-emitter drive from the MCU; that is, drive-high
for ON and float for OFF.
Parts:
- added JP6: Jumper_2_Bridged, Connector_PinHeader_2.54mm:PinHeader_1x02_P2.54mm_Vertical, F.Cu at (183.5, 65.4)
- moved R6 11.4 mm to (177.2, 65.4)
Connections:
- R6 pad 1: +5V_STB -> /PWR_ON
- R6 pad 2: /PWR_ON -> GND
Routing:
- net +5V: track 2218.7 -> 2215.6 mm
- net +5V_STB: track 24.2 -> 26.7 mm
- net /PWR_ON: track 35.9 -> 37.9 mm
- net Net-(U43-~{RESET}/PB5): track 331.1 -> 329.4 mm
- net Net-(D4-K): track 19.6 -> 18.1 mm
- net ~{RST}: track 614.1 -> 613.0 mm
- net Net-(J9-Pin_3): track 7.15 -> 6.13 mm
- net Net-(U33-Pad13): track 28.7 -> 27.7 mm
- net Net-(R8-Pad1): track 7.88 -> 6.99 mm
- net /CPU_TC: track 438.1 -> 437.2 mm
- net Net-(U3-Pad10): track 104.0 -> 103.1 mm
- net /ISA_IRQ2: track 256.7 -> 255.9 mm
- net GND: track 3283.6 -> 3284.4 mm
- net Net-(J7-Pin_1): track 101.0 -> 100.3 mm
- net /BUF_D7: track 352.1 -> 351.4 mm
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Other:
- board text added: "PWR OVERRIDE"

Commit message: Moved internal USB connector to create more USB routing clearance.
Parts:
- moved C74 12.1 mm to (262.8, 147.9), turned to 0 degrees
- moved J7 12.0 mm to (263.5, 142.9)
Routing:
- net Net-(J7-Pin_1): track 100.3 -> 114.3 mm
- net /USB/USB_DN_INT_D+: track 48.7 -> 60.2 mm
- net /USB/USB_DN_INT_D-: track 49.3 -> 60.9 mm
- net GND: track 3284.4 -> 3277.9 mm, vias 16 -> 15
- net Net-(U43-~{RESET}/PB5): track 329.4 -> 332.7 mm
- net Net-(U24-R1OUT): track 261.9 -> 264.9 mm
- net /MIO/SER_TXD: track 253.1 -> 256.1 mm
- net /VIDEO_DDC_SCL: track 272.0 -> 275.0 mm
- net /PG: track 269.7 -> 272.7 mm
- net Net-(U24-R2OUT): track 161.4 -> 164.4 mm
- net /MIO/USB_CLK: track 179.0 -> 182.0 mm
- net /MIO/SER_RTS: track 247.8 -> 250.8 mm
- net /VIDEO_HPD: track 295.2 -> 298.2 mm
- net /VIDEO_DDC_SDA: track 292.7 -> 295.0 mm
- net /I2C_SDA: track 410.9 -> 413.2 mm
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