File: boards/a1_micro_atx/cpu.kicad_sch (KiCad schematic)
At the start: 2 parts, among them U19 ESPRESSO

Commit message: Fixed 3.3V for SDCARD; more beautification.
Other:
- company: (none) -> Modular Circuits
- title: Anachron CPU -> Anachron uATX CPU
Changed lines of the file:
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@@
   (paper "A")
   (title_block
-    (title "Anachron CPU")
+    (title "Anachron uATX CPU")
+    (date "2024-02-07")
+    (company "Modular Circuits")
   )
   (bus_entry (at 58.42 86.36) (size 2.54 2.54)
