File: boards/a1_micro_atx/memory.kicad_sch (KiCad schematic)
At the start: 4 parts, among them U21 SIMM-30x2

Commit message: Major schematic beautification.
Other:
- note added: "DRAM: There's one FPM DRAM from ISSI still in production: IS41LV16105D. This is a 1Mx16bit (3.3V) part. To mount it on a SIMM, one would need to: - Implement level-shifters - Add a 3.3V LDO - Add a single-bit flop to capture A10 on falling edge of RAS - Add a demux to select LCAS/HCAS based on captured A10"
- note added: "SIMM socket source: https://www.peconnectors.com/sockets-pga-cpu-and-memory/hws9594/"
Changed lines of the file:
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@@
     (effects (font (face "LM Mono 10") (size 1.27 1.27)) (justify left bottom))
+  )
+  (text "DRAM: There's one FPM DRAM from ISSI still in production: IS41LV16105D.\nThis is a 1Mx16bit (3.3V) part. To mount it on a SIMM, one would need to:\n- Implement level-shifters\n- Add a 3.3V LDO\n- Add a single-bit flop to capture A10 on falling edge of RAS\n- Add a demux to select LCAS/HCAS based on captured A10"
+    (at 53.34 26.67 0)
+    (effects (font (size 1.27 1.27)) (justify left bottom))
+  )
+  (text "SIMM socket source: https://www.peconnectors.com/sockets-pga-cpu-and-memory/hws9594/"
+    (at 38.1 166.37 0)
+    (effects (font (size 1.27 1.27)) (justify left bottom))
   )
   (label "A9" (at 88.9 71.12 0) (fields_autoplaced)
@@
     (pin "1")
     (instances
-      (project "a1_mini"
+      (project "a1_micro_atx"
         (path "/3257e1ae-50a8-410a-87c3-a39d96a2c51a/74914ce5-2001-49ca-8f09-c71b1f2944ab"
           (reference "#PWR0124") (unit 1)
@@
     (pin "1")
     (instances
-      (project "a1_mini"
+      (project "a1_micro_atx"
         (path "/3257e1ae-50a8-410a-87c3-a39d96a2c51a/74914ce5-2001-49ca-8f09-c71b1f2944ab"
           (reference "#PWR0115") (unit 1)
@@
     (pin "1")
     (instances
-      (project "a1_mini"
+      (project "a1_micro_atx"
         (path "/3257e1ae-50a8-410a-87c3-a39d96a2c51a/74914ce5-2001-49ca-8f09-c71b1f2944ab"
           (reference "#PWR0116") (unit 1)
@@
     (pin "1")
     (instances
-      (project "a1_mini"
+      (project "a1_micro_atx"
         (path "/3257e1ae-50a8-410a-87c3-a39d96a2c51a/74914ce5-2001-49ca-8f09-c71b1f2944ab"
           (reference "#PWR0117") (unit 1)
@@
     (pin "1")
     (instances
-      (project "a1_mini"
+      (project "a1_micro_atx"
         (path "/3257e1ae-50a8-410a-87c3-a39d96a2c51a/74914ce5-2001-49ca-8f09-c71b1f2944ab"
           (reference "#PWR0118") (unit 1)
@@
     (pin "1")
     (instances
-      (project "a1_mini"
+      (project "a1_micro_atx"
         (path "/3257e1ae-50a8-410a-87c3-a39d96a2c51a/74914ce5-2001-49ca-8f09-c71b1f2944ab"
           (reference "C23") (unit 1)
@@
     (pin "1")
     (instances
-      (project "a1_mini"
+      (project "a1_micro_atx"
         (path "/3257e1ae-50a8-410a-87c3-a39d96a2c51a/74914ce5-2001-49ca-8f09-c71b1f2944ab"
           (reference "#PWR0114") (unit 1)
@@
     (pin "1")
     (instances
-      (project "a1_mini"
+      (project "a1_micro_atx"
         (path "/3257e1ae-50a8-410a-87c3-a39d96a2c51a/74914ce5-2001-49ca-8f09-c71b1f2944ab"
           (reference "C22") (unit 1)
@@
     (pin "A29")
     (instances
-      (project "a1_mini"
+      (project "a1_micro_atx"
         (path "/3257e1ae-50a8-410a-87c3-a39d96a2c51a/58d11f1c-6aae-4928-b318-2d07bb2e6df5"
           (reference "U21") (unit 1)
@@
   )
   (symbol (lib_id "anachron:SIMM-30x2") (at 152.4 129.54 0) (unit 2)
-    (in_bom yes) (on_board yes) (dnp no) (fields_autoplaced)
-    (property "Reference" "U21" (at 157.1341 104.14 0)
-      (effects (font (size 1.27 1.27)) (justify left))
-    )
-    (property "Value" "SIMM-30x2" (at 157.1341 106.68 0)
+    (in_bom yes) (on_board yes) (dnp no)
+    (property "Reference" "U21" (at 156.21 104.14 0)
+      (effects (font (size 1.27 1.27)) (justify left))
+    )
+    (property "Value" "SIMM-30x2" (at 156.21 106.68 0)
       (effects (font (size 1.27 1.27)) (justify left))
     )
@@
     (pin "A29")
     (instances
-      (project "a1_mini"
+      (project "a1_micro_atx"
         (path "/3257e1ae-50a8-410a-87c3-a39d96a2c51a/58d11f1c-6aae-4928-b318-2d07bb2e6df5"
           (reference "U21") (unit 2)
@@
     (pin "1")
     (instances
-      (project "a1_mini"
+      (project "a1_micro_atx"
         (path "/3257e1ae-50a8-410a-87c3-a39d96a2c51a/74914ce5-2001-49ca-8f09-c71b1f2944ab"
           (reference "#PWR0121") (unit 1)
@@
     (pin "1")
     (instances
-      (project "a1_mini"
+      (project "a1_micro_atx"
         (path "/3257e1ae-50a8-410a-87c3-a39d96a2c51a/74914ce5-2001-49ca-8f09-c71b1f2944ab"
           (reference "C21") (unit 1)
@@
     (pin "1")
     (instances
-      (project "a1_mini"
+      (project "a1_micro_atx"
         (path "/3257e1ae-50a8-410a-87c3-a39d96a2c51a/74914ce5-2001-49ca-8f09-c71b1f2944ab"
           (reference "#PWR0126") (unit 1)
@@
     (pin "1")
     (instances
-      (project "a1_mini"
+      (project "a1_micro_atx"
         (path "/3257e1ae-50a8-410a-87c3-a39d96a2c51a/74914ce5-2001-49ca-8f09-c71b1f2944ab"
           (reference "#PWR0123") (unit 1)
@@
     (pin "1")
     (instances
-      (project "a1_mini"
+      (project "a1_micro_atx"
         (path "/3257e1ae-50a8-410a-87c3-a39d96a2c51a/74914ce5-2001-49ca-8f09-c71b1f2944ab"
           (reference "#PWR0125") (unit 1)
@@
     (pin "1")
     (instances
-      (project "a1_mini"
+      (project "a1_micro_atx"
         (path "/3257e1ae-50a8-410a-87c3-a39d96a2c51a/74914ce5-2001-49ca-8f09-c71b1f2944ab"
           (reference "#PWR0111") (unit 1)
@@
     (pin "1")
     (instances
-      (project "a1_mini"
+      (project "a1_micro_atx"
         (path "/3257e1ae-50a8-410a-87c3-a39d96a2c51a/74914ce5-2001-49ca-8f09-c71b1f2944ab"
           (reference "#PWR0112") (unit 1)
@@
     (pin "1")
     (instances
-      (project "a1_mini"
+      (project "a1_micro_atx"
         (path "/3257e1ae-50a8-410a-87c3-a39d96a2c51a/74914ce5-2001-49ca-8f09-c71b1f2944ab"
           (reference "#PWR0113") (unit 1)
@@
     (pin "1")
     (instances
-      (project "a1_mini"
+      (project "a1_micro_atx"
         (path "/3257e1ae-50a8-410a-87c3-a39d96a2c51a/74914ce5-2001-49ca-8f09-c71b1f2944ab"
           (reference "#PWR0122") (unit 1)

Commit message: Fixed 3.3V for SDCARD; more beautification.
Other:
- company: (none) -> Modular Circuits
- title: Anachron RAM bank -> Anachron uATX RAM Bank
Changed lines of the file:
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@@
   (paper "A")
   (title_block
-    (title "Anachron RAM bank")
+    (title "Anachron uATX RAM Bank")
+    (date "2024-02-07")
+    (company "Modular Circuits")
   )
   (junction (at 154.94 30.48) (diameter 0) (color 0 0 0 0)
