File: boards/a1_micro_atx/isa.kicad_sch (KiCad schematic)
At the start: 36 parts, among them J18 Bus_ISA_8bit, J19 Bus_ISA_8bit, U31 74LS14, U32 74LS139, U33 4075, U34 MC33063AP, U35 MC33063AP, U36 L79L05_TO92, X4 14.31818MHz

Commit message: Major schematic beautification.
Parts:
- added unit 1 of U32
Connections:
- net GND: now also U31.5, U32.1 (E), U32.2 (A0), U32.3 (A1)
- net ~{INT}: now also U31.2
Other:
- note added: "Optional oscillator in case there's a bunch of problems with feeding just SYS_CLK to ISA_OSC."
- note removed: "Optional oscillator in case there's a bunch of problems with feeding just SYS_CLK to this ISA pin."
- moved on the sheet: C54, C55, C56, C57, C58, C59, C60, C61, C62, C63, C64, C65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

Commit message: Fixed 3.3V for SDCARD; more beautification.
Other:
- company: (none) -> Modular Circuits
- title: Anachron ISA bus interface -> Anachron ISA Bus Interface
Changed lines of the file:
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@@
   (paper "B")
   (title_block
-    (title "Anachron ISA bus interface")
+    (title "Anachron ISA Bus Interface")
+    (date "2024-02-07")
+    (company "Modular Circuits")
   )
   (junction (at 279.4 208.28) (diameter 0) (color 0 0 0 0)

Commit message: Lots of ISA fixes and introduction of 16-bit slots.
These 16-bit slots only support 8-bit transfers, but they do so in a 16-bit
compatible fashion. 16-bit DMAs, upper IRQs and higher addresses are
not supported.

Th PCB is not yet updated and the schematic is ugly. Still the logic should be
there.
Parts:
- added C68, C69, C70, C71: 1uF, Capacitor_THT:C_Disc_D4.7mm_W2.5mm_P5.00mm, symbol Device:C
- added J20, J21: Bus_ISA_16bit, anachron:BUS_AT_CONN, symbol Connector:Bus_ISA_16bit
- added U30, U37: 74AHCT245, Package_DIP:DIP-20_W7.62mm_LongPads, symbol 74xx:74LS245
- added U38: 74HCT153, Package_DIP:CERDIP-16_W7.62mm_SideBrazed_LongPads_Socket, symbol 74xx:74LS153
- added U41: 74LS00, Package_DIP:CERDIP-14_W7.62mm_SideBrazed_LongPads_Socket, symbol 74xx:74LS00
- U31: value 74LS14 -> 74AHCT14
- U32: value 74LS139 -> 74AHCT139
Connections:
- net +12V: now also J20.9 (+12V), J21.9 (+12V)
- net +5V: now also C68.1, C69.1, C70.1, C71.1, J20.29 (VCC), J20.3 (+5V), J20.78 (+5V), J21.29 (VCC), J21.3 (+5V), J21.78 (+5V), U30.20 (VCC), U37.20 (VCC), U38.10 (I0b), U38.11 (I1b), U38.12 (I2b), U38.13 (I3b), U38.16 (VCC), U38.3 (I3a), U38.4 (I2a), U41.14 (VCC), U41.4
- net -12V: now also J20.7 (-12V), J21.7 (-12V)
- net CPU_~{DACK}: now also U41.9; no longer U31.9
- net DMA_TC: now also J20.27 (TC), J21.27 (TC)
- net DRQ1: now also J20.18 (DRQ1), J21.18 (DRQ1)
- net DRQ2: now also J20.6 (DRQ2), J21.6 (DRQ2)
- net DRQ3: now also J20.16 (DRQ3), J21.16 (DRQ3)
- net GND: now also C68.2, C69.2, C70.2, C71.2, J20.1 (GND), J20.10 (GND), J20.31 (GND), J20.70 (~{DACK0}), J20.72 (~{DACK5}), J20.74 (~{DACK6}), J20.76 (~{DACK7}), J20.80 (GND), J20.82 (LA23), J20.83 (LA22), J20.84 (LA21), J20.85 (LA20), J20.86 (LA19), J20.87 (LA18), J20.88 (LA17), J21.1 (GND), J21.10 (GND), J21.31 (GND), J21.70 (~{DACK0}), J21.72 (~{DACK5}), J21.74 (~{DACK6}), J21.76 (~{DACK7}), J21.80 (GND), J21.82 (LA23), J21.83 (LA22), J21.84 (LA21), J21.85 (LA20), J21.86 (LA19), J21.87 (LA18), J21.88 (LA17), U30.10 (GND), U38.1 (Ea), U38.8 (GND), U41.7 (GND); no longer U31.5, U32.1 (E), U32.3 (A1)
- net ISA_-5V: now also J20.5 (-5V), J21.5 (-5V)
- net ISA_A0: now also U31.5, J20.62 (BA00), J21.62 (BA00), U41.1
- net ISA_A1: now also J20.61 (BA01), J21.61 (BA01)
- net ISA_A10: now also J20.52 (BA10), J21.52 (BA10)
- net ISA_A11: now also J20.51 (BA11), J21.51 (BA11)
- net ISA_A12: now also J20.50 (BA12), J21.50 (BA12)
- net ISA_A13: now also J20.49 (BA13), J21.49 (BA13)
- net ISA_A14: now also J20.48 (BA14), J21.48 (BA14)
- net ISA_A15: now also J20.47 (BA15), J21.47 (BA15)
- net ISA_A16: now also J20.46 (BA16), J21.46 (BA16)
- net ISA_A17: now also J20.45 (BA17), J21.45 (BA17)
- net ISA_A18: now also J20.44 (BA18), J21.44 (BA18)
- net ISA_A19: now also J20.43 (BA19), J21.43 (BA19)
- net ISA_A2: now also J20.60 (BA02), J21.60 (BA02)
- net ISA_A20: now also U32.3 (A1), U38.14 (S0); no longer U32.13 (A1)
- net ISA_A3: now also J20.59 (BA03), J21.59 (BA03)
- net ISA_A4: now also J20.58 (BA04), J21.58 (BA04)
- net ISA_A5: now also J20.57 (BA05), J21.57 (BA05)
- net ISA_A6: now also J20.56 (BA06), J21.56 (BA06)
- net ISA_A7: now also J20.55 (BA07), J21.55 (BA07)
- net ISA_A8: now also J20.54 (BA08), J21.54 (BA08)
- net ISA_A9: now also J20.53 (BA09), J21.53 (BA09)
- net ISA_ALE: now also J20.28 (ALE), J21.28 (ALE), U41.13
- net ISA_D0: now also J20.40 (DB0), J21.40 (DB0), U30.11 (B7)
- net ISA_D1: now also J20.39 (DB1), J21.39 (DB1), U30.12 (B6)
- net ISA_D2: now also J20.38 (DB2), J21.38 (DB2), U30.13 (B5)
- net ISA_D3: now also J20.37 (DB3), J21.37 (DB3), U30.14 (B4)
- net ISA_D4: now also J20.36 (DB4), J21.36 (DB4), U30.15 (B3)
- net ISA_D5: now also J20.35 (DB5), J21.35 (DB5), U30.16 (B2)
- net ISA_D6: now also J20.34 (DB6), J21.34 (DB6), U30.17 (B1)
- net ISA_D7: now also J20.33 (DB7), J21.33 (DB7), U30.18 (B0)
- net ISA_IRQ2: now also J20.4 (IRQ2), J21.4 (IRQ2)
- net ISA_IRQ3: now also J20.25 (IRQ3), J21.25 (IRQ3)
- net ISA_IRQ4: now also J20.24 (IRQ4), J21.24 (IRQ4)
- net ISA_IRQ5: now also J20.23 (IRQ5), J21.23 (IRQ5)
- net ISA_IRQ6: now also J20.22 (IRQ6), J21.22 (IRQ6)
- net ISA_IRQ7: now also J20.21 (IRQ7), J21.21 (IRQ7)
- net ISA_OSC: now also J20.30 (OSC), J21.30 (OSC)
- net SYS_CLK: now also J20.20 (CLK), J21.20 (CLK)
- net ~{DACK1}: now also J20.17 (~{DACK1}), J21.17 (~{DACK1})
- net ~{DACK2}: now also J20.26 (~{DACK2}), J21.26 (~{DACK2})
- net ~{DACK3}: now also J20.15 (~{DACK3}), J21.15 (~{DACK3})
- net ~{ISA_0WS}: now also J20.8 (UNUSED), J21.8 (UNUSED)
- net ~{ISA_DACK0}: now also J20.19 (~{REFRESH}), J21.19 (~{REFRESH})
- net ~{ISA_IOR}: now also J20.14 (~{IOR}), J21.14 (~{IOR})
- net ~{ISA_IOW}: now also J20.13 (~{IOW}), J21.13 (~{IOW})
- net ~{ISA_IO_CH_CK}: now also J20.32 (IO), J21.32 (IO)
- net ~{ISA_MEMR}: now also J20.12 (~{SMEMR}), J20.89 (~{MEMR}), J21.12 (~{SMEMR}), J21.89 (~{MEMR})
- net ~{ISA_MEMW}: now also J20.11 (~{SMEMW}), J20.90 (~{MEMW}), J21.11 (~{SMEMW}), J21.90 (~{MEMW})
- net ~{ISA_SEL}: now also U38.2 (S1), U41.10; no longer U32.15 (E)
- net ~{WAIT}: now also J20.41 (IO_READY), J21.41 (IO_READY)
- net ~{WE}: now also U30.1 (A->B), U37.1 (A->B)
- net at U32.4 (O0): now also U32.13 (A1)
- net ISA_~{SBHE}: now reaches U31.6
- net ISA_~{SBHE}: now also J20.81 (SBHE), J21.81 (SBHE)
- net ISA_AEN renamed CPU_DACK
- net CPU_DACK: now also U32.1 (E), J20.42 (AEN), J21.42 (AEN); no longer U31.8
- net ISA_RST renamed RST
- net RST: now also J20.2 (RESET), J21.2 (RESET); no longer U31.10
- net ~{RST}: no longer names the net of U31.11
- net ~{RST}: now also U41.8
- new net: U31.10, U32.15 (E)
- new net D0: U30.9 (A7), U37.2 (A0)
- new net D1: U30.8 (A6), U37.3 (A1)
- new net D2: U30.7 (A5), U37.4 (A2)
- new net D3: U30.6 (A4), U37.5 (A3)
- new net D4: U30.5 (A3), U37.6 (A4)
- new net D5: U30.4 (A2), U37.7 (A5)
- new net D6: U30.3 (A1), U37.8 (A6)
- new net D7: U30.2 (A0), U37.9 (A7)
- new net ISA_CSH: U41.3, U41.5
- new net ISA_D10: J20.93 (D10), J21.93 (D10), U37.16 (B2)
- new net ISA_D11: J20.94 (D11), J21.94 (D11), U37.15 (B3)
- new net ISA_D12: J20.95 (D12), J21.95 (D12), U37.14 (B4)
- new net ISA_D13: J20.96 (D13), J21.96 (D13), U37.13 (B5)
- new net ISA_D14: J20.97 (D14), J21.97 (D14), U37.12 (B6)
- new net ISA_D15: J20.98 (D15), J21.98 (D15), U37.11 (B7)
- new net ISA_D8: J20.91 (D8), J21.91 (D8), U37.18 (B0)
- new net ISA_D9: J20.92 (D9), J21.92 (D9), U37.17 (B1)
- new net ISA_DRQ0: J20.71 (DRQ0), J21.71 (DRQ0)
- new net ISA_DRQ5: J20.73 (DRQ5), J21.73 (DRQ5)
- new net ISA_DRQ6: J20.75 (DRQ6), J21.75 (DRQ6)
- new net ISA_DRQ7: J20.77 (DRQ7), J21.77 (DRQ7)
- new net ISA_IRQ10: J20.65 (IRQ10), J21.65 (IRQ10)
- new net ISA_IRQ11: J20.66 (IRQ11), J21.66 (IRQ11)
- new net ISA_IRQ12: J20.67 (IRQ12), J21.67 (IRQ12)
- new net ISA_IRQ14: J20.69 (IRQ14), J21.69 (IRQ14)
- new net ISA_IRQ15: J20.68 (IRQ15), J21.68 (IRQ15)
- new net ISA_MASTER: J20.79 (MASTER), J21.79 (MASTER)
- new net ISA_TGR16: U31.8, U41.2
- new net ISA_~{CSH}: U37.19 (CE), U41.12, U41.6
- new net ISA_~{CSL}: U30.19 (CE), U41.11
- new net ISA_~{IOCS16}: J20.64 (~{IOCS16}), J21.64 (~{IOCS16}), U38.5 (I1a)
- new net ISA_~{MEMCS16}: J20.63 (~{MEMCS16}), J21.63 (~{MEMCS16}), U38.6 (I0a)
- new net ISA_~{TGR16}: U31.9, U38.15 (Eb), U38.7 (Za)
Other:
- note added: "For DMA transfers, we'll have to enable ~{ISA_IOW} or ~{ISA_IOR} depending on the transfer type. ~{WE} is already in the 'right' direction, that is, it's the inverted version of that of the CPU in case of DMAs."
- note added: "Truth table: ~ISA_SEL ~TRG16 ~SBHE A0 Low ~CS High ~CS Transfer type 0 0 1 0 0 1 D0-7 0 0 0 0 N/A N/A D0-15 (16-bit transfer) 0 0 1 1 N/A N/A Invalid 0 0 0 1 1 0 D7-15 0 1 1 0 0 1 D0-7 0 1 0 1 0 1 D0-7 1 X (1) X X 1 1 not addressed"
- note removed: "TODO: should we add a couple of 16-bit slots, where the appropriate signals are tied down to ensure that 16-bit cards don't accidentally assume 16-bit transactions just because of floating control pins?"
- moved on the sheet: C54, C55, C56, C57, C58, C59, C60, C61, C62, C63, C64, C65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

Commit message: A1 motherboard now has 16-bit ISA slot support.
Parts:
- removed C58, C59: 220uF, Capacitor_THT:CP_Radial_D7.5mm_P2.50mm, symbol Device:C_Polarized_Small_US
- removed C60: 302pF, Capacitor_THT:C_Disc_D4.7mm_W2.5mm_P5.00mm, symbol Device:C
- removed C61: 260p, Capacitor_THT:C_Disc_D4.7mm_W2.5mm_P5.00mm, symbol Device:C
- removed C62: 1000uF, Capacitor_THT:CP_Radial_D10.0mm_P5.00mm, symbol Device:C_Polarized_Small_US
- removed C63: 1500uF, Capacitor_THT:CP_Radial_D10.0mm_P5.00mm, symbol Device:C_Polarized_Small_US
- removed C64, C65: 1uF, Capacitor_THT:C_Disc_D4.7mm_W2.5mm_P5.00mm, symbol Device:C
- removed D4, D5: 1N5817, Diode_THT:D_DO-41_SOD81_P10.16mm_Horizontal, symbol Diode:1N5817
- removed JP5: Jumper_2_Bridged, Connector_PinHeader_2.54mm:PinHeader_1x02_P2.54mm_Vertical, symbol Jumper:Jumper_2_Bridged
- removed JP6: Jumper_2_Open, Connector_PinHeader_2.54mm:PinHeader_1x02_P2.54mm_Vertical, symbol Jumper:Jumper_2_Open
- removed L1: 25uH, Inductor_THT:L_Radial_D8.7mm_P5.00mm_Fastron_07HCP, symbol Device:L
- removed L2: 18uH, Inductor_THT:L_Radial_D8.7mm_P5.00mm_Fastron_07HCP, symbol Device:L
- removed R29: 0.244Ohm, Resistor_THT:R_Axial_DIN0204_L3.6mm_D1.6mm_P5.08mm_Horizontal, symbol Device:R_US
- removed R30: 0.211Ohm, Resistor_THT:R_Axial_DIN0204_L3.6mm_D1.6mm_P5.08mm_Horizontal, symbol Device:R_US
- removed R31: 180, Resistor_THT:R_Axial_DIN0204_L3.6mm_D1.6mm_P5.08mm_Horizontal, symbol Device:R_US
- removed R32, R35: 1.5k, Resistor_THT:R_Axial_DIN0204_L3.6mm_D1.6mm_P5.08mm_Horizontal, symbol Device:R_US
- removed R33, R34: 13k, Resistor_THT:R_Axial_DIN0204_L3.6mm_D1.6mm_P5.08mm_Horizontal, symbol Device:R_US
- removed U34, U35: MC33063AP, Package_DIP:DIP-8_W7.62mm, symbol Regulator_Switching:MC33063AP
- removed U36: L79L05_TO92, Package_TO_SOT_THT:TO-92_Inline, symbol Regulator_Linear:L79L05_TO92
- U38: footprint Package_DIP:CERDIP-16_W7.62mm_SideBrazed_LongPads_Socket -> Package_DIP:CERDIP-16_W7.62mm_SideBrazed_LongPads
- U41: footprint Package_DIP:CERDIP-14_W7.62mm_SideBrazed_LongPads_Socket -> Package_DIP:CERDIP-14_W7.62mm_SideBrazed_LongPads
Connections:
- net +5V: now also U38.15 (Eb)
- net D0: now also U30.2 (A0); no longer U30.9 (A7)
- net D1: now also U30.3 (A1); no longer U30.8 (A6)
- net D2: now also U30.4 (A2); no longer U30.7 (A5)
- net D3: now also U30.5 (A3); no longer U30.6 (A4)
- net D4: now also U30.6 (A4); no longer U30.5 (A3)
- net D5: now also U30.7 (A5); no longer U30.4 (A2)
- net D6: now also U30.8 (A6); no longer U30.3 (A1)
- net D7: now also U30.9 (A7); no longer U30.2 (A0)
- net GND: now also U37.10 (GND)
- net ISA_D0: now also U30.18 (B0); no longer U30.11 (B7)
- net ISA_D1: now also U30.17 (B1); no longer U30.12 (B6)
- net ISA_D2: now also U30.16 (B2); no longer U30.13 (B5)
- net ISA_D3: now also U30.15 (B3); no longer U30.14 (B4)
- net ISA_D4: now also U30.14 (B4); no longer U30.15 (B3)
- net ISA_D5: now also U30.13 (B5); no longer U30.16 (B2)
- net ISA_D6: now also U30.12 (B6); no longer U30.17 (B1)
- net ISA_D7: now also U30.11 (B7); no longer U30.18 (B0)
- net ISA_~{TGR16}: no longer U38.15 (Eb)
- net +12V renamed ISA_+12V
- net -12V renamed ISA_-12V
Other:
- note removed: "Designed using http://www.nomad.ee/micros/mc34063a/index.shtml"
- note removed: "Other supply options (dual channel): TPS6513x - this seems to fit the bill BD8316GWL - this can't generate -12, only about -9. R1283x - this seems to fit the bill MAX864 - switched capacitor +/-10V @ 100mA D81870EFV - seems to fit the bill ADP5071 - seems to fit the bill max743 - low current, expensive, but, in DIP PACKAGE!!!"
- note removed: "The original PC provided several amps on +12V. We obviously can't match that, but we don't expect much load on the +12V rail either."
- note removed: "The original PC supplied 0.3A on the -5V and 0.25 on the -12V rails. It had 5 expansion slots. We provide about half of that current for about half of the slots. However it is anticipated that -5V is not used at all and -12 is used by RS232 transceivers only."
- moved on the sheet: C54, C55, C56, C57, C68, C69, C70, C71, RN10, U30, U31D, U31E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

Commit message: Rotated last DIP package, fixed up a lot of violations and warnings.
Parts:
- U38: footprint Package_DIP:CERDIP-16_W7.62mm_SideBrazed_LongPads -> Package_DIP:DIP-16_W7.62mm_LongPads
- U41: footprint Package_DIP:CERDIP-14_W7.62mm_SideBrazed_LongPads -> Package_DIP:DIP-14_W7.62mm_LongPads
Changed lines of the file:
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@@
 			)
 		)
-		(property "Footprint" "Package_DIP:CERDIP-14_W7.62mm_SideBrazed_LongPads"
+		(property "Footprint" "Package_DIP:DIP-14_W7.62mm_LongPads"
 			(at 387.35 222.25 0)
 			(effects
@@
 			)
 		)
-		(property "Footprint" "Package_DIP:CERDIP-16_W7.62mm_SideBrazed_LongPads"
+		(property "Footprint" "Package_DIP:DIP-16_W7.62mm_LongPads"
 			(at 294.64 223.52 0)
 			(effects
@@
 			)
 		)
-		(property "Footprint" "Package_DIP:CERDIP-14_W7.62mm_SideBrazed_LongPads"
+		(property "Footprint" "Package_DIP:DIP-14_W7.62mm_LongPads"
 			(at 27.94 245.11 0)
 			(effects
@@
 			)
 		)
-		(property "Footprint" "Package_DIP:CERDIP-14_W7.62mm_SideBrazed_LongPads"
+		(property "Footprint" "Package_DIP:DIP-14_W7.62mm_LongPads"
 			(at 355.6 203.2 0)
 			(effects
@@
 			)
 		)
-		(property "Footprint" "Package_DIP:CERDIP-14_W7.62mm_SideBrazed_LongPads"
+		(property "Footprint" "Package_DIP:DIP-14_W7.62mm_LongPads"
 			(at 383.54 200.66 0)
 			(effects
@@
 			)
 		)
-		(property "Footprint" "Package_DIP:CERDIP-14_W7.62mm_SideBrazed_LongPads"
+		(property "Footprint" "Package_DIP:DIP-14_W7.62mm_LongPads"
 			(at 67.945 205.105 0)
 			(effects

Commit message: Missed a file...
Connections:
- net +5V: no longer U38.10 (I0b), U38.11 (I1b), U38.12 (I2b), U38.13 (I3b), U38.15 (Eb)
- net GND: now also U38.10 (I0b), U38.11 (I1b), U38.12 (I2b), U38.13 (I3b)
- net ISA_TGR16: now also U38.9 (Zb); no longer U31.8
- net ISA_~{TGR16}: now also U38.15 (Eb); no longer U31.9
- net RST renamed ISA_RST
- net ISA_RST: now also U31.8
- new net ~{RST}: U31.9
Other:
- note added: "Review: High and Low CS generation for both I/O, mem and DMA cycles"
- moved on the sheet: U31D
