File: boards/a1_micro_atx/a1_micro_atx.kicad_sch (KiCad schematic)
At the start: 67 parts, among them J1 Conn_01x01, J2 Conn_01x01, J3 Conn_01x01, J4 Conn_01x01, J5 Conn_01x02, J6 Jack-DC, J7 Conn_01x02, SW1 SW_DPDT_x2, SW2 SW_Push, SW3 SW_Push, U1 74LS08, U10 74AHCT245, U11 SST39SF040, U12 A1_POWER, U13 74AHCT245, U14 74AHCT245, U15 74AHCT245, U16 74LS273, U17 74LS273, U18 74LS273, U2 74LS86, U3 74LS00, U4 74LS273, U5 74LS574, U6 74LS139, U7 74LS14, U8 74LS126, U9 74AHCT245, X1 8MHz

Commit message: Major schematic beautification.
Parts:
- RN6: now not fitted
Connections:
- net +5V: now also U7.11
- net GND: now also J1.1 (Pin_1), J2.1 (Pin_1), J3.1 (Pin_1), J4.1 (Pin_1), U7.1
- net nNR_DECODE_EN renamed ~{NR_DECODE_EN}
- no-connect marks 0 -> 2
Other:
- note added: "TODO: - Should we add an ATX power connector?"
- note added: "TODO: check all bypass capacitors: do we have enough for everybody?"
- note added: "TODO: consider replacing '273-s with '574 ones. They seem to have a more forgiving pinout."
- note removed: "DRAM: There's one FPM DRAM from ISSI still in production: IS41LV16105D. This is a 1Mx16bit (3.3V) part but unfortunately it can't be used as such in a DDR setup. One also has to use ~{OE} to control output as ~{CAS} rising edge doesn't disable the output drivers. So each chip gives you a single 1MByte SIMM module."
- note removed: "One could also use the SIO10N268 ($10) which gives for UARTs and an FDD controller and it's in active production still. https://ww1.microchip.com/downloads/aemDocuments/documents/OTH/ProductDocuments/DataSheets/00001819A.pdf Or the FDC37C78 ($11), which is just a FDD controller and is not recommended for new designs and is not really in stock (big surprise)."
- note removed: "TODO: - Check and fix power jack and switch connectors - Add DC/DC converter to generate 5V"
- note removed: "These should be 3.3V parts to enable 3.3V DRAM modules. LVC devices with an A suffix are like that, and those still seem to come in DIP packages. So we need: SN74LVC245AN SN74AHC126N For full 3.3V conversion, 273 needs to be exchanged to 373 or even better, 574 chips. The AHC series seems to have similar properties, which is good as the SN74LVC139 is NOT available in DIP."
- note removed: "WiFi is difficult: The ESP32-based modules are cheap and available, but they really would like to see a UART interface (with an AT command set), which means very low data-rates. I think I'll punt on WiFi for now: it's wired LAN through something something Microchip."
- moved on the sheet: C1, C10, C11, C12, C13, C14, C15, C16, C17, C18, C19, C2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

Commit message: Fixed 3.3V for SDCARD; more beautification.
Other:
- company: (none) -> Modular Circuits
- title: Anachron -> Anachron uATX Main Sheet
Changed lines of the file:
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@@
   (paper "C")
   (title_block
-    (title "Anachron")
+    (title "Anachron uATX Main Sheet")
+    (date "2024-02-07")
+    (company "Modular Circuits")
   )
   (junction (at 171.45 383.54) (diameter 0) (color 0 0 0 0)

Commit message: Lots of ISA fixes and introduction of 16-bit slots.
These 16-bit slots only support 8-bit transfers, but they do so in a 16-bit
compatible fashion. 16-bit DMAs, upper IRQs and higher addresses are
not supported.

Th PCB is not yet updated and the schematic is ugly. Still the logic should be
there.
Parts:
- added J22, J23, J24: Conn_01x01, MountingHole:MountingHole_4.3mm_M4_DIN965_Pad, symbol Connector_Generic:Conn_01x01
Connections:
- net BUF_DIR: now also U7.9
- net BUF_~{EN}: now also U3.12
- net CPU_~{NREN}: no longer U3.12
- net CPU_~{WE}: no longer U7.9
- net GND: now also J22.1 (Pin_1), J23.1 (Pin_1), J24.1 (Pin_1); no longer U7.1
- net ~{RST}: now also U7.1
- net RST: now reaches U7.2
- no-connect marks 2 -> 1
Other:
- sheet ISA ports: added CPU_DACK, ISA_DACK; removed none
- note added: "We disable GFX~{BUSY} propagation to CPU_~{WAIT} when we do I/O or DMA cycles. This allows for peripherals to generate their own wait-states without the GFX chip interfering all the time. However, the control of the VRAM isolators from GFX_BUSY directly means we can't DMA into VRAM."
- note removed: "We disable GFX~{BUSY} propagation to CPU_~{WAIT} when we do I/O cycles. This allows for peripherals to generate their own wait-states without the GFX chip interfering all the time."
- moved on the sheet: J1, J2, J3, J4, R9, U7A

Commit message: A1 motherboard now has 16-bit ISA slot support.
Other:
- added sheet ISA power (isa_power.kicad_sch)

Commit message: Partially fixed GFX I/O access.
Connections:
- net +5V: no longer U3.9, U7.11
- net BUF_NREN: now also U7.10; no longer U3.8
- net BUF_~{EN}: now also U7.1; no longer U3.12
- net BUF_~{NREN}: now also U7.11; no longer U3.10
- net RST: no longer U7.2
- net ~{GFX_SEL}: now also U3.9
- net ~{RST}: no longer U7.1
- new net: U3.10, U7.2
- new net: U3.12, U3.8
Other:
- note added: "Review: Goal is to enable wait states for RAS and GFX I/O cycles."
- note added: "Review: Hopefully RST is no longer needed."
- note added: "TODO: fix on-off switch: as it is, things default to 'on'."
- moved on the sheet: U3C, U7A, U7E
Changed lines of the file:
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@@
 	(wire
 		(pts
+			(xy 104.14 114.3) (xy 115.57 114.3)
+		)
+		(stroke
+			(width 0)
+			(type default)
+		)
+	)
+	(wire
+		(pts
 			(xy 293.37 165.1) (xy 293.37 180.34)
 		)
@@
 	(wire
 		(pts
+			(xy 53.34 111.76) (xy 88.9 111.76)
+		)
+		(stroke
+			(width 0)
+			(type default)
+		)
+	)
+	(wire
+		(pts
 			(xy 463.55 52.07) (xy 477.52 52.07)
 		)
@@
 		)
 	)
+	(wire
+		(pts
+			(xy 53.34 123.19) (xy 68.58 123.19)
+		)
+		(stroke
+			(width 0)
+			(type default)
+		)
+	)
 	(bus
 		(pts
@@
 	(wire
 		(pts
+			(xy 83.82 116.84) (xy 88.9 116.84)
+		)
+		(stroke
+			(width 0)
+			(type default)
+		)
+	)
+	(wire
+		(pts
 			(xy 190.5 44.45) (xy 190.5 100.33)
 		)
@@
 	(wire
 		(pts
+			(xy 83.82 123.19) (xy 83.82 116.84)
+		)
+		(stroke
+			(width 0)
+			(type default)
+		)
+	)
+	(wire
+		(pts
 			(xy 128.27 283.21) (xy 143.51 283.21)
 		)
@@
 	(wire
 		(pts
-			(xy 115.57 121.92) (xy 115.57 96.52)
+			(xy 115.57 96.52) (xy 115.57 114.3)
 		)
 		(stroke
@@
 	(wire
 		(pts
+			(xy 328.93 361.95) (xy 328.93 370.84)
+		)
+		(stroke
+			(width 0)
+			(type default)
+		)
+	)
+	(wire
+		(pts
 			(xy 167.64 243.84) (xy 175.26 243.84)
 		)
@@
 		)
 	)
-	(wire
-		(pts
-			(xy 328.93 361.95) (xy 328.93 368.3)
-		)
-		(stroke
-			(width 0)
-			(type default)
-		)
-	)
 	(bus
 		(pts
@@
 		)
 	)
-	(wire
-		(pts
-			(xy 347.98 365.76) (xy 344.17 365.76)
-		)
-		(stroke
-			(width 0)
-			(type default)
-		)
-	)
 	(bus
 		(pts
@@
 		)
 	)
+	(text "Review: Hopefully RST is no longer needed."
+		(exclude_from_sim no)
+		(at 192.024 372.11 0)
+		(effects
+			(font
+				(size 3 3)
+				(thickness 0.6)
+				(bold yes)
+				(color 255 45 0 1)
+			)
+		)
+	)
 	(text "Data is captured on the falling edge of nWE | nCAS by the DRAM.\nThus, buffering either of those will not cause write-setup\nviolations. At the same time, read responses are delayed, but\nthat can be handled by slowing the clock down.\n\nSo, all in all, we can buffer control and address signals to\nthe DRAM without too much worry. Buffering data hopefully is\nnot necessary as there's only 4 loads on the bus.\n\nTons of DRAM datasheets: https://minuszerodegrees.net/memory/ram.htm\n\nEssentially everything supported page mode, no worries there.\n"
 		(exclude_from_sim no)
@@
 		)
 	)
+	(text "TODO: fix on-off switch: as it is, things default to 'on'."
+		(exclude_from_sim no)
+		(at 73.66 388.112 0)
+		(effects
+			(font
+				(size 3 3)
+				(thickness 0.6)
+				(bold yes)
+				(color 255 45 0 1)
+			)
+		)
+	)
 	(text "PWR LED"
 		(exclude_from_sim no)
@@
 		)
 	)
+	(text "Review: Goal is to enable wait states for RAS and GFX I/O cycles."
+		(exclude_from_sim no)
+		(at 78.74 118.364 0)
+		(effects
+			(font
+				(size 3 3)
+				(thickness 0.6)
+				(bold yes)
+				(color 255 45 0 1)
+			)
+		)
+	)
 	(text "BOOT SELECT"
 		(exclude_from_sim no)
@@
 		)
 	)
+	(label "~{GFX_SEL}"
+		(at 60.96 111.76 180)
+		(fields_autoplaced yes)
+		(effects
+			(font
+				(size 1.27 1.27)
+			)
+			(justify right bottom)
+		)
+	)
 	(label "VIDEO_DDC_SCL"
 		(at 25.4 175.26 0)
@@
 	)
 	(label "BUF_~{EN}"
-		(at 115.57 115.57 90)
+		(at 60.96 123.19 180)
 		(fields_autoplaced yes)
 		(effects
@@
 				(size 1.27 1.27)
 			)
-			(justify left bottom)
+			(justify right bottom)
 		)
 	)
@@
 	(symbol
 		(lib_id "74xx:74LS00")
-		(at 336.55 368.3 0)
-		(mirror y)
+		(at 96.52 114.3 0)
 		(unit 3)
 		(exclude_from_sim no)
@@
 		(on_board yes)
 		(dnp no)
-		(fields_autoplaced yes)
 		(property "Reference" "U3"
-			(at 336.5583 359.41 0)
+			(at 96.5117 105.41 0)
 			(effects
 				(font
@@
 		)
 		(property "Value" "74LS00"
-			(at 336.5583 361.95 0)
+			(at 96.5117 107.95 0)
 			(effects
 				(font
@@
 		)
 		(property "Footprint" "Package_DIP:DIP-14_W7.62mm_LongPads"
-			(at 336.55 368.3 0)
+			(at 96.52 114.3 0)
 			(effects
 				(font
@@
 		)
 		(property "Datasheet" "http://www.ti.com/lit/gpn/sn74ls00"
-			(at 336.55 368.3 0)
+			(at 96.52 114.3 0)
 			(effects
 				(font
@@
 		)
 		(property "Description" ""
-			(at 336.55 368.3 0)
+			(at 96.52 114.3 0)
 			(effects
 				(font
@@
 	(symbol
 		(lib_id "74xx:74LS14")
-		(at 214.63 373.38 0)
+		(at 76.2 123.19 0)
 		(unit 1)
 		(exclude_from_sim no)
@@
 		(fields_autoplaced yes)
 		(property "Reference" "U7"
-			(at 214.63 364.49 0)
+			(at 76.2 114.3 0)
 			(effects
 				(font
@@
 		)
 		(property "Value" "74LS14"
-			(at 214.63 367.03 0)
+			(at 76.2 116.84 0)
 			(effects
 				(font
@@
 		)
 		(property "Footprint" "Package_DIP:DIP-14_W7.62mm_LongPads"
-			(at 214.63 373.38 0)
+			(at 76.2 123.19 0)
 			(effects
 				(font
@@
 		)
 		(property "Datasheet" "http://www.ti.com/lit/gpn/sn74LS14"
-			(at 214.63 373.38 0)
+			(at 76.2 123.19 0)
 			(effects
 				(font
@@
 		)
 		(property "Description" ""
-			(at 214.63 373.38 0)
+			(at 76.2 123.19 0)
 			(effects
 				(font
@@
 	)
 	(symbol
-		(lib_id "power:+5V")
-		(at 347.98 365.76 0)
-		(mirror y)
-		(unit 1)
-		(exclude_from_sim no)
-		(in_bom yes)
-		(on_board yes)
-		(dnp no)
-		(fields_autoplaced yes)
-		(property "Reference" "#PWR091"
-			(at 347.98 369.57 0)
-			(effects
-				(font
-					(size 1.27 1.27)
-				)
-				(hide yes)
-			)
-		)
-		(property "Value" "+5V"
-			(at 347.98 360.68 0)
-			(effects
-				(font
-					(size 1.27 1.27)
-				)
-			)
-		)
-		(property "Footprint" ""
-			(at 347.98 365.76 0)
-			(effects
-				(font
-					(size 1.27 1.27)
-				)
-				(hide yes)
-			)
-		)
-		(property "Datasheet" ""
-			(at 347.98 365.76 0)
-			(effects
-				(font
-					(size 1.27 1.27)
-				)
-				(hide yes)
-			)
-		)
-		(property "Description" ""
-			(at 347.98 365.76 0)
-			(effects
-				(font
-					(size 1.27 1.27)
-				)
-				(hide yes)
-			)
-		)
-		(pin "1"
-		)
-		(instances
-			(project "a1_micro_atx"
-				(path "/3257e1ae-50a8-410a-87c3-a39d96a2c51a"
-					(reference "#PWR091")
-					(unit 1)
-				)
-			)
-		)
-	)
-	(symbol
 		(lib_id "Device:R_US")
 		(at 222.885 266.7 0)
@@
 	(symbol
 		(lib_id "74xx:74LS14")
-		(at 505.46 302.26 0)
+		(at 336.55 370.84 180)
 		(unit 5)
 		(exclude_from_sim no)
@@
 		(fields_autoplaced yes)
 		(property "Reference" "U7"
-			(at 505.46 293.37 0)
+			(at 336.55 361.95 0)
 			(effects
 				(font
@@
 		)
 		(property "Value" "74LS14"
-			(at 505.46 295.91 0)
+			(at 336.55 364.49 0)
 			(effects
 				(font
@@
 		)
 		(property "Footprint" "Package_DIP:DIP-14_W7.62mm_LongPads"
-			(at 505.46 302.26 0)
+			(at 336.55 370.84 0)
 			(effects
 				(font
@@
 		)
 		(property "Datasheet" "http://www.ti.com/lit/gpn/sn74LS14"
-			(at 505.46 302.26 0)
+			(at 336.55 370.84 0)
 			(effects
 				(font
@@
 		)
 		(property "Description" ""
-			(at 505.46 302.26 0)
+			(at 336.55 370.84 0)
 			(effects
 				(font

Commit message: Updated PCB to latest schematic changes.
Also removed 12V boost bypass: that option would also bypass the on-off switch; not good.
Connections:
- no-connect marks 1 -> 0
Changed lines of the file:
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@@
 		(color 0 0 0 0)
 	)
-	(no_connect
-		(at 513.08 302.26)
-	)
 	(bus_entry
 		(at 280.035 308.61)
@@
 					(unit 1)
 				)
-			)
-		)
-	)
-	(symbol
-		(lib_id "power:+5V")
-		(at 497.84 302.26 0)
-		(unit 1)
-		(exclude_from_sim no)
-		(in_bom yes)
-		(on_board yes)
-		(dnp no)
-		(fields_autoplaced yes)
-		(property "Reference" "#PWR0209"
-			(at 497.84 306.07 0)
-			(effects
-				(font
-					(size 1.27 1.27)
-				)
-				(hide yes)
-			)
-		)
-		(property "Value" "+5V"
-			(at 497.84 297.18 0)
-			(effects
-				(font
-					(size 1.27 1.27)
-				)
-			)
-		)
-		(property "Footprint" ""
-			(at 497.84 302.26 0)
-			(effects
-				(font
-					(size 1.27 1.27)
-				)
-				(hide yes)
-			)
-		)
-		(property "Datasheet" ""
-			(at 497.84 302.26 0)
-			(effects
-				(font
-					(size 1.27 1.27)
-				)
-				(hide yes)
-			)
-		)
-		(property "Description" ""
-			(at 497.84 302.26 0)
-			(effects
-				(font
-					(size 1.27 1.27)
-				)
-				(hide yes)
-			)
-		)
-		(pin "1"
-		)
-		(instances
-			(project "a1_micro_atx"
-				(path "/3257e1ae-50a8-410a-87c3-a39d96a2c51a"
-					(reference "#PWR0209")
-					(unit 1)
-				)

Commit message: Added ATX-style power button.
This also involves a management ATTiny because discrete logic just simply doesn't fit.

Power can be turned-off by I2C transactions and by press-and-hold the power SW.
The power switch can also generate an interrupt. Finally, the MCU monitors ~RST
so it can ignore I2C transactions when their pull-ups are inactive due to lack of power.
Parts:
- removed J7: Conn_01x02, Connector_PinHeader_2.54mm:PinHeader_1x02_P2.54mm_Vertical, symbol Connector_Generic:Conn_01x02
- removed SW1: SW_DPDT_x2, Button_Switch_THT:SW_CuK_JS202011CQN_DPDT_Straight, symbol Switch:SW_DPDT_x2
- added C72, C73: 1uF, Capacitor_THT:C_Disc_D4.7mm_W2.5mm_P5.00mm, symbol Device:C
- added R36: 10k, Resistor_THT:R_Axial_DIN0204_L3.6mm_D1.6mm_P5.08mm_Horizontal, symbol Device:R_US
- added SW4: SW_Push, Connector_PinHeader_2.54mm:PinHeader_1x02_P2.54mm_Vertical, symbol Switch:SW_Push
- added SW5: SW_Push, Button_Switch_THT:SW_PUSH_6mm, symbol Switch:SW_Push
- added U40: L78L05_TO92, Package_TO_SOT_THT:TO-92_Inline, symbol Regulator_Linear:L78L05_TO92
- added U43: ATtiny25-20P, Package_DIP:DIP-8_W7.62mm_LongPads, symbol MCU_Microchip_ATtiny:ATtiny25-20P
Connections:
- net GND: now also R6.1, C72.2, C73.2, SW4.1, SW5.1, U40.2 (GND), U43.4 (GND)
- net I2C_SCL: now also U43.7 (PB2)
- net I2C_SDA: now also U43.5 (AREF/PB0)
- net PWR_IN: now also C72.1, U40.3 (VI); no longer R6.1
- net PWR_ON: now reaches R6.2, U12.9 (EN)
- net PWR_ON: now also U43.2 (XTAL1/PB3)
- new net: R36.2, SW4.2, SW5.2, U43.1 (~{RESET}/PB5)
- new net +5V_STB: C73.1, R36.1, U40.1 (VO), U43.8 (VCC)
- new net I2C_~{INT}: U43.6 (PB1)
Other:
- sheet MIO ports: added I2C_~{INT}; removed none
- note added: "POWER BTN"
- note removed: "Review: Hopefully RST is no longer needed."
- note removed: "TODO: - Should we add an ATX power connector?"
- note removed: "TODO: fix on-off switch: as it is, things default to 'on'."
- moved on the sheet: R6

Commit message: Missed a file...
Connections:
- net ~{RST}: now also U43.3 (XTAL2/PB4)
- net PG: now reaches JP1.1 (A), U12.12 (PG)
Other:
- moved on the sheet: C72, C73, J1, J2, J22, J23, J24, J3, J4, JP1, R36, SW4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
