File: boards/a1_micro_atx/a1_micro_atx.kicad_sch (KiCad schematic)
At the start: 75 parts, among them J1 Conn_01x01, J2 Conn_01x01, J22 Conn_01x01, J23 Conn_01x01, J24 Conn_01x01, J3 Conn_01x01, J4 Conn_01x01, J5 Conn_01x02, J6 Jack-DC, SW2 SW_Push, SW3 SW_Push, SW4 SW_Push, SW5 SW_Push, U1 74LS08, U10 74AHCT245, U11 SST39SF040, U12 A1_POWER, U13 74AHCT245, U14 74AHCT245, U15 74AHCT245, U16 74LS273, U17 74LS273, U18 74LS273, U2 74LS86, U3 74LS00, U4 74LS273, U40 L78L05_TO92, U43 ATtiny25-20P, U5 74LS574, U6 74LS139, U7 74LS14, U8 74LS126, U9 74AHCT245, X1 8MHz

Commit message: Added reverse-power protection to HDMI; small cleanup
- Reverse-current protection on HDMI (via simple diode)
- Cleaned up diff-pair annotation on schematic
- Added proper 3D shape for AT connector
Other:
- note added: "For ~{DACK} cycles: ~{WAIT} is not driven; GFX_~{BUSY} must be high."
- note added: "For ~{GFX_SEL} cycles: ~{WAIT} is driven; GFX_~{BUSY} must be high."
- note added: "For ~{NRAM} cycles: ~{WAIT} is not driven; GFX_~{BUSY} must be high."
- note added: "For ~{RAS_x} cycles: ~{WAIT} is driven"
- note added: "We disable GFX~{BUSY} propagation to CPU_~{WAIT} when we do I/O or DMA cycles. This allows for peripherals to generate their own wait-states without the GFX chip interfering all the time."
- note removed: "Review: Goal is to enable wait states for RAS and GFX I/O cycles."
- note removed: "We disable GFX~{BUSY} propagation to CPU_~{WAIT} when we do I/O or DMA cycles. This allows for peripherals to generate their own wait-states without the GFX chip interfering all the time. However, the control of the VRAM isolators from GFX_BUSY directly means we can't DMA into VRAM."
Changed lines of the file:
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@@
+		)
+	)
+	(text "For ~{GFX_SEL} cycles: ~{WAIT} is driven; GFX_~{BUSY} must be high."
+		(exclude_from_sim no)
+		(at 15.24 104.14 0)
+		(effects
+			(font
+				(size 1.27 1.27)
+			)
+			(justify left)
+		)
+	)
+	(text "For ~{NRAM} cycles: ~{WAIT} is not driven; GFX_~{BUSY} must be high."
+		(exclude_from_sim no)
+		(at 15.24 101.6 0)
+		(effects
+			(font
+				(size 1.27 1.27)
+			)
+			(justify left)
 		)
 	)
@@
 		)
 	)
+	(text "For ~{RAS_x} cycles: ~{WAIT} is driven"
+		(exclude_from_sim no)
+		(at 15.24 106.68 0)
+		(effects
+			(font
+				(size 1.27 1.27)
+			)
+			(justify left)
+		)
+	)
 	(text "ACTIVITY\nLED"
 		(exclude_from_sim no)
@@
 		)
 	)
-	(text "We disable GFX~{BUSY} propagation to CPU_~{WAIT}\nwhen we do I/O or DMA cycles. This allows for\nperipherals to generate their own wait-states\nwithout the GFX chip interfering all the time.\nHowever, the control of the VRAM isolators from\nGFX_BUSY directly means we can't DMA into VRAM."
+	(text "We disable GFX~{BUSY} propagation to CPU_~{WAIT}\nwhen we do I/O or DMA cycles. This allows for\nperipherals to generate their own wait-states\nwithout the GFX chip interfering all the time.\n"
 		(exclude_from_sim no)
 		(at 55.88 93.98 0)
@@
 		)
 	)
-	(text "Review: Goal is to enable wait states for RAS and GFX I/O cycles."
+	(text "For ~{DACK} cycles: ~{WAIT} is not driven; GFX_~{BUSY} must be high."
 		(exclude_from_sim no)
-		(at 78.74 118.364 0)
+		(at 15.24 99.06 0)
 		(effects
 			(font
-				(size 3 3)
-				(thickness 0.6)
-				(bold yes)
-				(color 255 45 0 1)
+				(size 1.27 1.27)
 			)
+			(justify left)
 		)
 	)
