File: boards/a1_micro_atx/a1_micro_atx.kicad_sch (KiCad schematic)
At the start: 75 parts, among them J1 Conn_01x01, J2 Conn_01x01, J22 Conn_01x01, J23 Conn_01x01, J24 Conn_01x01, J3 Conn_01x01, J4 Conn_01x01, J5 Conn_01x02, J6 Jack-DC, SW2 SW_Push, SW3 SW_Push, SW4 SW_Push, SW5 SW_Push, U1 74LS08, U10 74AHCT245, U11 SST39SF040, U12 A1_POWER, U13 74AHCT245, U14 74AHCT245, U15 74AHCT245, U16 74LS273, U17 74LS273, U18 74LS273, U2 74LS86, U3 74LS00, U4 74LS273, U40 L78L05_TO92, U43 ATtiny25-20P, U5 74LS574, U6 74LS139, U7 74LS14, U8 74LS126, U9 74AHCT245, X1 8MHz

Commit message: Small fixes and improvements
- Speaker connector is now PC-compatible
- Added internal USB connector for the 7th USB port
- If MCU is not programmed, power defaults to ON
Connections:
- net +5V_STB: now also R6.1
- net GND: no longer R6.1
Other:
- moved on the sheet: R6
Changed lines of the file:
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@@
 	)
 	(junction
+		(at 519.43 290.83)
+		(diameter 0)
+		(color 0 0 0 0)
+	)
+	(junction
 		(at 69.85 373.38)
 		(diameter 0)
@@
 	)
 	(junction
-		(at 58.42 381)
-		(diameter 0)
-		(color 0 0 0 0)
-	)
-	(junction
 		(at 138.43 190.5)
 		(diameter 0)
@@
 	(wire
 		(pts
-			(xy 58.42 396.24) (xy 58.42 397.51)
-		)
-		(stroke
-			(width 0)
-			(type default)
-		)
-	)
-	(wire
-		(pts
 			(xy 151.13 85.09) (xy 151.13 100.33)
 		)
@@
 	(wire
 		(pts
+			(xy 514.35 300.99) (xy 514.35 314.96)
+		)
+		(stroke
+			(width 0)
+			(type default)
+		)
+	)
+	(wire
+		(pts
 			(xy 21.59 182.88) (xy 41.91 182.88)
 		)
@@
 	(wire
 		(pts
-			(xy 45.72 381) (xy 58.42 381)
+			(xy 45.72 381) (xy 69.85 381)
 		)
 		(stroke
@@
 	(wire
 		(pts
+			(xy 519.43 290.83) (xy 519.43 293.37)
+		)
+		(stroke
+			(width 0)
+			(type default)
+		)
+	)
+	(wire
+		(pts
 			(xy 128.27 317.5) (xy 143.51 317.5)
 		)
@@
 	(wire
 		(pts
+			(xy 519.43 288.29) (xy 519.43 290.83)
+		)
+		(stroke
+			(width 0)
+			(type default)
+		)
+	)
+	(wire
+		(pts
 			(xy 106.68 74.93) (xy 106.68 77.47)
 		)
@@
 		)
 	)
-	(bus
+	(wire
 		(pts
-			(xy 455.93 209.55) (xy 455.93 212.09)
+			(xy 514.35 293.37) (xy 514.35 290.83)
 		)
 		(stroke
@@
 	(bus
 		(pts
-			(xy 250.19 149.86) (xy 247.65 149.86)
+			(xy 455.93 209.55) (xy 455.93 212.09)
 		)
 		(stroke
@@
 	(bus
 		(pts
-			(xy 365.76 261.62) (xy 365.76 264.16)
+			(xy 250.19 149.86) (xy 247.65 149.86)
 		)
 		(stroke
@@
 	(bus
 		(pts
-			(xy 463.55 123.19) (xy 463.55 125.73)
+			(xy 365.76 261.62) (xy 365.76 264.16)
 		)
 		(stroke
@@
 	(bus
 		(pts
-			(xy 280.035 256.54) (xy 280.035 259.08)
+			(xy 463.55 123.19) (xy 463.55 125.73)
 		)
 		(stroke
@@
 		)
 	)
-	(wire
+	(bus
 		(pts
-			(xy 287.02 292.1) (xy 316.23 292.1)
+			(xy 280.035 256.54) (xy 280.035 259.08)
 		)
 		(stroke
@@
 	(wire
 		(pts
-			(xy 58.42 381) (xy 58.42 388.62)
+			(xy 287.02 292.1) (xy 316.23 292.1)
 		)
 		(stroke
@@
 	(wire
 		(pts
-			(xy 496.57 314.96) (xy 511.81 314.96)
+			(xy 496.57 314.96) (xy 514.35 314.96)
 		)
 		(stroke
@@
 	(wire
 		(pts
-			(xy 58.42 381) (xy 69.85 381)
-		)
-		(stroke
-			(width 0)
-			(type default)
-		)
-	)
-	(wire
-		(pts
 			(xy 228.6 306.07) (xy 193.04 306.07)
 		)
@@
 	(wire
 		(pts
+			(xy 514.35 290.83) (xy 519.43 290.83)
+		)
+		(stroke
+			(width 0)
+			(type default)
+		)
+	)
+	(wire
+		(pts
 			(xy 322.58 54.61) (xy 334.01 54.61)
 		)
@@
 	(symbol
 		(lib_id "Device:R_US")
-		(at 58.42 392.43 180)
+		(at 514.35 297.18 0)
 		(unit 1)
 		(exclude_from_sim no)
@@
 		(dnp no)
 		(property "Reference" "R6"
-			(at 60.96 391.16 90)
+			(at 511.81 298.45 90)
 			(effects
 				(font
@@
 		)
 		(property "Value" "10k"
-			(at 55.88 391.16 90)
+			(at 516.89 298.45 90)
 			(effects
 				(font
@@
 		)
 		(property "Footprint" "Resistor_THT:R_Axial_DIN0204_L3.6mm_D1.6mm_P5.08mm_Horizontal"
-			(at 57.404 392.176 90)
+			(at 515.366 297.434 90)
 			(effects
 				(font
@@
 		)
 		(property "Datasheet" "~"
-			(at 58.42 392.43 0)
+			(at 514.35 297.18 0)
 			(effects
 				(font
@@
 		)
 		(property "Description" ""
-			(at 58.42 392.43 0)
+			(at 514.35 297.18 0)
 			(effects
 				(font
@@
 	(symbol
 		(lib_id "power:+5VL")
-		(at 519.43 293.37 0)
+		(at 519.43 288.29 0)
 		(mirror y)
 		(unit 1)
@@
 		(fields_autoplaced yes)
 		(property "Reference" "#PWR0280"
-			(at 519.43 297.18 0)
+			(at 519.43 292.1 0)
 			(effects
 				(font
@@
 		)
 		(property "Value" "+5V_STB"
-			(at 519.43 288.29 0)
+			(at 519.43 283.21 0)
 			(effects
 				(font
@@
 		)
 		(property "Footprint" ""
-			(at 519.43 293.37 0)
+			(at 519.43 288.29 0)
 			(effects
 				(font
@@
 		)
 		(property "Datasheet" ""
-			(at 519.43 293.37 0)
+			(at 519.43 288.29 0)
 			(effects
 				(font
@@
 		)
 		(property "Description" "Power symbol creates a global label with name \"+5V_STB\""
-			(at 519.43 293.37 0)
+			(at 519.43 288.29 0)
 			(effects
 				(font
@@
 					(unit 1)
 				)
-			)
-		)
-	)
-	(symbol
-		(lib_id "power:GND")
-		(at 58.42 397.51 0)
-		(unit 1)
-		(exclude_from_sim no)
-		(in_bom yes)
-		(on_board yes)
-		(dnp no)
-		(fields_autoplaced yes)
-		(property "Reference" "#PWR048"
-			(at 58.42 403.86 0)
-			(effects
-				(font
-					(size 1.27 1.27)
-				)
-				(hide yes)
-			)
-		)
-		(property "Value" "GND"
-			(at 58.42 402.59 0)
-			(effects
-				(font
-					(size 1.27 1.27)
-				)
-			)
-		)
-		(property "Footprint" ""
-			(at 58.42 397.51 0)
-			(effects
-				(font
-					(size 1.27 1.27)
-				)
-				(hide yes)
-			)
-		)
-		(property "Datasheet" ""
-			(at 58.42 397.51 0)
-			(effects
-				(font
-					(size 1.27 1.27)
-				)
-				(hide yes)
-			)
-		)
-		(property "Description" ""
-			(at 58.42 397.51 0)
-			(effects
-				(font
-					(size 1.27 1.27)
-				)
-				(hide yes)
-			)
-		)
-		(pin "1"
-		)
-		(instances
-			(project "a1_micro_atx"
-				(path "/3257e1ae-50a8-410a-87c3-a39d96a2c51a"
-					(reference "#PWR048")
-					(unit 1)
-				)

Commit message: Reversed default power-on.
The problem with defaulting to power-on-by-default is that there is a short
on transient while the MCU is booting and gets to override the pull-up. This
is mitigated now by a pull-down and an override jumper. The existence of the
jumper now necessitates an open-emitter drive from the MCU; that is, drive-high
for ON and float for OFF.
Parts:
- added JP6: Jumper_2_Bridged, Connector_PinHeader_2.54mm:PinHeader_1x02_P2.54mm_Vertical, symbol Jumper:Jumper_2_Open
Connections:
- net +5V_STB: now also JP6.2 (B); no longer R6.1
- net GND: now also R6.2
- net PWR_ON: now also R6.1, JP6.1 (A); no longer R6.2
Other:
- moved on the sheet: R6
Changed lines of the file:
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@@
 	)
 	(junction
+		(at 55.88 381)
+		(diameter 0)
+		(color 0 0 0 0)
+	)
+	(junction
 		(at 171.45 383.54)
 		(diameter 0)
@@
 	(wire
 		(pts
+			(xy 55.88 381) (xy 69.85 381)
+		)
+		(stroke
+			(width 0)
+			(type default)
+		)
+	)
+	(wire
+		(pts
 			(xy 250.19 85.09) (xy 250.19 100.33)
 		)
@@
 	(wire
 		(pts
-			(xy 514.35 300.99) (xy 514.35 314.96)
-		)
-		(stroke
-			(width 0)
-			(type default)
-		)
-	)
-	(wire
-		(pts
 			(xy 21.59 182.88) (xy 41.91 182.88)
 		)
@@
 	(wire
 		(pts
-			(xy 45.72 381) (xy 69.85 381)
+			(xy 45.72 381) (xy 55.88 381)
 		)
 		(stroke
@@
 		)
 	)
-	(wire
-		(pts
-			(xy 514.35 293.37) (xy 514.35 290.83)
-		)
-		(stroke
-			(width 0)
-			(type default)
-		)
-	)
 	(bus
 		(pts
@@
 		)
 	)
+	(wire
+		(pts
+			(xy 55.88 381) (xy 55.88 388.62)
+		)
+		(stroke
+			(width 0)
+			(type default)
+		)
+	)
 	(bus
 		(pts
@@
 		)
 	)
+	(wire
+		(pts
+			(xy 55.88 396.24) (xy 55.88 397.51)
+		)
+		(stroke
+			(width 0)
+			(type default)
+		)
+	)
 	(bus
 		(pts
@@
 	(wire
 		(pts
+			(xy 514.35 300.99) (xy 514.35 314.96)
+		)
+		(stroke
+			(width 0)
+			(type default)
+		)
+	)
+	(wire
+		(pts
 			(xy 195.58 308.61) (xy 195.58 322.58)
 		)
@@
 	)
 	(symbol
+		(lib_id "power:GND")
+		(at 55.88 397.51 0)
+		(unit 1)
+		(exclude_from_sim no)
+		(in_bom yes)
+		(on_board yes)
+		(dnp no)
+		(fields_autoplaced yes)
+		(property "Reference" "#PWR048"
+			(at 55.88 403.86 0)
+			(effects
+				(font
+					(size 1.27 1.27)
+				)
+				(hide yes)
+			)
+		)
+		(property "Value" "GND"
+			(at 55.88 402.59 0)
+			(effects
+				(font
+					(size 1.27 1.27)
+				)
+			)
+		)
+		(property "Footprint" ""
+			(at 55.88 397.51 0)
+			(effects
+				(font
+					(size 1.27 1.27)
+				)
+				(hide yes)
+			)
+		)
+		(property "Datasheet" ""
+			(at 55.88 397.51 0)
+			(effects
+				(font
+					(size 1.27 1.27)
+				)
+				(hide yes)
+			)
+		)
+		(property "Description" ""
+			(at 55.88 397.51 0)
+			(effects
+				(font
+					(size 1.27 1.27)
+				)
+				(hide yes)
+			)
+		)
+		(pin "1"
+		)
+		(instances
+			(project "a1_micro_atx"
+				(path "/3257e1ae-50a8-410a-87c3-a39d96a2c51a"
+					(reference "#PWR048")
+					(unit 1)
+				)
+			)
+		)
+	)
+	(symbol
 		(lib_id "74xx:74LS14")
 		(at 265.43 86.36 270)
@@
 	(symbol
 		(lib_id "Device:R_US")
-		(at 514.35 297.18 0)
+		(at 55.88 392.43 0)
 		(unit 1)
 		(exclude_from_sim no)
@@
 		(dnp no)
 		(property "Reference" "R6"
-			(at 511.81 298.45 90)
+			(at 53.34 393.7 90)
 			(effects
 				(font
@@
 		)
 		(property "Value" "10k"
-			(at 516.89 298.45 90)
+			(at 58.42 393.7 90)
 			(effects
 				(font
@@
 		)
 		(property "Footprint" "Resistor_THT:R_Axial_DIN0204_L3.6mm_D1.6mm_P5.08mm_Horizontal"
-			(at 515.366 297.434 90)
+			(at 56.896 392.684 90)
 			(effects
 				(font
@@
 		)
 		(property "Datasheet" "~"
-			(at 514.35 297.18 0)
+			(at 55.88 392.43 0)
 			(effects
 				(font
@@
 		)
 		(property "Description" ""
-			(at 514.35 297.18 0)
+			(at 55.88 392.43 0)
 			(effects
 				(font
@@
 				)
 			)
+		)
+	)
+	(symbol
+		(lib_id "Jumper:Jumper_2_Open")
+		(at 514.35 295.91 90)
+		(unit 1)
+		(exclude_from_sim no)
+		(in_bom yes)
+		(on_board yes)
+		(dnp no)
+		(property "Reference" "JP6"
+			(at 508 294.64 90)
+			(effects
+				(font
+					(size 1.27 1.27)
+				)
+				(justify right)
+			)
+		)
+		(property "Value" "Jumper_2_Bridged"
+			(at 494.03 297.18 90)
+			(effects
+				(font
+					(size 1.27 1.27)
+				)
+				(justify right)
+			)
+		)
+		(property "Footprint" "Connector_PinHeader_2.54mm:PinHeader_1x02_P2.54mm_Vertical"
+			(at 514.35 295.91 0)
+			(effects
+				(font
+					(size 1.27 1.27)
+				)
+				(hide yes)
+			)
+		)
+		(property "Datasheet" "~"
+			(at 514.35 295.91 0)
+			(effects
+				(font
+					(size 1.27 1.27)
+				)
+				(hide yes)
+			)
+		)
+		(property "Description" ""
+			(at 514.35 295.91 0)
+			(effects
+				(font
+					(size 1.27 1.27)
+				)
+				(hide yes)
+			)
+		)
+		(pin "2"
+		)
+		(pin "1"
+		)
+		(instances
+			(project "a1_micro_atx"
+				(path "/3257e1ae-50a8-410a-87c3-a39d96a2c51a"
+					(reference "JP6")
+					(unit 1)
+				)
+			)
