File: boards/a1_micro_atx/ethernet.kicad_sch (KiCad schematic)
At the start: 15 parts, among them U27 KSZ8851-11MLL, Y2 25MHz

Commit message: Major schematic beautification.
Other:
- moved on the sheet: C39, C40, C41, C42, C43, J14, R22, R23, R24, R25, R26, R27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

Commit message: Fixed 3.3V for SDCARD; more beautification.
Other:
- company: (none) -> Modular Circuits
- title: (none) -> Anachron uATX Ethernet Interface
Changed lines of the file:
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@@
 (kicad_sch (version 20230121) (generator eeschema)
   (paper "A")
+  (title_block
+    (title "Anachron uATX Ethernet Interface")
+    (date "2024-02-07")
+    (company "Modular Circuits")
+  )
   (junction (at 186.69 99.06) (diameter 0) (color 0 0 0 0)
   )
