File: boards/a1_micro_atx/mio.kicad_sch (KiCad schematic)
At the start: 27 parts, among them J12 DE9_Plug, J13 Micro_SD_Card, U24 MAX232, U25 MIO, U26 DS1307+, X3 24MHz, Y1 32768Hz

Commit message: Major schematic beautification.
Other:
- note added: "One could use the SIO10N268 ($10) which gives four UARTs and an FDD controller and it's in active production still. https://ww1.microchip.com/downloads/aemDocuments/documents/OTH/ProductDocuments/DataSheets/00001819A.pdf"
- note removed: "DRQ signals must be open-SOURCE and DACK must be ignored when DRQ is not active!!!"

Commit message: Fixed 3.3V for SDCARD; more beautification.
Parts:
- added C66, C67: 1uF, Capacitor_THT:C_Disc_D4.7mm_W2.5mm_P5.00mm, symbol Device:C
- added U29: L78L33ABZ-AP, Package_TO_SOT_THT:TO-92_Inline, symbol Regulator_Linear:L78L05_TO92
Connections:
- net +5V: now also C66.1, U29.3 (VI); no longer J13.4 (VDD), R20.2, RN8.1 (common), RN9.1 (common)
- net GND: now also C66.2, C67.2, U29.2 (GND)
- new net VCC_SD: C67.1, J13.4 (VDD), R20.2, RN8.1 (common), RN9.1 (common), U29.1 (VO)
Other:
- note removed: "TODO: SD-card pull-ups should go to 3.3V!!!!!!"
- company: (none) -> Modular Circuits
- title: Anachron Main I/O Interfaces -> Anachron uATX Main I/O Interfaces
- moved on the sheet: BT1, C36, C37, C38, J13, R20, R21, RN7, RN8, RN9, U25, U26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

Commit message: Added ATX-style power button.
This also involves a management ATTiny because discrete logic just simply doesn't fit.

Power can be turned-off by I2C transactions and by press-and-hold the power SW.
The power switch can also generate an interrupt. Finally, the MCU monitors ~RST
so it can ignore I2C transactions when their pull-ups are inactive due to lack of power.
Connections:
- net ~{RTC_INT} renamed I2C_~{INT}
Changed lines of the file:
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@@
 	(wire
 		(pts
-			(xy 109.22 91.44) (xy 124.46 91.44)
+			(xy 109.22 91.44) (xy 135.89 91.44)
 		)
 		(stroke
@@
 		(fields_autoplaced yes)
 		(effects
+			(font
+				(size 1.27 1.27)
+			)
+			(justify left)
+		)
+	)
+	(hierarchical_label "I2C_~{INT}"
+		(shape input)
+		(at 135.89 91.44 0)
+		(fields_autoplaced yes)
+		(effects

Commit message: Added reverse-power protection to HDMI; small cleanup
- Reverse-current protection on HDMI (via simple diode)
- Cleaned up diff-pair annotation on schematic
- Added proper 3D shape for AT connector
Changed lines of the file:
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@@
 	)
 	(label "USB_D+"
-		(at 114.3 101.6 0)
+		(at 116.84 101.6 0)
 		(fields_autoplaced yes)
 		(effects
@@
 	)
 	(label "USB_D-"
-		(at 114.3 104.14 0)
+		(at 116.84 104.14 0)
 		(fields_autoplaced yes)
 		(effects
@@
 	)
 	(netclass_flag ""
-		(length 2.54)
+		(length 1.27)
 		(shape round)
-		(at 114.3 104.14 0)
+		(at 110.49 104.14 0)
 		(fields_autoplaced yes)
 		(effects
@@
 		)
 		(property "Netclass" "USB"
-			(at 114.9985 101.6 0)
+			(at 111.1885 102.87 0)
 			(effects
 				(font
@@
 	)
 	(netclass_flag ""
-		(length 2.54)
+		(length 1.27)
 		(shape round)
-		(at 111.76 101.6 0)
+		(at 110.49 101.6 0)
 		(fields_autoplaced yes)
 		(effects
@@
 		)
 		(property "Netclass" "USB"
-			(at 112.4585 99.06 0)
+			(at 111.1885 100.33 0)
 			(effects
 				(font
