File: boards/a1_micro_atx/graphics.kicad_sch (KiCad schematic)
At the start: 40 parts, among them J10 HDMI_A, J11 SJ1-3535NG-BE, J8 SJ1-3535NG-BE, J9 Conn_01x02, U22 DISCO, U23 A1_CODEC, X2 CXO_DIP14

Commit message: Fixed 3.3V for SDCARD; more beautification.
Other:
- company: (none) -> Modular Circuits
- title: Anachron Graphics and Audio -> Anachron uATX Graphics and Audio
Changed lines of the file:
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@@
   (paper "A")
   (title_block
-    (title "Anachron Graphics and Audio")
+    (title "Anachron uATX Graphics and Audio")
+    (date "2024-02-07")
+    (company "Modular Circuits")
   )
   (junction (at 246.38 109.22) (diameter 0) (color 0 0 0 0)

Commit message: Added reverse-power protection to HDMI; small cleanup
- Reverse-current protection on HDMI (via simple diode)
- Cleaned up diff-pair annotation on schematic
- Added proper 3D shape for AT connector
Parts:
- added D6: 1N5817, Diode_THT:D_DO-41_SOD81_P10.16mm_Horizontal, symbol Diode:1N5817
Connections:
- net +5V: now also D6.2 (A); no longer F1.2
- new net: D6.1 (K), F1.2
Changed lines of the file:
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@@
+	(wire
+		(pts
+			(xy 238.76 31.75) (xy 238.76 34.29)
+		)
+		(stroke
+			(width 0)
+			(type default)
+		)
+	)
 	(wire
 		(pts
@@
 	(wire
 		(pts
-			(xy 238.76 30.48) (xy 238.76 34.29)
+			(xy 238.76 21.59) (xy 238.76 24.13)
 		)
 		(stroke
@@
 	)
 	(netclass_flag ""
-		(length 2.54)
+		(length 1.27)
 		(shape round)
-		(at 165.1 60.96 0)
+		(at 158.75 60.96 0)
 		(fields_autoplaced yes)
 		(effects
@@
 		)
 		(property "Netclass" "HDMI"
-			(at 165.7985 58.42 0)
+			(at 159.4485 59.69 0)
 			(effects
 				(font
@@
 	)
 	(netclass_flag ""
-		(length 2.54)
+		(length 1.27)
 		(shape round)
-		(at 165.1 66.04 0)
+		(at 158.75 66.04 0)
 		(fields_autoplaced yes)
 		(effects
@@
 		)
 		(property "Netclass" "HDMI"
-			(at 165.7985 63.5 0)
+			(at 159.4485 64.77 0)
 			(effects
 				(font
@@
 	)
 	(netclass_flag ""
-		(length 2.54)
+		(length 1.27)
 		(shape round)
 		(at 158.75 76.2 0)
@@
 		)
 		(property "Netclass" "HDMI"
-			(at 159.4485 73.66 0)
+			(at 159.4485 74.93 0)
 			(effects
 				(font
@@
 	)
 	(netclass_flag ""
-		(length 2.54)
+		(length 1.27)
 		(shape round)
-		(at 165.1 71.12 0)
+		(at 158.75 71.12 0)
 		(fields_autoplaced yes)
 		(effects
@@
 		)
 		(property "Netclass" "HDMI"
-			(at 165.7985 68.58 0)
+			(at 159.4485 69.85 0)
 			(effects
 				(font
@@
 	)
 	(netclass_flag ""
-		(length 2.54)
+		(length 1.27)
 		(shape round)
 		(at 158.75 68.58 0)
@@
 		)
 		(property "Netclass" "HDMI"
-			(at 159.4485 66.04 0)
+			(at 159.4485 67.31 0)
 			(effects
 				(font
@@
 	)
 	(netclass_flag ""
-		(length 2.54)
+		(length 1.27)
 		(shape round)
 		(at 158.75 63.5 0)
@@
 		)
 		(property "Netclass" "HDMI"
-			(at 159.4485 60.96 0)
+			(at 159.4485 62.23 0)
 			(effects
 				(font
@@
 	)
 	(netclass_flag ""
-		(length 2.54)
+		(length 1.27)
 		(shape round)
 		(at 158.75 58.42 0)
@@
 		)
 		(property "Netclass" "HDMI"
-			(at 159.4485 55.88 0)
+			(at 159.4485 57.15 0)
 			(effects
 				(font
@@
 	)
 	(netclass_flag ""
-		(length 2.54)
+		(length 1.27)
 		(shape round)
-		(at 165.1 78.74 0)
+		(at 158.75 78.74 0)
 		(fields_autoplaced yes)
 		(effects
@@
 		)
 		(property "Netclass" "HDMI"
-			(at 165.7985 76.2 0)
+			(at 159.4485 77.47 0)
 			(effects
 				(font
@@
 	(symbol
 		(lib_id "power:+5V")
-		(at 238.76 30.48 0)
+		(at 238.76 21.59 0)
 		(unit 1)
 		(exclude_from_sim no)
@@
 		(fields_autoplaced yes)
 		(property "Reference" "#PWR0150"
-			(at 238.76 34.29 0)
+			(at 238.76 25.4 0)
 			(effects
 				(font
@@
 		)
 		(property "Value" "+5V"
-			(at 238.76 25.4 0)
+			(at 238.76 16.51 0)
 			(effects
 				(font
@@
 		)
 		(property "Footprint" ""
-			(at 238.76 30.48 0)
+			(at 238.76 21.59 0)
 			(effects
 				(font
@@
 		)
 		(property "Datasheet" ""
-			(at 238.76 30.48 0)
+			(at 238.76 21.59 0)
 			(effects
 				(font
@@
 		)
 		(property "Description" ""
-			(at 238.76 30.48 0)
+			(at 238.76 21.59 0)
 			(effects
 				(font
@@
 					(unit 1)
 				)
+			)
+		)
+	)
+	(symbol
+		(lib_id "Diode:1N5817")
+		(at 238.76 27.94 90)
+		(unit 1)
+		(exclude_from_sim no)
+		(in_bom yes)
+		(on_board yes)
+		(dnp no)
+		(fields_autoplaced yes)
+		(property "Reference" "D6"
+			(at 241.3 26.9874 90)
+			(effects
+				(font
+					(size 1.27 1.27)
+				)
+				(justify right)
+			)
+		)
+		(property "Value" "1N5817"
+			(at 241.3 29.5274 90)
+			(effects
+				(font
+					(size 1.27 1.27)
+				)
+				(justify right)
+			)
+		)
+		(property "Footprint" "Diode_THT:D_DO-41_SOD81_P10.16mm_Horizontal"
+			(at 243.205 27.94 0)
+			(effects
+				(font
+					(size 1.27 1.27)
+				)
+				(hide yes)
+			)
+		)
+		(property "Datasheet" "http://www.vishay.com/docs/88525/1n5817.pdf"
+			(at 238.76 27.94 0)
+			(effects
+				(font
+					(size 1.27 1.27)
+				)
+				(hide yes)
+			)
+		)
+		(property "Description" "20V 1A Schottky Barrier Rectifier Diode, DO-41"
+			(at 238.76 27.94 0)
+			(effects
+				(font
+					(size 1.27 1.27)
+				)
+				(hide yes)
+			)
+		)
+		(pin "1"
+		)
+		(pin "2"
+		)
+		(instances
+			(project "a1_micro_atx"
+				(path "/3257e1ae-50a8-410a-87c3-a39d96a2c51a/ca3554d2-b22b-4135-824b-57937af5503f"
+					(reference "D6")
+					(unit 1)
+				)

Commit message: Small fixes and improvements
- Speaker connector is now PC-compatible
- Added internal USB connector for the 7th USB port
- If MCU is not programmed, power defaults to ON
Parts:
- J9: footprint Connector_PinHeader_2.54mm:PinHeader_1x02_P2.54mm_Vertical -> Connector_PinHeader_2.54mm:PinHeader_1x04_P2.54mm_Vertical; symbol Connector_Generic:Conn_01x02 -> Connector_Generic:Conn_01x04
Connections:
- net at U23.11 (RSPKOUT): now also J9.3 (Pin_3), J9.4 (Pin_4); no longer J9.2 (Pin_2)
- net at J9.1 (Pin_1), U23.12 (LSPKOUT): now also J9.2 (Pin_2)
Changed lines of the file:
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@@
 	)
 	(junction
+		(at 158.75 130.81)
+		(diameter 0)
+		(color 0 0 0 0)
+	)
+	(junction
 		(at 91.44 179.07)
 		(diameter 0)
@@
 	)
 	(junction
+		(at 158.75 128.27)
+		(diameter 0)
+		(color 0 0 0 0)
+	)
+	(junction
 		(at 139.7 114.3)
 		(diameter 0)
@@
 	(wire
 		(pts
+			(xy 158.75 130.81) (xy 158.75 133.35)
+		)
+		(stroke
+			(width 0)
+			(type default)
+		)
+	)
+	(wire
+		(pts
 			(xy 154.94 114.3) (xy 154.94 115.57)
 		)
@@
 	(wire
 		(pts
-			(xy 154.94 128.27) (xy 147.32 128.27)
+			(xy 161.29 128.27) (xy 158.75 128.27)
 		)
 		(stroke
@@
 	(wire
 		(pts
-			(xy 154.94 130.81) (xy 147.32 130.81)
+			(xy 161.29 130.81) (xy 158.75 130.81)
+		)
+		(stroke
+			(width 0)
+			(type default)
+		)
+	)
+	(wire
+		(pts
+			(xy 158.75 128.27) (xy 147.32 128.27)
 		)
 		(stroke
@@
 	(wire
 		(pts
+			(xy 158.75 130.81) (xy 147.32 130.81)
+		)
+		(stroke
+			(width 0)
+			(type default)
+		)
+	)
+	(wire
+		(pts
 			(xy 80.01 171.45) (xy 80.01 173.99)
 		)
@@
 	(wire
 		(pts
+			(xy 161.29 125.73) (xy 158.75 125.73)
+		)
+		(stroke
+			(width 0)
+			(type default)
+		)
+	)
+	(wire
+		(pts
 			(xy 118.11 38.1) (xy 138.43 38.1)
 		)
@@
 	(wire
 		(pts
+			(xy 161.29 133.35) (xy 158.75 133.35)
+		)
+		(stroke
+			(width 0)
+			(type default)
+		)
+	)
+	(wire
+		(pts
 			(xy 176.53 71.12) (xy 176.53 68.58)
 		)
@@
 	(wire
 		(pts
+			(xy 158.75 125.73) (xy 158.75 128.27)
+		)
+		(stroke
+			(width 0)
+			(type default)
+		)
+	)
+	(wire
+		(pts
 			(xy 73.66 138.43) (xy 85.09 138.43)
 		)
@@
 	)
 	(symbol
-		(lib_id "Connector_Generic:Conn_01x02")
-		(at 160.02 128.27 0)
+		(lib_id "Connector_Generic:Conn_01x04")
+		(at 166.37 128.27 0)
 		(unit 1)
 		(exclude_from_sim no)
@@
 		(on_board yes)
 		(dnp no)
-		(fields_autoplaced yes)
 		(property "Reference" "J9"
-			(at 162.56 128.27 0)
+			(at 165.1 120.65 0)
 			(effects
 				(font
@@
 		)
 		(property "Value" "Conn_01x02"
-			(at 162.56 130.81 0)
+			(at 165.1 123.19 0)
 			(effects
 				(font
@@
 			)
 		)
-		(property "Footprint" "Connector_PinHeader_2.54mm:PinHeader_1x02_P2.54mm_Vertical"
-			(at 160.02 128.27 0)
+		(property "Footprint" "Connector_PinHeader_2.54mm:PinHeader_1x04_P2.54mm_Vertical"
+			(at 166.37 128.27 0)
 			(effects
 				(font
@@
 		)
 		(property "Datasheet" "~"
-			(at 160.02 128.27 0)
+			(at 166.37 128.27 0)
 			(effects
 				(font
@@
 			)
 		)
-		(property "Description" ""
-			(at 160.02 128.27 0)
+		(property "Description" "Generic connector, single row, 01x04, script generated (kicad-library-utils/schlib/autogen/connector/)"
+			(at 166.37 128.27 0)
 			(effects
 				(font
@@
 		(pin "2"
 		)
+		(pin "4"
+		)
+		(pin "3"
+		)
 		(instances
