File: boards/a1_micro_atx/usb.kicad_sch (KiCad schematic)
At the start: 24 parts, among them J15 USB_A_Stacked, J16 USB_A_Stacked, J17 USB_A_Stacked, U28 A1_USBHUB

Commit message: Major schematic beautification.
Changed lines of the file:
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@@
 (kicad_sch (version 20230121) (generator eeschema)
-  (paper "A4")
+  (paper "A")
   (junction (at 113.03 111.76) (diameter 0) (color 0 0 0 0)
   )
@@
     (pin "1")
     (instances
-      (project "a1_mini"
+      (project "a1_micro_atx"
         (path "/3257e1ae-50a8-410a-87c3-a39d96a2c51a/77f1c88a-ea71-40c5-9918-dee285c676a1"
           (reference "#PWR0198") (unit 1)
@@
     (pin "10")
     (instances
-      (project "a1_mini"
+      (project "a1_micro_atx"
         (path "/3257e1ae-50a8-410a-87c3-a39d96a2c51a/77f1c88a-ea71-40c5-9918-dee285c676a1"
           (reference "U28") (unit 1)
@@
     (pin "2")
     (instances
-      (project "a1_mini"
+      (project "a1_micro_atx"
         (path "/3257e1ae-50a8-410a-87c3-a39d96a2c51a/77f1c88a-ea71-40c5-9918-dee285c676a1"
           (reference "CMC5") (unit 1)
@@
     (pin "1")
     (instances
-      (project "a1_mini"
+      (project "a1_micro_atx"
         (path "/3257e1ae-50a8-410a-87c3-a39d96a2c51a/77f1c88a-ea71-40c5-9918-dee285c676a1"
           (reference "FB17") (unit 1)
@@
   )
   (symbol (lib_id "Connector:USB_A_Stacked") (at 246.38 41.91 0) (mirror y) (unit 1)
-    (in_bom yes) (on_board yes) (dnp no) (fields_autoplaced)
-    (property "Reference" "J16" (at 255.27 40.64 0)
+    (in_bom yes) (on_board yes) (dnp no)
+    (property "Reference" "J16" (at 238.76 25.4 0)
       (effects (font (size 1.27 1.27)) (justify right))
     )
-    (property "Value" "USB_A_Stacked" (at 255.27 43.18 0)
+    (property "Value" "USB_A_Stacked" (at 238.76 27.94 0)
       (effects (font (size 1.27 1.27)) (justify right))
     )
@@
     (pin "7")
     (instances
-      (project "a1_mini"
+      (project "a1_micro_atx"
         (path "/3257e1ae-50a8-410a-87c3-a39d96a2c51a/77f1c88a-ea71-40c5-9918-dee285c676a1"
           (reference "J16") (unit 1)
@@
     (pin "2")
     (instances
-      (project "a1_mini"
+      (project "a1_micro_atx"
         (path "/3257e1ae-50a8-410a-87c3-a39d96a2c51a/77f1c88a-ea71-40c5-9918-dee285c676a1"
           (reference "C46") (unit 1)
@@
     (pin "1")
     (instances
-      (project "a1_mini"
+      (project "a1_micro_atx"
         (path "/3257e1ae-50a8-410a-87c3-a39d96a2c51a/77f1c88a-ea71-40c5-9918-dee285c676a1"
           (reference "FB18") (unit 1)
@@
     (pin "1")
     (instances
-      (project "a1_mini"
+      (project "a1_micro_atx"
         (path "/3257e1ae-50a8-410a-87c3-a39d96a2c51a/77f1c88a-ea71-40c5-9918-dee285c676a1"
           (reference "FB15") (unit 1)
@@
     (pin "2")
     (instances
-      (project "a1_mini"
+      (project "a1_micro_atx"
         (path "/3257e1ae-50a8-410a-87c3-a39d96a2c51a/77f1c88a-ea71-40c5-9918-dee285c676a1"
           (reference "CMC7") (unit 1)
@@
     (pin "1")
     (instances
-      (project "a1_mini"
+      (project "a1_micro_atx"
         (path "/3257e1ae-50a8-410a-87c3-a39d96a2c51a/77f1c88a-ea71-40c5-9918-dee285c676a1"
           (reference "#PWR0199") (unit 1)
@@
     (pin "1")
     (instances
-      (project "a1_mini"
+      (project "a1_micro_atx"
         (path "/3257e1ae-50a8-410a-87c3-a39d96a2c51a/77f1c88a-ea71-40c5-9918-dee285c676a1"
           (reference "FB16") (unit 1)
@@
     (pin "1")
     (instances
-      (project "a1_mini"
+      (project "a1_micro_atx"
         (path "/3257e1ae-50a8-410a-87c3-a39d96a2c51a/77f1c88a-ea71-40c5-9918-dee285c676a1"
           (reference "#PWR0196") (unit 1)
@@
     (pin "1")
     (instances
-      (project "a1_mini"
+      (project "a1_micro_atx"
         (path "/3257e1ae-50a8-410a-87c3-a39d96a2c51a/77f1c88a-ea71-40c5-9918-dee285c676a1"
           (reference "#PWR0193") (unit 1)
@@
   )
   (symbol (lib_id "Connector:USB_A_Stacked") (at 246.38 86.36 0) (mirror y) (unit 1)
-    (in_bom yes) (on_board yes) (dnp no) (fields_autoplaced)
-    (property "Reference" "J17" (at 255.27 85.09 0)
+    (in_bom yes) (on_board yes) (dnp no)
+    (property "Reference" "J17" (at 238.76 69.85 0)
       (effects (font (size 1.27 1.27)) (justify right))
     )
-    (property "Value" "USB_A_Stacked" (at 255.27 87.63 0)
+    (property "Value" "USB_A_Stacked" (at 238.76 72.39 0)
       (effects (font (size 1.27 1.27)) (justify right))
     )
@@
     (pin "7")
     (instances
-      (project "a1_mini"
+      (project "a1_micro_atx"
         (path "/3257e1ae-50a8-410a-87c3-a39d96a2c51a/77f1c88a-ea71-40c5-9918-dee285c676a1"
           (reference "J17") (unit 1)
@@
     (pin "2")
     (instances
-      (project "a1_mini"
+      (project "a1_micro_atx"
         (path "/3257e1ae-50a8-410a-87c3-a39d96a2c51a/77f1c88a-ea71-40c5-9918-dee285c676a1"
           (reference "CMC9") (unit 1)
@@
     (pin "2")
     (instances
-      (project "a1_mini"
+      (project "a1_micro_atx"
         (path "/3257e1ae-50a8-410a-87c3-a39d96a2c51a/77f1c88a-ea71-40c5-9918-dee285c676a1"
           (reference "C47") (unit 1)
@@
     (pin "1")
     (instances
-      (project "a1_mini"
+      (project "a1_micro_atx"
         (path "/3257e1ae-50a8-410a-87c3-a39d96a2c51a/77f1c88a-ea71-40c5-9918-dee285c676a1"
           (reference "#PWR0197") (unit 1)
@@
     (pin "1")
     (instances
-      (project "a1_mini"
+      (project "a1_micro_atx"
         (path "/3257e1ae-50a8-410a-87c3-a39d96a2c51a/77f1c88a-ea71-40c5-9918-dee285c676a1"
           (reference "#PWR0194") (unit 1)
@@
     (pin "1")
     (instances
-      (project "a1_mini"
+      (project "a1_micro_atx"
         (path "/3257e1ae-50a8-410a-87c3-a39d96a2c51a/77f1c88a-ea71-40c5-9918-dee285c676a1"
           (reference "JP3") (unit 1)
@@
     (pin "1")
     (instances
-      (project "a1_mini"
+      (project "a1_micro_atx"
         (path "/3257e1ae-50a8-410a-87c3-a39d96a2c51a/77f1c88a-ea71-40c5-9918-dee285c676a1"
           (reference "#PWR0195") (unit 1)
@@
     (pin "2")
     (instances
-      (project "a1_mini"
+      (project "a1_micro_atx"
         (path "/3257e1ae-50a8-410a-87c3-a39d96a2c51a/77f1c88a-ea71-40c5-9918-dee285c676a1"
           (reference "CMC6") (unit 1)
@@
     (pin "2")
     (instances
-      (project "a1_mini"
+      (project "a1_micro_atx"
         (path "/3257e1ae-50a8-410a-87c3-a39d96a2c51a/77f1c88a-ea71-40c5-9918-dee285c676a1"
           (reference "CMC8") (unit 1)
@@
     (pin "2")
     (instances
-      (project "a1_mini"
+      (project "a1_micro_atx"
         (path "/3257e1ae-50a8-410a-87c3-a39d96a2c51a/77f1c88a-ea71-40c5-9918-dee285c676a1"
           (reference "C48") (unit 1)
@@
     (pin "1")
     (instances
-      (project "a1_mini"
+      (project "a1_micro_atx"
         (path "/3257e1ae-50a8-410a-87c3-a39d96a2c51a/77f1c88a-ea71-40c5-9918-dee285c676a1"
           (reference "FB19") (unit 1)
@@
     (pin "1")
     (instances
-      (project "a1_mini"
+      (project "a1_micro_atx"
         (path "/3257e1ae-50a8-410a-87c3-a39d96a2c51a/77f1c88a-ea71-40c5-9918-dee285c676a1"
           (reference "FB20") (unit 1)
@@
     (pin "2")
     (instances
-      (project "a1_mini"
+      (project "a1_micro_atx"
         (path "/3257e1ae-50a8-410a-87c3-a39d96a2c51a/77f1c88a-ea71-40c5-9918-dee285c676a1"
           (reference "C45") (unit 1)
@@
     (pin "2")
     (instances
-      (project "a1_mini"
+      (project "a1_micro_atx"
         (path "/3257e1ae-50a8-410a-87c3-a39d96a2c51a/77f1c88a-ea71-40c5-9918-dee285c676a1"
           (reference "CMC10") (unit 1)
@@
   )
   (symbol (lib_id "Connector:USB_A_Stacked") (at 245.11 130.81 0) (mirror y) (unit 1)
-    (in_bom yes) (on_board yes) (dnp no) (fields_autoplaced)
-    (property "Reference" "J15" (at 254 129.54 0)
+    (in_bom yes) (on_board yes) (dnp no)
+    (property "Reference" "J15" (at 237.49 114.3 0)
       (effects (font (size 1.27 1.27)) (justify right))
     )
-    (property "Value" "USB_A_Stacked" (at 254 132.08 0)
+    (property "Value" "USB_A_Stacked" (at 237.49 116.84 0)
       (effects (font (size 1.27 1.27)) (justify right))
     )
@@
     (pin "7")
     (instances
-      (project "a1_mini"
+      (project "a1_micro_atx"
         (path "/3257e1ae-50a8-410a-87c3-a39d96a2c51a/77f1c88a-ea71-40c5-9918-dee285c676a1"
           (reference "J15") (unit 1)
@@
     (pin "2")
     (instances
-      (project "a1_mini"
+      (project "a1_micro_atx"
         (path "/3257e1ae-50a8-410a-87c3-a39d96a2c51a/77f1c88a-ea71-40c5-9918-dee285c676a1"
           (reference "C49") (unit 1)
@@
     (pin "1")
     (instances
-      (project "a1_mini"
+      (project "a1_micro_atx"
         (path "/3257e1ae-50a8-410a-87c3-a39d96a2c51a/77f1c88a-ea71-40c5-9918-dee285c676a1"
           (reference "C44") (unit 1)
@@
     (pin "1")
     (instances
-      (project "a1_mini"
+      (project "a1_micro_atx"
         (path "/3257e1ae-50a8-410a-87c3-a39d96a2c51a/77f1c88a-ea71-40c5-9918-dee285c676a1"
           (reference "#PWR0200") (unit 1)
@@
     (pin "2")
     (instances
-      (project "a1_mini"
+      (project "a1_micro_atx"
         (path "/3257e1ae-50a8-410a-87c3-a39d96a2c51a/77f1c88a-ea71-40c5-9918-dee285c676a1"
           (reference "C50") (unit 1)

Commit message: Fixed 3.3V for SDCARD; more beautification.
Other:
- company: (none) -> Modular Circuits
- title: (none) -> Anachron uATX USB HUB
Changed lines of the file:
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@@
 (kicad_sch (version 20230121) (generator eeschema)
   (paper "A")
+  (title_block
+    (title "Anachron uATX USB HUB")
+    (date "2024-02-07")
+    (company "Modular Circuits")
+  )
   (junction (at 113.03 111.76) (diameter 0) (color 0 0 0 0)
   )

Commit message: Moved USB HUB ports around.
Connections:
- net USB_DN6_D+: now also CMC10.1, U28.24 (USBDN1_DP); no longer CMC9.1, U28.15 (USBDN6_DP)
- net USB_DN6_D-: now also CMC10.4, U28.23 (USBDN1_DM); no longer CMC9.4, U28.14 (USBDN6_DM)
- net USB_DN7_D+: now also CMC9.1; no longer CMC10.1
- net USB_DN7_D-: now also CMC9.4; no longer CMC10.4
- net at U28.1 (VBUS6): no longer FB19.1
- net at U28.3 (VBUS7): now also FB19.1; no longer FB20.1
- net at U28.4 (VBUS1): now also FB20.1
Other:
- moved on the sheet: CMC10, CMC9, FB19, FB20

Commit message: Rotated last DIP package, fixed up a lot of violations and warnings.
Parts:
- U28: footprint Package_DIP:DIP-40_W15.24mm_LongPads -> anachron:DIP-40_W15.24mm_Socket
Changed lines of the file:
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@@
 			)
 		)
-		(property "Footprint" "Package_DIP:DIP-40_W15.24mm_LongPads"
+		(property "Footprint" "anachron:DIP-40_W15.24mm_Socket"
 			(at 107.95 54.61 0)
 			(effects

Commit message: Added reverse-power protection to HDMI; small cleanup
- Reverse-current protection on HDMI (via simple diode)
- Cleaned up diff-pair annotation on schematic
- Added proper 3D shape for AT connector
Changed lines of the file:
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@@
 	)
 	(netclass_flag ""
-		(length 2.54)
+		(length 1.27)
 		(shape round)
-		(at 165.1 106.68 0)
+		(at 161.29 106.68 0)
 		(fields_autoplaced yes)
 		(effects
@@
 		)
 		(property "Netclass" "USB2"
-			(at 165.7985 104.14 0)
+			(at 161.9885 105.41 0)
 			(effects
 				(font
@@
 	)
 	(netclass_flag ""
-		(length 2.54)
+		(length 1.27)
 		(shape round)
 		(at 161.29 63.5 0)
@@
 		)
 		(property "Netclass" "USB2"
-			(at 161.9885 60.96 0)
+			(at 161.9885 62.23 0)
 			(effects
 				(font
@@
 	)
 	(netclass_flag ""
-		(length 2.54)
+		(length 1.27)
 		(shape round)
 		(at 161.29 83.82 0)
@@
 		)
 		(property "Netclass" "USB2"
-			(at 161.9885 81.28 0)
+			(at 161.9885 82.55 0)
 			(effects
 				(font
@@
 	)
 	(netclass_flag ""
-		(length 2.54)
+		(length 1.27)
 		(shape round)
 		(at 161.29 104.14 0)
@@
 		)
 		(property "Netclass" "USB2"
-			(at 161.9885 101.6 0)
+			(at 161.9885 102.87 0)
 			(effects
 				(font
@@
 	)
 	(netclass_flag ""
-		(length 2.54)
+		(length 1.27)
 		(shape round)
-		(at 165.1 55.88 0)
+		(at 161.29 55.88 0)
 		(fields_autoplaced yes)
 		(effects
@@
 		)
 		(property "Netclass" "USB2"
-			(at 165.7985 53.34 0)
+			(at 161.9885 54.61 0)
 			(effects
 				(font
@@
 	)
 	(netclass_flag ""
-		(length 2.54)
+		(length 1.27)
 		(shape round)
 		(at 161.29 53.34 0)
@@
 		)
 		(property "Netclass" "USB2"
-			(at 161.9885 50.8 0)
+			(at 161.9885 52.07 0)
 			(effects
 				(font
@@
 	)
 	(netclass_flag ""
-		(length 2.54)
+		(length 1.27)
 		(shape round)
-		(at 165.1 45.72 0)
+		(at 161.29 45.72 0)
 		(fields_autoplaced yes)
 		(effects
@@
 		)
 		(property "Netclass" "USB2"
-			(at 165.7985 43.18 0)
+			(at 161.9885 44.45 0)
 			(effects
 				(font
@@
 	)
 	(netclass_flag ""
-		(length 2.54)
+		(length 1.27)
 		(shape round)
 		(at 161.29 73.66 0)
@@
 		)
 		(property "Netclass" "USB2"
-			(at 161.9885 71.12 0)
+			(at 161.9885 72.39 0)
 			(effects
 				(font
@@
 	)
 	(netclass_flag ""
-		(length 2.54)
+		(length 1.27)
 		(shape round)
-		(at 165.1 66.04 0)
+		(at 161.29 66.04 0)
 		(fields_autoplaced yes)
 		(effects
@@
 		)
 		(property "Netclass" "USB2"
-			(at 165.7985 63.5 0)
+			(at 161.9885 64.77 0)
 			(effects
 				(font
@@
 	)
 	(netclass_flag ""
-		(length 2.54)
+		(length 1.27)
 		(shape round)
-		(at 165.1 86.36 0)
+		(at 161.29 86.36 0)
 		(fields_autoplaced yes)
 		(effects
@@
 		)
 		(property "Netclass" "USB2"
-			(at 165.7985 83.82 0)
+			(at 161.9885 85.09 0)
 			(effects
 				(font
@@
 	)
 	(netclass_flag ""
-		(length 2.54)
+		(length 1.27)
 		(shape round)
-		(at 165.1 76.2 0)
+		(at 161.29 76.2 0)
 		(fields_autoplaced yes)
 		(effects
@@
 		)
 		(property "Netclass" "USB2"
-			(at 165.7985 73.66 0)
+			(at 161.9885 74.93 0)
 			(effects
 				(font
@@
 	)
 	(netclass_flag ""
-		(length 2.54)
+		(length 1.27)
 		(shape round)
 		(at 161.29 43.18 0)
@@
 		)
 		(property "Netclass" "USB2"
-			(at 161.9885 40.64 0)
+			(at 161.9885 41.91 0)
 			(effects
 				(font
@@
 		(dnp no)
 		(property "Reference" "CMC5"
-			(at 170.18 54.61 0)
+			(at 175.26 57.15 0)
 			(effects
 				(font
@@
 		(dnp no)
 		(property "Reference" "FB17"
-			(at 173.99 69.85 90)
+			(at 172.72 69.85 90)
 			(effects
 				(font
@@
 		(dnp no)
 		(property "Reference" "FB18"
-			(at 173.99 80.01 90)
+			(at 172.72 80.01 90)
 			(effects
 				(font
@@
 		(dnp no)
 		(property "Reference" "FB15"
-			(at 173.99 49.53 90)
+			(at 172.72 49.53 90)
 			(effects
 				(font
@@
 		(dnp no)
 		(property "Reference" "CMC7"
-			(at 170.18 74.93 0)
+			(at 176.53 77.47 0)
 			(effects
 				(font
@@
 		(dnp no)
 		(property "Reference" "FB16"
-			(at 173.99 59.69 90)
+			(at 172.72 59.69 90)
 			(effects
 				(font
@@
 		(dnp no)
 		(property "Reference" "CMC9"
-			(at 170.18 105.41 0)
+			(at 176.53 107.95 0)
 			(effects
 				(font
@@
 		(dnp no)
 		(property "Reference" "CMC6"
-			(at 170.18 64.77 0)
+			(at 176.53 67.31 0)
 			(effects
 				(font
@@
 		(dnp no)
 		(property "Reference" "CMC8"
-			(at 170.18 85.09 0)
+			(at 176.53 87.63 0)
 			(effects
 				(font
@@
 		(dnp no)
 		(property "Reference" "FB19"
-			(at 173.99 100.33 90)
+			(at 172.72 100.33 90)
 			(effects
 				(font
@@
 		(dnp no)
 		(property "Reference" "FB20"
-			(at 173.99 39.37 90)
+			(at 172.72 39.37 90)
 			(effects
 				(font
@@
 		(dnp no)
 		(property "Reference" "CMC10"
-			(at 170.18 44.45 0)
-			(effects
-				(font
+			(at 175.26 46.99 0)
+			(effects
+				(font

Commit message: Small fixes and improvements
- Speaker connector is now PC-compatible
- Added internal USB connector for the 7th USB port
- If MCU is not programmed, power defaults to ON
Parts:
- added C74: 100uF, Capacitor_THT:CP_Radial_D5.0mm_P2.00mm, symbol Device:C_Polarized_Small_US
- added J7: Conn_02x05_Odd_Even, Connector_PinHeader_2.54mm:PinHeader_2x05_P2.54mm_Vertical, symbol Connector_Generic:Conn_2Rows-09Pins
Connections:
- net GND: now also C74.2, J7.7 (Pin_7)
- net at U28.1 (VBUS6): now also C74.1, J7.1 (Pin_1)
- net USB_DN_INT_D+: now reaches U28.14 (USBDN6_DM)
- net USB_DN_INT_D+: now also J7.3 (Pin_3)
- net USB_DN_INT_D-: now reaches U28.15 (USBDN6_DP)
- net USB_DN_INT_D-: now also J7.5 (Pin_5)
